File: KiCad/ClockFOUR.kicad_pcb (KiCad board)
At the start: 2 copper layers, 0 parts

Commit message: Schematic updated, board started
Parts:
- added S1, S2, S3, S4: CONN_1, 1pin, F.Cu at (279.4, 268.1)
- added SW1: SW_RST, SW_PUSH_SMALL, F.Cu at (279.4, 268.1)
- added U1: DS3231N, so-16, F.Cu at (279.4, 268.1)
Other:
- board outline added: 220 x 240 mm
