File: KiCad/ClockFOUR.kicad_pcb (KiCad board)
At the start: 2 copper layers, 210 x 228 mm, 406 parts, among them P1 ICSP, P2 FTDI, P3 LDR_header, P4 Button_Header, P5 BARREL_JACK, SW1 SW_RST, U1 ATMEGA328P, U2 DS3231N, X1 CRYSTAL

Commit message: PCB layout, work in progress
Parts:
- added L1: OSHW, C4_Pretty:Logo_silk_OSHW_6x6mm, F.Cu at (229.5, 261.9)
- added L2: Wyolum, C4_Pretty:Logo-WL3, F.Cu at (236.5, 259.2)
- added LDR1: LDR, C4_Pretty:r_0805, F.Cu at (195.2, 48.0)
- BT1: value BATT_RTC -> Batt_RTC; footprint C4_Modules:CR2032 -> C4_Pretty:CR2032_SMD
- C1, C11, C2, C3, C4, C5, C6, C7, C8, C9: footprint C4_Modules:SM0805 -> C4_Pretty:c_0805
- C10, C194, C195, C196: footprint C4_Modules:c_2917 -> C4_Pretty:c_2917
- C100, C101, C102, C103, C104, C105, C106, C107, C108, C109, C110, C111, C112, C113, C114, C115, C116, C117, C118, C119, C12, C120, C121, C122, C123, C124, C125, C126, C127, C128, C129, C13, C130, C131, C132, C133, C134, C135, C136, C137, C138, C139, C14, C140, C141, C142, C143, C144, C145, C146, C147, C148, C149, C15, C150, C151, C152, C153, C154, C155, C156, C157, C158, C159, C16, C160, C161, C162, C163, C164, C165, C166, C167, C168, C169, C17, C170, C171, C172, C173, C174, C175, C176, C177, C178, C179, C18, C180, C181, C182, C183, C184, C185, C186, C187, C188, C189, C19, C190, C191, C192, C193, C20, C21, C22, C23, C24, C25, C26, C27, C28, C29, C30, C31, C32, C33, C34, C35, C36, C37, C38, C39, C40, C41, C42, C43, C44, C45, C46, C47, C48, C49, C50, C51, C52, C53, C54, C55, C56, C57, C58, C59, C60, C61, C62, C63, C64, C65, C66, C67, C68, C69, C70, C71, C72, C73, C74, C75, C76, C77, C78, C79, C80, C81, C82, C83, C84, C85, C86, C87, C88, C89, C90, C91, C92, C93, C94, C95, C96, C97, C98, C99: footprint C4_Modules:C4_SM0805 -> C4_Pretty:c_0805
- LED1, LED10, LED100, LED101, LED102, LED103, LED104, LED105, LED106, LED107, LED108, LED109, LED11, LED110, LED111, LED112, LED113, LED114, LED115, LED116, LED117, LED118, LED119, LED12, LED120, LED121, LED122, LED123, LED124, LED125, LED126, LED127, LED128, LED129, LED13, LED130, LED131, LED132, LED133, LED134, LED135, LED136, LED137, LED138, LED139, LED14, LED140, LED141, LED142, LED143, LED144, LED145, LED146, LED147, LED148, LED149, LED15, LED150, LED151, LED152, LED153, LED154, LED155, LED156, LED157, LED158, LED159, LED16, LED160, LED161, LED162, LED163, LED164, LED165, LED166, LED167, LED168, LED169, LED17, LED170, LED171, LED172, LED173, LED174, LED175, LED176, LED177, LED178, LED179, LED18, LED180, LED181, LED182, LED19, LED2, LED20, LED21, LED22, LED23, LED24, LED25, LED26, LED27, LED28, LED29, LED3, LED30, LED31, LED32, LED33, LED34, LED35, LED36, LED37, LED38, LED39, LED4, LED40, LED41, LED42, LED43, LED44, LED45, LED46, LED47, LED48, LED49, LED5, LED50, LED51, LED52, LED53, LED54, LED55, LED56, LED57, LED58, LED59, LED6, LED60, LED61, LED62, LED63, LED64, LED65, LED66, LED67, LED68, LED69, LED7, LED70, LED71, LED72, LED73, LED74, LED75, LED76, LED77, LED78, LED79, LED8, LED80, LED81, LED82, LED83, LED84, LED85, LED86, LED87, LED88, LED89, LED9, LED90, LED91, LED92, LED93, LED94, LED95, LED96, LED97, LED98, LED99: footprint C4_Modules:WS2812B -> C4_Pretty:RGB_WS2811B
- P1: footprint Header_ISP -> C4_Pretty:ISP
- P2: footprint Header_FTDI -> C4_Pretty:Header_FTDI
- P3, P4: footprint SIL-2 -> C4_Pretty:SIL-2
- P5: footprint JACK_PJ-047a -> C4_Pretty:JACK_PJ-047a
- R1, R2, R3, R4, R5, R6, R7, R8, R9: footprint C4_Modules:SM0805 -> C4_Pretty:r_0805
- S1, S2, S3, S4: footprint C4_Modules:1pin -> C4_Pretty:Screw_3mm
- S5, S6, S7, S8, S9: footprint PIN_ARRAY_1 -> C4_Pretty:BreakOutPad
- SW1: footprint SW_PUSH_SMALL -> C4_Pretty:SW_PB_V_H; moved to B.Cu
- U1: footprint TQFP32 -> C4_Pretty:TQFP32
- U2: footprint DS3231 -> C4_Pretty:DS3231
- X1: value CRYSTAL -> 16MHz; footprint Xtal_SMD -> C4_Pretty:Xtal_SMD3
- moved P5 13.5 mm to (151.0, 264.0), turned to 0 degrees
- moved C5 8.61 mm to (131.4, 90.8), turned to 90 degrees
- moved C7 7.67 mm to (131.4, 83.8), turned to 90 degrees
- moved C8 7.47 mm to (121.4, 44.0)
- moved C9 5.96 mm to (104.0, 50.3), turned to 180 degrees
- moved SW1 2.95 mm to (241.5, 43.3), turned to 270 degrees
- moved X1 2.35 mm to (131.4, 87.2)
- moved R8 1.80 mm to (100.8, 74.4), turned to 270 degrees
- moved BT1 1.70 mm to (84.0, 50.2)
- moved R6 1.50 mm to (81.0, 70.0), turned to 180 degrees
- moved U2 1.40 mm to (91.3, 68.4)
- moved R7 1.10 mm to (81.0, 73.1), turned to 180 degrees
- moved C6 1.00 mm to (230.0, 46.2), turned to 0 degrees
- moved R9 1.00 mm to (100.8, 70.0), turned to 90 degrees
- moved R2 0.80 mm to (234.7, 46.0), turned to 270 degrees
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Connections:
- C5 pad 1: N-000003 -> Net-(C5-Pad1)
- C7 pad 2: N-000002 -> Net-(C7-Pad2)
- LED182 pad 2: (no net) -> /Row_M/DO_M
- S1 pad 1: (no net) -> Net-(S1-Pad1)
- S2 pad 1: (no net) -> Net-(S2-Pad1)
- S3 pad 1: (no net) -> Net-(S3-Pad1)
- S4 pad 1: (no net) -> Net-(S4-Pad1)
- SW1 pad 1: GND -> /RESET
- SW1 pad 2: /RESET -> GND
- U1 pad 12: (no net) -> Net-(U1-Pad12)
- U1 pad 13: (no net) -> Net-(U1-Pad13)
- U1 pad 14: (no net) -> Net-(U1-Pad14)
- U1 pad 19: (no net) -> Net-(U1-Pad19)
- U1 pad 22: (no net) -> Net-(U1-Pad22)
- U1 pad 7: N-000003 -> Net-(C5-Pad1)
- U1 pad 8: N-000002 -> Net-(C7-Pad2)
- X1 pad 1: N-000002 -> Net-(C5-Pad1)
- X1 pad 2: N-000003 -> Net-(C7-Pad2)
Routing:
- net GND: track 26.4 -> 1446.5 mm, vias 2 -> 4
- net N-000002: track 16.8 -> 0.00 mm
- net 5V: track 4428.6 -> 4444.5 mm
- net N-000003: track 14.4 -> 0.00 mm
- net Net-(C5-Pad1): track 0.00 -> 13.3 mm
- net Net-(C7-Pad2): track 0.00 -> 10.0 mm
- net Net-(BT1-Pad1): track 87.4 -> 97.3 mm
- net /LDR_PIN: track 79.4 -> 83.3 mm
- net /SCL: track 91.4 -> 93.0 mm
- net /SDA: track 88.4 -> 89.6 mm
- net Net-(C6-Pad2): track 7.42 -> 6.42 mm
- net /BUTTON_L: track 39.5 -> 40.1 mm
