File: KiCad/Row_A.sch (KiCad schematic (older format))
At the start: 29 parts

Commit message: Schematic updated
Parts:
- removed C117: 47u,8V, TinyTiM_Lib:c_2917, symbol C_POL_1
- gave numbers to parts that had none: 27
Connections:
- wire segments 84 -> 82
Changed lines of the file:
@@
 LIBS:valves
 LIBS:TinyTiM-cache
+LIBS:TiNA_sym
 LIBS:ClockFOUR-cache
 EELAYER 27 0
@@
 Sheet 2 14
 Title "ClockFOUR"
-Date "26 sep 2014"
+Date "29 sep 2014"
 Rev ""
 Comp "WyoLum"
 Comment1 "www.wyolum.com"
-Comment2 ""
+Comment2 "David Pincus"
 Comment3 ""
 Comment4 ""
 $EndDescr
-Text Label 950  900  0    60   ~ 0
-DI_A
 Text HLabel 950  5250 0    60   Output ~ 0
 DO_A
@@
 Text HLabel 950  2750 0    60   Input ~ 0
 5V
-Text Label 950  2350 0    60   ~ 0
-GND
-Text Label 950  2750 0    60   ~ 0
-5V
-$Comp
-L GND #PWR011
+$Comp
+L GND #PWR6
 U 1 1 5116893B
 P 1150 2400
-F 0 "#PWR011" H 1150 2400 30  0001 C CNN
+F 0 "#PWR6" H 1150 2400 30  0001 C CNN
 F 1 "GND" H 1150 2330 30  0001 C CNN
 F 2 "" H 1150 2400 60  0001 C CNN
 F 3 "" H 1150 2400 60  0001 C CNN
 	1    1150 2400
-	1    0    0    -1
-$EndComp
-Text Label 1900 5900 0    60   ~ 0
-5V
-Text Label 1900 6750 0    60   ~ 0
-GND
-$Comp
-L C_POL_1 C117
-U 1 1 5118AB5E
-P 1900 6300
-F 0 "C117" H 2025 6275 50  0000 L CNN
-F 1 "47u,8V" H 2025 6175 50  0000 L CNN
-F 2 "TinyTiM_Lib:c_2917" H 1900 6250 50  0001 C CNN
-F 3 "" H 1900 6300 60  0001 C CNN
-F 4 "CAP ALUM 47UF 8V 20% SMD" H 1900 6500 60  0001 L CNN "Field4"
-F 5 "47u,8V" H 1900 6600 60  0001 L CNN "Field5"
-F 6 "2917 (7343 Metric)" H 1900 6700 60  0001 L CNN "Field6"
-F 7 "Panasonic Electronic Components" H 1900 6800 60  0001 L CNN "Field7"
-F 8 "EEF-CD0K470R" H 1900 6900 60  0001 L CNN "Field8"
-F 9 "Digikey" H 1900 7000 60  0001 L CNN "Field9"
-F 10 "PCE3606CT-ND" H 1900 7100 60  0001 L CNN "Field10"
-F 11 "http://www.digikey.com/product-detail/en/EEF-CD0K470R/PCE3606CT-ND/614442" H 1900 7200 60  0001 L CNN "Field11"
-	1    1900 6300
 	1    0    0    -1
 $EndComp
@@
 $EndComp
 $Comp
-L RGB_WS2812B U?
+L RGB_WS2812B U3
 U 1 1 5424CDC4
 P 1525 1575
-F 0 "U?" V 1275 1575 60  0000 C CNN
+F 0 "U3" V 1275 1575 60  0000 C CNN
 F 1 "RGB_WS2812B" V 1925 1575 60  0000 C CNN
 F 2 "" H 1525 1575 60  0000 C CNN
@@
 $EndComp
 $Comp
-L RGB_WS2812B U?
+L RGB_WS2812B U5
 U 1 1 5424CE47
 P 2925 1575
-F 0 "U?" V 2675 1575 60  0000 C CNN
+F 0 "U5" V 2675 1575 60  0000 C CNN
 F 1 "RGB_WS2812B" V 3325 1575 60  0000 C CNN
 F 2 "" H 2925 1575 60  0000 C CNN
@@
 $EndComp
 $Comp
-L RGB_WS2812B U?
+L RGB_WS2812B U7
 U 1 1 5424CE4D
 P 4325 1575
-F 0 "U?" V 4075 1575 60  0000 C CNN
+F 0 "U7" V 4075 1575 60  0000 C CNN
 F 1 "RGB_WS2812B" V 4725 1575 60  0000 C CNN
 F 2 "" H 4325 1575 60  0000 C CNN
@@
 $EndComp
 $Comp
-L RGB_WS2812B U?
+L RGB_WS2812B U9
 U 1 1 5424CE53
 P 5725 1575
-F 0 "U?" V 5475 1575 60  0000 C CNN
+F 0 "U9" V 5475 1575 60  0000 C CNN
 F 1 "RGB_WS2812B" V 6125 1575 60  0000 C CNN
 F 2 "" H 5725 1575 60  0000 C CNN
@@
 $EndComp
 $Comp
-L RGB_WS2812B U?
+L RGB_WS2812B U11
 U 1 1 5424CE59
 P 7125 1575
-F 0 "U?" V 6875 1575 60  0000 C CNN
+F 0 "U11" V 6875 1575 60  0000 C CNN
 F 1 "RGB_WS2812B" V 7525 1575 60  0000 C CNN
 F 2 "" H 7125 1575 60  0000 C CNN
@@
 $EndComp
 $Comp
-L RGB_WS2812B U?
+L RGB_WS2812B U13
 U 1 1 5424CE5F
 P 8525 1575
-F 0 "U?" V 8275 1575 60  0000 C CNN
+F 0 "U13" V 8275 1575 60  0000 C CNN
 F 1 "RGB_WS2812B" V 8925 1575 60  0000 C CNN
 F 2 "" H 8525 1575 60  0000 C CNN
@@
 $EndComp
 $Comp
-L RGB_WS2812B U?
+L RGB_WS2812B U15
 U 1 1 5424CE65
 P 9925 1575
-F 0 "U?" V 9675 1575 60  0000 C CNN
+F 0 "U15" V 9675 1575 60  0000 C CNN
 F 1 "RGB_WS2812B" V 10325 1575 60  0000 C CNN
 F 2 "" H 9925 1575 60  0000 C CNN
@@
 $EndComp
 $Comp
-L RGB_WS2812B U?
+L RGB_WS2812B U4
 U 1 1 5424CE6B
 P 1525 3975
-F 0 "U?" V 1275 3975 60  0000 C CNN
+F 0 "U4" V 1275 3975 60  0000 C CNN
 F 1 "RGB_WS2812B" V 1925 3975 60  0000 C CNN
 F 2 "" H 1525 3975 60  0000 C CNN
@@
 $EndComp
 $Comp
-L RGB_WS2812B U?
+L RGB_WS2812B U6
 U 1 1 5424CE71
 P 2925 3975
-F 0 "U?" V 2675 3975 60  0000 C CNN
+F 0 "U6" V 2675 3975 60  0000 C CNN
 F 1 "RGB_WS2812B" V 3325 3975 60  0000 C CNN
 F 2 "" H 2925 3975 60  0000 C CNN
@@
 $EndComp
 $Comp
-L RGB_WS2812B U?
+L RGB_WS2812B U8
 U 1 1 5424CE77
 P 4325 3975
-F 0 "U?" V 4075 3975 60  0000 C CNN
+F 0 "U8" V 4075 3975 60  0000 C CNN
 F 1 "RGB_WS2812B" V 4725 3975 60  0000 C CNN
 F 2 "" H 4325 3975 60  0000 C CNN
@@
 $EndComp
 $Comp
-L RGB_WS2812B U?
+L RGB_WS2812B U10
 U 1 1 5424CE7D
 P 5725 3975
-F 0 "U?" V 5475 3975 60  0000 C CNN
+F 0 "U10" V 5475 3975 60  0000 C CNN
 F 1 "RGB_WS2812B" V 6125 3975 60  0000 C CNN
 F 2 "" H 5725 3975 60  0000 C CNN
@@
 $EndComp
 $Comp
-L RGB_WS2812B U?
+L RGB_WS2812B U12
 U 1 1 5424CE83
 P 7125 3975
-F 0 "U?" V 6875 3975 60  0000 C CNN
+F 0 "U12" V 6875 3975 60  0000 C CNN
 F 1 "RGB_WS2812B" V 7525 3975 60  0000 C CNN
 F 2 "" H 7125 3975 60  0000 C CNN
@@
 $EndComp
 $Comp
-L RGB_WS2812B U?
+L RGB_WS2812B U14
 U 1 1 5424CE89
 P 8525 3975
-F 0 "U?" V 8275 3975 60  0000 C CNN
+F 0 "U14" V 8275 3975 60  0000 C CNN
 F 1 "RGB_WS2812B" V 8925 3975 60  0000 C CNN
 F 2 "" H 8525 3975 60  0000 C CNN
@@
 $EndComp
 $Comp
-L RGB_WS2812B U?
+L RGB_WS2812B U16
 U 1 1 5424CE8F
 P 9925 3975
-F 0 "U?" V 9675 3975 60  0000 C CNN
+F 0 "U16" V 9675 3975 60  0000 C CNN
 F 1 "RGB_WS2812B" V 10325 3975 60  0000 C CNN
 F 2 "" H 9925 3975 60  0000 C CNN
@@
 $EndComp
 Wire Wire Line
-	1900 6550 1900 6750
-Wire Wire Line
 	1150 2350 1150 2400
 Wire Wire Line
@@
 Connection ~ 1150 2350
 Wire Wire Line
-	1900 6100 1900 5900
-Wire Wire Line
 	1800 1000 1800 900
 Wire Wire Line
@@
 Connection ~ 1600 2750
 $Comp
-L C2 C?
+L C2 C6
 U 1 1 5424D6B9
 P 3100 2550
-F 0 "C?" H 3125 2650 50  0000 L CNN
+F 0 "C6" H 3125 2650 50  0000 L CNN
 F 1 "100n" H 3125 2450 50  0000 L CNN
 F 2 "TinyTiM_Lib:c_0805" H 3100 2550 50  0001 C CNN
@@
 $EndComp
 $Comp
-L C2 C?
+L C2 C8
 U 1 1 5424D6C7
 P 4500 2550
-F 0 "C?" H 4525 2650 50  0000 L CNN
+F 0 "C8" H 4525 2650 50  0000 L CNN
 F 1 "100n" H 4525 2450 50  0000 L CNN
 F 2 "TinyTiM_Lib:c_0805" H 4500 2550 50  0001 C CNN
@@
 $EndComp
 $Comp
-L C2 C?
+L C2 C10
 U 1 1 5424D6D5
 P 5900 2550
-F 0 "C?" H 5925 2650 50  0000 L CNN
+F 0 "C10" H 5925 2650 50  0000 L CNN
 F 1 "100n" H 5925 2450 50  0000 L CNN
 F 2 "TinyTiM_Lib:c_0805" H 5900 2550 50  0001 C CNN
@@
 $EndComp
 $Comp
-L C2 C?
+L C2 C12
 U 1 1 5424D6E3
 P 7300 2550
-F 0 "C?" H 7325 2650 50  0000 L CNN
+F 0 "C12" H 7325 2650 50  0000 L CNN
 F 1 "100n" H 7325 2450 50  0000 L CNN
 F 2 "TinyTiM_Lib:c_0805" H 7300 2550 50  0001 C CNN
@@
 $EndComp
 $Comp
-L C2 C?
+L C2 C14
 U 1 1 5424D6F1
 P 8700 2550
-F 0 "C?" H 8725 2650 50  0000 L CNN
+F 0 "C14" H 8725 2650 50  0000 L CNN
 F 1 "100n" H 8725 2450 50  0000 L CNN
 F 2 "TinyTiM_Lib:c_0805" H 8700 2550 50  0001 C CNN
@@
 $EndComp
 $Comp
-L C2 C?
+L C2 C16
 U 1 1 5424D6FF
 P 10100 2550
-F 0 "C?" H 10125 2650 50  0000 L CNN
+F 0 "C16" H 10125 2650 50  0000 L CNN
 F 1 "100n" H 10125 2450 50  0000 L CNN
 F 2 "TinyTiM_Lib:c_0805" H 10100 2550 50  0001 C CNN
@@
 Connection ~ 10000 2750
 $Comp
-L C2 C?
+L C2 C5
 U 1 1 5424D75D
 P 1700 4900
-F 0 "C?" H 1725 5000 50  0000 L CNN
+F 0 "C5" H 1725 5000 50  0000 L CNN
 F 1 "100n" H 1725 4800 50  0000 L CNN
 F 2 "TinyTiM_Lib:c_0805" H 1700 4900 50  0001 C CNN
@@
 Connection ~ 1600 5100
 $Comp
-L C2 C?
+L C2 C7
 U 1 1 5424DFA1
 P 3100 4900
-F 0 "C?" H 3125 5000 50  0000 L CNN
+F 0 "C7" H 3125 5000 50  0000 L CNN
 F 1 "100n" H 3125 4800 50  0000 L CNN
 F 2 "TinyTiM_Lib:c_0805" H 3100 4900 50  0001 C CNN
@@
 $EndComp
 $Comp
-L C2 C?
+L C2 C9
 U 1 1 5424DFAF
 P 4500 4900
-F 0 "C?" H 4525 5000 50  0000 L CNN
+F 0 "C9" H 4525 5000 50  0000 L CNN
 F 1 "100n" H 4525 4800 50  0000 L CNN
 F 2 "TinyTiM_Lib:c_0805" H 4500 4900 50  0001 C CNN
@@
 $EndComp
 $Comp
-L C2 C?
+L C2 C11
 U 1 1 5424DFBD
 P 5900 4900
-F 0 "C?" H 5925 5000 50  0000 L CNN
+F 0 "C11" H 5925 5000 50  0000 L CNN
 F 1 "100n" H 5925 4800 50  0000 L CNN
 F 2 "TinyTiM_Lib:c_0805" H 5900 4900 50  0001 C CNN
@@
 $EndComp
 $Comp
-L C2 C?
+L C2 C13
 U 1 1 5424DFCB
 P 7300 4900
-F 0 "C?" H 7325 5000 50  0000 L CNN
+F 0 "C13" H 7325 5000 50  0000 L CNN
 F 1 "100n" H 7325 4800 50  0000 L CNN
 F 2 "TinyTiM_Lib:c_0805" H 7300 4900 50  0001 C CNN
@@
 $EndComp
 $Comp
-L C2 C?
+L C2 C15
 U 1 1 5424DFD9
 P 8700 4900
-F 0 "C?" H 8725 5000 50  0000 L CNN
+F 0 "C15" H 8725 5000 50  0000 L CNN
 F 1 "100n" H 8725 4800 50  0000 L CNN
 F 2 "TinyTiM_Lib:c_0805" H 8700 4900 50  0001 C CNN
@@
 $EndComp
 $Comp
-L C2 C?
+L C2 C17
 U 1 1 5424DFE7
 P 10100 4900
-F 0 "C?" H 10125 5000 50  0000 L CNN
+F 0 "C17" H 10125 5000 50  0000 L CNN
 F 1 "100n" H 10125 4800 50  0000 L CNN
 F 2 "TinyTiM_Lib:c_0805" H 10100 4900 50  0001 C CNN
@@
 Connection ~ 3100 5100
 Connection ~ 3100 4700
+Connection ~ 1250 2350
 $EndSCHEMATC

Commit message: Schematic updated
Changed lines of the file:
@@
 Sheet 2 14
 Title "ClockFOUR"
-Date "29 sep 2014"
+Date "30 sep 2014"
 Rev ""
 Comp "WyoLum"
@@
 5V
 $Comp
-L GND #PWR6
+L GND #PWR012
 U 1 1 5116893B
 P 1150 2400
-F 0 "#PWR6" H 1150 2400 30  0001 C CNN
+F 0 "#PWR012" H 1150 2400 30  0001 C CNN
 F 1 "GND" H 1150 2330 30  0001 C CNN
 F 2 "" H 1150 2400 60  0001 C CNN
@@
 Connection ~ 3100 4700
 Connection ~ 1250 2350
+Connection ~ 10000 5100
 $EndSCHEMATC

Commit message: Schematic updated, board started
Parts:
- C11: renamed from C101; Field5 100nF, 25V -> 100n, 25V
- C13: renamed from C8; Field5 100nF, 25V -> 100n, 25V
- C15: renamed from C12; Field5 100nF, 25V -> 100n, 25V
- C17: renamed from C16; Field5 100nF, 25V -> 100n, 25V
- C19: renamed from C7; Field5 100nF, 25V -> 100n, 25V
- C21: renamed from C11; Field5 100nF, 25V -> 100n, 25V
- C23: renamed from C15; Field5 100nF, 25V -> 100n, 25V
- U2: renamed from U3; footprint (none) -> ~
- renumbered C6 to C12, C10 to C14, C14 to C16, C5 to C18, C9 to C20, C13 to C22, C17 to C24, U6 to U10, U8 to U11, U10 to U12, U12 to U13, U16 to U15, U5 to U3, U7 to U4, U9 to U5, U11 to U6, U13 to U7, U15 to U8, U4 to U9
Changed lines of the file:
@@
 LIBS:contrib
 LIBS:valves
-LIBS:TinyTiM-cache
-LIBS:TiNA_sym
+LIBS:ClockFOUR
 LIBS:ClockFOUR-cache
 EELAYER 27 0
@@
 Sheet 2 14
 Title "ClockFOUR"
-Date "30 sep 2014"
+Date "1 oct 2014"
 Rev ""
 Comp "WyoLum"
@@
 5V
 $Comp
-L GND #PWR012
+L GND #PWR014
 U 1 1 5116893B
 P 1150 2400
-F 0 "#PWR012" H 1150 2400 30  0001 C CNN
+F 0 "#PWR014" H 1150 2400 30  0001 C CNN
 F 1 "GND" H 1150 2330 30  0001 C CNN
 F 2 "" H 1150 2400 60  0001 C CNN
@@
 $EndComp
 $Comp
-L C2 C101
+L C2 C11
 U 1 1 5118AB57
 P 1700 2550
-F 0 "C101" H 1725 2650 50  0000 L CNN
+F 0 "C11" H 1725 2650 50  0000 L CNN
 F 1 "100n" H 1725 2450 50  0000 L CNN
 F 2 "TinyTiM_Lib:c_0805" H 1700 2550 50  0001 C CNN
 F 3 "" H 1700 2550 60  0001 C CNN
 F 4 "CAP CER 0.1UF 25V 10% X7R 0805" H 1700 2750 60  0001 L CNN "Field4"
-F 5 "100nF, 25V" H 1700 2850 60  0001 L CNN "Field5"
+F 5 "100n, 25V" H 1700 2850 60  0001 L CNN "Field5"
 F 6 "Surface Mount, MLCC" H 1700 2950 60  0001 L CNN "Field6"
 F 7 "Kemet" H 1700 3050 60  0001 L CNN "Field7"
@@
 $EndComp
 $Comp
-L RGB_WS2812B U3
+L RGB_WS2812B U2
 U 1 1 5424CDC4
 P 1525 1575
-F 0 "U3" V 1275 1575 60  0000 C CNN
+F 0 "U2" V 1275 1575 60  0000 C CNN
 F 1 "RGB_WS2812B" V 1925 1575 60  0000 C CNN
-F 2 "" H 1525 1575 60  0000 C CNN
+F 2 "~" H 1525 1575 60  0000 C CNN
 F 3 "" H 1525 1575 60  0000 C CNN
 	1    1525 1575
@@
 $EndComp
 $Comp
-L RGB_WS2812B U5
+L RGB_WS2812B U3
 U 1 1 5424CE47
 P 2925 1575
-F 0 "U5" V 2675 1575 60  0000 C CNN
+F 0 "U3" V 2675 1575 60  0000 C CNN
 F 1 "RGB_WS2812B" V 3325 1575 60  0000 C CNN
 F 2 "" H 2925 1575 60  0000 C CNN
@@
 $EndComp
 $Comp
-L RGB_WS2812B U7
+L RGB_WS2812B U4
 U 1 1 5424CE4D
 P 4325 1575
-F 0 "U7" V 4075 1575 60  0000 C CNN
+F 0 "U4" V 4075 1575 60  0000 C CNN
 F 1 "RGB_WS2812B" V 4725 1575 60  0000 C CNN
 F 2 "" H 4325 1575 60  0000 C CNN
@@
 $EndComp
 $Comp
-L RGB_WS2812B U9
+L RGB_WS2812B U5
 U 1 1 5424CE53
 P 5725 1575
-F 0 "U9" V 5475 1575 60  0000 C CNN
+F 0 "U5" V 5475 1575 60  0000 C CNN
 F 1 "RGB_WS2812B" V 6125 1575 60  0000 C CNN
 F 2 "" H 5725 1575 60  0000 C CNN
@@
 $EndComp
 $Comp
-L RGB_WS2812B U11
+L RGB_WS2812B U6
 U 1 1 5424CE59
 P 7125 1575
-F 0 "U11" V 6875 1575 60  0000 C CNN
+F 0 "U6" V 6875 1575 60  0000 C CNN
 F 1 "RGB_WS2812B" V 7525 1575 60  0000 C CNN
 F 2 "" H 7125 1575 60  0000 C CNN
@@
 $EndComp
 $Comp
-L RGB_WS2812B U13
+L RGB_WS2812B U7
 U 1 1 5424CE5F
 P 8525 1575
-F 0 "U13" V 8275 1575 60  0000 C CNN
+F 0 "U7" V 8275 1575 60  0000 C CNN
 F 1 "RGB_WS2812B" V 8925 1575 60  0000 C CNN
 F 2 "" H 8525 1575 60  0000 C CNN
@@
 $EndComp
 $Comp
-L RGB_WS2812B U15
+L RGB_WS2812B U8
 U 1 1 5424CE65
 P 9925 1575
-F 0 "U15" V 9675 1575 60  0000 C CNN
+F 0 "U8" V 9675 1575 60  0000 C CNN
 F 1 "RGB_WS2812B" V 10325 1575 60  0000 C CNN
 F 2 "" H 9925 1575 60  0000 C CNN
@@
 $EndComp
 $Comp
-L RGB_WS2812B U4
+L RGB_WS2812B U9
 U 1 1 5424CE6B
 P 1525 3975
-F 0 "U4" V 1275 3975 60  0000 C CNN
+F 0 "U9" V 1275 3975 60  0000 C CNN
 F 1 "RGB_WS2812B" V 1925 3975 60  0000 C CNN
 F 2 "" H 1525 3975 60  0000 C CNN
@@
 $EndComp
 $Comp
-L RGB_WS2812B U6
+L RGB_WS2812B U10
 U 1 1 5424CE71
 P 2925 3975
-F 0 "U6" V 2675 3975 60  0000 C CNN
+F 0 "U10" V 2675 3975 60  0000 C CNN
 F 1 "RGB_WS2812B" V 3325 3975 60  0000 C CNN
 F 2 "" H 2925 3975 60  0000 C CNN
@@
 $EndComp
 $Comp
-L RGB_WS2812B U8
+L RGB_WS2812B U11
 U 1 1 5424CE77
 P 4325 3975
-F 0 "U8" V 4075 3975 60  0000 C CNN
+F 0 "U11" V 4075 3975 60  0000 C CNN
 F 1 "RGB_WS2812B" V 4725 3975 60  0000 C CNN
 F 2 "" H 4325 3975 60  0000 C CNN
@@
 $EndComp
 $Comp
-L RGB_WS2812B U10
+L RGB_WS2812B U12
 U 1 1 5424CE7D
 P 5725 3975
-F 0 "U10" V 5475 3975 60  0000 C CNN
+F 0 "U12" V 5475 3975 60  0000 C CNN
 F 1 "RGB_WS2812B" V 6125 3975 60  0000 C CNN
 F 2 "" H 5725 3975 60  0000 C CNN
@@
 $EndComp
 $Comp
-L RGB_WS2812B U12
+L RGB_WS2812B U13
 U 1 1 5424CE83
 P 7125 3975
-F 0 "U12" V 6875 3975 60  0000 C CNN
+F 0 "U13" V 6875 3975 60  0000 C CNN
 F 1 "RGB_WS2812B" V 7525 3975 60  0000 C CNN
 F 2 "" H 7125 3975 60  0000 C CNN
@@
 $EndComp
 $Comp
-L RGB_WS2812B U16
+L RGB_WS2812B U15
 U 1 1 5424CE8F
 P 9925 3975
-F 0 "U16" V 9675 3975 60  0000 C CNN
+F 0 "U15" V 9675 3975 60  0000 C CNN
 F 1 "RGB_WS2812B" V 10325 3975 60  0000 C CNN
 F 2 "" H 9925 3975 60  0000 C CNN
@@
 Connection ~ 1600 2750
 $Comp
-L C2 C6
+L C2 C12
 U 1 1 5424D6B9
 P 3100 2550
-F 0 "C6" H 3125 2650 50  0000 L CNN
+F 0 "C12" H 3125 2650 50  0000 L CNN
 F 1 "100n" H 3125 2450 50  0000 L CNN
 F 2 "TinyTiM_Lib:c_0805" H 3100 2550 50  0001 C CNN
@@
 $EndComp
 $Comp
-L C2 C8
+L C2 C13
 U 1 1 5424D6C7
 P 4500 2550
-F 0 "C8" H 4525 2650 50  0000 L CNN
+F 0 "C13" H 4525 2650 50  0000 L CNN
 F 1 "100n" H 4525 2450 50  0000 L CNN
 F 2 "TinyTiM_Lib:c_0805" H 4500 2550 50  0001 C CNN
 F 3 "" H 4500 2550 60  0001 C CNN
 F 4 "CAP CER 0.1UF 25V 10% X7R 0805" H 4500 2750 60  0001 L CNN "Field4"
-F 5 "100nF, 25V" H 4500 2850 60  0001 L CNN "Field5"
+F 5 "100n, 25V" H 4500 2850 60  0001 L CNN "Field5"
 F 6 "Surface Mount, MLCC" H 4500 2950 60  0001 L CNN "Field6"
 F 7 "Kemet" H 4500 3050 60  0001 L CNN "Field7"
@@
 $EndComp
 $Comp
-L C2 C10
+L C2 C14
 U 1 1 5424D6D5
 P 5900 2550
-F 0 "C10" H 5925 2650 50  0000 L CNN
+F 0 "C14" H 5925 2650 50  0000 L CNN
 F 1 "100n" H 5925 2450 50  0000 L CNN
 F 2 "TinyTiM_Lib:c_0805" H 5900 2550 50  0001 C CNN
@@
 $EndComp
 $Comp
-L C2 C12
+L C2 C15
 U 1 1 5424D6E3
 P 7300 2550
-F 0 "C12" H 7325 2650 50  0000 L CNN
+F 0 "C15" H 7325 2650 50  0000 L CNN
 F 1 "100n" H 7325 2450 50  0000 L CNN
 F 2 "TinyTiM_Lib:c_0805" H 7300 2550 50  0001 C CNN
 F 3 "" H 7300 2550 60  0001 C CNN
 F 4 "CAP CER 0.1UF 25V 10% X7R 0805" H 7300 2750 60  0001 L CNN "Field4"
-F 5 "100nF, 25V" H 7300 2850 60  0001 L CNN "Field5"
+F 5 "100n, 25V" H 7300 2850 60  0001 L CNN "Field5"
 F 6 "Surface Mount, MLCC" H 7300 2950 60  0001 L CNN "Field6"
 F 7 "Kemet" H 7300 3050 60  0001 L CNN "Field7"
@@
 $EndComp
 $Comp
-L C2 C14
+L C2 C16
 U 1 1 5424D6F1
 P 8700 2550
-F 0 "C14" H 8725 2650 50  0000 L CNN
+F 0 "C16" H 8725 2650 50  0000 L CNN
 F 1 "100n" H 8725 2450 50  0000 L CNN
 F 2 "TinyTiM_Lib:c_0805" H 8700 2550 50  0001 C CNN
@@
 $EndComp
 $Comp
-L C2 C16
+L C2 C17
 U 1 1 5424D6FF
 P 10100 2550
-F 0 "C16" H 10125 2650 50  0000 L CNN
+F 0 "C17" H 10125 2650 50  0000 L CNN
 F 1 "100n" H 10125 2450 50  0000 L CNN
 F 2 "TinyTiM_Lib:c_0805" H 10100 2550 50  0001 C CNN
 F 3 "" H 10100 2550 60  0001 C CNN
 F 4 "CAP CER 0.1UF 25V 10% X7R 0805" H 10100 2750 60  0001 L CNN "Field4"
-F 5 "100nF, 25V" H 10100 2850 60  0001 L CNN "Field5"
+F 5 "100n, 25V" H 10100 2850 60  0001 L CNN "Field5"
 F 6 "Surface Mount, MLCC" H 10100 2950 60  0001 L CNN "Field6"
 F 7 "Kemet" H 10100 3050 60  0001 L CNN "Field7"
@@
 Connection ~ 10000 2750
 $Comp
-L C2 C5
+L C2 C18
 U 1 1 5424D75D
 P 1700 4900
-F 0 "C5" H 1725 5000 50  0000 L CNN
+F 0 "C18" H 1725 5000 50  0000 L CNN
 F 1 "100n" H 1725 4800 50  0000 L CNN
 F 2 "TinyTiM_Lib:c_0805" H 1700 4900 50  0001 C CNN
@@
 Connection ~ 1600 5100
 $Comp
-L C2 C7
+L C2 C19
 U 1 1 5424DFA1
 P 3100 4900
-F 0 "C7" H 3125 5000 50  0000 L CNN
+F 0 "C19" H 3125 5000 50  0000 L CNN
 F 1 "100n" H 3125 4800 50  0000 L CNN
 F 2 "TinyTiM_Lib:c_0805" H 3100 4900 50  0001 C CNN
 F 3 "" H 3100 4900 60  0001 C CNN
 F 4 "CAP CER 0.1UF 25V 10% X7R 0805" H 3100 5100 60  0001 L CNN "Field4"
-F 5 "100nF, 25V" H 3100 5200 60  0001 L CNN "Field5"
+F 5 "100n, 25V" H 3100 5200 60  0001 L CNN "Field5"
 F 6 "Surface Mount, MLCC" H 3100 5300 60  0001 L CNN "Field6"
 F 7 "Kemet" H 3100 5400 60  0001 L CNN "Field7"
@@
 $EndComp
 $Comp
-L C2 C9
+L C2 C20
 U 1 1 5424DFAF
 P 4500 4900
-F 0 "C9" H 4525 5000 50  0000 L CNN
+F 0 "C20" H 4525 5000 50  0000 L CNN
 F 1 "100n" H 4525 4800 50  0000 L CNN
 F 2 "TinyTiM_Lib:c_0805" H 4500 4900 50  0001 C CNN
@@
 $EndComp
 $Comp
-L C2 C11
+L C2 C21
 U 1 1 5424DFBD
 P 5900 4900
-F 0 "C11" H 5925 5000 50  0000 L CNN
+F 0 "C21" H 5925 5000 50  0000 L CNN
 F 1 "100n" H 5925 4800 50  0000 L CNN
 F 2 "TinyTiM_Lib:c_0805" H 5900 4900 50  0001 C CNN
 F 3 "" H 5900 4900 60  0001 C CNN
 F 4 "CAP CER 0.1UF 25V 10% X7R 0805" H 5900 5100 60  0001 L CNN "Field4"
-F 5 "100nF, 25V" H 5900 5200 60  0001 L CNN "Field5"
+F 5 "100n, 25V" H 5900 5200 60  0001 L CNN "Field5"
 F 6 "Surface Mount, MLCC" H 5900 5300 60  0001 L CNN "Field6"
 F 7 "Kemet" H 5900 5400 60  0001 L CNN "Field7"
@@
 $EndComp
 $Comp
-L C2 C13
+L C2 C22
 U 1 1 5424DFCB
 P 7300 4900
-F 0 "C13" H 7325 5000 50  0000 L CNN
+F 0 "C22" H 7325 5000 50  0000 L CNN
 F 1 "100n" H 7325 4800 50  0000 L CNN
 F 2 "TinyTiM_Lib:c_0805" H 7300 4900 50  0001 C CNN
@@
 $EndComp
 $Comp
-L C2 C15
+L C2 C23
 U 1 1 5424DFD9
 P 8700 4900
-F 0 "C15" H 8725 5000 50  0000 L CNN
+F 0 "C23" H 8725 5000 50  0000 L CNN
 F 1 "100n" H 8725 4800 50  0000 L CNN
 F 2 "TinyTiM_Lib:c_0805" H 8700 4900 50  0001 C CNN
 F 3 "" H 8700 4900 60  0001 C CNN
 F 4 "CAP CER 0.1UF 25V 10% X7R 0805" H 8700 5100 60  0001 L CNN "Field4"
-F 5 "100nF, 25V" H 8700 5200 60  0001 L CNN "Field5"
+F 5 "100n, 25V" H 8700 5200 60  0001 L CNN "Field5"
 F 6 "Surface Mount, MLCC" H 8700 5300 60  0001 L CNN "Field6"
 F 7 "Kemet" H 8700 5400 60  0001 L CNN "Field7"
@@
 $EndComp
 $Comp
-L C2 C17
+L C2 C24
 U 1 1 5424DFE7
 P 10100 4900
-F 0 "C17" H 10125 5000 50  0000 L CNN
+F 0 "C24" H 10125 5000 50  0000 L CNN
 F 1 "100n" H 10125 4800 50  0000 L CNN
 F 2 "TinyTiM_Lib:c_0805" H 10100 4900 50  0001 C CNN
