File: KiCad/Row_A.sch (KiCad schematic (older format))
At the start: 28 parts

Commit message: PCB layout, work in progress
Parts:
- C12, C13, C14, C15, C16, C17, C18, C19, C20, C21, C22, C23, C24, C25: footprint TinyTiM_Lib:c_0805 -> C4_Pretty:c_0805
- LED1, LED10, LED11, LED12, LED13, LED14, LED2, LED3, LED4, LED5, LED6, LED7, LED8, LED9: footprint ~ -> C4_Pretty:RGB_WS2811B
Changed lines of the file:
@@
 F 0 "C12" H 1725 2650 50  0000 L CNN
 F 1 "100n" H 1725 2450 50  0000 L CNN
-F 2 "TinyTiM_Lib:c_0805" H 1700 2550 50  0001 C CNN
+F 2 "C4_Pretty:c_0805" H 1700 2550 50  0001 C CNN
 F 3 "" H 1700 2550 60  0001 C CNN
 F 4 "CAP CER 0.1UF 25V 10% X7R 0805" H 1700 2750 60  0001 L CNN "Field4"
@@
 F 0 "C13" H 3125 2650 50  0000 L CNN
 F 1 "100n" H 3125 2450 50  0000 L CNN
-F 2 "TinyTiM_Lib:c_0805" H 3100 2550 50  0001 C CNN
+F 2 "C4_Pretty:c_0805" H 3100 2550 50  0001 C CNN
 F 3 "" H 3100 2550 60  0001 C CNN
 F 4 "CAP CER 0.1UF 25V 10% X7R 0805" H 3100 2750 60  0001 L CNN "Field4"
@@
 F 0 "C14" H 4525 2650 50  0000 L CNN
 F 1 "100n" H 4525 2450 50  0000 L CNN
-F 2 "TinyTiM_Lib:c_0805" H 4500 2550 50  0001 C CNN
+F 2 "C4_Pretty:c_0805" H 4500 2550 50  0001 C CNN
 F 3 "" H 4500 2550 60  0001 C CNN
 F 4 "CAP CER 0.1UF 25V 10% X7R 0805" H 4500 2750 60  0001 L CNN "Field4"
@@
 F 0 "C15" H 5925 2650 50  0000 L CNN
 F 1 "100n" H 5925 2450 50  0000 L CNN
-F 2 "TinyTiM_Lib:c_0805" H 5900 2550 50  0001 C CNN
+F 2 "C4_Pretty:c_0805" H 5900 2550 50  0001 C CNN
 F 3 "" H 5900 2550 60  0001 C CNN
 F 4 "CAP CER 0.1UF 25V 10% X7R 0805" H 5900 2750 60  0001 L CNN "Field4"
@@
 F 0 "C16" H 7325 2650 50  0000 L CNN
 F 1 "100n" H 7325 2450 50  0000 L CNN
-F 2 "TinyTiM_Lib:c_0805" H 7300 2550 50  0001 C CNN
+F 2 "C4_Pretty:c_0805" H 7300 2550 50  0001 C CNN
 F 3 "" H 7300 2550 60  0001 C CNN
 F 4 "CAP CER 0.1UF 25V 10% X7R 0805" H 7300 2750 60  0001 L CNN "Field4"
@@
 F 0 "C17" H 8725 2650 50  0000 L CNN
 F 1 "100n" H 8725 2450 50  0000 L CNN
-F 2 "TinyTiM_Lib:c_0805" H 8700 2550 50  0001 C CNN
+F 2 "C4_Pretty:c_0805" H 8700 2550 50  0001 C CNN
 F 3 "" H 8700 2550 60  0001 C CNN
 F 4 "CAP CER 0.1UF 25V 10% X7R 0805" H 8700 2750 60  0001 L CNN "Field4"
@@
 F 0 "C18" H 10125 2650 50  0000 L CNN
 F 1 "100n" H 10125 2450 50  0000 L CNN
-F 2 "TinyTiM_Lib:c_0805" H 10100 2550 50  0001 C CNN
+F 2 "C4_Pretty:c_0805" H 10100 2550 50  0001 C CNN
 F 3 "" H 10100 2550 60  0001 C CNN
 F 4 "CAP CER 0.1UF 25V 10% X7R 0805" H 10100 2750 60  0001 L CNN "Field4"
@@
 F 0 "C19" H 1725 5000 50  0000 L CNN
 F 1 "100n" H 1725 4800 50  0000 L CNN
-F 2 "TinyTiM_Lib:c_0805" H 1700 4900 50  0001 C CNN
+F 2 "C4_Pretty:c_0805" H 1700 4900 50  0001 C CNN
 F 3 "" H 1700 4900 60  0001 C CNN
 F 4 "CAP CER 0.1UF 25V 10% X7R 0805" H 1700 5100 60  0001 L CNN "Field4"
@@
 F 0 "C20" H 3125 5000 50  0000 L CNN
 F 1 "100n" H 3125 4800 50  0000 L CNN
-F 2 "TinyTiM_Lib:c_0805" H 3100 4900 50  0001 C CNN
+F 2 "C4_Pretty:c_0805" H 3100 4900 50  0001 C CNN
 F 3 "" H 3100 4900 60  0001 C CNN
 F 4 "CAP CER 0.1UF 25V 10% X7R 0805" H 3100 5100 60  0001 L CNN "Field4"
@@
 F 0 "C21" H 4525 5000 50  0000 L CNN
 F 1 "100n" H 4525 4800 50  0000 L CNN
-F 2 "TinyTiM_Lib:c_0805" H 4500 4900 50  0001 C CNN
+F 2 "C4_Pretty:c_0805" H 4500 4900 50  0001 C CNN
 F 3 "" H 4500 4900 60  0001 C CNN
 F 4 "CAP CER 0.1UF 25V 10% X7R 0805" H 4500 5100 60  0001 L CNN "Field4"
@@
 F 0 "C22" H 5925 5000 50  0000 L CNN
 F 1 "100n" H 5925 4800 50  0000 L CNN
-F 2 "TinyTiM_Lib:c_0805" H 5900 4900 50  0001 C CNN
+F 2 "C4_Pretty:c_0805" H 5900 4900 50  0001 C CNN
 F 3 "" H 5900 4900 60  0001 C CNN
 F 4 "CAP CER 0.1UF 25V 10% X7R 0805" H 5900 5100 60  0001 L CNN "Field4"
@@
 F 0 "C23" H 7325 5000 50  0000 L CNN
 F 1 "100n" H 7325 4800 50  0000 L CNN
-F 2 "TinyTiM_Lib:c_0805" H 7300 4900 50  0001 C CNN
+F 2 "C4_Pretty:c_0805" H 7300 4900 50  0001 C CNN
 F 3 "" H 7300 4900 60  0001 C CNN
 F 4 "CAP CER 0.1UF 25V 10% X7R 0805" H 7300 5100 60  0001 L CNN "Field4"
@@
 F 0 "C24" H 8725 5000 50  0000 L CNN
 F 1 "100n" H 8725 4800 50  0000 L CNN
-F 2 "TinyTiM_Lib:c_0805" H 8700 4900 50  0001 C CNN
+F 2 "C4_Pretty:c_0805" H 8700 4900 50  0001 C CNN
 F 3 "" H 8700 4900 60  0001 C CNN
 F 4 "CAP CER 0.1UF 25V 10% X7R 0805" H 8700 5100 60  0001 L CNN "Field4"
@@
 F 0 "C25" H 10125 5000 50  0000 L CNN
 F 1 "100n" H 10125 4800 50  0000 L CNN
-F 2 "TinyTiM_Lib:c_0805" H 10100 4900 50  0001 C CNN
+F 2 "C4_Pretty:c_0805" H 10100 4900 50  0001 C CNN
 F 3 "" H 10100 4900 60  0001 C CNN
 F 4 "CAP CER 0.1UF 25V 10% X7R 0805" H 10100 5100 60  0001 L CNN "Field4"
@@
 F 0 "LED1" V 1275 1575 60  0000 C CNN
 F 1 "WS2812B" V 1925 1575 60  0001 C CNN
-F 2 "~" H 1525 1575 60  0000 C CNN
+F 2 "C4_Pretty:RGB_WS2811B" H 1525 1575 60  0001 C CNN
 F 3 "~" H 1525 1575 60  0000 C CNN
 	1    1525 1575
@@
 F 0 "LED2" V 2675 1575 60  0000 C CNN
 F 1 "WS2812B" V 3325 1575 60  0001 C CNN
-F 2 "~" H 2925 1575 60  0000 C CNN
+F 2 "C4_Pretty:RGB_WS2811B" H 2925 1575 60  0001 C CNN
 F 3 "~" H 2925 1575 60  0000 C CNN
 	1    2925 1575
@@
 F 0 "LED3" V 4075 1575 60  0000 C CNN
 F 1 "WS2812B" V 4725 1575 60  0001 C CNN
-F 2 "~" H 4325 1575 60  0000 C CNN
+F 2 "C4_Pretty:RGB_WS2811B" H 4325 1575 60  0001 C CNN
 F 3 "~" H 4325 1575 60  0000 C CNN
 	1    4325 1575
@@
 F 0 "LED4" V 5475 1575 60  0000 C CNN
 F 1 "WS2812B" V 6125 1575 60  0001 C CNN
-F 2 "~" H 5725 1575 60  0000 C CNN
+F 2 "C4_Pretty:RGB_WS2811B" H 5725 1575 60  0001 C CNN
 F 3 "~" H 5725 1575 60  0000 C CNN
 	1    5725 1575
@@
 F 0 "LED5" V 6875 1575 60  0000 C CNN
 F 1 "WS2812B" V 7525 1575 60  0001 C CNN
-F 2 "~" H 7125 1575 60  0000 C CNN
+F 2 "C4_Pretty:RGB_WS2811B" H 7125 1575 60  0001 C CNN
 F 3 "~" H 7125 1575 60  0000 C CNN
 	1    7125 1575
@@
 F 0 "LED6" V 8275 1575 60  0000 C CNN
 F 1 "WS2812B" V 8925 1575 60  0001 C CNN
-F 2 "~" H 8525 1575 60  0000 C CNN
+F 2 "C4_Pretty:RGB_WS2811B" H 8525 1575 60  0001 C CNN
 F 3 "~" H 8525 1575 60  0000 C CNN
 	1    8525 1575
@@
 F 0 "LED7" V 9675 1575 60  0000 C CNN
 F 1 "WS2812B" V 10325 1575 60  0001 C CNN
-F 2 "~" H 9925 1575 60  0000 C CNN
+F 2 "C4_Pretty:RGB_WS2811B" H 9925 1575 60  0001 C CNN
 F 3 "~" H 9925 1575 60  0000 C CNN
 	1    9925 1575
@@
 F 0 "LED8" V 1275 3975 60  0000 C CNN
 F 1 "WS2812B" V 1925 3975 60  0001 C CNN
-F 2 "~" H 1525 3975 60  0000 C CNN
+F 2 "C4_Pretty:RGB_WS2811B" H 1525 3975 60  0001 C CNN
 F 3 "~" H 1525 3975 60  0000 C CNN
 	1    1525 3975
@@
 F 0 "LED9" V 2675 3975 60  0000 C CNN
 F 1 "WS2812B" V 3325 3975 60  0001 C CNN
-F 2 "~" H 2925 3975 60  0000 C CNN
+F 2 "C4_Pretty:RGB_WS2811B" H 2925 3975 60  0001 C CNN
 F 3 "~" H 2925 3975 60  0000 C CNN
 	1    2925 3975
@@
 F 0 "LED10" V 4075 3975 60  0000 C CNN
 F 1 "WS2812B" V 4725 3975 60  0001 C CNN
-F 2 "~" H 4325 3975 60  0000 C CNN
+F 2 "C4_Pretty:RGB_WS2811B" H 4325 3975 60  0001 C CNN
 F 3 "~" H 4325 3975 60  0000 C CNN
 	1    4325 3975
@@
 F 0 "LED11" V 5475 3975 60  0000 C CNN
 F 1 "WS2812B" V 6125 3975 60  0001 C CNN
-F 2 "~" H 5725 3975 60  0000 C CNN
+F 2 "C4_Pretty:RGB_WS2811B" H 5725 3975 60  0001 C CNN
 F 3 "~" H 5725 3975 60  0000 C CNN
 	1    5725 3975
@@
 F 0 "LED12" V 6875 3975 60  0000 C CNN
 F 1 "WS2812B" V 7525 3975 60  0001 C CNN
-F 2 "~" H 7125 3975 60  0000 C CNN
+F 2 "C4_Pretty:RGB_WS2811B" H 7125 3975 60  0001 C CNN
 F 3 "~" H 7125 3975 60  0000 C CNN
 	1    7125 3975
@@
 F 0 "LED13" V 8275 3975 60  0000 C CNN
 F 1 "WS2812B" V 8925 3975 60  0001 C CNN
-F 2 "~" H 8525 3975 60  0000 C CNN
+F 2 "C4_Pretty:RGB_WS2811B" H 8525 3975 60  0001 C CNN
 F 3 "~" H 8525 3975 60  0000 C CNN
 	1    8525 3975
@@
 F 0 "LED14" V 9675 3975 60  0000 C CNN
 F 1 "WS2812B" V 10325 3975 60  0001 C CNN
-F 2 "~" H 9925 3975 60  0000 C CNN
+F 2 "C4_Pretty:RGB_WS2811B" H 9925 3975 60  0001 C CNN
 F 3 "~" H 9925 3975 60  0000 C CNN
 	1    9925 3975

Commit message: C4 PCB layout complete. Added Gerbers
Parts:
- C12, C13, C14, C15, C16, C17, C18, C19, C20, C21, C22, C23, C24, C25: footprint C4_Pretty:c_0805 -> C4_Pretty:c_0805_led
Changed lines of the file:
@@
 EESchema Schematic File Version 2
 LIBS:ClockFOUR
+LIBS:RowGB_sym
 LIBS:ClockFOUR-cache
 EELAYER 24 0
@@
 F 0 "C12" H 1725 2650 50  0000 L CNN
 F 1 "100n" H 1725 2450 50  0000 L CNN
-F 2 "C4_Pretty:c_0805" H 1700 2550 50  0001 C CNN
+F 2 "C4_Pretty:c_0805_led" H 1700 2550 50  0001 C CNN
 F 3 "" H 1700 2550 60  0001 C CNN
 F 4 "CAP CER 0.1UF 25V 10% X7R 0805" H 1700 2750 60  0001 L CNN "Field4"
@@
 F 0 "C13" H 3125 2650 50  0000 L CNN
 F 1 "100n" H 3125 2450 50  0000 L CNN
-F 2 "C4_Pretty:c_0805" H 3100 2550 50  0001 C CNN
+F 2 "C4_Pretty:c_0805_led" H 3100 2550 50  0001 C CNN
 F 3 "" H 3100 2550 60  0001 C CNN
 F 4 "CAP CER 0.1UF 25V 10% X7R 0805" H 3100 2750 60  0001 L CNN "Field4"
@@
 F 0 "C14" H 4525 2650 50  0000 L CNN
 F 1 "100n" H 4525 2450 50  0000 L CNN
-F 2 "C4_Pretty:c_0805" H 4500 2550 50  0001 C CNN
+F 2 "C4_Pretty:c_0805_led" H 4500 2550 50  0001 C CNN
 F 3 "" H 4500 2550 60  0001 C CNN
 F 4 "CAP CER 0.1UF 25V 10% X7R 0805" H 4500 2750 60  0001 L CNN "Field4"
@@
 F 0 "C15" H 5925 2650 50  0000 L CNN
 F 1 "100n" H 5925 2450 50  0000 L CNN
-F 2 "C4_Pretty:c_0805" H 5900 2550 50  0001 C CNN
+F 2 "C4_Pretty:c_0805_led" H 5900 2550 50  0001 C CNN
 F 3 "" H 5900 2550 60  0001 C CNN
 F 4 "CAP CER 0.1UF 25V 10% X7R 0805" H 5900 2750 60  0001 L CNN "Field4"
@@
 F 0 "C16" H 7325 2650 50  0000 L CNN
 F 1 "100n" H 7325 2450 50  0000 L CNN
-F 2 "C4_Pretty:c_0805" H 7300 2550 50  0001 C CNN
+F 2 "C4_Pretty:c_0805_led" H 7300 2550 50  0001 C CNN
 F 3 "" H 7300 2550 60  0001 C CNN
 F 4 "CAP CER 0.1UF 25V 10% X7R 0805" H 7300 2750 60  0001 L CNN "Field4"
@@
 F 0 "C17" H 8725 2650 50  0000 L CNN
 F 1 "100n" H 8725 2450 50  0000 L CNN
-F 2 "C4_Pretty:c_0805" H 8700 2550 50  0001 C CNN
+F 2 "C4_Pretty:c_0805_led" H 8700 2550 50  0001 C CNN
 F 3 "" H 8700 2550 60  0001 C CNN
 F 4 "CAP CER 0.1UF 25V 10% X7R 0805" H 8700 2750 60  0001 L CNN "Field4"
@@
 F 0 "C18" H 10125 2650 50  0000 L CNN
 F 1 "100n" H 10125 2450 50  0000 L CNN
-F 2 "C4_Pretty:c_0805" H 10100 2550 50  0001 C CNN
+F 2 "C4_Pretty:c_0805_led" H 10100 2550 50  0001 C CNN
 F 3 "" H 10100 2550 60  0001 C CNN
 F 4 "CAP CER 0.1UF 25V 10% X7R 0805" H 10100 2750 60  0001 L CNN "Field4"
@@
 F 0 "C19" H 1725 5000 50  0000 L CNN
 F 1 "100n" H 1725 4800 50  0000 L CNN
-F 2 "C4_Pretty:c_0805" H 1700 4900 50  0001 C CNN
+F 2 "C4_Pretty:c_0805_led" H 1700 4900 50  0001 C CNN
 F 3 "" H 1700 4900 60  0001 C CNN
 F 4 "CAP CER 0.1UF 25V 10% X7R 0805" H 1700 5100 60  0001 L CNN "Field4"
@@
 F 0 "C20" H 3125 5000 50  0000 L CNN
 F 1 "100n" H 3125 4800 50  0000 L CNN
-F 2 "C4_Pretty:c_0805" H 3100 4900 50  0001 C CNN
+F 2 "C4_Pretty:c_0805_led" H 3100 4900 50  0001 C CNN
 F 3 "" H 3100 4900 60  0001 C CNN
 F 4 "CAP CER 0.1UF 25V 10% X7R 0805" H 3100 5100 60  0001 L CNN "Field4"
@@
 F 0 "C21" H 4525 5000 50  0000 L CNN
 F 1 "100n" H 4525 4800 50  0000 L CNN
-F 2 "C4_Pretty:c_0805" H 4500 4900 50  0001 C CNN
+F 2 "C4_Pretty:c_0805_led" H 4500 4900 50  0001 C CNN
 F 3 "" H 4500 4900 60  0001 C CNN
 F 4 "CAP CER 0.1UF 25V 10% X7R 0805" H 4500 5100 60  0001 L CNN "Field4"
@@
 F 0 "C22" H 5925 5000 50  0000 L CNN
 F 1 "100n" H 5925 4800 50  0000 L CNN
-F 2 "C4_Pretty:c_0805" H 5900 4900 50  0001 C CNN
+F 2 "C4_Pretty:c_0805_led" H 5900 4900 50  0001 C CNN
 F 3 "" H 5900 4900 60  0001 C CNN
 F 4 "CAP CER 0.1UF 25V 10% X7R 0805" H 5900 5100 60  0001 L CNN "Field4"
@@
 F 0 "C23" H 7325 5000 50  0000 L CNN
 F 1 "100n" H 7325 4800 50  0000 L CNN
-F 2 "C4_Pretty:c_0805" H 7300 4900 50  0001 C CNN
+F 2 "C4_Pretty:c_0805_led" H 7300 4900 50  0001 C CNN
 F 3 "" H 7300 4900 60  0001 C CNN
 F 4 "CAP CER 0.1UF 25V 10% X7R 0805" H 7300 5100 60  0001 L CNN "Field4"
@@
 F 0 "C24" H 8725 5000 50  0000 L CNN
 F 1 "100n" H 8725 4800 50  0000 L CNN
-F 2 "C4_Pretty:c_0805" H 8700 4900 50  0001 C CNN
+F 2 "C4_Pretty:c_0805_led" H 8700 4900 50  0001 C CNN
 F 3 "" H 8700 4900 60  0001 C CNN
 F 4 "CAP CER 0.1UF 25V 10% X7R 0805" H 8700 5100 60  0001 L CNN "Field4"
@@
 F 0 "C25" H 10125 5000 50  0000 L CNN
 F 1 "100n" H 10125 4800 50  0000 L CNN
-F 2 "C4_Pretty:c_0805" H 10100 4900 50  0001 C CNN
+F 2 "C4_Pretty:c_0805_led" H 10100 4900 50  0001 C CNN
 F 3 "" H 10100 4900 60  0001 C CNN
 F 4 "CAP CER 0.1UF 25V 10% X7R 0805" H 10100 5100 60  0001 L CNN "Field4"
