File: KiCad/Row_C.sch (KiCad schematic (older format))
At the start: 14 parts, among them U101 RGB_WS2811B, U102 RGB_WS2811B, U103 RGB_WS2811B, U104 RGB_WS2811B, U105 RGB_WS2811B, U106 RGB_WS2811B, U107 RGB_WS2811B, U108 RGB_WS2811B

Commit message: Schematic updated
Parts:
- removed C101: 100n, TinyTiM_Lib:c_0805, symbol C2
- removed C117: 47u,8V, TinyTiM_Lib:c_2917, symbol C_POL_1
- removed S101, S102, S103, S104: CONN_1, TinyTiM_Lib:Screw, symbol CONN_1
- removed U101, U102, U103, U104, U105, U106, U107, U108: RGB_WS2811B, TinyTiM_Lib:RGB_WS2811B, symbol RGB_WS2811B
Connections:
- net labels removed: 5V, A_02, A_03, A_04, A_05, A_06, A_07, A_08, A_09, DI_A, DO_A, GND
- wire segments 49 -> 0
- no-connect marks 4 -> 0
Other:
- note removed: "Mounting Screws"

Commit message: Schematic updated
Parts:
- added C37, C38, C39, C40, C41, C42, C43, C44, C45, C46, C47, C48, C49, C50: 100n, TinyTiM_Lib:c_0805, symbol C2
- added U32, U33, U34, U35, U36, U37, U38, U39, U40, U41, U42, U43, U44, U45: RGB_WS2812B, symbol RGB_WS2812B
Connections:
- net labels added: 5V, DI_C, DO_C, GND
- wire segments 0 -> 82

Commit message: Schematic updated, board started
Parts:
- C39: renamed from C37; Field5 100nF, 25V -> 100n, 25V
- C41: Field5 100nF, 25V -> 100n, 25V
- C43: renamed from C45; Field5 100nF, 25V -> 100n, 25V
- C45: renamed from C49; Field5 100nF, 25V -> 100n, 25V
- C47: renamed from C40; Field5 100nF, 25V -> 100n, 25V
- C49: renamed from C44; Field5 100nF, 25V -> 100n, 25V
- C51: renamed from C48; Field5 100nF, 25V -> 100n, 25V
- renumbered C39 to C40, C43 to C42, C47 to C44, C38 to C46, C42 to C48, C46 to C50, C50 to C52, U32 to U30, U34 to U31, U36 to U32, U38 to U33, U40 to U34, U42 to U35, U44 to U36, U33 to U37, U35 to U38, U37 to U39, U39 to U40, U43 to U42, U45 to U43
Changed lines of the file:
@@
 LIBS:contrib
 LIBS:valves
-LIBS:TinyTiM-cache
-LIBS:TiNA_sym
+LIBS:ClockFOUR
 LIBS:ClockFOUR-cache
 EELAYER 27 0
@@
 Sheet 4 14
 Title "ClockFOUR"
-Date "30 sep 2014"
+Date "1 oct 2014"
 Rev ""
 Comp "WyoLum"
@@
 5V
 $Comp
-L GND #PWR014
+L GND #PWR016
 U 1 1 542C08DE
 P 1400 2650
-F 0 "#PWR014" H 1400 2650 30  0001 C CNN
+F 0 "#PWR016" H 1400 2650 30  0001 C CNN
 F 1 "GND" H 1400 2580 30  0001 C CNN
 F 2 "" H 1400 2650 60  0001 C CNN
@@
 $EndComp
 $Comp
-L C2 C37
+L C2 C39
 U 1 1 542C08EC
 P 1950 2800
-F 0 "C37" H 1975 2900 50  0000 L CNN
+F 0 "C39" H 1975 2900 50  0000 L CNN
 F 1 "100n" H 1975 2700 50  0000 L CNN
 F 2 "TinyTiM_Lib:c_0805" H 1950 2800 50  0001 C CNN
 F 3 "" H 1950 2800 60  0001 C CNN
 F 4 "CAP CER 0.1UF 25V 10% X7R 0805" H 1950 3000 60  0001 L CNN "Field4"
-F 5 "100nF, 25V" H 1950 3100 60  0001 L CNN "Field5"
+F 5 "100n, 25V" H 1950 3100 60  0001 L CNN "Field5"
 F 6 "Surface Mount, MLCC" H 1950 3200 60  0001 L CNN "Field6"
 F 7 "Kemet" H 1950 3300 60  0001 L CNN "Field7"
@@
 $EndComp
 $Comp
-L RGB_WS2812B U32
+L RGB_WS2812B U30
 U 1 1 542C08F2
 P 1775 1825
-F 0 "U32" V 1525 1825 60  0000 C CNN
+F 0 "U30" V 1525 1825 60  0000 C CNN
 F 1 "RGB_WS2812B" V 2175 1825 60  0000 C CNN
 F 2 "" H 1775 1825 60  0000 C CNN
@@
 $EndComp
 $Comp
-L RGB_WS2812B U34
+L RGB_WS2812B U31
 U 1 1 542C08F8
 P 3175 1825
-F 0 "U34" V 2925 1825 60  0000 C CNN
+F 0 "U31" V 2925 1825 60  0000 C CNN
 F 1 "RGB_WS2812B" V 3575 1825 60  0000 C CNN
 F 2 "" H 3175 1825 60  0000 C CNN
@@
 $EndComp
 $Comp
-L RGB_WS2812B U36
+L RGB_WS2812B U32
 U 1 1 542C08FE
 P 4575 1825
-F 0 "U36" V 4325 1825 60  0000 C CNN
+F 0 "U32" V 4325 1825 60  0000 C CNN
 F 1 "RGB_WS2812B" V 4975 1825 60  0000 C CNN
 F 2 "" H 4575 1825 60  0000 C CNN
@@
 $EndComp
 $Comp
-L RGB_WS2812B U38
+L RGB_WS2812B U33
 U 1 1 542C0904
 P 5975 1825
-F 0 "U38" V 5725 1825 60  0000 C CNN
+F 0 "U33" V 5725 1825 60  0000 C CNN
 F 1 "RGB_WS2812B" V 6375 1825 60  0000 C CNN
 F 2 "" H 5975 1825 60  0000 C CNN
@@
 $EndComp
 $Comp
-L RGB_WS2812B U40
+L RGB_WS2812B U34
 U 1 1 542C090A
 P 7375 1825
-F 0 "U40" V 7125 1825 60  0000 C CNN
+F 0 "U34" V 7125 1825 60  0000 C CNN
 F 1 "RGB_WS2812B" V 7775 1825 60  0000 C CNN
 F 2 "" H 7375 1825 60  0000 C CNN
@@
 $EndComp
 $Comp
-L RGB_WS2812B U42
+L RGB_WS2812B U35
 U 1 1 542C0910
 P 8775 1825
-F 0 "U42" V 8525 1825 60  0000 C CNN
+F 0 "U35" V 8525 1825 60  0000 C CNN
 F 1 "RGB_WS2812B" V 9175 1825 60  0000 C CNN
 F 2 "" H 8775 1825 60  0000 C CNN
@@
 $EndComp
 $Comp
-L RGB_WS2812B U44
+L RGB_WS2812B U36
 U 1 1 542C0916
 P 10175 1825
-F 0 "U44" V 9925 1825 60  0000 C CNN
+F 0 "U36" V 9925 1825 60  0000 C CNN
 F 1 "RGB_WS2812B" V 10575 1825 60  0000 C CNN
 F 2 "" H 10175 1825 60  0000 C CNN
@@
 $EndComp
 $Comp
-L RGB_WS2812B U33
+L RGB_WS2812B U37
 U 1 1 542C091C
 P 1775 4225
-F 0 "U33" V 1525 4225 60  0000 C CNN
+F 0 "U37" V 1525 4225 60  0000 C CNN
 F 1 "RGB_WS2812B" V 2175 4225 60  0000 C CNN
 F 2 "" H 1775 4225 60  0000 C CNN
@@
 $EndComp
 $Comp
-L RGB_WS2812B U35
+L RGB_WS2812B U38
 U 1 1 542C0922
 P 3175 4225
-F 0 "U35" V 2925 4225 60  0000 C CNN
+F 0 "U38" V 2925 4225 60  0000 C CNN
 F 1 "RGB_WS2812B" V 3575 4225 60  0000 C CNN
 F 2 "" H 3175 4225 60  0000 C CNN
@@
 $EndComp
 $Comp
-L RGB_WS2812B U37
+L RGB_WS2812B U39
 U 1 1 542C0928
 P 4575 4225
-F 0 "U37" V 4325 4225 60  0000 C CNN
+F 0 "U39" V 4325 4225 60  0000 C CNN
 F 1 "RGB_WS2812B" V 4975 4225 60  0000 C CNN
 F 2 "" H 4575 4225 60  0000 C CNN
@@
 $EndComp
 $Comp
-L RGB_WS2812B U39
+L RGB_WS2812B U40
 U 1 1 542C092E
 P 5975 4225
-F 0 "U39" V 5725 4225 60  0000 C CNN
+F 0 "U40" V 5725 4225 60  0000 C CNN
 F 1 "RGB_WS2812B" V 6375 4225 60  0000 C CNN
 F 2 "" H 5975 4225 60  0000 C CNN
@@
 $EndComp
 $Comp
-L RGB_WS2812B U43
+L RGB_WS2812B U42
 U 1 1 542C093A
 P 8775 4225
-F 0 "U43" V 8525 4225 60  0000 C CNN
+F 0 "U42" V 8525 4225 60  0000 C CNN
 F 1 "RGB_WS2812B" V 9175 4225 60  0000 C CNN
 F 2 "" H 8775 4225 60  0000 C CNN
@@
 $EndComp
 $Comp
-L RGB_WS2812B U45
+L RGB_WS2812B U43
 U 1 1 542C0940
 P 10175 4225
-F 0 "U45" V 9925 4225 60  0000 C CNN
+F 0 "U43" V 9925 4225 60  0000 C CNN
 F 1 "RGB_WS2812B" V 10575 4225 60  0000 C CNN
 F 2 "" H 10175 4225 60  0000 C CNN
@@
 Connection ~ 1850 3000
 $Comp
-L C2 C39
+L C2 C40
 U 1 1 542C099B
 P 3350 2800
-F 0 "C39" H 3375 2900 50  0000 L CNN
+F 0 "C40" H 3375 2900 50  0000 L CNN
 F 1 "100n" H 3375 2700 50  0000 L CNN
 F 2 "TinyTiM_Lib:c_0805" H 3350 2800 50  0001 C CNN
@@
 F 3 "" H 4750 2800 60  0001 C CNN
 F 4 "CAP CER 0.1UF 25V 10% X7R 0805" H 4750 3000 60  0001 L CNN "Field4"
-F 5 "100nF, 25V" H 4750 3100 60  0001 L CNN "Field5"
+F 5 "100n, 25V" H 4750 3100 60  0001 L CNN "Field5"
 F 6 "Surface Mount, MLCC" H 4750 3200 60  0001 L CNN "Field6"
 F 7 "Kemet" H 4750 3300 60  0001 L CNN "Field7"
@@
 $EndComp
 $Comp
-L C2 C43
+L C2 C42
 U 1 1 542C09B7
 P 6150 2800
-F 0 "C43" H 6175 2900 50  0000 L CNN
+F 0 "C42" H 6175 2900 50  0000 L CNN
 F 1 "100n" H 6175 2700 50  0000 L CNN
 F 2 "TinyTiM_Lib:c_0805" H 6150 2800 50  0001 C CNN
@@
 $EndComp
 $Comp
-L C2 C45
+L C2 C43
 U 1 1 542C09C5
 P 7550 2800
-F 0 "C45" H 7575 2900 50  0000 L CNN
+F 0 "C43" H 7575 2900 50  0000 L CNN
 F 1 "100n" H 7575 2700 50  0000 L CNN
 F 2 "TinyTiM_Lib:c_0805" H 7550 2800 50  0001 C CNN
 F 3 "" H 7550 2800 60  0001 C CNN
 F 4 "CAP CER 0.1UF 25V 10% X7R 0805" H 7550 3000 60  0001 L CNN "Field4"
-F 5 "100nF, 25V" H 7550 3100 60  0001 L CNN "Field5"
+F 5 "100n, 25V" H 7550 3100 60  0001 L CNN "Field5"
 F 6 "Surface Mount, MLCC" H 7550 3200 60  0001 L CNN "Field6"
 F 7 "Kemet" H 7550 3300 60  0001 L CNN "Field7"
@@
 $EndComp
 $Comp
-L C2 C47
+L C2 C44
 U 1 1 542C09D3
 P 8950 2800
-F 0 "C47" H 8975 2900 50  0000 L CNN
+F 0 "C44" H 8975 2900 50  0000 L CNN
 F 1 "100n" H 8975 2700 50  0000 L CNN
 F 2 "TinyTiM_Lib:c_0805" H 8950 2800 50  0001 C CNN
@@
 $EndComp
 $Comp
-L C2 C49
+L C2 C45
 U 1 1 542C09E1
 P 10350 2800
-F 0 "C49" H 10375 2900 50  0000 L CNN
+F 0 "C45" H 10375 2900 50  0000 L CNN
 F 1 "100n" H 10375 2700 50  0000 L CNN
 F 2 "TinyTiM_Lib:c_0805" H 10350 2800 50  0001 C CNN
 F 3 "" H 10350 2800 60  0001 C CNN
 F 4 "CAP CER 0.1UF 25V 10% X7R 0805" H 10350 3000 60  0001 L CNN "Field4"
-F 5 "100nF, 25V" H 10350 3100 60  0001 L CNN "Field5"
+F 5 "100n, 25V" H 10350 3100 60  0001 L CNN "Field5"
 F 6 "Surface Mount, MLCC" H 10350 3200 60  0001 L CNN "Field6"
 F 7 "Kemet" H 10350 3300 60  0001 L CNN "Field7"
@@
 Connection ~ 10250 3000
 $Comp
-L C2 C38
+L C2 C46
 U 1 1 542C09F0
 P 1950 5150
-F 0 "C38" H 1975 5250 50  0000 L CNN
+F 0 "C46" H 1975 5250 50  0000 L CNN
 F 1 "100n" H 1975 5050 50  0000 L CNN
 F 2 "TinyTiM_Lib:c_0805" H 1950 5150 50  0001 C CNN
@@
 Connection ~ 1850 5350
 $Comp
-L C2 C40
+L C2 C47
 U 1 1 542C0A2D
 P 3350 5150
-F 0 "C40" H 3375 5250 50  0000 L CNN
+F 0 "C47" H 3375 5250 50  0000 L CNN
 F 1 "100n" H 3375 5050 50  0000 L CNN
 F 2 "TinyTiM_Lib:c_0805" H 3350 5150 50  0001 C CNN
 F 3 "" H 3350 5150 60  0001 C CNN
 F 4 "CAP CER 0.1UF 25V 10% X7R 0805" H 3350 5350 60  0001 L CNN "Field4"
-F 5 "100nF, 25V" H 3350 5450 60  0001 L CNN "Field5"
+F 5 "100n, 25V" H 3350 5450 60  0001 L CNN "Field5"
 F 6 "Surface Mount, MLCC" H 3350 5550 60  0001 L CNN "Field6"
 F 7 "Kemet" H 3350 5650 60  0001 L CNN "Field7"
@@
 $EndComp
 $Comp
-L C2 C42
+L C2 C48
 U 1 1 542C0A3B
 P 4750 5150
-F 0 "C42" H 4775 5250 50  0000 L CNN
+F 0 "C48" H 4775 5250 50  0000 L CNN
 F 1 "100n" H 4775 5050 50  0000 L CNN
 F 2 "TinyTiM_Lib:c_0805" H 4750 5150 50  0001 C CNN
@@
 $EndComp
 $Comp
-L C2 C44
+L C2 C49
 U 1 1 542C0A49
 P 6150 5150
-F 0 "C44" H 6175 5250 50  0000 L CNN
+F 0 "C49" H 6175 5250 50  0000 L CNN
 F 1 "100n" H 6175 5050 50  0000 L CNN
 F 2 "TinyTiM_Lib:c_0805" H 6150 5150 50  0001 C CNN
 F 3 "" H 6150 5150 60  0001 C CNN
 F 4 "CAP CER 0.1UF 25V 10% X7R 0805" H 6150 5350 60  0001 L CNN "Field4"
-F 5 "100nF, 25V" H 6150 5450 60  0001 L CNN "Field5"
+F 5 "100n, 25V" H 6150 5450 60  0001 L CNN "Field5"
 F 6 "Surface Mount, MLCC" H 6150 5550 60  0001 L CNN "Field6"
 F 7 "Kemet" H 6150 5650 60  0001 L CNN "Field7"
@@
 $EndComp
 $Comp
-L C2 C46
+L C2 C50
 U 1 1 542C0A57
 P 7550 5150
-F 0 "C46" H 7575 5250 50  0000 L CNN
+F 0 "C50" H 7575 5250 50  0000 L CNN
 F 1 "100n" H 7575 5050 50  0000 L CNN
 F 2 "TinyTiM_Lib:c_0805" H 7550 5150 50  0001 C CNN
@@
 $EndComp
 $Comp
-L C2 C48
+L C2 C51
 U 1 1 542C0A65
 P 8950 5150
-F 0 "C48" H 8975 5250 50  0000 L CNN
+F 0 "C51" H 8975 5250 50  0000 L CNN
 F 1 "100n" H 8975 5050 50  0000 L CNN
 F 2 "TinyTiM_Lib:c_0805" H 8950 5150 50  0001 C CNN
 F 3 "" H 8950 5150 60  0001 C CNN
 F 4 "CAP CER 0.1UF 25V 10% X7R 0805" H 8950 5350 60  0001 L CNN "Field4"
-F 5 "100nF, 25V" H 8950 5450 60  0001 L CNN "Field5"
+F 5 "100n, 25V" H 8950 5450 60  0001 L CNN "Field5"
 F 6 "Surface Mount, MLCC" H 8950 5550 60  0001 L CNN "Field6"
 F 7 "Kemet" H 8950 5650 60  0001 L CNN "Field7"
@@
 $EndComp
 $Comp
-L C2 C50
+L C2 C52
 U 1 1 542C0A73
 P 10350 5150
-F 0 "C50" H 10375 5250 50  0000 L CNN
+F 0 "C52" H 10375 5250 50  0000 L CNN
 F 1 "100n" H 10375 5050 50  0000 L CNN
 F 2 "TinyTiM_Lib:c_0805" H 10350 5150 50  0001 C CNN

Commit message: Board layout updated
Parts:
- removed U30, U31, U32, U33, U34, U35, U36, U37, U38, U39, U40, U41, U42, U43: RGB_WS2812B, symbol RGB_WS2812B
- added LED29, LED30, LED31, LED32, LED33, LED34, LED35, LED36, LED37, LED38, LED39, LED40, LED41, LED42: RGB_WS2812B, ~, symbol RGB_WS2812B

Commit message: Board layout updated
Matrix placed and wired. Added RTC.
Parts:
- removed C39: 100n, TinyTiM_Lib:c_0805, symbol C2
- removed LED29, LED30, LED31, LED32, LED33, LED34, LED35, LED36, LED37, LED38, LED39, LED40, LED41, LED42: RGB_WS2812B, ~, symbol RGB_WS2812B
- added C53: 100n, TinyTiM_Lib:c_0805, symbol C2
- added LED29, LED30, LED31, LED32, LED33, LED34, LED35, LED36, LED37, LED38, LED39, LED40, LED41, LED42: WS2812B, ~, symbol WS2812B
- C40, C42, C44, C46, C48, C50, C52: Field5 100nF, 25V -> 100n, 25V
- C41, C43, C45, C47, C49, C51: Field5 100n, 25V -> 100nF, 25V
