File: KiCad/Row_C.sch (KiCad schematic (older format))
At the start: 28 parts

Commit message: PCB layout, work in progress
Parts:
- C40, C41, C42, C43, C44, C45, C46, C47, C48, C49, C50, C51, C52, C53: footprint TinyTiM_Lib:c_0805 -> C4_Pretty:c_0805
- LED29, LED30, LED31, LED32, LED33, LED34, LED35, LED36, LED37, LED38, LED39, LED40, LED41, LED42: footprint ~ -> C4_Pretty:RGB_WS2811B
Changed lines of the file:
@@
 F 0 "C40" H 1875 2800 50  0000 L CNN
 F 1 "100n" H 1875 2600 50  0000 L CNN
-F 2 "TinyTiM_Lib:c_0805" H 1850 2700 50  0001 C CNN
+F 2 "C4_Pretty:c_0805" H 1850 2700 50  0001 C CNN
 F 3 "" H 1850 2700 60  0001 C CNN
 F 4 "CAP CER 0.1UF 25V 10% X7R 0805" H 1850 2900 60  0001 L CNN "Field4"
@@
 F 0 "C41" H 3275 2800 50  0000 L CNN
 F 1 "100n" H 3275 2600 50  0000 L CNN
-F 2 "TinyTiM_Lib:c_0805" H 3250 2700 50  0001 C CNN
+F 2 "C4_Pretty:c_0805" H 3250 2700 50  0001 C CNN
 F 3 "" H 3250 2700 60  0001 C CNN
 F 4 "CAP CER 0.1UF 25V 10% X7R 0805" H 3250 2900 60  0001 L CNN "Field4"
@@
 F 0 "C42" H 4675 2800 50  0000 L CNN
 F 1 "100n" H 4675 2600 50  0000 L CNN
-F 2 "TinyTiM_Lib:c_0805" H 4650 2700 50  0001 C CNN
+F 2 "C4_Pretty:c_0805" H 4650 2700 50  0001 C CNN
 F 3 "" H 4650 2700 60  0001 C CNN
 F 4 "CAP CER 0.1UF 25V 10% X7R 0805" H 4650 2900 60  0001 L CNN "Field4"
@@
 F 0 "C43" H 6075 2800 50  0000 L CNN
 F 1 "100n" H 6075 2600 50  0000 L CNN
-F 2 "TinyTiM_Lib:c_0805" H 6050 2700 50  0001 C CNN
+F 2 "C4_Pretty:c_0805" H 6050 2700 50  0001 C CNN
 F 3 "" H 6050 2700 60  0001 C CNN
 F 4 "CAP CER 0.1UF 25V 10% X7R 0805" H 6050 2900 60  0001 L CNN "Field4"
@@
 F 0 "C44" H 7475 2800 50  0000 L CNN
 F 1 "100n" H 7475 2600 50  0000 L CNN
-F 2 "TinyTiM_Lib:c_0805" H 7450 2700 50  0001 C CNN
+F 2 "C4_Pretty:c_0805" H 7450 2700 50  0001 C CNN
 F 3 "" H 7450 2700 60  0001 C CNN
 F 4 "CAP CER 0.1UF 25V 10% X7R 0805" H 7450 2900 60  0001 L CNN "Field4"
@@
 F 0 "C45" H 8875 2800 50  0000 L CNN
 F 1 "100n" H 8875 2600 50  0000 L CNN
-F 2 "TinyTiM_Lib:c_0805" H 8850 2700 50  0001 C CNN
+F 2 "C4_Pretty:c_0805" H 8850 2700 50  0001 C CNN
 F 3 "" H 8850 2700 60  0001 C CNN
 F 4 "CAP CER 0.1UF 25V 10% X7R 0805" H 8850 2900 60  0001 L CNN "Field4"
@@
 F 0 "C46" H 10275 2800 50  0000 L CNN
 F 1 "100n" H 10275 2600 50  0000 L CNN
-F 2 "TinyTiM_Lib:c_0805" H 10250 2700 50  0001 C CNN
+F 2 "C4_Pretty:c_0805" H 10250 2700 50  0001 C CNN
 F 3 "" H 10250 2700 60  0001 C CNN
 F 4 "CAP CER 0.1UF 25V 10% X7R 0805" H 10250 2900 60  0001 L CNN "Field4"
@@
 F 0 "C47" H 1875 5150 50  0000 L CNN
 F 1 "100n" H 1875 4950 50  0000 L CNN
-F 2 "TinyTiM_Lib:c_0805" H 1850 5050 50  0001 C CNN
+F 2 "C4_Pretty:c_0805" H 1850 5050 50  0001 C CNN
 F 3 "" H 1850 5050 60  0001 C CNN
 F 4 "CAP CER 0.1UF 25V 10% X7R 0805" H 1850 5250 60  0001 L CNN "Field4"
@@
 F 0 "C48" H 3275 5150 50  0000 L CNN
 F 1 "100n" H 3275 4950 50  0000 L CNN
-F 2 "TinyTiM_Lib:c_0805" H 3250 5050 50  0001 C CNN
+F 2 "C4_Pretty:c_0805" H 3250 5050 50  0001 C CNN
 F 3 "" H 3250 5050 60  0001 C CNN
 F 4 "CAP CER 0.1UF 25V 10% X7R 0805" H 3250 5250 60  0001 L CNN "Field4"
@@
 F 0 "C49" H 4675 5150 50  0000 L CNN
 F 1 "100n" H 4675 4950 50  0000 L CNN
-F 2 "TinyTiM_Lib:c_0805" H 4650 5050 50  0001 C CNN
+F 2 "C4_Pretty:c_0805" H 4650 5050 50  0001 C CNN
 F 3 "" H 4650 5050 60  0001 C CNN
 F 4 "CAP CER 0.1UF 25V 10% X7R 0805" H 4650 5250 60  0001 L CNN "Field4"
@@
 F 0 "C50" H 6075 5150 50  0000 L CNN
 F 1 "100n" H 6075 4950 50  0000 L CNN
-F 2 "TinyTiM_Lib:c_0805" H 6050 5050 50  0001 C CNN
+F 2 "C4_Pretty:c_0805" H 6050 5050 50  0001 C CNN
 F 3 "" H 6050 5050 60  0001 C CNN
 F 4 "CAP CER 0.1UF 25V 10% X7R 0805" H 6050 5250 60  0001 L CNN "Field4"
@@
 F 0 "C51" H 7475 5150 50  0000 L CNN
 F 1 "100n" H 7475 4950 50  0000 L CNN
-F 2 "TinyTiM_Lib:c_0805" H 7450 5050 50  0001 C CNN
+F 2 "C4_Pretty:c_0805" H 7450 5050 50  0001 C CNN
 F 3 "" H 7450 5050 60  0001 C CNN
 F 4 "CAP CER 0.1UF 25V 10% X7R 0805" H 7450 5250 60  0001 L CNN "Field4"
@@
 F 0 "C52" H 8875 5150 50  0000 L CNN
 F 1 "100n" H 8875 4950 50  0000 L CNN
-F 2 "TinyTiM_Lib:c_0805" H 8850 5050 50  0001 C CNN
+F 2 "C4_Pretty:c_0805" H 8850 5050 50  0001 C CNN
 F 3 "" H 8850 5050 60  0001 C CNN
 F 4 "CAP CER 0.1UF 25V 10% X7R 0805" H 8850 5250 60  0001 L CNN "Field4"
@@
 F 0 "C53" H 10275 5150 50  0000 L CNN
 F 1 "100n" H 10275 4950 50  0000 L CNN
-F 2 "TinyTiM_Lib:c_0805" H 10250 5050 50  0001 C CNN
+F 2 "C4_Pretty:c_0805" H 10250 5050 50  0001 C CNN
 F 3 "" H 10250 5050 60  0001 C CNN
 F 4 "CAP CER 0.1UF 25V 10% X7R 0805" H 10250 5250 60  0001 L CNN "Field4"
@@
 F 0 "LED29" V 1425 1725 60  0000 C CNN
 F 1 "WS2812B" V 2075 1725 60  0001 C CNN
-F 2 "~" H 1675 1725 60  0000 C CNN
+F 2 "C4_Pretty:RGB_WS2811B" H 1675 1725 60  0001 C CNN
 F 3 "~" H 1675 1725 60  0000 C CNN
 	1    1675 1725
@@
 F 0 "LED30" V 2825 1725 60  0000 C CNN
 F 1 "WS2812B" V 3475 1725 60  0001 C CNN
-F 2 "~" H 3075 1725 60  0000 C CNN
+F 2 "C4_Pretty:RGB_WS2811B" H 3075 1725 60  0001 C CNN
 F 3 "~" H 3075 1725 60  0000 C CNN
 	1    3075 1725
@@
 F 0 "LED31" V 4225 1725 60  0000 C CNN
 F 1 "WS2812B" V 4875 1725 60  0001 C CNN
-F 2 "~" H 4475 1725 60  0000 C CNN
+F 2 "C4_Pretty:RGB_WS2811B" H 4475 1725 60  0001 C CNN
 F 3 "~" H 4475 1725 60  0000 C CNN
 	1    4475 1725
@@
 F 0 "LED32" V 5625 1725 60  0000 C CNN
 F 1 "WS2812B" V 6275 1725 60  0001 C CNN
-F 2 "~" H 5875 1725 60  0000 C CNN
+F 2 "C4_Pretty:RGB_WS2811B" H 5875 1725 60  0001 C CNN
 F 3 "~" H 5875 1725 60  0000 C CNN
 	1    5875 1725
@@
 F 0 "LED33" V 7025 1725 60  0000 C CNN
 F 1 "WS2812B" V 7675 1725 60  0001 C CNN
-F 2 "~" H 7275 1725 60  0000 C CNN
+F 2 "C4_Pretty:RGB_WS2811B" H 7275 1725 60  0001 C CNN
 F 3 "~" H 7275 1725 60  0000 C CNN
 	1    7275 1725
@@
 F 0 "LED34" V 8425 1725 60  0000 C CNN
 F 1 "WS2812B" V 9075 1725 60  0001 C CNN
-F 2 "~" H 8675 1725 60  0000 C CNN
+F 2 "C4_Pretty:RGB_WS2811B" H 8675 1725 60  0001 C CNN
 F 3 "~" H 8675 1725 60  0000 C CNN
 	1    8675 1725
@@
 F 0 "LED35" V 9825 1725 60  0000 C CNN
 F 1 "WS2812B" V 10475 1725 60  0001 C CNN
-F 2 "~" H 10075 1725 60  0000 C CNN
+F 2 "C4_Pretty:RGB_WS2811B" H 10075 1725 60  0001 C CNN
 F 3 "~" H 10075 1725 60  0000 C CNN
 	1    10075 1725
@@
 F 0 "LED36" V 1425 4125 60  0000 C CNN
 F 1 "WS2812B" V 2075 4125 60  0001 C CNN
-F 2 "~" H 1675 4125 60  0000 C CNN
+F 2 "C4_Pretty:RGB_WS2811B" H 1675 4125 60  0001 C CNN
 F 3 "~" H 1675 4125 60  0000 C CNN
 	1    1675 4125
@@
 F 0 "LED37" V 2825 4125 60  0000 C CNN
 F 1 "WS2812B" V 3475 4125 60  0001 C CNN
-F 2 "~" H 3075 4125 60  0000 C CNN
+F 2 "C4_Pretty:RGB_WS2811B" H 3075 4125 60  0001 C CNN
 F 3 "~" H 3075 4125 60  0000 C CNN
 	1    3075 4125
@@
 F 0 "LED38" V 4225 4125 60  0000 C CNN
 F 1 "WS2812B" V 4875 4125 60  0001 C CNN
-F 2 "~" H 4475 4125 60  0000 C CNN
+F 2 "C4_Pretty:RGB_WS2811B" H 4475 4125 60  0001 C CNN
 F 3 "~" H 4475 4125 60  0000 C CNN
 	1    4475 4125
@@
 F 0 "LED39" V 5625 4125 60  0000 C CNN
 F 1 "WS2812B" V 6275 4125 60  0001 C CNN
-F 2 "~" H 5875 4125 60  0000 C CNN
+F 2 "C4_Pretty:RGB_WS2811B" H 5875 4125 60  0001 C CNN
 F 3 "~" H 5875 4125 60  0000 C CNN
 	1    5875 4125
@@
 F 0 "LED40" V 7025 4125 60  0000 C CNN
 F 1 "WS2812B" V 7675 4125 60  0001 C CNN
-F 2 "~" H 7275 4125 60  0000 C CNN
+F 2 "C4_Pretty:RGB_WS2811B" H 7275 4125 60  0001 C CNN
 F 3 "~" H 7275 4125 60  0000 C CNN
 	1    7275 4125
@@
 F 0 "LED41" V 8425 4125 60  0000 C CNN
 F 1 "WS2812B" V 9075 4125 60  0001 C CNN
-F 2 "~" H 8675 4125 60  0000 C CNN
+F 2 "C4_Pretty:RGB_WS2811B" H 8675 4125 60  0001 C CNN
 F 3 "~" H 8675 4125 60  0000 C CNN
 	1    8675 4125
@@
 F 0 "LED42" V 9825 4125 60  0000 C CNN
 F 1 "WS2812B" V 10475 4125 60  0001 C CNN
-F 2 "~" H 10075 4125 60  0000 C CNN
+F 2 "C4_Pretty:RGB_WS2811B" H 10075 4125 60  0001 C CNN
 F 3 "~" H 10075 4125 60  0000 C CNN
 	1    10075 4125

Commit message: C4 PCB layout complete. Added Gerbers
Parts:
- C40, C41, C42, C43, C44, C45, C46, C47, C48, C49, C50, C51, C52, C53: footprint C4_Pretty:c_0805 -> C4_Pretty:c_0805_led
Changed lines of the file:
@@
 EESchema Schematic File Version 2
 LIBS:ClockFOUR
+LIBS:RowGB_sym
 LIBS:ClockFOUR-cache
 EELAYER 24 0
@@
 F 0 "C40" H 1875 2800 50  0000 L CNN
 F 1 "100n" H 1875 2600 50  0000 L CNN
-F 2 "C4_Pretty:c_0805" H 1850 2700 50  0001 C CNN
+F 2 "C4_Pretty:c_0805_led" H 1850 2700 50  0001 C CNN
 F 3 "" H 1850 2700 60  0001 C CNN
 F 4 "CAP CER 0.1UF 25V 10% X7R 0805" H 1850 2900 60  0001 L CNN "Field4"
@@
 F 0 "C41" H 3275 2800 50  0000 L CNN
 F 1 "100n" H 3275 2600 50  0000 L CNN
-F 2 "C4_Pretty:c_0805" H 3250 2700 50  0001 C CNN
+F 2 "C4_Pretty:c_0805_led" H 3250 2700 50  0001 C CNN
 F 3 "" H 3250 2700 60  0001 C CNN
 F 4 "CAP CER 0.1UF 25V 10% X7R 0805" H 3250 2900 60  0001 L CNN "Field4"
@@
 F 0 "C42" H 4675 2800 50  0000 L CNN
 F 1 "100n" H 4675 2600 50  0000 L CNN
-F 2 "C4_Pretty:c_0805" H 4650 2700 50  0001 C CNN
+F 2 "C4_Pretty:c_0805_led" H 4650 2700 50  0001 C CNN
 F 3 "" H 4650 2700 60  0001 C CNN
 F 4 "CAP CER 0.1UF 25V 10% X7R 0805" H 4650 2900 60  0001 L CNN "Field4"
@@
 F 0 "C43" H 6075 2800 50  0000 L CNN
 F 1 "100n" H 6075 2600 50  0000 L CNN
-F 2 "C4_Pretty:c_0805" H 6050 2700 50  0001 C CNN
+F 2 "C4_Pretty:c_0805_led" H 6050 2700 50  0001 C CNN
 F 3 "" H 6050 2700 60  0001 C CNN
 F 4 "CAP CER 0.1UF 25V 10% X7R 0805" H 6050 2900 60  0001 L CNN "Field4"
@@
 F 0 "C44" H 7475 2800 50  0000 L CNN
 F 1 "100n" H 7475 2600 50  0000 L CNN
-F 2 "C4_Pretty:c_0805" H 7450 2700 50  0001 C CNN
+F 2 "C4_Pretty:c_0805_led" H 7450 2700 50  0001 C CNN
 F 3 "" H 7450 2700 60  0001 C CNN
 F 4 "CAP CER 0.1UF 25V 10% X7R 0805" H 7450 2900 60  0001 L CNN "Field4"
@@
 F 0 "C45" H 8875 2800 50  0000 L CNN
 F 1 "100n" H 8875 2600 50  0000 L CNN
-F 2 "C4_Pretty:c_0805" H 8850 2700 50  0001 C CNN
+F 2 "C4_Pretty:c_0805_led" H 8850 2700 50  0001 C CNN
 F 3 "" H 8850 2700 60  0001 C CNN
 F 4 "CAP CER 0.1UF 25V 10% X7R 0805" H 8850 2900 60  0001 L CNN "Field4"
@@
 F 0 "C46" H 10275 2800 50  0000 L CNN
 F 1 "100n" H 10275 2600 50  0000 L CNN
-F 2 "C4_Pretty:c_0805" H 10250 2700 50  0001 C CNN
+F 2 "C4_Pretty:c_0805_led" H 10250 2700 50  0001 C CNN
 F 3 "" H 10250 2700 60  0001 C CNN
 F 4 "CAP CER 0.1UF 25V 10% X7R 0805" H 10250 2900 60  0001 L CNN "Field4"
@@
 F 0 "C47" H 1875 5150 50  0000 L CNN
 F 1 "100n" H 1875 4950 50  0000 L CNN
-F 2 "C4_Pretty:c_0805" H 1850 5050 50  0001 C CNN
+F 2 "C4_Pretty:c_0805_led" H 1850 5050 50  0001 C CNN
 F 3 "" H 1850 5050 60  0001 C CNN
 F 4 "CAP CER 0.1UF 25V 10% X7R 0805" H 1850 5250 60  0001 L CNN "Field4"
@@
 F 0 "C48" H 3275 5150 50  0000 L CNN
 F 1 "100n" H 3275 4950 50  0000 L CNN
-F 2 "C4_Pretty:c_0805" H 3250 5050 50  0001 C CNN
+F 2 "C4_Pretty:c_0805_led" H 3250 5050 50  0001 C CNN
 F 3 "" H 3250 5050 60  0001 C CNN
 F 4 "CAP CER 0.1UF 25V 10% X7R 0805" H 3250 5250 60  0001 L CNN "Field4"
@@
 F 0 "C49" H 4675 5150 50  0000 L CNN
 F 1 "100n" H 4675 4950 50  0000 L CNN
-F 2 "C4_Pretty:c_0805" H 4650 5050 50  0001 C CNN
+F 2 "C4_Pretty:c_0805_led" H 4650 5050 50  0001 C CNN
 F 3 "" H 4650 5050 60  0001 C CNN
 F 4 "CAP CER 0.1UF 25V 10% X7R 0805" H 4650 5250 60  0001 L CNN "Field4"
@@
 F 0 "C50" H 6075 5150 50  0000 L CNN
 F 1 "100n" H 6075 4950 50  0000 L CNN
-F 2 "C4_Pretty:c_0805" H 6050 5050 50  0001 C CNN
+F 2 "C4_Pretty:c_0805_led" H 6050 5050 50  0001 C CNN
 F 3 "" H 6050 5050 60  0001 C CNN
 F 4 "CAP CER 0.1UF 25V 10% X7R 0805" H 6050 5250 60  0001 L CNN "Field4"
@@
 F 0 "C51" H 7475 5150 50  0000 L CNN
 F 1 "100n" H 7475 4950 50  0000 L CNN
-F 2 "C4_Pretty:c_0805" H 7450 5050 50  0001 C CNN
+F 2 "C4_Pretty:c_0805_led" H 7450 5050 50  0001 C CNN
 F 3 "" H 7450 5050 60  0001 C CNN
 F 4 "CAP CER 0.1UF 25V 10% X7R 0805" H 7450 5250 60  0001 L CNN "Field4"
@@
 F 0 "C52" H 8875 5150 50  0000 L CNN
 F 1 "100n" H 8875 4950 50  0000 L CNN
-F 2 "C4_Pretty:c_0805" H 8850 5050 50  0001 C CNN
+F 2 "C4_Pretty:c_0805_led" H 8850 5050 50  0001 C CNN
 F 3 "" H 8850 5050 60  0001 C CNN
 F 4 "CAP CER 0.1UF 25V 10% X7R 0805" H 8850 5250 60  0001 L CNN "Field4"
@@
 F 0 "C53" H 10275 5150 50  0000 L CNN
 F 1 "100n" H 10275 4950 50  0000 L CNN
-F 2 "C4_Pretty:c_0805" H 10250 5050 50  0001 C CNN
+F 2 "C4_Pretty:c_0805_led" H 10250 5050 50  0001 C CNN
 F 3 "" H 10250 5050 60  0001 C CNN
 F 4 "CAP CER 0.1UF 25V 10% X7R 0805" H 10250 5250 60  0001 L CNN "Field4"
