File: KiCad/Row_D.sch (KiCad schematic (older format))
At the start: 14 parts, among them U101 RGB_WS2811B, U102 RGB_WS2811B, U103 RGB_WS2811B, U104 RGB_WS2811B, U105 RGB_WS2811B, U106 RGB_WS2811B, U107 RGB_WS2811B, U108 RGB_WS2811B

Commit message: Schematic updated
Parts:
- removed C101: 100n, TinyTiM_Lib:c_0805, symbol C2
- removed C117: 47u,8V, TinyTiM_Lib:c_2917, symbol C_POL_1
- removed S101, S102, S103, S104: CONN_1, TinyTiM_Lib:Screw, symbol CONN_1
- removed U101, U102, U103, U104, U105, U106, U107, U108: RGB_WS2811B, TinyTiM_Lib:RGB_WS2811B, symbol RGB_WS2811B
Connections:
- net labels removed: 5V, A_02, A_03, A_04, A_05, A_06, A_07, A_08, A_09, DI_A, DO_A, GND
- wire segments 49 -> 0
- no-connect marks 4 -> 0
Other:
- note removed: "Mounting Screws"

Commit message: Schematic updated
Parts:
- added C51, C52, C53, C54, C55, C56, C57, C58, C59, C60, C61, C62, C63, C64: 100n, TinyTiM_Lib:c_0805, symbol C2
- added U46, U47, U48, U49, U50, U51, U52, U53, U54, U55, U56, U57, U58, U59: RGB_WS2812B, symbol RGB_WS2812B
Connections:
- net labels added: 5V, DI_D, DO_D, GND
- wire segments 0 -> 82

Commit message: Schematic updated, board started
Parts:
- C53: renamed from C51; Field5 100nF, 25V -> 100n, 25V
- C55: Field5 100nF, 25V -> 100n, 25V
- C57: renamed from C59; Field5 100nF, 25V -> 100n, 25V
- C59: renamed from C63; Field5 100nF, 25V -> 100n, 25V
- C61: renamed from C54; Field5 100nF, 25V -> 100n, 25V
- C63: renamed from C58; Field5 100nF, 25V -> 100n, 25V
- C65: renamed from C62; Field5 100nF, 25V -> 100n, 25V
- renumbered C53 to C54, C57 to C56, C61 to C58, C52 to C60, C56 to C62, C60 to C64, C64 to C66, U46 to U44, U48 to U45, U50 to U46, U52 to U47, U54 to U48, U56 to U49, U58 to U50, U47 to U51, U49 to U52, U51 to U53, U53 to U54, U57 to U56, U59 to U57
Changed lines of the file:
@@
 LIBS:contrib
 LIBS:valves
-LIBS:TinyTiM-cache
-LIBS:TiNA_sym
+LIBS:ClockFOUR
 LIBS:ClockFOUR-cache
 EELAYER 27 0
@@
 Sheet 5 14
 Title "ClockFOUR"
-Date "30 sep 2014"
+Date "1 oct 2014"
 Rev ""
 Comp "WyoLum"
@@
 5V
 $Comp
-L GND #PWR015
+L GND #PWR017
 U 1 1 542C0A8B
 P 1450 2600
-F 0 "#PWR015" H 1450 2600 30  0001 C CNN
+F 0 "#PWR017" H 1450 2600 30  0001 C CNN
 F 1 "GND" H 1450 2530 30  0001 C CNN
 F 2 "" H 1450 2600 60  0001 C CNN
@@
 $EndComp
 $Comp
-L C2 C51
+L C2 C53
 U 1 1 542C0A99
 P 2000 2750
-F 0 "C51" H 2025 2850 50  0000 L CNN
+F 0 "C53" H 2025 2850 50  0000 L CNN
 F 1 "100n" H 2025 2650 50  0000 L CNN
 F 2 "TinyTiM_Lib:c_0805" H 2000 2750 50  0001 C CNN
 F 3 "" H 2000 2750 60  0001 C CNN
 F 4 "CAP CER 0.1UF 25V 10% X7R 0805" H 2000 2950 60  0001 L CNN "Field4"
-F 5 "100nF, 25V" H 2000 3050 60  0001 L CNN "Field5"
+F 5 "100n, 25V" H 2000 3050 60  0001 L CNN "Field5"
 F 6 "Surface Mount, MLCC" H 2000 3150 60  0001 L CNN "Field6"
 F 7 "Kemet" H 2000 3250 60  0001 L CNN "Field7"
@@
 $EndComp
 $Comp
-L RGB_WS2812B U46
+L RGB_WS2812B U44
 U 1 1 542C0A9F
 P 1825 1775
-F 0 "U46" V 1575 1775 60  0000 C CNN
+F 0 "U44" V 1575 1775 60  0000 C CNN
 F 1 "RGB_WS2812B" V 2225 1775 60  0000 C CNN
 F 2 "" H 1825 1775 60  0000 C CNN
@@
 $EndComp
 $Comp
-L RGB_WS2812B U48
+L RGB_WS2812B U45
 U 1 1 542C0AA5
 P 3225 1775
-F 0 "U48" V 2975 1775 60  0000 C CNN
+F 0 "U45" V 2975 1775 60  0000 C CNN
 F 1 "RGB_WS2812B" V 3625 1775 60  0000 C CNN
 F 2 "" H 3225 1775 60  0000 C CNN
@@
 $EndComp
 $Comp
-L RGB_WS2812B U50
+L RGB_WS2812B U46
 U 1 1 542C0AAB
 P 4625 1775
-F 0 "U50" V 4375 1775 60  0000 C CNN
+F 0 "U46" V 4375 1775 60  0000 C CNN
 F 1 "RGB_WS2812B" V 5025 1775 60  0000 C CNN
 F 2 "" H 4625 1775 60  0000 C CNN
@@
 $EndComp
 $Comp
-L RGB_WS2812B U52
+L RGB_WS2812B U47
 U 1 1 542C0AB1
 P 6025 1775
-F 0 "U52" V 5775 1775 60  0000 C CNN
+F 0 "U47" V 5775 1775 60  0000 C CNN
 F 1 "RGB_WS2812B" V 6425 1775 60  0000 C CNN
 F 2 "" H 6025 1775 60  0000 C CNN
@@
 $EndComp
 $Comp
-L RGB_WS2812B U54
+L RGB_WS2812B U48
 U 1 1 542C0AB7
 P 7425 1775
-F 0 "U54" V 7175 1775 60  0000 C CNN
+F 0 "U48" V 7175 1775 60  0000 C CNN
 F 1 "RGB_WS2812B" V 7825 1775 60  0000 C CNN
 F 2 "" H 7425 1775 60  0000 C CNN
@@
 $EndComp
 $Comp
-L RGB_WS2812B U56
+L RGB_WS2812B U49
 U 1 1 542C0ABD
 P 8825 1775
-F 0 "U56" V 8575 1775 60  0000 C CNN
+F 0 "U49" V 8575 1775 60  0000 C CNN
 F 1 "RGB_WS2812B" V 9225 1775 60  0000 C CNN
 F 2 "" H 8825 1775 60  0000 C CNN
@@
 $EndComp
 $Comp
-L RGB_WS2812B U58
+L RGB_WS2812B U50
 U 1 1 542C0AC3
 P 10225 1775
-F 0 "U58" V 9975 1775 60  0000 C CNN
+F 0 "U50" V 9975 1775 60  0000 C CNN
 F 1 "RGB_WS2812B" V 10625 1775 60  0000 C CNN
 F 2 "" H 10225 1775 60  0000 C CNN
@@
 $EndComp
 $Comp
-L RGB_WS2812B U47
+L RGB_WS2812B U51
 U 1 1 542C0AC9
 P 1825 4175
-F 0 "U47" V 1575 4175 60  0000 C CNN
+F 0 "U51" V 1575 4175 60  0000 C CNN
 F 1 "RGB_WS2812B" V 2225 4175 60  0000 C CNN
 F 2 "" H 1825 4175 60  0000 C CNN
@@
 $EndComp
 $Comp
-L RGB_WS2812B U49
+L RGB_WS2812B U52
 U 1 1 542C0ACF
 P 3225 4175
-F 0 "U49" V 2975 4175 60  0000 C CNN
+F 0 "U52" V 2975 4175 60  0000 C CNN
 F 1 "RGB_WS2812B" V 3625 4175 60  0000 C CNN
 F 2 "" H 3225 4175 60  0000 C CNN
@@
 $EndComp
 $Comp
-L RGB_WS2812B U51
+L RGB_WS2812B U53
 U 1 1 542C0AD5
 P 4625 4175
-F 0 "U51" V 4375 4175 60  0000 C CNN
+F 0 "U53" V 4375 4175 60  0000 C CNN
 F 1 "RGB_WS2812B" V 5025 4175 60  0000 C CNN
 F 2 "" H 4625 4175 60  0000 C CNN
@@
 $EndComp
 $Comp
-L RGB_WS2812B U53
+L RGB_WS2812B U54
 U 1 1 542C0ADB
 P 6025 4175
-F 0 "U53" V 5775 4175 60  0000 C CNN
+F 0 "U54" V 5775 4175 60  0000 C CNN
 F 1 "RGB_WS2812B" V 6425 4175 60  0000 C CNN
 F 2 "" H 6025 4175 60  0000 C CNN
@@
 $EndComp
 $Comp
-L RGB_WS2812B U57
+L RGB_WS2812B U56
 U 1 1 542C0AE7
 P 8825 4175
-F 0 "U57" V 8575 4175 60  0000 C CNN
+F 0 "U56" V 8575 4175 60  0000 C CNN
 F 1 "RGB_WS2812B" V 9225 4175 60  0000 C CNN
 F 2 "" H 8825 4175 60  0000 C CNN
@@
 $EndComp
 $Comp
-L RGB_WS2812B U59
+L RGB_WS2812B U57
 U 1 1 542C0AED
 P 10225 4175
-F 0 "U59" V 9975 4175 60  0000 C CNN
+F 0 "U57" V 9975 4175 60  0000 C CNN
 F 1 "RGB_WS2812B" V 10625 4175 60  0000 C CNN
 F 2 "" H 10225 4175 60  0000 C CNN
@@
 Connection ~ 1900 2950
 $Comp
-L C2 C53
+L C2 C54
 U 1 1 542C0B48
 P 3400 2750
-F 0 "C53" H 3425 2850 50  0000 L CNN
+F 0 "C54" H 3425 2850 50  0000 L CNN
 F 1 "100n" H 3425 2650 50  0000 L CNN
 F 2 "TinyTiM_Lib:c_0805" H 3400 2750 50  0001 C CNN
@@
 F 3 "" H 4800 2750 60  0001 C CNN
 F 4 "CAP CER 0.1UF 25V 10% X7R 0805" H 4800 2950 60  0001 L CNN "Field4"
-F 5 "100nF, 25V" H 4800 3050 60  0001 L CNN "Field5"
+F 5 "100n, 25V" H 4800 3050 60  0001 L CNN "Field5"
 F 6 "Surface Mount, MLCC" H 4800 3150 60  0001 L CNN "Field6"
 F 7 "Kemet" H 4800 3250 60  0001 L CNN "Field7"
@@
 $EndComp
 $Comp
-L C2 C57
+L C2 C56
 U 1 1 542C0B64
 P 6200 2750
-F 0 "C57" H 6225 2850 50  0000 L CNN
+F 0 "C56" H 6225 2850 50  0000 L CNN
 F 1 "100n" H 6225 2650 50  0000 L CNN
 F 2 "TinyTiM_Lib:c_0805" H 6200 2750 50  0001 C CNN
@@
 $EndComp
 $Comp
-L C2 C59
+L C2 C57
 U 1 1 542C0B72
 P 7600 2750
-F 0 "C59" H 7625 2850 50  0000 L CNN
+F 0 "C57" H 7625 2850 50  0000 L CNN
 F 1 "100n" H 7625 2650 50  0000 L CNN
 F 2 "TinyTiM_Lib:c_0805" H 7600 2750 50  0001 C CNN
 F 3 "" H 7600 2750 60  0001 C CNN
 F 4 "CAP CER 0.1UF 25V 10% X7R 0805" H 7600 2950 60  0001 L CNN "Field4"
-F 5 "100nF, 25V" H 7600 3050 60  0001 L CNN "Field5"
+F 5 "100n, 25V" H 7600 3050 60  0001 L CNN "Field5"
 F 6 "Surface Mount, MLCC" H 7600 3150 60  0001 L CNN "Field6"
 F 7 "Kemet" H 7600 3250 60  0001 L CNN "Field7"
@@
 $EndComp
 $Comp
-L C2 C61
+L C2 C58
 U 1 1 542C0B80
 P 9000 2750
-F 0 "C61" H 9025 2850 50  0000 L CNN
+F 0 "C58" H 9025 2850 50  0000 L CNN
 F 1 "100n" H 9025 2650 50  0000 L CNN
 F 2 "TinyTiM_Lib:c_0805" H 9000 2750 50  0001 C CNN
@@
 $EndComp
 $Comp
-L C2 C63
+L C2 C59
 U 1 1 542C0B8E
 P 10400 2750
-F 0 "C63" H 10425 2850 50  0000 L CNN
+F 0 "C59" H 10425 2850 50  0000 L CNN
 F 1 "100n" H 10425 2650 50  0000 L CNN
 F 2 "TinyTiM_Lib:c_0805" H 10400 2750 50  0001 C CNN
 F 3 "" H 10400 2750 60  0001 C CNN
 F 4 "CAP CER 0.1UF 25V 10% X7R 0805" H 10400 2950 60  0001 L CNN "Field4"
-F 5 "100nF, 25V" H 10400 3050 60  0001 L CNN "Field5"
+F 5 "100n, 25V" H 10400 3050 60  0001 L CNN "Field5"
 F 6 "Surface Mount, MLCC" H 10400 3150 60  0001 L CNN "Field6"
 F 7 "Kemet" H 10400 3250 60  0001 L CNN "Field7"
@@
 Connection ~ 10300 2950
 $Comp
-L C2 C52
+L C2 C60
 U 1 1 542C0B9D
 P 2000 5100
-F 0 "C52" H 2025 5200 50  0000 L CNN
+F 0 "C60" H 2025 5200 50  0000 L CNN
 F 1 "100n" H 2025 5000 50  0000 L CNN
 F 2 "TinyTiM_Lib:c_0805" H 2000 5100 50  0001 C CNN
@@
 Connection ~ 1900 5300
 $Comp
-L C2 C54
+L C2 C61
 U 1 1 542C0BDA
 P 3400 5100
-F 0 "C54" H 3425 5200 50  0000 L CNN
+F 0 "C61" H 3425 5200 50  0000 L CNN
 F 1 "100n" H 3425 5000 50  0000 L CNN
 F 2 "TinyTiM_Lib:c_0805" H 3400 5100 50  0001 C CNN
 F 3 "" H 3400 5100 60  0001 C CNN
 F 4 "CAP CER 0.1UF 25V 10% X7R 0805" H 3400 5300 60  0001 L CNN "Field4"
-F 5 "100nF, 25V" H 3400 5400 60  0001 L CNN "Field5"
+F 5 "100n, 25V" H 3400 5400 60  0001 L CNN "Field5"
 F 6 "Surface Mount, MLCC" H 3400 5500 60  0001 L CNN "Field6"
 F 7 "Kemet" H 3400 5600 60  0001 L CNN "Field7"
@@
 $EndComp
 $Comp
-L C2 C56
+L C2 C62
 U 1 1 542C0BE8
 P 4800 5100
-F 0 "C56" H 4825 5200 50  0000 L CNN
+F 0 "C62" H 4825 5200 50  0000 L CNN
 F 1 "100n" H 4825 5000 50  0000 L CNN
 F 2 "TinyTiM_Lib:c_0805" H 4800 5100 50  0001 C CNN
@@
 $EndComp
 $Comp
-L C2 C58
+L C2 C63
 U 1 1 542C0BF6
 P 6200 5100
-F 0 "C58" H 6225 5200 50  0000 L CNN
+F 0 "C63" H 6225 5200 50  0000 L CNN
 F 1 "100n" H 6225 5000 50  0000 L CNN
 F 2 "TinyTiM_Lib:c_0805" H 6200 5100 50  0001 C CNN
 F 3 "" H 6200 5100 60  0001 C CNN
 F 4 "CAP CER 0.1UF 25V 10% X7R 0805" H 6200 5300 60  0001 L CNN "Field4"
-F 5 "100nF, 25V" H 6200 5400 60  0001 L CNN "Field5"
+F 5 "100n, 25V" H 6200 5400 60  0001 L CNN "Field5"
 F 6 "Surface Mount, MLCC" H 6200 5500 60  0001 L CNN "Field6"
 F 7 "Kemet" H 6200 5600 60  0001 L CNN "Field7"
@@
 $EndComp
 $Comp
-L C2 C60
+L C2 C64
 U 1 1 542C0C04
 P 7600 5100
-F 0 "C60" H 7625 5200 50  0000 L CNN
+F 0 "C64" H 7625 5200 50  0000 L CNN
 F 1 "100n" H 7625 5000 50  0000 L CNN
 F 2 "TinyTiM_Lib:c_0805" H 7600 5100 50  0001 C CNN
@@
 $EndComp
 $Comp
-L C2 C62
+L C2 C65
 U 1 1 542C0C12
 P 9000 5100
-F 0 "C62" H 9025 5200 50  0000 L CNN
+F 0 "C65" H 9025 5200 50  0000 L CNN
 F 1 "100n" H 9025 5000 50  0000 L CNN
 F 2 "TinyTiM_Lib:c_0805" H 9000 5100 50  0001 C CNN
 F 3 "" H 9000 5100 60  0001 C CNN
 F 4 "CAP CER 0.1UF 25V 10% X7R 0805" H 9000 5300 60  0001 L CNN "Field4"
-F 5 "100nF, 25V" H 9000 5400 60  0001 L CNN "Field5"
+F 5 "100n, 25V" H 9000 5400 60  0001 L CNN "Field5"
 F 6 "Surface Mount, MLCC" H 9000 5500 60  0001 L CNN "Field6"
 F 7 "Kemet" H 9000 5600 60  0001 L CNN "Field7"
@@
 $EndComp
 $Comp
-L C2 C64
+L C2 C66
 U 1 1 542C0C20
 P 10400 5100
-F 0 "C64" H 10425 5200 50  0000 L CNN
+F 0 "C66" H 10425 5200 50  0000 L CNN
 F 1 "100n" H 10425 5000 50  0000 L CNN
 F 2 "TinyTiM_Lib:c_0805" H 10400 5100 50  0001 C CNN

Commit message: Board layout updated
Parts:
- removed U44, U45, U46, U47, U48, U49, U50, U51, U52, U53, U54, U55, U56, U57: RGB_WS2812B, symbol RGB_WS2812B
- added LED43, LED44, LED45, LED46, LED47, LED48, LED49, LED50, LED51, LED52, LED53, LED54, LED55, LED56: RGB_WS2812B, ~, symbol RGB_WS2812B

Commit message: Board layout updated
Matrix placed and wired. Added RTC.
Parts:
- removed C53: 100n, TinyTiM_Lib:c_0805, symbol C2
- removed LED43, LED44, LED45, LED46, LED47, LED48, LED49, LED50, LED51, LED52, LED53, LED54, LED55, LED56: RGB_WS2812B, ~, symbol RGB_WS2812B
- added C67: 100n, TinyTiM_Lib:c_0805, symbol C2
- added LED43, LED44, LED45, LED46, LED47, LED48, LED49, LED50, LED51, LED52, LED53, LED54, LED55, LED56: WS2812B, ~, symbol WS2812B
- C54, C56, C58, C60, C62, C64, C66: Field5 100nF, 25V -> 100n, 25V
- C55, C57, C59, C61, C63, C65: Field5 100n, 25V -> 100nF, 25V
