File: KiCad/Row_D.sch (KiCad schematic (older format))
At the start: 28 parts

Commit message: PCB layout, work in progress
Parts:
- C54, C55, C56, C57, C58, C59, C60, C61, C62, C63, C64, C65, C66, C67: footprint TinyTiM_Lib:c_0805 -> C4_Pretty:c_0805
- LED43, LED44, LED45, LED46, LED47, LED48, LED49, LED50, LED51, LED52, LED53, LED54, LED55, LED56: footprint ~ -> C4_Pretty:RGB_WS2811B
Changed lines of the file:
@@
 F 0 "C54" H 1875 3200 50  0000 L CNN
 F 1 "100n" H 1875 3000 50  0000 L CNN
-F 2 "TinyTiM_Lib:c_0805" H 1850 3100 50  0001 C CNN
+F 2 "C4_Pretty:c_0805" H 1850 3100 50  0001 C CNN
 F 3 "" H 1850 3100 60  0001 C CNN
 F 4 "CAP CER 0.1UF 25V 10% X7R 0805" H 1850 3300 60  0001 L CNN "Field4"
@@
 F 0 "C55" H 3275 3200 50  0000 L CNN
 F 1 "100n" H 3275 3000 50  0000 L CNN
-F 2 "TinyTiM_Lib:c_0805" H 3250 3100 50  0001 C CNN
+F 2 "C4_Pretty:c_0805" H 3250 3100 50  0001 C CNN
 F 3 "" H 3250 3100 60  0001 C CNN
 F 4 "CAP CER 0.1UF 25V 10% X7R 0805" H 3250 3300 60  0001 L CNN "Field4"
@@
 F 0 "C56" H 4675 3200 50  0000 L CNN
 F 1 "100n" H 4675 3000 50  0000 L CNN
-F 2 "TinyTiM_Lib:c_0805" H 4650 3100 50  0001 C CNN
+F 2 "C4_Pretty:c_0805" H 4650 3100 50  0001 C CNN
 F 3 "" H 4650 3100 60  0001 C CNN
 F 4 "CAP CER 0.1UF 25V 10% X7R 0805" H 4650 3300 60  0001 L CNN "Field4"
@@
 F 0 "C57" H 6075 3200 50  0000 L CNN
 F 1 "100n" H 6075 3000 50  0000 L CNN
-F 2 "TinyTiM_Lib:c_0805" H 6050 3100 50  0001 C CNN
+F 2 "C4_Pretty:c_0805" H 6050 3100 50  0001 C CNN
 F 3 "" H 6050 3100 60  0001 C CNN
 F 4 "CAP CER 0.1UF 25V 10% X7R 0805" H 6050 3300 60  0001 L CNN "Field4"
@@
 F 0 "C58" H 7475 3200 50  0000 L CNN
 F 1 "100n" H 7475 3000 50  0000 L CNN
-F 2 "TinyTiM_Lib:c_0805" H 7450 3100 50  0001 C CNN
+F 2 "C4_Pretty:c_0805" H 7450 3100 50  0001 C CNN
 F 3 "" H 7450 3100 60  0001 C CNN
 F 4 "CAP CER 0.1UF 25V 10% X7R 0805" H 7450 3300 60  0001 L CNN "Field4"
@@
 F 0 "C59" H 8875 3200 50  0000 L CNN
 F 1 "100n" H 8875 3000 50  0000 L CNN
-F 2 "TinyTiM_Lib:c_0805" H 8850 3100 50  0001 C CNN
+F 2 "C4_Pretty:c_0805" H 8850 3100 50  0001 C CNN
 F 3 "" H 8850 3100 60  0001 C CNN
 F 4 "CAP CER 0.1UF 25V 10% X7R 0805" H 8850 3300 60  0001 L CNN "Field4"
@@
 F 0 "C60" H 10275 3200 50  0000 L CNN
 F 1 "100n" H 10275 3000 50  0000 L CNN
-F 2 "TinyTiM_Lib:c_0805" H 10250 3100 50  0001 C CNN
+F 2 "C4_Pretty:c_0805" H 10250 3100 50  0001 C CNN
 F 3 "" H 10250 3100 60  0001 C CNN
 F 4 "CAP CER 0.1UF 25V 10% X7R 0805" H 10250 3300 60  0001 L CNN "Field4"
@@
 F 0 "C61" H 1875 5550 50  0000 L CNN
 F 1 "100n" H 1875 5350 50  0000 L CNN
-F 2 "TinyTiM_Lib:c_0805" H 1850 5450 50  0001 C CNN
+F 2 "C4_Pretty:c_0805" H 1850 5450 50  0001 C CNN
 F 3 "" H 1850 5450 60  0001 C CNN
 F 4 "CAP CER 0.1UF 25V 10% X7R 0805" H 1850 5650 60  0001 L CNN "Field4"
@@
 F 0 "C62" H 3275 5550 50  0000 L CNN
 F 1 "100n" H 3275 5350 50  0000 L CNN
-F 2 "TinyTiM_Lib:c_0805" H 3250 5450 50  0001 C CNN
+F 2 "C4_Pretty:c_0805" H 3250 5450 50  0001 C CNN
 F 3 "" H 3250 5450 60  0001 C CNN
 F 4 "CAP CER 0.1UF 25V 10% X7R 0805" H 3250 5650 60  0001 L CNN "Field4"
@@
 F 0 "C63" H 4675 5550 50  0000 L CNN
 F 1 "100n" H 4675 5350 50  0000 L CNN
-F 2 "TinyTiM_Lib:c_0805" H 4650 5450 50  0001 C CNN
+F 2 "C4_Pretty:c_0805" H 4650 5450 50  0001 C CNN
 F 3 "" H 4650 5450 60  0001 C CNN
 F 4 "CAP CER 0.1UF 25V 10% X7R 0805" H 4650 5650 60  0001 L CNN "Field4"
@@
 F 0 "C64" H 6075 5550 50  0000 L CNN
 F 1 "100n" H 6075 5350 50  0000 L CNN
-F 2 "TinyTiM_Lib:c_0805" H 6050 5450 50  0001 C CNN
+F 2 "C4_Pretty:c_0805" H 6050 5450 50  0001 C CNN
 F 3 "" H 6050 5450 60  0001 C CNN
 F 4 "CAP CER 0.1UF 25V 10% X7R 0805" H 6050 5650 60  0001 L CNN "Field4"
@@
 F 0 "C65" H 7475 5550 50  0000 L CNN
 F 1 "100n" H 7475 5350 50  0000 L CNN
-F 2 "TinyTiM_Lib:c_0805" H 7450 5450 50  0001 C CNN
+F 2 "C4_Pretty:c_0805" H 7450 5450 50  0001 C CNN
 F 3 "" H 7450 5450 60  0001 C CNN
 F 4 "CAP CER 0.1UF 25V 10% X7R 0805" H 7450 5650 60  0001 L CNN "Field4"
@@
 F 0 "C66" H 8875 5550 50  0000 L CNN
 F 1 "100n" H 8875 5350 50  0000 L CNN
-F 2 "TinyTiM_Lib:c_0805" H 8850 5450 50  0001 C CNN
+F 2 "C4_Pretty:c_0805" H 8850 5450 50  0001 C CNN
 F 3 "" H 8850 5450 60  0001 C CNN
 F 4 "CAP CER 0.1UF 25V 10% X7R 0805" H 8850 5650 60  0001 L CNN "Field4"
@@
 F 0 "C67" H 10275 5550 50  0000 L CNN
 F 1 "100n" H 10275 5350 50  0000 L CNN
-F 2 "TinyTiM_Lib:c_0805" H 10250 5450 50  0001 C CNN
+F 2 "C4_Pretty:c_0805" H 10250 5450 50  0001 C CNN
 F 3 "" H 10250 5450 60  0001 C CNN
 F 4 "CAP CER 0.1UF 25V 10% X7R 0805" H 10250 5650 60  0001 L CNN "Field4"
@@
 F 0 "LED43" V 1425 2125 60  0000 C CNN
 F 1 "WS2812B" V 2075 2125 60  0001 C CNN
-F 2 "~" H 1675 2125 60  0000 C CNN
+F 2 "C4_Pretty:RGB_WS2811B" H 1675 2125 60  0001 C CNN
 F 3 "~" H 1675 2125 60  0000 C CNN
 	1    1675 2125
@@
 F 0 "LED44" V 2825 2125 60  0000 C CNN
 F 1 "WS2812B" V 3475 2125 60  0001 C CNN
-F 2 "~" H 3075 2125 60  0000 C CNN
+F 2 "C4_Pretty:RGB_WS2811B" H 3075 2125 60  0001 C CNN
 F 3 "~" H 3075 2125 60  0000 C CNN
 	1    3075 2125
@@
 F 0 "LED45" V 4225 2125 60  0000 C CNN
 F 1 "WS2812B" V 4875 2125 60  0001 C CNN
-F 2 "~" H 4475 2125 60  0000 C CNN
+F 2 "C4_Pretty:RGB_WS2811B" H 4475 2125 60  0001 C CNN
 F 3 "~" H 4475 2125 60  0000 C CNN
 	1    4475 2125
@@
 F 0 "LED46" V 5625 2125 60  0000 C CNN
 F 1 "WS2812B" V 6275 2125 60  0001 C CNN
-F 2 "~" H 5875 2125 60  0000 C CNN
+F 2 "C4_Pretty:RGB_WS2811B" H 5875 2125 60  0001 C CNN
 F 3 "~" H 5875 2125 60  0000 C CNN
 	1    5875 2125
@@
 F 0 "LED47" V 7025 2125 60  0000 C CNN
 F 1 "WS2812B" V 7675 2125 60  0001 C CNN
-F 2 "~" H 7275 2125 60  0000 C CNN
+F 2 "C4_Pretty:RGB_WS2811B" H 7275 2125 60  0001 C CNN
 F 3 "~" H 7275 2125 60  0000 C CNN
 	1    7275 2125
@@
 F 0 "LED48" V 8425 2125 60  0000 C CNN
 F 1 "WS2812B" V 9075 2125 60  0001 C CNN
-F 2 "~" H 8675 2125 60  0000 C CNN
+F 2 "C4_Pretty:RGB_WS2811B" H 8675 2125 60  0001 C CNN
 F 3 "~" H 8675 2125 60  0000 C CNN
 	1    8675 2125
@@
 F 0 "LED49" V 9825 2125 60  0000 C CNN
 F 1 "WS2812B" V 10475 2125 60  0001 C CNN
-F 2 "~" H 10075 2125 60  0000 C CNN
+F 2 "C4_Pretty:RGB_WS2811B" H 10075 2125 60  0001 C CNN
 F 3 "~" H 10075 2125 60  0000 C CNN
 	1    10075 2125
@@
 F 0 "LED50" V 1425 4525 60  0000 C CNN
 F 1 "WS2812B" V 2075 4525 60  0001 C CNN
-F 2 "~" H 1675 4525 60  0000 C CNN
+F 2 "C4_Pretty:RGB_WS2811B" H 1675 4525 60  0001 C CNN
 F 3 "~" H 1675 4525 60  0000 C CNN
 	1    1675 4525
@@
 F 0 "LED51" V 2825 4525 60  0000 C CNN
 F 1 "WS2812B" V 3475 4525 60  0001 C CNN
-F 2 "~" H 3075 4525 60  0000 C CNN
+F 2 "C4_Pretty:RGB_WS2811B" H 3075 4525 60  0001 C CNN
 F 3 "~" H 3075 4525 60  0000 C CNN
 	1    3075 4525
@@
 F 0 "LED52" V 4225 4525 60  0000 C CNN
 F 1 "WS2812B" V 4875 4525 60  0001 C CNN
-F 2 "~" H 4475 4525 60  0000 C CNN
+F 2 "C4_Pretty:RGB_WS2811B" H 4475 4525 60  0001 C CNN
 F 3 "~" H 4475 4525 60  0000 C CNN
 	1    4475 4525
@@
 F 0 "LED53" V 5625 4525 60  0000 C CNN
 F 1 "WS2812B" V 6275 4525 60  0001 C CNN
-F 2 "~" H 5875 4525 60  0000 C CNN
+F 2 "C4_Pretty:RGB_WS2811B" H 5875 4525 60  0001 C CNN
 F 3 "~" H 5875 4525 60  0000 C CNN
 	1    5875 4525
@@
 F 0 "LED54" V 7025 4525 60  0000 C CNN
 F 1 "WS2812B" V 7675 4525 60  0001 C CNN
-F 2 "~" H 7275 4525 60  0000 C CNN
+F 2 "C4_Pretty:RGB_WS2811B" H 7275 4525 60  0001 C CNN
 F 3 "~" H 7275 4525 60  0000 C CNN
 	1    7275 4525
@@
 F 0 "LED55" V 8425 4525 60  0000 C CNN
 F 1 "WS2812B" V 9075 4525 60  0001 C CNN
-F 2 "~" H 8675 4525 60  0000 C CNN
+F 2 "C4_Pretty:RGB_WS2811B" H 8675 4525 60  0001 C CNN
 F 3 "~" H 8675 4525 60  0000 C CNN
 	1    8675 4525
@@
 F 0 "LED56" V 9825 4525 60  0000 C CNN
 F 1 "WS2812B" V 10475 4525 60  0001 C CNN
-F 2 "~" H 10075 4525 60  0000 C CNN
+F 2 "C4_Pretty:RGB_WS2811B" H 10075 4525 60  0001 C CNN
 F 3 "~" H 10075 4525 60  0000 C CNN
 	1    10075 4525

Commit message: C4 PCB layout complete. Added Gerbers
Parts:
- C54, C55, C56, C57, C58, C59, C60, C61, C62, C63, C64, C65, C66, C67: footprint C4_Pretty:c_0805 -> C4_Pretty:c_0805_led
Changed lines of the file:
@@
 EESchema Schematic File Version 2
 LIBS:ClockFOUR
+LIBS:RowGB_sym
 LIBS:ClockFOUR-cache
 EELAYER 24 0
@@
 F 0 "C54" H 1875 3200 50  0000 L CNN
 F 1 "100n" H 1875 3000 50  0000 L CNN
-F 2 "C4_Pretty:c_0805" H 1850 3100 50  0001 C CNN
+F 2 "C4_Pretty:c_0805_led" H 1850 3100 50  0001 C CNN
 F 3 "" H 1850 3100 60  0001 C CNN
 F 4 "CAP CER 0.1UF 25V 10% X7R 0805" H 1850 3300 60  0001 L CNN "Field4"
@@
 F 0 "C55" H 3275 3200 50  0000 L CNN
 F 1 "100n" H 3275 3000 50  0000 L CNN
-F 2 "C4_Pretty:c_0805" H 3250 3100 50  0001 C CNN
+F 2 "C4_Pretty:c_0805_led" H 3250 3100 50  0001 C CNN
 F 3 "" H 3250 3100 60  0001 C CNN
 F 4 "CAP CER 0.1UF 25V 10% X7R 0805" H 3250 3300 60  0001 L CNN "Field4"
@@
 F 0 "C56" H 4675 3200 50  0000 L CNN
 F 1 "100n" H 4675 3000 50  0000 L CNN
-F 2 "C4_Pretty:c_0805" H 4650 3100 50  0001 C CNN
+F 2 "C4_Pretty:c_0805_led" H 4650 3100 50  0001 C CNN
 F 3 "" H 4650 3100 60  0001 C CNN
 F 4 "CAP CER 0.1UF 25V 10% X7R 0805" H 4650 3300 60  0001 L CNN "Field4"
@@
 F 0 "C57" H 6075 3200 50  0000 L CNN
 F 1 "100n" H 6075 3000 50  0000 L CNN
-F 2 "C4_Pretty:c_0805" H 6050 3100 50  0001 C CNN
+F 2 "C4_Pretty:c_0805_led" H 6050 3100 50  0001 C CNN
 F 3 "" H 6050 3100 60  0001 C CNN
 F 4 "CAP CER 0.1UF 25V 10% X7R 0805" H 6050 3300 60  0001 L CNN "Field4"
@@
 F 0 "C58" H 7475 3200 50  0000 L CNN
 F 1 "100n" H 7475 3000 50  0000 L CNN
-F 2 "C4_Pretty:c_0805" H 7450 3100 50  0001 C CNN
+F 2 "C4_Pretty:c_0805_led" H 7450 3100 50  0001 C CNN
 F 3 "" H 7450 3100 60  0001 C CNN
 F 4 "CAP CER 0.1UF 25V 10% X7R 0805" H 7450 3300 60  0001 L CNN "Field4"
@@
 F 0 "C59" H 8875 3200 50  0000 L CNN
 F 1 "100n" H 8875 3000 50  0000 L CNN
-F 2 "C4_Pretty:c_0805" H 8850 3100 50  0001 C CNN
+F 2 "C4_Pretty:c_0805_led" H 8850 3100 50  0001 C CNN
 F 3 "" H 8850 3100 60  0001 C CNN
 F 4 "CAP CER 0.1UF 25V 10% X7R 0805" H 8850 3300 60  0001 L CNN "Field4"
@@
 F 0 "C60" H 10275 3200 50  0000 L CNN
 F 1 "100n" H 10275 3000 50  0000 L CNN
-F 2 "C4_Pretty:c_0805" H 10250 3100 50  0001 C CNN
+F 2 "C4_Pretty:c_0805_led" H 10250 3100 50  0001 C CNN
 F 3 "" H 10250 3100 60  0001 C CNN
 F 4 "CAP CER 0.1UF 25V 10% X7R 0805" H 10250 3300 60  0001 L CNN "Field4"
@@
 F 0 "C61" H 1875 5550 50  0000 L CNN
 F 1 "100n" H 1875 5350 50  0000 L CNN
-F 2 "C4_Pretty:c_0805" H 1850 5450 50  0001 C CNN
+F 2 "C4_Pretty:c_0805_led" H 1850 5450 50  0001 C CNN
 F 3 "" H 1850 5450 60  0001 C CNN
 F 4 "CAP CER 0.1UF 25V 10% X7R 0805" H 1850 5650 60  0001 L CNN "Field4"
@@
 F 0 "C62" H 3275 5550 50  0000 L CNN
 F 1 "100n" H 3275 5350 50  0000 L CNN
-F 2 "C4_Pretty:c_0805" H 3250 5450 50  0001 C CNN
+F 2 "C4_Pretty:c_0805_led" H 3250 5450 50  0001 C CNN
 F 3 "" H 3250 5450 60  0001 C CNN
 F 4 "CAP CER 0.1UF 25V 10% X7R 0805" H 3250 5650 60  0001 L CNN "Field4"
@@
 F 0 "C63" H 4675 5550 50  0000 L CNN
 F 1 "100n" H 4675 5350 50  0000 L CNN
-F 2 "C4_Pretty:c_0805" H 4650 5450 50  0001 C CNN
+F 2 "C4_Pretty:c_0805_led" H 4650 5450 50  0001 C CNN
 F 3 "" H 4650 5450 60  0001 C CNN
 F 4 "CAP CER 0.1UF 25V 10% X7R 0805" H 4650 5650 60  0001 L CNN "Field4"
@@
 F 0 "C64" H 6075 5550 50  0000 L CNN
 F 1 "100n" H 6075 5350 50  0000 L CNN
-F 2 "C4_Pretty:c_0805" H 6050 5450 50  0001 C CNN
+F 2 "C4_Pretty:c_0805_led" H 6050 5450 50  0001 C CNN
 F 3 "" H 6050 5450 60  0001 C CNN
 F 4 "CAP CER 0.1UF 25V 10% X7R 0805" H 6050 5650 60  0001 L CNN "Field4"
@@
 F 0 "C65" H 7475 5550 50  0000 L CNN
 F 1 "100n" H 7475 5350 50  0000 L CNN
-F 2 "C4_Pretty:c_0805" H 7450 5450 50  0001 C CNN
+F 2 "C4_Pretty:c_0805_led" H 7450 5450 50  0001 C CNN
 F 3 "" H 7450 5450 60  0001 C CNN
 F 4 "CAP CER 0.1UF 25V 10% X7R 0805" H 7450 5650 60  0001 L CNN "Field4"
@@
 F 0 "C66" H 8875 5550 50  0000 L CNN
 F 1 "100n" H 8875 5350 50  0000 L CNN
-F 2 "C4_Pretty:c_0805" H 8850 5450 50  0001 C CNN
+F 2 "C4_Pretty:c_0805_led" H 8850 5450 50  0001 C CNN
 F 3 "" H 8850 5450 60  0001 C CNN
 F 4 "CAP CER 0.1UF 25V 10% X7R 0805" H 8850 5650 60  0001 L CNN "Field4"
@@
 F 0 "C67" H 10275 5550 50  0000 L CNN
 F 1 "100n" H 10275 5350 50  0000 L CNN
-F 2 "C4_Pretty:c_0805" H 10250 5450 50  0001 C CNN
+F 2 "C4_Pretty:c_0805_led" H 10250 5450 50  0001 C CNN
 F 3 "" H 10250 5450 60  0001 C CNN
 F 4 "CAP CER 0.1UF 25V 10% X7R 0805" H 10250 5650 60  0001 L CNN "Field4"
