File: KiCad/Row_E.sch (KiCad schematic (older format))
At the start: 14 parts, among them U101 RGB_WS2811B, U102 RGB_WS2811B, U103 RGB_WS2811B, U104 RGB_WS2811B, U105 RGB_WS2811B, U106 RGB_WS2811B, U107 RGB_WS2811B, U108 RGB_WS2811B

Commit message: Schematic updated
Parts:
- removed C101: 100n, TinyTiM_Lib:c_0805, symbol C2
- removed C117: 47u,8V, TinyTiM_Lib:c_2917, symbol C_POL_1
- removed S101, S102, S103, S104: CONN_1, TinyTiM_Lib:Screw, symbol CONN_1
- removed U101, U102, U103, U104, U105, U106, U107, U108: RGB_WS2811B, TinyTiM_Lib:RGB_WS2811B, symbol RGB_WS2811B
Connections:
- net labels removed: 5V, A_02, A_03, A_04, A_05, A_06, A_07, A_08, A_09, DI_A, DO_A, GND
- wire segments 49 -> 0
- no-connect marks 4 -> 0
Other:
- note removed: "Mounting Screws"

Commit message: Schematic updated
Parts:
- added C65, C66, C67, C68, C69, C70, C71, C72, C73, C74, C75, C76, C77, C78: 100n, TinyTiM_Lib:c_0805, symbol C2
- added U60, U61, U62, U63, U64, U65, U66, U67, U68, U69, U70, U71, U72, U73: RGB_WS2812B, symbol RGB_WS2812B
Connections:
- net labels added: 5V, DI_E, DO_E, GND
- wire segments 0 -> 82

Commit message: Schematic updated, board started
Parts:
- C67: renamed from C65; Field5 100nF, 25V -> 100n, 25V
- C69: Field5 100nF, 25V -> 100n, 25V
- C71: renamed from C73; Field5 100nF, 25V -> 100n, 25V
- C73: renamed from C77; Field5 100nF, 25V -> 100n, 25V
- C75: renamed from C68; Field5 100nF, 25V -> 100n, 25V
- C77: renamed from C72; Field5 100nF, 25V -> 100n, 25V
- C79: renamed from C76; Field5 100nF, 25V -> 100n, 25V
- renumbered C67 to C68, C71 to C70, C75 to C72, C66 to C74, C70 to C76, C74 to C78, C78 to C80, U60 to U58, U62 to U59, U64 to U60, U66 to U61, U68 to U62, U70 to U63, U72 to U64, U61 to U65, U63 to U66, U65 to U67, U67 to U68, U71 to U70, U73 to U71
Changed lines of the file:
@@
 LIBS:contrib
 LIBS:valves
-LIBS:TinyTiM-cache
-LIBS:TiNA_sym
+LIBS:ClockFOUR
 LIBS:ClockFOUR-cache
 EELAYER 27 0
@@
 Sheet 6 14
 Title "ClockFOUR"
-Date "30 sep 2014"
+Date "1 oct 2014"
 Rev ""
 Comp "WyoLum"
@@
 5V
 $Comp
-L GND #PWR016
+L GND #PWR018
 U 1 1 542C0C38
 P 1450 2600
-F 0 "#PWR016" H 1450 2600 30  0001 C CNN
+F 0 "#PWR018" H 1450 2600 30  0001 C CNN
 F 1 "GND" H 1450 2530 30  0001 C CNN
 F 2 "" H 1450 2600 60  0001 C CNN
@@
 $EndComp
 $Comp
-L C2 C65
+L C2 C67
 U 1 1 542C0C46
 P 2000 2750
-F 0 "C65" H 2025 2850 50  0000 L CNN
+F 0 "C67" H 2025 2850 50  0000 L CNN
 F 1 "100n" H 2025 2650 50  0000 L CNN
 F 2 "TinyTiM_Lib:c_0805" H 2000 2750 50  0001 C CNN
 F 3 "" H 2000 2750 60  0001 C CNN
 F 4 "CAP CER 0.1UF 25V 10% X7R 0805" H 2000 2950 60  0001 L CNN "Field4"
-F 5 "100nF, 25V" H 2000 3050 60  0001 L CNN "Field5"
+F 5 "100n, 25V" H 2000 3050 60  0001 L CNN "Field5"
 F 6 "Surface Mount, MLCC" H 2000 3150 60  0001 L CNN "Field6"
 F 7 "Kemet" H 2000 3250 60  0001 L CNN "Field7"
@@
 $EndComp
 $Comp
-L RGB_WS2812B U60
+L RGB_WS2812B U58
 U 1 1 542C0C4C
 P 1825 1775
-F 0 "U60" V 1575 1775 60  0000 C CNN
+F 0 "U58" V 1575 1775 60  0000 C CNN
 F 1 "RGB_WS2812B" V 2225 1775 60  0000 C CNN
 F 2 "" H 1825 1775 60  0000 C CNN
@@
 $EndComp
 $Comp
-L RGB_WS2812B U62
+L RGB_WS2812B U59
 U 1 1 542C0C52
 P 3225 1775
-F 0 "U62" V 2975 1775 60  0000 C CNN
+F 0 "U59" V 2975 1775 60  0000 C CNN
 F 1 "RGB_WS2812B" V 3625 1775 60  0000 C CNN
 F 2 "" H 3225 1775 60  0000 C CNN
@@
 $EndComp
 $Comp
-L RGB_WS2812B U64
+L RGB_WS2812B U60
 U 1 1 542C0C58
 P 4625 1775
-F 0 "U64" V 4375 1775 60  0000 C CNN
+F 0 "U60" V 4375 1775 60  0000 C CNN
 F 1 "RGB_WS2812B" V 5025 1775 60  0000 C CNN
 F 2 "" H 4625 1775 60  0000 C CNN
@@
 $EndComp
 $Comp
-L RGB_WS2812B U66
+L RGB_WS2812B U61
 U 1 1 542C0C5E
 P 6025 1775
-F 0 "U66" V 5775 1775 60  0000 C CNN
+F 0 "U61" V 5775 1775 60  0000 C CNN
 F 1 "RGB_WS2812B" V 6425 1775 60  0000 C CNN
 F 2 "" H 6025 1775 60  0000 C CNN
@@
 $EndComp
 $Comp
-L RGB_WS2812B U68
+L RGB_WS2812B U62
 U 1 1 542C0C64
 P 7425 1775
-F 0 "U68" V 7175 1775 60  0000 C CNN
+F 0 "U62" V 7175 1775 60  0000 C CNN
 F 1 "RGB_WS2812B" V 7825 1775 60  0000 C CNN
 F 2 "" H 7425 1775 60  0000 C CNN
@@
 $EndComp
 $Comp
-L RGB_WS2812B U70
+L RGB_WS2812B U63
 U 1 1 542C0C6A
 P 8825 1775
-F 0 "U70" V 8575 1775 60  0000 C CNN
+F 0 "U63" V 8575 1775 60  0000 C CNN
 F 1 "RGB_WS2812B" V 9225 1775 60  0000 C CNN
 F 2 "" H 8825 1775 60  0000 C CNN
@@
 $EndComp
 $Comp
-L RGB_WS2812B U72
+L RGB_WS2812B U64
 U 1 1 542C0C70
 P 10225 1775
-F 0 "U72" V 9975 1775 60  0000 C CNN
+F 0 "U64" V 9975 1775 60  0000 C CNN
 F 1 "RGB_WS2812B" V 10625 1775 60  0000 C CNN
 F 2 "" H 10225 1775 60  0000 C CNN
@@
 $EndComp
 $Comp
-L RGB_WS2812B U61
+L RGB_WS2812B U65
 U 1 1 542C0C76
 P 1825 4175
-F 0 "U61" V 1575 4175 60  0000 C CNN
+F 0 "U65" V 1575 4175 60  0000 C CNN
 F 1 "RGB_WS2812B" V 2225 4175 60  0000 C CNN
 F 2 "" H 1825 4175 60  0000 C CNN
@@
 $EndComp
 $Comp
-L RGB_WS2812B U63
+L RGB_WS2812B U66
 U 1 1 542C0C7C
 P 3225 4175
-F 0 "U63" V 2975 4175 60  0000 C CNN
+F 0 "U66" V 2975 4175 60  0000 C CNN
 F 1 "RGB_WS2812B" V 3625 4175 60  0000 C CNN
 F 2 "" H 3225 4175 60  0000 C CNN
@@
 $EndComp
 $Comp
-L RGB_WS2812B U65
+L RGB_WS2812B U67
 U 1 1 542C0C82
 P 4625 4175
-F 0 "U65" V 4375 4175 60  0000 C CNN
+F 0 "U67" V 4375 4175 60  0000 C CNN
 F 1 "RGB_WS2812B" V 5025 4175 60  0000 C CNN
 F 2 "" H 4625 4175 60  0000 C CNN
@@
 $EndComp
 $Comp
-L RGB_WS2812B U67
+L RGB_WS2812B U68
 U 1 1 542C0C88
 P 6025 4175
-F 0 "U67" V 5775 4175 60  0000 C CNN
+F 0 "U68" V 5775 4175 60  0000 C CNN
 F 1 "RGB_WS2812B" V 6425 4175 60  0000 C CNN
 F 2 "" H 6025 4175 60  0000 C CNN
@@
 $EndComp
 $Comp
-L RGB_WS2812B U71
+L RGB_WS2812B U70
 U 1 1 542C0C94
 P 8825 4175
-F 0 "U71" V 8575 4175 60  0000 C CNN
+F 0 "U70" V 8575 4175 60  0000 C CNN
 F 1 "RGB_WS2812B" V 9225 4175 60  0000 C CNN
 F 2 "" H 8825 4175 60  0000 C CNN
@@
 $EndComp
 $Comp
-L RGB_WS2812B U73
+L RGB_WS2812B U71
 U 1 1 542C0C9A
 P 10225 4175
-F 0 "U73" V 9975 4175 60  0000 C CNN
+F 0 "U71" V 9975 4175 60  0000 C CNN
 F 1 "RGB_WS2812B" V 10625 4175 60  0000 C CNN
 F 2 "" H 10225 4175 60  0000 C CNN
@@
 Connection ~ 1900 2950
 $Comp
-L C2 C67
+L C2 C68
 U 1 1 542C0CF5
 P 3400 2750
-F 0 "C67" H 3425 2850 50  0000 L CNN
+F 0 "C68" H 3425 2850 50  0000 L CNN
 F 1 "100n" H 3425 2650 50  0000 L CNN
 F 2 "TinyTiM_Lib:c_0805" H 3400 2750 50  0001 C CNN
@@
 F 3 "" H 4800 2750 60  0001 C CNN
 F 4 "CAP CER 0.1UF 25V 10% X7R 0805" H 4800 2950 60  0001 L CNN "Field4"
-F 5 "100nF, 25V" H 4800 3050 60  0001 L CNN "Field5"
+F 5 "100n, 25V" H 4800 3050 60  0001 L CNN "Field5"
 F 6 "Surface Mount, MLCC" H 4800 3150 60  0001 L CNN "Field6"
 F 7 "Kemet" H 4800 3250 60  0001 L CNN "Field7"
@@
 $EndComp
 $Comp
-L C2 C71
+L C2 C70
 U 1 1 542C0D11
 P 6200 2750
-F 0 "C71" H 6225 2850 50  0000 L CNN
+F 0 "C70" H 6225 2850 50  0000 L CNN
 F 1 "100n" H 6225 2650 50  0000 L CNN
 F 2 "TinyTiM_Lib:c_0805" H 6200 2750 50  0001 C CNN
@@
 $EndComp
 $Comp
-L C2 C73
+L C2 C71
 U 1 1 542C0D1F
 P 7600 2750
-F 0 "C73" H 7625 2850 50  0000 L CNN
+F 0 "C71" H 7625 2850 50  0000 L CNN
 F 1 "100n" H 7625 2650 50  0000 L CNN
 F 2 "TinyTiM_Lib:c_0805" H 7600 2750 50  0001 C CNN
 F 3 "" H 7600 2750 60  0001 C CNN
 F 4 "CAP CER 0.1UF 25V 10% X7R 0805" H 7600 2950 60  0001 L CNN "Field4"
-F 5 "100nF, 25V" H 7600 3050 60  0001 L CNN "Field5"
+F 5 "100n, 25V" H 7600 3050 60  0001 L CNN "Field5"
 F 6 "Surface Mount, MLCC" H 7600 3150 60  0001 L CNN "Field6"
 F 7 "Kemet" H 7600 3250 60  0001 L CNN "Field7"
@@
 $EndComp
 $Comp
-L C2 C75
+L C2 C72
 U 1 1 542C0D2D
 P 9000 2750
-F 0 "C75" H 9025 2850 50  0000 L CNN
+F 0 "C72" H 9025 2850 50  0000 L CNN
 F 1 "100n" H 9025 2650 50  0000 L CNN
 F 2 "TinyTiM_Lib:c_0805" H 9000 2750 50  0001 C CNN
@@
 $EndComp
 $Comp
-L C2 C77
+L C2 C73
 U 1 1 542C0D3B
 P 10400 2750
-F 0 "C77" H 10425 2850 50  0000 L CNN
+F 0 "C73" H 10425 2850 50  0000 L CNN
 F 1 "100n" H 10425 2650 50  0000 L CNN
 F 2 "TinyTiM_Lib:c_0805" H 10400 2750 50  0001 C CNN
 F 3 "" H 10400 2750 60  0001 C CNN
 F 4 "CAP CER 0.1UF 25V 10% X7R 0805" H 10400 2950 60  0001 L CNN "Field4"
-F 5 "100nF, 25V" H 10400 3050 60  0001 L CNN "Field5"
+F 5 "100n, 25V" H 10400 3050 60  0001 L CNN "Field5"
 F 6 "Surface Mount, MLCC" H 10400 3150 60  0001 L CNN "Field6"
 F 7 "Kemet" H 10400 3250 60  0001 L CNN "Field7"
@@
 Connection ~ 10300 2950
 $Comp
-L C2 C66
+L C2 C74
 U 1 1 542C0D4A
 P 2000 5100
-F 0 "C66" H 2025 5200 50  0000 L CNN
+F 0 "C74" H 2025 5200 50  0000 L CNN
 F 1 "100n" H 2025 5000 50  0000 L CNN
 F 2 "TinyTiM_Lib:c_0805" H 2000 5100 50  0001 C CNN
@@
 Connection ~ 1900 5300
 $Comp
-L C2 C68
+L C2 C75
 U 1 1 542C0D87
 P 3400 5100
-F 0 "C68" H 3425 5200 50  0000 L CNN
+F 0 "C75" H 3425 5200 50  0000 L CNN
 F 1 "100n" H 3425 5000 50  0000 L CNN
 F 2 "TinyTiM_Lib:c_0805" H 3400 5100 50  0001 C CNN
 F 3 "" H 3400 5100 60  0001 C CNN
 F 4 "CAP CER 0.1UF 25V 10% X7R 0805" H 3400 5300 60  0001 L CNN "Field4"
-F 5 "100nF, 25V" H 3400 5400 60  0001 L CNN "Field5"
+F 5 "100n, 25V" H 3400 5400 60  0001 L CNN "Field5"
 F 6 "Surface Mount, MLCC" H 3400 5500 60  0001 L CNN "Field6"
 F 7 "Kemet" H 3400 5600 60  0001 L CNN "Field7"
@@
 $EndComp
 $Comp
-L C2 C70
+L C2 C76
 U 1 1 542C0D95
 P 4800 5100
-F 0 "C70" H 4825 5200 50  0000 L CNN
+F 0 "C76" H 4825 5200 50  0000 L CNN
 F 1 "100n" H 4825 5000 50  0000 L CNN
 F 2 "TinyTiM_Lib:c_0805" H 4800 5100 50  0001 C CNN
@@
 $EndComp
 $Comp
-L C2 C72
+L C2 C77
 U 1 1 542C0DA3
 P 6200 5100
-F 0 "C72" H 6225 5200 50  0000 L CNN
+F 0 "C77" H 6225 5200 50  0000 L CNN
 F 1 "100n" H 6225 5000 50  0000 L CNN
 F 2 "TinyTiM_Lib:c_0805" H 6200 5100 50  0001 C CNN
 F 3 "" H 6200 5100 60  0001 C CNN
 F 4 "CAP CER 0.1UF 25V 10% X7R 0805" H 6200 5300 60  0001 L CNN "Field4"
-F 5 "100nF, 25V" H 6200 5400 60  0001 L CNN "Field5"
+F 5 "100n, 25V" H 6200 5400 60  0001 L CNN "Field5"
 F 6 "Surface Mount, MLCC" H 6200 5500 60  0001 L CNN "Field6"
 F 7 "Kemet" H 6200 5600 60  0001 L CNN "Field7"
@@
 $EndComp
 $Comp
-L C2 C74
+L C2 C78
 U 1 1 542C0DB1
 P 7600 5100
-F 0 "C74" H 7625 5200 50  0000 L CNN
+F 0 "C78" H 7625 5200 50  0000 L CNN
 F 1 "100n" H 7625 5000 50  0000 L CNN
 F 2 "TinyTiM_Lib:c_0805" H 7600 5100 50  0001 C CNN
@@
 $EndComp
 $Comp
-L C2 C76
+L C2 C79
 U 1 1 542C0DBF
 P 9000 5100
-F 0 "C76" H 9025 5200 50  0000 L CNN
+F 0 "C79" H 9025 5200 50  0000 L CNN
 F 1 "100n" H 9025 5000 50  0000 L CNN
 F 2 "TinyTiM_Lib:c_0805" H 9000 5100 50  0001 C CNN
 F 3 "" H 9000 5100 60  0001 C CNN
 F 4 "CAP CER 0.1UF 25V 10% X7R 0805" H 9000 5300 60  0001 L CNN "Field4"
-F 5 "100nF, 25V" H 9000 5400 60  0001 L CNN "Field5"
+F 5 "100n, 25V" H 9000 5400 60  0001 L CNN "Field5"
 F 6 "Surface Mount, MLCC" H 9000 5500 60  0001 L CNN "Field6"
 F 7 "Kemet" H 9000 5600 60  0001 L CNN "Field7"
@@
 $EndComp
 $Comp
-L C2 C78
+L C2 C80
 U 1 1 542C0DCD
 P 10400 5100
-F 0 "C78" H 10425 5200 50  0000 L CNN
+F 0 "C80" H 10425 5200 50  0000 L CNN
 F 1 "100n" H 10425 5000 50  0000 L CNN
 F 2 "TinyTiM_Lib:c_0805" H 10400 5100 50  0001 C CNN

Commit message: Board layout updated
Parts:
- removed U58, U59, U60, U61, U62, U63, U64, U65, U66, U67, U68, U69, U70, U71: RGB_WS2812B, symbol RGB_WS2812B
- added LED57, LED58, LED59, LED60, LED61, LED62, LED63, LED64, LED65, LED66, LED67, LED68, LED69, LED70: RGB_WS2812B, ~, symbol RGB_WS2812B

Commit message: Board layout updated
Matrix placed and wired. Added RTC.
Parts:
- removed C67: 100n, TinyTiM_Lib:c_0805, symbol C2
- removed LED57, LED58, LED59, LED60, LED61, LED62, LED63, LED64, LED65, LED66, LED67, LED68, LED69, LED70: RGB_WS2812B, ~, symbol RGB_WS2812B
- added C81: 100n, TinyTiM_Lib:c_0805, symbol C2
- added LED57, LED58, LED59, LED60, LED61, LED62, LED63, LED64, LED65, LED66, LED67, LED68, LED69, LED70: WS2812B, ~, symbol WS2812B
- C68, C70, C72, C74, C76, C78, C80: Field5 100nF, 25V -> 100n, 25V
- C69, C71, C73, C75, C77, C79: Field5 100n, 25V -> 100nF, 25V
