File: KiCad/Row_E.sch (KiCad schematic (older format))
At the start: 28 parts

Commit message: PCB layout, work in progress
Parts:
- C68, C69, C70, C71, C72, C73, C74, C75, C76, C77, C78, C79, C80, C81: footprint TinyTiM_Lib:c_0805 -> C4_Pretty:c_0805
- LED57, LED58, LED59, LED60, LED61, LED62, LED63, LED64, LED65, LED66, LED67, LED68, LED69, LED70: footprint ~ -> C4_Pretty:RGB_WS2811B
Changed lines of the file:
@@
 F 0 "C68" H 1975 2750 50  0000 L CNN
 F 1 "100n" H 1975 2550 50  0000 L CNN
-F 2 "TinyTiM_Lib:c_0805" H 1950 2650 50  0001 C CNN
+F 2 "C4_Pretty:c_0805" H 1950 2650 50  0001 C CNN
 F 3 "" H 1950 2650 60  0001 C CNN
 F 4 "CAP CER 0.1UF 25V 10% X7R 0805" H 1950 2850 60  0001 L CNN "Field4"
@@
 F 0 "C69" H 3375 2750 50  0000 L CNN
 F 1 "100n" H 3375 2550 50  0000 L CNN
-F 2 "TinyTiM_Lib:c_0805" H 3350 2650 50  0001 C CNN
+F 2 "C4_Pretty:c_0805" H 3350 2650 50  0001 C CNN
 F 3 "" H 3350 2650 60  0001 C CNN
 F 4 "CAP CER 0.1UF 25V 10% X7R 0805" H 3350 2850 60  0001 L CNN "Field4"
@@
 F 0 "C70" H 4775 2750 50  0000 L CNN
 F 1 "100n" H 4775 2550 50  0000 L CNN
-F 2 "TinyTiM_Lib:c_0805" H 4750 2650 50  0001 C CNN
+F 2 "C4_Pretty:c_0805" H 4750 2650 50  0001 C CNN
 F 3 "" H 4750 2650 60  0001 C CNN
 F 4 "CAP CER 0.1UF 25V 10% X7R 0805" H 4750 2850 60  0001 L CNN "Field4"
@@
 F 0 "C71" H 6175 2750 50  0000 L CNN
 F 1 "100n" H 6175 2550 50  0000 L CNN
-F 2 "TinyTiM_Lib:c_0805" H 6150 2650 50  0001 C CNN
+F 2 "C4_Pretty:c_0805" H 6150 2650 50  0001 C CNN
 F 3 "" H 6150 2650 60  0001 C CNN
 F 4 "CAP CER 0.1UF 25V 10% X7R 0805" H 6150 2850 60  0001 L CNN "Field4"
@@
 F 0 "C72" H 7575 2750 50  0000 L CNN
 F 1 "100n" H 7575 2550 50  0000 L CNN
-F 2 "TinyTiM_Lib:c_0805" H 7550 2650 50  0001 C CNN
+F 2 "C4_Pretty:c_0805" H 7550 2650 50  0001 C CNN
 F 3 "" H 7550 2650 60  0001 C CNN
 F 4 "CAP CER 0.1UF 25V 10% X7R 0805" H 7550 2850 60  0001 L CNN "Field4"
@@
 F 0 "C73" H 8975 2750 50  0000 L CNN
 F 1 "100n" H 8975 2550 50  0000 L CNN
-F 2 "TinyTiM_Lib:c_0805" H 8950 2650 50  0001 C CNN
+F 2 "C4_Pretty:c_0805" H 8950 2650 50  0001 C CNN
 F 3 "" H 8950 2650 60  0001 C CNN
 F 4 "CAP CER 0.1UF 25V 10% X7R 0805" H 8950 2850 60  0001 L CNN "Field4"
@@
 F 0 "C74" H 10375 2750 50  0000 L CNN
 F 1 "100n" H 10375 2550 50  0000 L CNN
-F 2 "TinyTiM_Lib:c_0805" H 10350 2650 50  0001 C CNN
+F 2 "C4_Pretty:c_0805" H 10350 2650 50  0001 C CNN
 F 3 "" H 10350 2650 60  0001 C CNN
 F 4 "CAP CER 0.1UF 25V 10% X7R 0805" H 10350 2850 60  0001 L CNN "Field4"
@@
 F 0 "C75" H 1975 5100 50  0000 L CNN
 F 1 "100n" H 1975 4900 50  0000 L CNN
-F 2 "TinyTiM_Lib:c_0805" H 1950 5000 50  0001 C CNN
+F 2 "C4_Pretty:c_0805" H 1950 5000 50  0001 C CNN
 F 3 "" H 1950 5000 60  0001 C CNN
 F 4 "CAP CER 0.1UF 25V 10% X7R 0805" H 1950 5200 60  0001 L CNN "Field4"
@@
 F 0 "C76" H 3375 5100 50  0000 L CNN
 F 1 "100n" H 3375 4900 50  0000 L CNN
-F 2 "TinyTiM_Lib:c_0805" H 3350 5000 50  0001 C CNN
+F 2 "C4_Pretty:c_0805" H 3350 5000 50  0001 C CNN
 F 3 "" H 3350 5000 60  0001 C CNN
 F 4 "CAP CER 0.1UF 25V 10% X7R 0805" H 3350 5200 60  0001 L CNN "Field4"
@@
 F 0 "C77" H 4775 5100 50  0000 L CNN
 F 1 "100n" H 4775 4900 50  0000 L CNN
-F 2 "TinyTiM_Lib:c_0805" H 4750 5000 50  0001 C CNN
+F 2 "C4_Pretty:c_0805" H 4750 5000 50  0001 C CNN
 F 3 "" H 4750 5000 60  0001 C CNN
 F 4 "CAP CER 0.1UF 25V 10% X7R 0805" H 4750 5200 60  0001 L CNN "Field4"
@@
 F 0 "C78" H 6175 5100 50  0000 L CNN
 F 1 "100n" H 6175 4900 50  0000 L CNN
-F 2 "TinyTiM_Lib:c_0805" H 6150 5000 50  0001 C CNN
+F 2 "C4_Pretty:c_0805" H 6150 5000 50  0001 C CNN
 F 3 "" H 6150 5000 60  0001 C CNN
 F 4 "CAP CER 0.1UF 25V 10% X7R 0805" H 6150 5200 60  0001 L CNN "Field4"
@@
 F 0 "C79" H 7575 5100 50  0000 L CNN
 F 1 "100n" H 7575 4900 50  0000 L CNN
-F 2 "TinyTiM_Lib:c_0805" H 7550 5000 50  0001 C CNN
+F 2 "C4_Pretty:c_0805" H 7550 5000 50  0001 C CNN
 F 3 "" H 7550 5000 60  0001 C CNN
 F 4 "CAP CER 0.1UF 25V 10% X7R 0805" H 7550 5200 60  0001 L CNN "Field4"
@@
 F 0 "C80" H 8975 5100 50  0000 L CNN
 F 1 "100n" H 8975 4900 50  0000 L CNN
-F 2 "TinyTiM_Lib:c_0805" H 8950 5000 50  0001 C CNN
+F 2 "C4_Pretty:c_0805" H 8950 5000 50  0001 C CNN
 F 3 "" H 8950 5000 60  0001 C CNN
 F 4 "CAP CER 0.1UF 25V 10% X7R 0805" H 8950 5200 60  0001 L CNN "Field4"
@@
 F 0 "C81" H 10375 5100 50  0000 L CNN
 F 1 "100n" H 10375 4900 50  0000 L CNN
-F 2 "TinyTiM_Lib:c_0805" H 10350 5000 50  0001 C CNN
+F 2 "C4_Pretty:c_0805" H 10350 5000 50  0001 C CNN
 F 3 "" H 10350 5000 60  0001 C CNN
 F 4 "CAP CER 0.1UF 25V 10% X7R 0805" H 10350 5200 60  0001 L CNN "Field4"
@@
 F 0 "LED57" V 1525 1675 60  0000 C CNN
 F 1 "WS2812B" V 2175 1675 60  0001 C CNN
-F 2 "~" H 1775 1675 60  0000 C CNN
+F 2 "C4_Pretty:RGB_WS2811B" H 1775 1675 60  0001 C CNN
 F 3 "~" H 1775 1675 60  0000 C CNN
 	1    1775 1675
@@
 F 0 "LED58" V 2925 1675 60  0000 C CNN
 F 1 "WS2812B" V 3575 1675 60  0001 C CNN
-F 2 "~" H 3175 1675 60  0000 C CNN
+F 2 "C4_Pretty:RGB_WS2811B" H 3175 1675 60  0001 C CNN
 F 3 "~" H 3175 1675 60  0000 C CNN
 	1    3175 1675
@@
 F 0 "LED59" V 4325 1675 60  0000 C CNN
 F 1 "WS2812B" V 4975 1675 60  0001 C CNN
-F 2 "~" H 4575 1675 60  0000 C CNN
+F 2 "C4_Pretty:RGB_WS2811B" H 4575 1675 60  0001 C CNN
 F 3 "~" H 4575 1675 60  0000 C CNN
 	1    4575 1675
@@
 F 0 "LED60" V 5725 1675 60  0000 C CNN
 F 1 "WS2812B" V 6375 1675 60  0001 C CNN
-F 2 "~" H 5975 1675 60  0000 C CNN
+F 2 "C4_Pretty:RGB_WS2811B" H 5975 1675 60  0001 C CNN
 F 3 "~" H 5975 1675 60  0000 C CNN
 	1    5975 1675
@@
 F 0 "LED61" V 7125 1675 60  0000 C CNN
 F 1 "WS2812B" V 7775 1675 60  0001 C CNN
-F 2 "~" H 7375 1675 60  0000 C CNN
+F 2 "C4_Pretty:RGB_WS2811B" H 7375 1675 60  0001 C CNN
 F 3 "~" H 7375 1675 60  0000 C CNN
 	1    7375 1675
@@
 F 0 "LED62" V 8525 1675 60  0000 C CNN
 F 1 "WS2812B" V 9175 1675 60  0001 C CNN
-F 2 "~" H 8775 1675 60  0000 C CNN
+F 2 "C4_Pretty:RGB_WS2811B" H 8775 1675 60  0001 C CNN
 F 3 "~" H 8775 1675 60  0000 C CNN
 	1    8775 1675
@@
 F 0 "LED63" V 9925 1675 60  0000 C CNN
 F 1 "WS2812B" V 10575 1675 60  0001 C CNN
-F 2 "~" H 10175 1675 60  0000 C CNN
+F 2 "C4_Pretty:RGB_WS2811B" H 10175 1675 60  0001 C CNN
 F 3 "~" H 10175 1675 60  0000 C CNN
 	1    10175 1675
@@
 F 0 "LED64" V 1525 4075 60  0000 C CNN
 F 1 "WS2812B" V 2175 4075 60  0001 C CNN
-F 2 "~" H 1775 4075 60  0000 C CNN
+F 2 "C4_Pretty:RGB_WS2811B" H 1775 4075 60  0001 C CNN
 F 3 "~" H 1775 4075 60  0000 C CNN
 	1    1775 4075
@@
 F 0 "LED65" V 2925 4075 60  0000 C CNN
 F 1 "WS2812B" V 3575 4075 60  0001 C CNN
-F 2 "~" H 3175 4075 60  0000 C CNN
+F 2 "C4_Pretty:RGB_WS2811B" H 3175 4075 60  0001 C CNN
 F 3 "~" H 3175 4075 60  0000 C CNN
 	1    3175 4075
@@
 F 0 "LED66" V 4325 4075 60  0000 C CNN
 F 1 "WS2812B" V 4975 4075 60  0001 C CNN
-F 2 "~" H 4575 4075 60  0000 C CNN
+F 2 "C4_Pretty:RGB_WS2811B" H 4575 4075 60  0001 C CNN
 F 3 "~" H 4575 4075 60  0000 C CNN
 	1    4575 4075
@@
 F 0 "LED67" V 5725 4075 60  0000 C CNN
 F 1 "WS2812B" V 6375 4075 60  0001 C CNN
-F 2 "~" H 5975 4075 60  0000 C CNN
+F 2 "C4_Pretty:RGB_WS2811B" H 5975 4075 60  0001 C CNN
 F 3 "~" H 5975 4075 60  0000 C CNN
 	1    5975 4075
@@
 F 0 "LED68" V 7125 4075 60  0000 C CNN
 F 1 "WS2812B" V 7775 4075 60  0001 C CNN
-F 2 "~" H 7375 4075 60  0000 C CNN
+F 2 "C4_Pretty:RGB_WS2811B" H 7375 4075 60  0001 C CNN
 F 3 "~" H 7375 4075 60  0000 C CNN
 	1    7375 4075
@@
 F 0 "LED69" V 8525 4075 60  0000 C CNN
 F 1 "WS2812B" V 9175 4075 60  0001 C CNN
-F 2 "~" H 8775 4075 60  0000 C CNN
+F 2 "C4_Pretty:RGB_WS2811B" H 8775 4075 60  0001 C CNN
 F 3 "~" H 8775 4075 60  0000 C CNN
 	1    8775 4075
@@
 F 0 "LED70" V 9925 4075 60  0000 C CNN
 F 1 "WS2812B" V 10575 4075 60  0001 C CNN
-F 2 "~" H 10175 4075 60  0000 C CNN
+F 2 "C4_Pretty:RGB_WS2811B" H 10175 4075 60  0001 C CNN
 F 3 "~" H 10175 4075 60  0000 C CNN
 	1    10175 4075

Commit message: C4 PCB layout complete. Added Gerbers
Parts:
- C68, C69, C70, C71, C72, C73, C74, C75, C76, C77, C78, C79, C80, C81: footprint C4_Pretty:c_0805 -> C4_Pretty:c_0805_led
Changed lines of the file:
@@
 EESchema Schematic File Version 2
 LIBS:ClockFOUR
+LIBS:RowGB_sym
 LIBS:ClockFOUR-cache
 EELAYER 24 0
@@
 F 0 "C68" H 1975 2750 50  0000 L CNN
 F 1 "100n" H 1975 2550 50  0000 L CNN
-F 2 "C4_Pretty:c_0805" H 1950 2650 50  0001 C CNN
+F 2 "C4_Pretty:c_0805_led" H 1950 2650 50  0001 C CNN
 F 3 "" H 1950 2650 60  0001 C CNN
 F 4 "CAP CER 0.1UF 25V 10% X7R 0805" H 1950 2850 60  0001 L CNN "Field4"
@@
 F 0 "C69" H 3375 2750 50  0000 L CNN
 F 1 "100n" H 3375 2550 50  0000 L CNN
-F 2 "C4_Pretty:c_0805" H 3350 2650 50  0001 C CNN
+F 2 "C4_Pretty:c_0805_led" H 3350 2650 50  0001 C CNN
 F 3 "" H 3350 2650 60  0001 C CNN
 F 4 "CAP CER 0.1UF 25V 10% X7R 0805" H 3350 2850 60  0001 L CNN "Field4"
@@
 F 0 "C70" H 4775 2750 50  0000 L CNN
 F 1 "100n" H 4775 2550 50  0000 L CNN
-F 2 "C4_Pretty:c_0805" H 4750 2650 50  0001 C CNN
+F 2 "C4_Pretty:c_0805_led" H 4750 2650 50  0001 C CNN
 F 3 "" H 4750 2650 60  0001 C CNN
 F 4 "CAP CER 0.1UF 25V 10% X7R 0805" H 4750 2850 60  0001 L CNN "Field4"
@@
 F 0 "C71" H 6175 2750 50  0000 L CNN
 F 1 "100n" H 6175 2550 50  0000 L CNN
-F 2 "C4_Pretty:c_0805" H 6150 2650 50  0001 C CNN
+F 2 "C4_Pretty:c_0805_led" H 6150 2650 50  0001 C CNN
 F 3 "" H 6150 2650 60  0001 C CNN
 F 4 "CAP CER 0.1UF 25V 10% X7R 0805" H 6150 2850 60  0001 L CNN "Field4"
@@
 F 0 "C72" H 7575 2750 50  0000 L CNN
 F 1 "100n" H 7575 2550 50  0000 L CNN
-F 2 "C4_Pretty:c_0805" H 7550 2650 50  0001 C CNN
+F 2 "C4_Pretty:c_0805_led" H 7550 2650 50  0001 C CNN
 F 3 "" H 7550 2650 60  0001 C CNN
 F 4 "CAP CER 0.1UF 25V 10% X7R 0805" H 7550 2850 60  0001 L CNN "Field4"
@@
 F 0 "C73" H 8975 2750 50  0000 L CNN
 F 1 "100n" H 8975 2550 50  0000 L CNN
-F 2 "C4_Pretty:c_0805" H 8950 2650 50  0001 C CNN
+F 2 "C4_Pretty:c_0805_led" H 8950 2650 50  0001 C CNN
 F 3 "" H 8950 2650 60  0001 C CNN
 F 4 "CAP CER 0.1UF 25V 10% X7R 0805" H 8950 2850 60  0001 L CNN "Field4"
@@
 F 0 "C74" H 10375 2750 50  0000 L CNN
 F 1 "100n" H 10375 2550 50  0000 L CNN
-F 2 "C4_Pretty:c_0805" H 10350 2650 50  0001 C CNN
+F 2 "C4_Pretty:c_0805_led" H 10350 2650 50  0001 C CNN
 F 3 "" H 10350 2650 60  0001 C CNN
 F 4 "CAP CER 0.1UF 25V 10% X7R 0805" H 10350 2850 60  0001 L CNN "Field4"
@@
 F 0 "C75" H 1975 5100 50  0000 L CNN
 F 1 "100n" H 1975 4900 50  0000 L CNN
-F 2 "C4_Pretty:c_0805" H 1950 5000 50  0001 C CNN
+F 2 "C4_Pretty:c_0805_led" H 1950 5000 50  0001 C CNN
 F 3 "" H 1950 5000 60  0001 C CNN
 F 4 "CAP CER 0.1UF 25V 10% X7R 0805" H 1950 5200 60  0001 L CNN "Field4"
@@
 F 0 "C76" H 3375 5100 50  0000 L CNN
 F 1 "100n" H 3375 4900 50  0000 L CNN
-F 2 "C4_Pretty:c_0805" H 3350 5000 50  0001 C CNN
+F 2 "C4_Pretty:c_0805_led" H 3350 5000 50  0001 C CNN
 F 3 "" H 3350 5000 60  0001 C CNN
 F 4 "CAP CER 0.1UF 25V 10% X7R 0805" H 3350 5200 60  0001 L CNN "Field4"
@@
 F 0 "C77" H 4775 5100 50  0000 L CNN
 F 1 "100n" H 4775 4900 50  0000 L CNN
-F 2 "C4_Pretty:c_0805" H 4750 5000 50  0001 C CNN
+F 2 "C4_Pretty:c_0805_led" H 4750 5000 50  0001 C CNN
 F 3 "" H 4750 5000 60  0001 C CNN
 F 4 "CAP CER 0.1UF 25V 10% X7R 0805" H 4750 5200 60  0001 L CNN "Field4"
@@
 F 0 "C78" H 6175 5100 50  0000 L CNN
 F 1 "100n" H 6175 4900 50  0000 L CNN
-F 2 "C4_Pretty:c_0805" H 6150 5000 50  0001 C CNN
+F 2 "C4_Pretty:c_0805_led" H 6150 5000 50  0001 C CNN
 F 3 "" H 6150 5000 60  0001 C CNN
 F 4 "CAP CER 0.1UF 25V 10% X7R 0805" H 6150 5200 60  0001 L CNN "Field4"
@@
 F 0 "C79" H 7575 5100 50  0000 L CNN
 F 1 "100n" H 7575 4900 50  0000 L CNN
-F 2 "C4_Pretty:c_0805" H 7550 5000 50  0001 C CNN
+F 2 "C4_Pretty:c_0805_led" H 7550 5000 50  0001 C CNN
 F 3 "" H 7550 5000 60  0001 C CNN
 F 4 "CAP CER 0.1UF 25V 10% X7R 0805" H 7550 5200 60  0001 L CNN "Field4"
@@
 F 0 "C80" H 8975 5100 50  0000 L CNN
 F 1 "100n" H 8975 4900 50  0000 L CNN
-F 2 "C4_Pretty:c_0805" H 8950 5000 50  0001 C CNN
+F 2 "C4_Pretty:c_0805_led" H 8950 5000 50  0001 C CNN
 F 3 "" H 8950 5000 60  0001 C CNN
 F 4 "CAP CER 0.1UF 25V 10% X7R 0805" H 8950 5200 60  0001 L CNN "Field4"
@@
 F 0 "C81" H 10375 5100 50  0000 L CNN
 F 1 "100n" H 10375 4900 50  0000 L CNN
-F 2 "C4_Pretty:c_0805" H 10350 5000 50  0001 C CNN
+F 2 "C4_Pretty:c_0805_led" H 10350 5000 50  0001 C CNN
 F 3 "" H 10350 5000 60  0001 C CNN
 F 4 "CAP CER 0.1UF 25V 10% X7R 0805" H 10350 5200 60  0001 L CNN "Field4"
