File: KiCad/Row_F.sch (KiCad schematic (older format))
At the start: 0 parts

Commit message: Schematic updated
Parts:
- added C79, C80, C81, C82, C83, C84, C85, C86, C87, C88, C89, C90, C91, C92: 100n, TinyTiM_Lib:c_0805, symbol C2
- added U74, U75, U76, U77, U78, U79, U80, U81, U82, U83, U84, U85, U86, U87: RGB_WS2812B, symbol RGB_WS2812B
Connections:
- net labels added: 5V, DI_F, DO_F, GND
- wire segments 0 -> 82

Commit message: Schematic updated, board started
Parts:
- C81: renamed from C79; Field5 100nF, 25V -> 100n, 25V
- C83: Field5 100nF, 25V -> 100n, 25V
- C85: renamed from C87; Field5 100nF, 25V -> 100n, 25V
- C87: renamed from C91; Field5 100nF, 25V -> 100n, 25V
- C89: renamed from C82; Field5 100nF, 25V -> 100n, 25V
- C91: renamed from C86; Field5 100nF, 25V -> 100n, 25V
- C93: renamed from C90; Field5 100nF, 25V -> 100n, 25V
- renumbered C81 to C82, C85 to C84, C89 to C86, C80 to C88, C84 to C90, C88 to C92, C92 to C94, U74 to U72, U76 to U73, U78 to U74, U80 to U75, U82 to U76, U84 to U77, U86 to U78, U75 to U79, U77 to U80, U79 to U81, U81 to U82, U85 to U84, U87 to U85
Changed lines of the file:
@@
 LIBS:contrib
 LIBS:valves
-LIBS:TinyTiM-cache
-LIBS:TiNA_sym
+LIBS:ClockFOUR
 LIBS:ClockFOUR-cache
 EELAYER 27 0
@@
 Sheet 7 14
 Title "ClockFOUR"
-Date "30 sep 2014"
+Date "1 oct 2014"
 Rev ""
 Comp "WyoLum"
@@
 5V
 $Comp
-L GND #PWR017
+L GND #PWR019
 U 1 1 542C0DE5
 P 1400 2650
-F 0 "#PWR017" H 1400 2650 30  0001 C CNN
+F 0 "#PWR019" H 1400 2650 30  0001 C CNN
 F 1 "GND" H 1400 2580 30  0001 C CNN
 F 2 "" H 1400 2650 60  0001 C CNN
@@
 $EndComp
 $Comp
-L C2 C79
+L C2 C81
 U 1 1 542C0DF3
 P 1950 2800
-F 0 "C79" H 1975 2900 50  0000 L CNN
+F 0 "C81" H 1975 2900 50  0000 L CNN
 F 1 "100n" H 1975 2700 50  0000 L CNN
 F 2 "TinyTiM_Lib:c_0805" H 1950 2800 50  0001 C CNN
 F 3 "" H 1950 2800 60  0001 C CNN
 F 4 "CAP CER 0.1UF 25V 10% X7R 0805" H 1950 3000 60  0001 L CNN "Field4"
-F 5 "100nF, 25V" H 1950 3100 60  0001 L CNN "Field5"
+F 5 "100n, 25V" H 1950 3100 60  0001 L CNN "Field5"
 F 6 "Surface Mount, MLCC" H 1950 3200 60  0001 L CNN "Field6"
 F 7 "Kemet" H 1950 3300 60  0001 L CNN "Field7"
@@
 $EndComp
 $Comp
-L RGB_WS2812B U74
+L RGB_WS2812B U72
 U 1 1 542C0DF9
 P 1775 1825
-F 0 "U74" V 1525 1825 60  0000 C CNN
+F 0 "U72" V 1525 1825 60  0000 C CNN
 F 1 "RGB_WS2812B" V 2175 1825 60  0000 C CNN
 F 2 "" H 1775 1825 60  0000 C CNN
@@
 $EndComp
 $Comp
-L RGB_WS2812B U76
+L RGB_WS2812B U73
 U 1 1 542C0DFF
 P 3175 1825
-F 0 "U76" V 2925 1825 60  0000 C CNN
+F 0 "U73" V 2925 1825 60  0000 C CNN
 F 1 "RGB_WS2812B" V 3575 1825 60  0000 C CNN
 F 2 "" H 3175 1825 60  0000 C CNN
@@
 $EndComp
 $Comp
-L RGB_WS2812B U78
+L RGB_WS2812B U74
 U 1 1 542C0E05
 P 4575 1825
-F 0 "U78" V 4325 1825 60  0000 C CNN
+F 0 "U74" V 4325 1825 60  0000 C CNN
 F 1 "RGB_WS2812B" V 4975 1825 60  0000 C CNN
 F 2 "" H 4575 1825 60  0000 C CNN
@@
 $EndComp
 $Comp
-L RGB_WS2812B U80
+L RGB_WS2812B U75
 U 1 1 542C0E0B
 P 5975 1825
-F 0 "U80" V 5725 1825 60  0000 C CNN
+F 0 "U75" V 5725 1825 60  0000 C CNN
 F 1 "RGB_WS2812B" V 6375 1825 60  0000 C CNN
 F 2 "" H 5975 1825 60  0000 C CNN
@@
 $EndComp
 $Comp
-L RGB_WS2812B U82
+L RGB_WS2812B U76
 U 1 1 542C0E11
 P 7375 1825
-F 0 "U82" V 7125 1825 60  0000 C CNN
+F 0 "U76" V 7125 1825 60  0000 C CNN
 F 1 "RGB_WS2812B" V 7775 1825 60  0000 C CNN
 F 2 "" H 7375 1825 60  0000 C CNN
@@
 $EndComp
 $Comp
-L RGB_WS2812B U84
+L RGB_WS2812B U77
 U 1 1 542C0E17
 P 8775 1825
-F 0 "U84" V 8525 1825 60  0000 C CNN
+F 0 "U77" V 8525 1825 60  0000 C CNN
 F 1 "RGB_WS2812B" V 9175 1825 60  0000 C CNN
 F 2 "" H 8775 1825 60  0000 C CNN
@@
 $EndComp
 $Comp
-L RGB_WS2812B U86
+L RGB_WS2812B U78
 U 1 1 542C0E1D
 P 10175 1825
-F 0 "U86" V 9925 1825 60  0000 C CNN
+F 0 "U78" V 9925 1825 60  0000 C CNN
 F 1 "RGB_WS2812B" V 10575 1825 60  0000 C CNN
 F 2 "" H 10175 1825 60  0000 C CNN
@@
 $EndComp
 $Comp
-L RGB_WS2812B U75
+L RGB_WS2812B U79
 U 1 1 542C0E23
 P 1775 4225
-F 0 "U75" V 1525 4225 60  0000 C CNN
+F 0 "U79" V 1525 4225 60  0000 C CNN
 F 1 "RGB_WS2812B" V 2175 4225 60  0000 C CNN
 F 2 "" H 1775 4225 60  0000 C CNN
@@
 $EndComp
 $Comp
-L RGB_WS2812B U77
+L RGB_WS2812B U80
 U 1 1 542C0E29
 P 3175 4225
-F 0 "U77" V 2925 4225 60  0000 C CNN
+F 0 "U80" V 2925 4225 60  0000 C CNN
 F 1 "RGB_WS2812B" V 3575 4225 60  0000 C CNN
 F 2 "" H 3175 4225 60  0000 C CNN
@@
 $EndComp
 $Comp
-L RGB_WS2812B U79
+L RGB_WS2812B U81
 U 1 1 542C0E2F
 P 4575 4225
-F 0 "U79" V 4325 4225 60  0000 C CNN
+F 0 "U81" V 4325 4225 60  0000 C CNN
 F 1 "RGB_WS2812B" V 4975 4225 60  0000 C CNN
 F 2 "" H 4575 4225 60  0000 C CNN
@@
 $EndComp
 $Comp
-L RGB_WS2812B U81
+L RGB_WS2812B U82
 U 1 1 542C0E35
 P 5975 4225
-F 0 "U81" V 5725 4225 60  0000 C CNN
+F 0 "U82" V 5725 4225 60  0000 C CNN
 F 1 "RGB_WS2812B" V 6375 4225 60  0000 C CNN
 F 2 "" H 5975 4225 60  0000 C CNN
@@
 $EndComp
 $Comp
-L RGB_WS2812B U85
+L RGB_WS2812B U84
 U 1 1 542C0E41
 P 8775 4225
-F 0 "U85" V 8525 4225 60  0000 C CNN
+F 0 "U84" V 8525 4225 60  0000 C CNN
 F 1 "RGB_WS2812B" V 9175 4225 60  0000 C CNN
 F 2 "" H 8775 4225 60  0000 C CNN
@@
 $EndComp
 $Comp
-L RGB_WS2812B U87
+L RGB_WS2812B U85
 U 1 1 542C0E47
 P 10175 4225
-F 0 "U87" V 9925 4225 60  0000 C CNN
+F 0 "U85" V 9925 4225 60  0000 C CNN
 F 1 "RGB_WS2812B" V 10575 4225 60  0000 C CNN
 F 2 "" H 10175 4225 60  0000 C CNN
@@
 Connection ~ 1850 3000
 $Comp
-L C2 C81
+L C2 C82
 U 1 1 542C0EA2
 P 3350 2800
-F 0 "C81" H 3375 2900 50  0000 L CNN
+F 0 "C82" H 3375 2900 50  0000 L CNN
 F 1 "100n" H 3375 2700 50  0000 L CNN
 F 2 "TinyTiM_Lib:c_0805" H 3350 2800 50  0001 C CNN
@@
 F 3 "" H 4750 2800 60  0001 C CNN
 F 4 "CAP CER 0.1UF 25V 10% X7R 0805" H 4750 3000 60  0001 L CNN "Field4"
-F 5 "100nF, 25V" H 4750 3100 60  0001 L CNN "Field5"
+F 5 "100n, 25V" H 4750 3100 60  0001 L CNN "Field5"
 F 6 "Surface Mount, MLCC" H 4750 3200 60  0001 L CNN "Field6"
 F 7 "Kemet" H 4750 3300 60  0001 L CNN "Field7"
@@
 $EndComp
 $Comp
-L C2 C85
+L C2 C84
 U 1 1 542C0EBE
 P 6150 2800
-F 0 "C85" H 6175 2900 50  0000 L CNN
+F 0 "C84" H 6175 2900 50  0000 L CNN
 F 1 "100n" H 6175 2700 50  0000 L CNN
 F 2 "TinyTiM_Lib:c_0805" H 6150 2800 50  0001 C CNN
@@
 $EndComp
 $Comp
-L C2 C87
+L C2 C85
 U 1 1 542C0ECC
 P 7550 2800
-F 0 "C87" H 7575 2900 50  0000 L CNN
+F 0 "C85" H 7575 2900 50  0000 L CNN
 F 1 "100n" H 7575 2700 50  0000 L CNN
 F 2 "TinyTiM_Lib:c_0805" H 7550 2800 50  0001 C CNN
 F 3 "" H 7550 2800 60  0001 C CNN
 F 4 "CAP CER 0.1UF 25V 10% X7R 0805" H 7550 3000 60  0001 L CNN "Field4"
-F 5 "100nF, 25V" H 7550 3100 60  0001 L CNN "Field5"
+F 5 "100n, 25V" H 7550 3100 60  0001 L CNN "Field5"
 F 6 "Surface Mount, MLCC" H 7550 3200 60  0001 L CNN "Field6"
 F 7 "Kemet" H 7550 3300 60  0001 L CNN "Field7"
@@
 $EndComp
 $Comp
-L C2 C89
+L C2 C86
 U 1 1 542C0EDA
 P 8950 2800
-F 0 "C89" H 8975 2900 50  0000 L CNN
+F 0 "C86" H 8975 2900 50  0000 L CNN
 F 1 "100n" H 8975 2700 50  0000 L CNN
 F 2 "TinyTiM_Lib:c_0805" H 8950 2800 50  0001 C CNN
@@
 $EndComp
 $Comp
-L C2 C91
+L C2 C87
 U 1 1 542C0EE8
 P 10350 2800
-F 0 "C91" H 10375 2900 50  0000 L CNN
+F 0 "C87" H 10375 2900 50  0000 L CNN
 F 1 "100n" H 10375 2700 50  0000 L CNN
 F 2 "TinyTiM_Lib:c_0805" H 10350 2800 50  0001 C CNN
 F 3 "" H 10350 2800 60  0001 C CNN
 F 4 "CAP CER 0.1UF 25V 10% X7R 0805" H 10350 3000 60  0001 L CNN "Field4"
-F 5 "100nF, 25V" H 10350 3100 60  0001 L CNN "Field5"
+F 5 "100n, 25V" H 10350 3100 60  0001 L CNN "Field5"
 F 6 "Surface Mount, MLCC" H 10350 3200 60  0001 L CNN "Field6"
 F 7 "Kemet" H 10350 3300 60  0001 L CNN "Field7"
@@
 Connection ~ 10250 3000
 $Comp
-L C2 C80
+L C2 C88
 U 1 1 542C0EF7
 P 1950 5150
-F 0 "C80" H 1975 5250 50  0000 L CNN
+F 0 "C88" H 1975 5250 50  0000 L CNN
 F 1 "100n" H 1975 5050 50  0000 L CNN
 F 2 "TinyTiM_Lib:c_0805" H 1950 5150 50  0001 C CNN
@@
 Connection ~ 1850 5350
 $Comp
-L C2 C82
+L C2 C89
 U 1 1 542C0F34
 P 3350 5150
-F 0 "C82" H 3375 5250 50  0000 L CNN
+F 0 "C89" H 3375 5250 50  0000 L CNN
 F 1 "100n" H 3375 5050 50  0000 L CNN
 F 2 "TinyTiM_Lib:c_0805" H 3350 5150 50  0001 C CNN
 F 3 "" H 3350 5150 60  0001 C CNN
 F 4 "CAP CER 0.1UF 25V 10% X7R 0805" H 3350 5350 60  0001 L CNN "Field4"
-F 5 "100nF, 25V" H 3350 5450 60  0001 L CNN "Field5"
+F 5 "100n, 25V" H 3350 5450 60  0001 L CNN "Field5"
 F 6 "Surface Mount, MLCC" H 3350 5550 60  0001 L CNN "Field6"
 F 7 "Kemet" H 3350 5650 60  0001 L CNN "Field7"
@@
 $EndComp
 $Comp
-L C2 C84
+L C2 C90
 U 1 1 542C0F42
 P 4750 5150
-F 0 "C84" H 4775 5250 50  0000 L CNN
+F 0 "C90" H 4775 5250 50  0000 L CNN
 F 1 "100n" H 4775 5050 50  0000 L CNN
 F 2 "TinyTiM_Lib:c_0805" H 4750 5150 50  0001 C CNN
@@
 $EndComp
 $Comp
-L C2 C86
+L C2 C91
 U 1 1 542C0F50
 P 6150 5150
-F 0 "C86" H 6175 5250 50  0000 L CNN
+F 0 "C91" H 6175 5250 50  0000 L CNN
 F 1 "100n" H 6175 5050 50  0000 L CNN
 F 2 "TinyTiM_Lib:c_0805" H 6150 5150 50  0001 C CNN
 F 3 "" H 6150 5150 60  0001 C CNN
 F 4 "CAP CER 0.1UF 25V 10% X7R 0805" H 6150 5350 60  0001 L CNN "Field4"
-F 5 "100nF, 25V" H 6150 5450 60  0001 L CNN "Field5"
+F 5 "100n, 25V" H 6150 5450 60  0001 L CNN "Field5"
 F 6 "Surface Mount, MLCC" H 6150 5550 60  0001 L CNN "Field6"
 F 7 "Kemet" H 6150 5650 60  0001 L CNN "Field7"
@@
 $EndComp
 $Comp
-L C2 C88
+L C2 C92
 U 1 1 542C0F5E
 P 7550 5150
-F 0 "C88" H 7575 5250 50  0000 L CNN
+F 0 "C92" H 7575 5250 50  0000 L CNN
 F 1 "100n" H 7575 5050 50  0000 L CNN
 F 2 "TinyTiM_Lib:c_0805" H 7550 5150 50  0001 C CNN
@@
 $EndComp
 $Comp
-L C2 C90
+L C2 C93
 U 1 1 542C0F6C
 P 8950 5150
-F 0 "C90" H 8975 5250 50  0000 L CNN
+F 0 "C93" H 8975 5250 50  0000 L CNN
 F 1 "100n" H 8975 5050 50  0000 L CNN
 F 2 "TinyTiM_Lib:c_0805" H 8950 5150 50  0001 C CNN
 F 3 "" H 8950 5150 60  0001 C CNN
 F 4 "CAP CER 0.1UF 25V 10% X7R 0805" H 8950 5350 60  0001 L CNN "Field4"
-F 5 "100nF, 25V" H 8950 5450 60  0001 L CNN "Field5"
+F 5 "100n, 25V" H 8950 5450 60  0001 L CNN "Field5"
 F 6 "Surface Mount, MLCC" H 8950 5550 60  0001 L CNN "Field6"
 F 7 "Kemet" H 8950 5650 60  0001 L CNN "Field7"
@@
 $EndComp
 $Comp
-L C2 C92
+L C2 C94
 U 1 1 542C0F7A
 P 10350 5150
-F 0 "C92" H 10375 5250 50  0000 L CNN
+F 0 "C94" H 10375 5250 50  0000 L CNN
 F 1 "100n" H 10375 5050 50  0000 L CNN
 F 2 "TinyTiM_Lib:c_0805" H 10350 5150 50  0001 C CNN

Commit message: Board layout updated
Parts:
- removed U72, U73, U74, U75, U76, U77, U78, U79, U80, U81, U82, U83, U84, U85: RGB_WS2812B, symbol RGB_WS2812B
- added LED71, LED72, LED73, LED74, LED75, LED76, LED77, LED78, LED79, LED80, LED81, LED82, LED83, LED84: RGB_WS2812B, ~, symbol RGB_WS2812B

Commit message: Board layout updated
Matrix placed and wired. Added RTC.
Parts:
- removed C81: 100n, TinyTiM_Lib:c_0805, symbol C2
- removed LED71, LED72, LED73, LED74, LED75, LED76, LED77, LED78, LED79, LED80, LED81, LED82, LED83, LED84: RGB_WS2812B, ~, symbol RGB_WS2812B
- added C95: 100n, TinyTiM_Lib:c_0805, symbol C2
- added LED71, LED72, LED73, LED74, LED75, LED76, LED77, LED78, LED79, LED80, LED81, LED82, LED83, LED84: WS2812B, ~, symbol WS2812B
- C82, C84, C86, C88, C90, C92, C94: Field5 100nF, 25V -> 100n, 25V
- C83, C85, C87, C89, C91, C93: Field5 100n, 25V -> 100nF, 25V
