File: KiCad/Row_F.sch (KiCad schematic (older format))
At the start: 28 parts

Commit message: PCB layout, work in progress
Parts:
- C82, C83, C84, C85, C86, C87, C88, C89, C90, C91, C92, C93, C94, C95: footprint TinyTiM_Lib:c_0805 -> C4_Pretty:c_0805
- LED71, LED72, LED73, LED74, LED75, LED76, LED77, LED78, LED79, LED80, LED81, LED82, LED83, LED84: footprint ~ -> C4_Pretty:RGB_WS2811B
Changed lines of the file:
@@
 F 0 "C82" H 1775 2900 50  0000 L CNN
 F 1 "100n" H 1775 2700 50  0000 L CNN
-F 2 "TinyTiM_Lib:c_0805" H 1750 2800 50  0001 C CNN
+F 2 "C4_Pretty:c_0805" H 1750 2800 50  0001 C CNN
 F 3 "" H 1750 2800 60  0001 C CNN
 F 4 "CAP CER 0.1UF 25V 10% X7R 0805" H 1750 3000 60  0001 L CNN "Field4"
@@
 F 0 "C83" H 3175 2900 50  0000 L CNN
 F 1 "100n" H 3175 2700 50  0000 L CNN
-F 2 "TinyTiM_Lib:c_0805" H 3150 2800 50  0001 C CNN
+F 2 "C4_Pretty:c_0805" H 3150 2800 50  0001 C CNN
 F 3 "" H 3150 2800 60  0001 C CNN
 F 4 "CAP CER 0.1UF 25V 10% X7R 0805" H 3150 3000 60  0001 L CNN "Field4"
@@
 F 0 "C84" H 4575 2900 50  0000 L CNN
 F 1 "100n" H 4575 2700 50  0000 L CNN
-F 2 "TinyTiM_Lib:c_0805" H 4550 2800 50  0001 C CNN
+F 2 "C4_Pretty:c_0805" H 4550 2800 50  0001 C CNN
 F 3 "" H 4550 2800 60  0001 C CNN
 F 4 "CAP CER 0.1UF 25V 10% X7R 0805" H 4550 3000 60  0001 L CNN "Field4"
@@
 F 0 "C85" H 5975 2900 50  0000 L CNN
 F 1 "100n" H 5975 2700 50  0000 L CNN
-F 2 "TinyTiM_Lib:c_0805" H 5950 2800 50  0001 C CNN
+F 2 "C4_Pretty:c_0805" H 5950 2800 50  0001 C CNN
 F 3 "" H 5950 2800 60  0001 C CNN
 F 4 "CAP CER 0.1UF 25V 10% X7R 0805" H 5950 3000 60  0001 L CNN "Field4"
@@
 F 0 "C86" H 7375 2900 50  0000 L CNN
 F 1 "100n" H 7375 2700 50  0000 L CNN
-F 2 "TinyTiM_Lib:c_0805" H 7350 2800 50  0001 C CNN
+F 2 "C4_Pretty:c_0805" H 7350 2800 50  0001 C CNN
 F 3 "" H 7350 2800 60  0001 C CNN
 F 4 "CAP CER 0.1UF 25V 10% X7R 0805" H 7350 3000 60  0001 L CNN "Field4"
@@
 F 0 "C87" H 8775 2900 50  0000 L CNN
 F 1 "100n" H 8775 2700 50  0000 L CNN
-F 2 "TinyTiM_Lib:c_0805" H 8750 2800 50  0001 C CNN
+F 2 "C4_Pretty:c_0805" H 8750 2800 50  0001 C CNN
 F 3 "" H 8750 2800 60  0001 C CNN
 F 4 "CAP CER 0.1UF 25V 10% X7R 0805" H 8750 3000 60  0001 L CNN "Field4"
@@
 F 0 "C88" H 10175 2900 50  0000 L CNN
 F 1 "100n" H 10175 2700 50  0000 L CNN
-F 2 "TinyTiM_Lib:c_0805" H 10150 2800 50  0001 C CNN
+F 2 "C4_Pretty:c_0805" H 10150 2800 50  0001 C CNN
 F 3 "" H 10150 2800 60  0001 C CNN
 F 4 "CAP CER 0.1UF 25V 10% X7R 0805" H 10150 3000 60  0001 L CNN "Field4"
@@
 F 0 "C89" H 1775 5250 50  0000 L CNN
 F 1 "100n" H 1775 5050 50  0000 L CNN
-F 2 "TinyTiM_Lib:c_0805" H 1750 5150 50  0001 C CNN
+F 2 "C4_Pretty:c_0805" H 1750 5150 50  0001 C CNN
 F 3 "" H 1750 5150 60  0001 C CNN
 F 4 "CAP CER 0.1UF 25V 10% X7R 0805" H 1750 5350 60  0001 L CNN "Field4"
@@
 F 0 "C90" H 3175 5250 50  0000 L CNN
 F 1 "100n" H 3175 5050 50  0000 L CNN
-F 2 "TinyTiM_Lib:c_0805" H 3150 5150 50  0001 C CNN
+F 2 "C4_Pretty:c_0805" H 3150 5150 50  0001 C CNN
 F 3 "" H 3150 5150 60  0001 C CNN
 F 4 "CAP CER 0.1UF 25V 10% X7R 0805" H 3150 5350 60  0001 L CNN "Field4"
@@
 F 0 "C91" H 4575 5250 50  0000 L CNN
 F 1 "100n" H 4575 5050 50  0000 L CNN
-F 2 "TinyTiM_Lib:c_0805" H 4550 5150 50  0001 C CNN
+F 2 "C4_Pretty:c_0805" H 4550 5150 50  0001 C CNN
 F 3 "" H 4550 5150 60  0001 C CNN
 F 4 "CAP CER 0.1UF 25V 10% X7R 0805" H 4550 5350 60  0001 L CNN "Field4"
@@
 F 0 "C92" H 5975 5250 50  0000 L CNN
 F 1 "100n" H 5975 5050 50  0000 L CNN
-F 2 "TinyTiM_Lib:c_0805" H 5950 5150 50  0001 C CNN
+F 2 "C4_Pretty:c_0805" H 5950 5150 50  0001 C CNN
 F 3 "" H 5950 5150 60  0001 C CNN
 F 4 "CAP CER 0.1UF 25V 10% X7R 0805" H 5950 5350 60  0001 L CNN "Field4"
@@
 F 0 "C93" H 7375 5250 50  0000 L CNN
 F 1 "100n" H 7375 5050 50  0000 L CNN
-F 2 "TinyTiM_Lib:c_0805" H 7350 5150 50  0001 C CNN
+F 2 "C4_Pretty:c_0805" H 7350 5150 50  0001 C CNN
 F 3 "" H 7350 5150 60  0001 C CNN
 F 4 "CAP CER 0.1UF 25V 10% X7R 0805" H 7350 5350 60  0001 L CNN "Field4"
@@
 F 0 "C94" H 8775 5250 50  0000 L CNN
 F 1 "100n" H 8775 5050 50  0000 L CNN
-F 2 "TinyTiM_Lib:c_0805" H 8750 5150 50  0001 C CNN
+F 2 "C4_Pretty:c_0805" H 8750 5150 50  0001 C CNN
 F 3 "" H 8750 5150 60  0001 C CNN
 F 4 "CAP CER 0.1UF 25V 10% X7R 0805" H 8750 5350 60  0001 L CNN "Field4"
@@
 F 0 "C95" H 10175 5250 50  0000 L CNN
 F 1 "100n" H 10175 5050 50  0000 L CNN
-F 2 "TinyTiM_Lib:c_0805" H 10150 5150 50  0001 C CNN
+F 2 "C4_Pretty:c_0805" H 10150 5150 50  0001 C CNN
 F 3 "" H 10150 5150 60  0001 C CNN
 F 4 "CAP CER 0.1UF 25V 10% X7R 0805" H 10150 5350 60  0001 L CNN "Field4"
@@
 F 0 "LED71" V 1325 1825 60  0000 C CNN
 F 1 "WS2812B" V 1975 1825 60  0001 C CNN
-F 2 "~" H 1575 1825 60  0000 C CNN
+F 2 "C4_Pretty:RGB_WS2811B" H 1575 1825 60  0001 C CNN
 F 3 "~" H 1575 1825 60  0000 C CNN
 	1    1575 1825
@@
 F 0 "LED72" V 2725 1825 60  0000 C CNN
 F 1 "WS2812B" V 3375 1825 60  0001 C CNN
-F 2 "~" H 2975 1825 60  0000 C CNN
+F 2 "C4_Pretty:RGB_WS2811B" H 2975 1825 60  0001 C CNN
 F 3 "~" H 2975 1825 60  0000 C CNN
 	1    2975 1825
@@
 F 0 "LED73" V 4125 1825 60  0000 C CNN
 F 1 "WS2812B" V 4775 1825 60  0001 C CNN
-F 2 "~" H 4375 1825 60  0000 C CNN
+F 2 "C4_Pretty:RGB_WS2811B" H 4375 1825 60  0001 C CNN
 F 3 "~" H 4375 1825 60  0000 C CNN
 	1    4375 1825
@@
 F 0 "LED74" V 5525 1825 60  0000 C CNN
 F 1 "WS2812B" V 6175 1825 60  0001 C CNN
-F 2 "~" H 5775 1825 60  0000 C CNN
+F 2 "C4_Pretty:RGB_WS2811B" H 5775 1825 60  0001 C CNN
 F 3 "~" H 5775 1825 60  0000 C CNN
 	1    5775 1825
@@
 F 0 "LED75" V 6925 1825 60  0000 C CNN
 F 1 "WS2812B" V 7575 1825 60  0001 C CNN
-F 2 "~" H 7175 1825 60  0000 C CNN
+F 2 "C4_Pretty:RGB_WS2811B" H 7175 1825 60  0001 C CNN
 F 3 "~" H 7175 1825 60  0000 C CNN
 	1    7175 1825
@@
 F 0 "LED76" V 8325 1825 60  0000 C CNN
 F 1 "WS2812B" V 8975 1825 60  0001 C CNN
-F 2 "~" H 8575 1825 60  0000 C CNN
+F 2 "C4_Pretty:RGB_WS2811B" H 8575 1825 60  0001 C CNN
 F 3 "~" H 8575 1825 60  0000 C CNN
 	1    8575 1825
@@
 F 0 "LED77" V 9725 1825 60  0000 C CNN
 F 1 "WS2812B" V 10375 1825 60  0001 C CNN
-F 2 "~" H 9975 1825 60  0000 C CNN
+F 2 "C4_Pretty:RGB_WS2811B" H 9975 1825 60  0001 C CNN
 F 3 "~" H 9975 1825 60  0000 C CNN
 	1    9975 1825
@@
 F 0 "LED78" V 1325 4225 60  0000 C CNN
 F 1 "WS2812B" V 1975 4225 60  0001 C CNN
-F 2 "~" H 1575 4225 60  0000 C CNN
+F 2 "C4_Pretty:RGB_WS2811B" H 1575 4225 60  0001 C CNN
 F 3 "~" H 1575 4225 60  0000 C CNN
 	1    1575 4225
@@
 F 0 "LED79" V 2725 4225 60  0000 C CNN
 F 1 "WS2812B" V 3375 4225 60  0001 C CNN
-F 2 "~" H 2975 4225 60  0000 C CNN
+F 2 "C4_Pretty:RGB_WS2811B" H 2975 4225 60  0001 C CNN
 F 3 "~" H 2975 4225 60  0000 C CNN
 	1    2975 4225
@@
 F 0 "LED80" V 4125 4225 60  0000 C CNN
 F 1 "WS2812B" V 4775 4225 60  0001 C CNN
-F 2 "~" H 4375 4225 60  0000 C CNN
+F 2 "C4_Pretty:RGB_WS2811B" H 4375 4225 60  0001 C CNN
 F 3 "~" H 4375 4225 60  0000 C CNN
 	1    4375 4225
@@
 F 0 "LED81" V 5525 4225 60  0000 C CNN
 F 1 "WS2812B" V 6175 4225 60  0001 C CNN
-F 2 "~" H 5775 4225 60  0000 C CNN
+F 2 "C4_Pretty:RGB_WS2811B" H 5775 4225 60  0001 C CNN
 F 3 "~" H 5775 4225 60  0000 C CNN
 	1    5775 4225
@@
 F 0 "LED82" V 6925 4225 60  0000 C CNN
 F 1 "WS2812B" V 7575 4225 60  0001 C CNN
-F 2 "~" H 7175 4225 60  0000 C CNN
+F 2 "C4_Pretty:RGB_WS2811B" H 7175 4225 60  0001 C CNN
 F 3 "~" H 7175 4225 60  0000 C CNN
 	1    7175 4225
@@
 F 0 "LED83" V 8325 4225 60  0000 C CNN
 F 1 "WS2812B" V 8975 4225 60  0001 C CNN
-F 2 "~" H 8575 4225 60  0000 C CNN
+F 2 "C4_Pretty:RGB_WS2811B" H 8575 4225 60  0001 C CNN
 F 3 "~" H 8575 4225 60  0000 C CNN
 	1    8575 4225
@@
 F 0 "LED84" V 9725 4225 60  0000 C CNN
 F 1 "WS2812B" V 10375 4225 60  0001 C CNN
-F 2 "~" H 9975 4225 60  0000 C CNN
+F 2 "C4_Pretty:RGB_WS2811B" H 9975 4225 60  0001 C CNN
 F 3 "~" H 9975 4225 60  0000 C CNN
 	1    9975 4225

Commit message: C4 PCB layout complete. Added Gerbers
Parts:
- C82, C83, C84, C85, C86, C87, C88, C89, C90, C91, C92, C93, C94, C95: footprint C4_Pretty:c_0805 -> C4_Pretty:c_0805_led
Changed lines of the file:
@@
 EESchema Schematic File Version 2
 LIBS:ClockFOUR
+LIBS:RowGB_sym
 LIBS:ClockFOUR-cache
 EELAYER 24 0
@@
 F 0 "C82" H 1775 2900 50  0000 L CNN
 F 1 "100n" H 1775 2700 50  0000 L CNN
-F 2 "C4_Pretty:c_0805" H 1750 2800 50  0001 C CNN
+F 2 "C4_Pretty:c_0805_led" H 1750 2800 50  0001 C CNN
 F 3 "" H 1750 2800 60  0001 C CNN
 F 4 "CAP CER 0.1UF 25V 10% X7R 0805" H 1750 3000 60  0001 L CNN "Field4"
@@
 F 0 "C83" H 3175 2900 50  0000 L CNN
 F 1 "100n" H 3175 2700 50  0000 L CNN
-F 2 "C4_Pretty:c_0805" H 3150 2800 50  0001 C CNN
+F 2 "C4_Pretty:c_0805_led" H 3150 2800 50  0001 C CNN
 F 3 "" H 3150 2800 60  0001 C CNN
 F 4 "CAP CER 0.1UF 25V 10% X7R 0805" H 3150 3000 60  0001 L CNN "Field4"
@@
 F 0 "C84" H 4575 2900 50  0000 L CNN
 F 1 "100n" H 4575 2700 50  0000 L CNN
-F 2 "C4_Pretty:c_0805" H 4550 2800 50  0001 C CNN
+F 2 "C4_Pretty:c_0805_led" H 4550 2800 50  0001 C CNN
 F 3 "" H 4550 2800 60  0001 C CNN
 F 4 "CAP CER 0.1UF 25V 10% X7R 0805" H 4550 3000 60  0001 L CNN "Field4"
@@
 F 0 "C85" H 5975 2900 50  0000 L CNN
 F 1 "100n" H 5975 2700 50  0000 L CNN
-F 2 "C4_Pretty:c_0805" H 5950 2800 50  0001 C CNN
+F 2 "C4_Pretty:c_0805_led" H 5950 2800 50  0001 C CNN
 F 3 "" H 5950 2800 60  0001 C CNN
 F 4 "CAP CER 0.1UF 25V 10% X7R 0805" H 5950 3000 60  0001 L CNN "Field4"
@@
 F 0 "C86" H 7375 2900 50  0000 L CNN
 F 1 "100n" H 7375 2700 50  0000 L CNN
-F 2 "C4_Pretty:c_0805" H 7350 2800 50  0001 C CNN
+F 2 "C4_Pretty:c_0805_led" H 7350 2800 50  0001 C CNN
 F 3 "" H 7350 2800 60  0001 C CNN
 F 4 "CAP CER 0.1UF 25V 10% X7R 0805" H 7350 3000 60  0001 L CNN "Field4"
@@
 F 0 "C87" H 8775 2900 50  0000 L CNN
 F 1 "100n" H 8775 2700 50  0000 L CNN
-F 2 "C4_Pretty:c_0805" H 8750 2800 50  0001 C CNN
+F 2 "C4_Pretty:c_0805_led" H 8750 2800 50  0001 C CNN
 F 3 "" H 8750 2800 60  0001 C CNN
 F 4 "CAP CER 0.1UF 25V 10% X7R 0805" H 8750 3000 60  0001 L CNN "Field4"
@@
 F 0 "C88" H 10175 2900 50  0000 L CNN
 F 1 "100n" H 10175 2700 50  0000 L CNN
-F 2 "C4_Pretty:c_0805" H 10150 2800 50  0001 C CNN
+F 2 "C4_Pretty:c_0805_led" H 10150 2800 50  0001 C CNN
 F 3 "" H 10150 2800 60  0001 C CNN
 F 4 "CAP CER 0.1UF 25V 10% X7R 0805" H 10150 3000 60  0001 L CNN "Field4"
@@
 F 0 "C89" H 1775 5250 50  0000 L CNN
 F 1 "100n" H 1775 5050 50  0000 L CNN
-F 2 "C4_Pretty:c_0805" H 1750 5150 50  0001 C CNN
+F 2 "C4_Pretty:c_0805_led" H 1750 5150 50  0001 C CNN
 F 3 "" H 1750 5150 60  0001 C CNN
 F 4 "CAP CER 0.1UF 25V 10% X7R 0805" H 1750 5350 60  0001 L CNN "Field4"
@@
 F 0 "C90" H 3175 5250 50  0000 L CNN
 F 1 "100n" H 3175 5050 50  0000 L CNN
-F 2 "C4_Pretty:c_0805" H 3150 5150 50  0001 C CNN
+F 2 "C4_Pretty:c_0805_led" H 3150 5150 50  0001 C CNN
 F 3 "" H 3150 5150 60  0001 C CNN
 F 4 "CAP CER 0.1UF 25V 10% X7R 0805" H 3150 5350 60  0001 L CNN "Field4"
@@
 F 0 "C91" H 4575 5250 50  0000 L CNN
 F 1 "100n" H 4575 5050 50  0000 L CNN
-F 2 "C4_Pretty:c_0805" H 4550 5150 50  0001 C CNN
+F 2 "C4_Pretty:c_0805_led" H 4550 5150 50  0001 C CNN
 F 3 "" H 4550 5150 60  0001 C CNN
 F 4 "CAP CER 0.1UF 25V 10% X7R 0805" H 4550 5350 60  0001 L CNN "Field4"
@@
 F 0 "C92" H 5975 5250 50  0000 L CNN
 F 1 "100n" H 5975 5050 50  0000 L CNN
-F 2 "C4_Pretty:c_0805" H 5950 5150 50  0001 C CNN
+F 2 "C4_Pretty:c_0805_led" H 5950 5150 50  0001 C CNN
 F 3 "" H 5950 5150 60  0001 C CNN
 F 4 "CAP CER 0.1UF 25V 10% X7R 0805" H 5950 5350 60  0001 L CNN "Field4"
@@
 F 0 "C93" H 7375 5250 50  0000 L CNN
 F 1 "100n" H 7375 5050 50  0000 L CNN
-F 2 "C4_Pretty:c_0805" H 7350 5150 50  0001 C CNN
+F 2 "C4_Pretty:c_0805_led" H 7350 5150 50  0001 C CNN
 F 3 "" H 7350 5150 60  0001 C CNN
 F 4 "CAP CER 0.1UF 25V 10% X7R 0805" H 7350 5350 60  0001 L CNN "Field4"
@@
 F 0 "C94" H 8775 5250 50  0000 L CNN
 F 1 "100n" H 8775 5050 50  0000 L CNN
-F 2 "C4_Pretty:c_0805" H 8750 5150 50  0001 C CNN
+F 2 "C4_Pretty:c_0805_led" H 8750 5150 50  0001 C CNN
 F 3 "" H 8750 5150 60  0001 C CNN
 F 4 "CAP CER 0.1UF 25V 10% X7R 0805" H 8750 5350 60  0001 L CNN "Field4"
@@
 F 0 "C95" H 10175 5250 50  0000 L CNN
 F 1 "100n" H 10175 5050 50  0000 L CNN
-F 2 "C4_Pretty:c_0805" H 10150 5150 50  0001 C CNN
+F 2 "C4_Pretty:c_0805_led" H 10150 5150 50  0001 C CNN
 F 3 "" H 10150 5150 60  0001 C CNN
 F 4 "CAP CER 0.1UF 25V 10% X7R 0805" H 10150 5350 60  0001 L CNN "Field4"
