File: KiCad/Row_G.sch (KiCad schematic (older format))
At the start: 0 parts

Commit message: Schematic updated
Parts:
- added C100, C102, C103, C104, C105, C106, C107, C93, C94, C95, C96, C97, C98, C99: 100n, TinyTiM_Lib:c_0805, symbol C2
- added U100, U101, U88, U89, U90, U91, U92, U93, U94, U95, U96, U97, U98, U99: RGB_WS2812B, symbol RGB_WS2812B
Connections:
- net labels added: 5V, DI_G, DO_G, GND
- wire segments 0 -> 82

Commit message: Schematic updated, board started
Parts:
- C101: renamed from C106; Field5 100nF, 25V -> 100n, 25V
- C103: renamed from C96; Field5 100nF, 25V -> 100n, 25V
- C105: renamed from C100; Field5 100nF, 25V -> 100n, 25V
- C107: renamed from C105; Field5 100nF, 25V -> 100n, 25V
- C95: renamed from C93; Field5 100nF, 25V -> 100n, 25V
- C97: Field5 100nF, 25V -> 100n, 25V
- C99: renamed from C102; Field5 100nF, 25V -> 100n, 25V
- renumbered C104 to C100, C94 to C102, C98 to C104, C103 to C106, C107 to C108, C95 to C96, C99 to C98, U88 to U86, U90 to U87, U92 to U88, U94 to U89, U96 to U90, U98 to U91, U100 to U92, U89 to U93, U91 to U94, U93 to U95, U95 to U96, U99 to U98, U101 to U99
Changed lines of the file:
@@
 LIBS:contrib
 LIBS:valves
-LIBS:TinyTiM-cache
-LIBS:TiNA_sym
+LIBS:ClockFOUR
 LIBS:ClockFOUR-cache
 EELAYER 27 0
@@
 Sheet 8 14
 Title "ClockFOUR"
-Date "30 sep 2014"
+Date "1 oct 2014"
 Rev ""
 Comp "WyoLum"
@@
 5V
 $Comp
-L GND #PWR018
+L GND #PWR020
 U 1 1 542C0F92
 P 1300 2550
-F 0 "#PWR018" H 1300 2550 30  0001 C CNN
+F 0 "#PWR020" H 1300 2550 30  0001 C CNN
 F 1 "GND" H 1300 2480 30  0001 C CNN
 F 2 "" H 1300 2550 60  0001 C CNN
@@
 $EndComp
 $Comp
-L C2 C93
+L C2 C95
 U 1 1 542C0FA0
 P 1850 2700
-F 0 "C93" H 1875 2800 50  0000 L CNN
+F 0 "C95" H 1875 2800 50  0000 L CNN
 F 1 "100n" H 1875 2600 50  0000 L CNN
 F 2 "TinyTiM_Lib:c_0805" H 1850 2700 50  0001 C CNN
 F 3 "" H 1850 2700 60  0001 C CNN
 F 4 "CAP CER 0.1UF 25V 10% X7R 0805" H 1850 2900 60  0001 L CNN "Field4"
-F 5 "100nF, 25V" H 1850 3000 60  0001 L CNN "Field5"
+F 5 "100n, 25V" H 1850 3000 60  0001 L CNN "Field5"
 F 6 "Surface Mount, MLCC" H 1850 3100 60  0001 L CNN "Field6"
 F 7 "Kemet" H 1850 3200 60  0001 L CNN "Field7"
@@
 $EndComp
 $Comp
-L RGB_WS2812B U88
+L RGB_WS2812B U86
 U 1 1 542C0FA6
 P 1675 1725
-F 0 "U88" V 1425 1725 60  0000 C CNN
+F 0 "U86" V 1425 1725 60  0000 C CNN
 F 1 "RGB_WS2812B" V 2075 1725 60  0000 C CNN
 F 2 "" H 1675 1725 60  0000 C CNN
@@
 $EndComp
 $Comp
-L RGB_WS2812B U90
+L RGB_WS2812B U87
 U 1 1 542C0FAC
 P 3075 1725
-F 0 "U90" V 2825 1725 60  0000 C CNN
+F 0 "U87" V 2825 1725 60  0000 C CNN
 F 1 "RGB_WS2812B" V 3475 1725 60  0000 C CNN
 F 2 "" H 3075 1725 60  0000 C CNN
@@
 $EndComp
 $Comp
-L RGB_WS2812B U92
+L RGB_WS2812B U88
 U 1 1 542C0FB2
 P 4475 1725
-F 0 "U92" V 4225 1725 60  0000 C CNN
+F 0 "U88" V 4225 1725 60  0000 C CNN
 F 1 "RGB_WS2812B" V 4875 1725 60  0000 C CNN
 F 2 "" H 4475 1725 60  0000 C CNN
@@
 $EndComp
 $Comp
-L RGB_WS2812B U94
+L RGB_WS2812B U89
 U 1 1 542C0FB8
 P 5875 1725
-F 0 "U94" V 5625 1725 60  0000 C CNN
+F 0 "U89" V 5625 1725 60  0000 C CNN
 F 1 "RGB_WS2812B" V 6275 1725 60  0000 C CNN
 F 2 "" H 5875 1725 60  0000 C CNN
@@
 $EndComp
 $Comp
-L RGB_WS2812B U96
+L RGB_WS2812B U90
 U 1 1 542C0FBE
 P 7275 1725
-F 0 "U96" V 7025 1725 60  0000 C CNN
+F 0 "U90" V 7025 1725 60  0000 C CNN
 F 1 "RGB_WS2812B" V 7675 1725 60  0000 C CNN
 F 2 "" H 7275 1725 60  0000 C CNN
@@
 $EndComp
 $Comp
-L RGB_WS2812B U98
+L RGB_WS2812B U91
 U 1 1 542C0FC4
 P 8675 1725
-F 0 "U98" V 8425 1725 60  0000 C CNN
+F 0 "U91" V 8425 1725 60  0000 C CNN
 F 1 "RGB_WS2812B" V 9075 1725 60  0000 C CNN
 F 2 "" H 8675 1725 60  0000 C CNN
@@
 $EndComp
 $Comp
-L RGB_WS2812B U100
+L RGB_WS2812B U92
 U 1 1 542C0FCA
 P 10075 1725
-F 0 "U100" V 9825 1725 60  0000 C CNN
+F 0 "U92" V 9825 1725 60  0000 C CNN
 F 1 "RGB_WS2812B" V 10475 1725 60  0000 C CNN
 F 2 "" H 10075 1725 60  0000 C CNN
@@
 $EndComp
 $Comp
-L RGB_WS2812B U89
+L RGB_WS2812B U93
 U 1 1 542C0FD0
 P 1675 4125
-F 0 "U89" V 1425 4125 60  0000 C CNN
+F 0 "U93" V 1425 4125 60  0000 C CNN
 F 1 "RGB_WS2812B" V 2075 4125 60  0000 C CNN
 F 2 "" H 1675 4125 60  0000 C CNN
@@
 $EndComp
 $Comp
-L RGB_WS2812B U91
+L RGB_WS2812B U94
 U 1 1 542C0FD6
 P 3075 4125
-F 0 "U91" V 2825 4125 60  0000 C CNN
+F 0 "U94" V 2825 4125 60  0000 C CNN
 F 1 "RGB_WS2812B" V 3475 4125 60  0000 C CNN
 F 2 "" H 3075 4125 60  0000 C CNN
@@
 $EndComp
 $Comp
-L RGB_WS2812B U93
+L RGB_WS2812B U95
 U 1 1 542C0FDC
 P 4475 4125
-F 0 "U93" V 4225 4125 60  0000 C CNN
+F 0 "U95" V 4225 4125 60  0000 C CNN
 F 1 "RGB_WS2812B" V 4875 4125 60  0000 C CNN
 F 2 "" H 4475 4125 60  0000 C CNN
@@
 $EndComp
 $Comp
-L RGB_WS2812B U95
+L RGB_WS2812B U96
 U 1 1 542C0FE2
 P 5875 4125
-F 0 "U95" V 5625 4125 60  0000 C CNN
+F 0 "U96" V 5625 4125 60  0000 C CNN
 F 1 "RGB_WS2812B" V 6275 4125 60  0000 C CNN
 F 2 "" H 5875 4125 60  0000 C CNN
@@
 $EndComp
 $Comp
-L RGB_WS2812B U99
+L RGB_WS2812B U98
 U 1 1 542C0FEE
 P 8675 4125
-F 0 "U99" V 8425 4125 60  0000 C CNN
+F 0 "U98" V 8425 4125 60  0000 C CNN
 F 1 "RGB_WS2812B" V 9075 4125 60  0000 C CNN
 F 2 "" H 8675 4125 60  0000 C CNN
@@
 $EndComp
 $Comp
-L RGB_WS2812B U101
+L RGB_WS2812B U99
 U 1 1 542C0FF4
 P 10075 4125
-F 0 "U101" V 9825 4125 60  0000 C CNN
+F 0 "U99" V 9825 4125 60  0000 C CNN
 F 1 "RGB_WS2812B" V 10475 4125 60  0000 C CNN
 F 2 "" H 10075 4125 60  0000 C CNN
@@
 Connection ~ 1750 2900
 $Comp
-L C2 C95
+L C2 C96
 U 1 1 542C104F
 P 3250 2700
-F 0 "C95" H 3275 2800 50  0000 L CNN
+F 0 "C96" H 3275 2800 50  0000 L CNN
 F 1 "100n" H 3275 2600 50  0000 L CNN
 F 2 "TinyTiM_Lib:c_0805" H 3250 2700 50  0001 C CNN
@@
 F 3 "" H 4650 2700 60  0001 C CNN
 F 4 "CAP CER 0.1UF 25V 10% X7R 0805" H 4650 2900 60  0001 L CNN "Field4"
-F 5 "100nF, 25V" H 4650 3000 60  0001 L CNN "Field5"
+F 5 "100n, 25V" H 4650 3000 60  0001 L CNN "Field5"
 F 6 "Surface Mount, MLCC" H 4650 3100 60  0001 L CNN "Field6"
 F 7 "Kemet" H 4650 3200 60  0001 L CNN "Field7"
@@
 $EndComp
 $Comp
-L C2 C99
+L C2 C98
 U 1 1 542C106B
 P 6050 2700
-F 0 "C99" H 6075 2800 50  0000 L CNN
+F 0 "C98" H 6075 2800 50  0000 L CNN
 F 1 "100n" H 6075 2600 50  0000 L CNN
 F 2 "TinyTiM_Lib:c_0805" H 6050 2700 50  0001 C CNN
@@
 $EndComp
 $Comp
-L C2 C102
+L C2 C99
 U 1 1 542C1079
 P 7450 2700
-F 0 "C102" H 7475 2800 50  0000 L CNN
+F 0 "C99" H 7475 2800 50  0000 L CNN
 F 1 "100n" H 7475 2600 50  0000 L CNN
 F 2 "TinyTiM_Lib:c_0805" H 7450 2700 50  0001 C CNN
 F 3 "" H 7450 2700 60  0001 C CNN
 F 4 "CAP CER 0.1UF 25V 10% X7R 0805" H 7450 2900 60  0001 L CNN "Field4"
-F 5 "100nF, 25V" H 7450 3000 60  0001 L CNN "Field5"
+F 5 "100n, 25V" H 7450 3000 60  0001 L CNN "Field5"
 F 6 "Surface Mount, MLCC" H 7450 3100 60  0001 L CNN "Field6"
 F 7 "Kemet" H 7450 3200 60  0001 L CNN "Field7"
@@
 $EndComp
 $Comp
-L C2 C104
+L C2 C100
 U 1 1 542C1087
 P 8850 2700
-F 0 "C104" H 8875 2800 50  0000 L CNN
+F 0 "C100" H 8875 2800 50  0000 L CNN
 F 1 "100n" H 8875 2600 50  0000 L CNN
 F 2 "TinyTiM_Lib:c_0805" H 8850 2700 50  0001 C CNN
@@
 $EndComp
 $Comp
-L C2 C106
+L C2 C101
 U 1 1 542C1095
 P 10250 2700
-F 0 "C106" H 10275 2800 50  0000 L CNN
+F 0 "C101" H 10275 2800 50  0000 L CNN
 F 1 "100n" H 10275 2600 50  0000 L CNN
 F 2 "TinyTiM_Lib:c_0805" H 10250 2700 50  0001 C CNN
 F 3 "" H 10250 2700 60  0001 C CNN
 F 4 "CAP CER 0.1UF 25V 10% X7R 0805" H 10250 2900 60  0001 L CNN "Field4"
-F 5 "100nF, 25V" H 10250 3000 60  0001 L CNN "Field5"
+F 5 "100n, 25V" H 10250 3000 60  0001 L CNN "Field5"
 F 6 "Surface Mount, MLCC" H 10250 3100 60  0001 L CNN "Field6"
 F 7 "Kemet" H 10250 3200 60  0001 L CNN "Field7"
@@
 Connection ~ 10150 2900
 $Comp
-L C2 C94
+L C2 C102
 U 1 1 542C10A4
 P 1850 5050
-F 0 "C94" H 1875 5150 50  0000 L CNN
+F 0 "C102" H 1875 5150 50  0000 L CNN
 F 1 "100n" H 1875 4950 50  0000 L CNN
 F 2 "TinyTiM_Lib:c_0805" H 1850 5050 50  0001 C CNN
@@
 Connection ~ 4550 5250
 Wire Wire Line
-	3150 4750 3150 5250
-Connection ~ 3150 5250
-Wire Wire Line
 	1750 4750 1750 5250
 Connection ~ 1750 5250
 $Comp
-L C2 C96
+L C2 C103
 U 1 1 542C10E1
 P 3250 5050
-F 0 "C96" H 3275 5150 50  0000 L CNN
+F 0 "C103" H 3275 5150 50  0000 L CNN
 F 1 "100n" H 3275 4950 50  0000 L CNN
 F 2 "TinyTiM_Lib:c_0805" H 3250 5050 50  0001 C CNN
 F 3 "" H 3250 5050 60  0001 C CNN
 F 4 "CAP CER 0.1UF 25V 10% X7R 0805" H 3250 5250 60  0001 L CNN "Field4"
-F 5 "100nF, 25V" H 3250 5350 60  0001 L CNN "Field5"
+F 5 "100n, 25V" H 3250 5350 60  0001 L CNN "Field5"
 F 6 "Surface Mount, MLCC" H 3250 5450 60  0001 L CNN "Field6"
 F 7 "Kemet" H 3250 5550 60  0001 L CNN "Field7"
@@
 $EndComp
 $Comp
-L C2 C98
+L C2 C104
 U 1 1 542C10EF
 P 4650 5050
-F 0 "C98" H 4675 5150 50  0000 L CNN
+F 0 "C104" H 4675 5150 50  0000 L CNN
 F 1 "100n" H 4675 4950 50  0000 L CNN
 F 2 "TinyTiM_Lib:c_0805" H 4650 5050 50  0001 C CNN
@@
 $EndComp
 $Comp
-L C2 C100
+L C2 C105
 U 1 1 542C10FD
 P 6050 5050
-F 0 "C100" H 6075 5150 50  0000 L CNN
+F 0 "C105" H 6075 5150 50  0000 L CNN
 F 1 "100n" H 6075 4950 50  0000 L CNN
 F 2 "TinyTiM_Lib:c_0805" H 6050 5050 50  0001 C CNN
 F 3 "" H 6050 5050 60  0001 C CNN
 F 4 "CAP CER 0.1UF 25V 10% X7R 0805" H 6050 5250 60  0001 L CNN "Field4"
-F 5 "100nF, 25V" H 6050 5350 60  0001 L CNN "Field5"
+F 5 "100n, 25V" H 6050 5350 60  0001 L CNN "Field5"
 F 6 "Surface Mount, MLCC" H 6050 5450 60  0001 L CNN "Field6"
 F 7 "Kemet" H 6050 5550 60  0001 L CNN "Field7"
@@
 $EndComp
 $Comp
-L C2 C103
+L C2 C106
 U 1 1 542C110B
 P 7450 5050
-F 0 "C103" H 7475 5150 50  0000 L CNN
+F 0 "C106" H 7475 5150 50  0000 L CNN
 F 1 "100n" H 7475 4950 50  0000 L CNN
 F 2 "TinyTiM_Lib:c_0805" H 7450 5050 50  0001 C CNN
@@
 $EndComp
 $Comp
-L C2 C105
+L C2 C107
 U 1 1 542C1119
 P 8850 5050
-F 0 "C105" H 8875 5150 50  0000 L CNN
+F 0 "C107" H 8875 5150 50  0000 L CNN
 F 1 "100n" H 8875 4950 50  0000 L CNN
 F 2 "TinyTiM_Lib:c_0805" H 8850 5050 50  0001 C CNN
 F 3 "" H 8850 5050 60  0001 C CNN
 F 4 "CAP CER 0.1UF 25V 10% X7R 0805" H 8850 5250 60  0001 L CNN "Field4"
-F 5 "100nF, 25V" H 8850 5350 60  0001 L CNN "Field5"
+F 5 "100n, 25V" H 8850 5350 60  0001 L CNN "Field5"
 F 6 "Surface Mount, MLCC" H 8850 5450 60  0001 L CNN "Field6"
 F 7 "Kemet" H 8850 5550 60  0001 L CNN "Field7"
@@
 $EndComp
 $Comp
-L C2 C107
+L C2 C108
 U 1 1 542C1127
 P 10250 5050
-F 0 "C107" H 10275 5150 50  0000 L CNN
+F 0 "C108" H 10275 5150 50  0000 L CNN
 F 1 "100n" H 10275 4950 50  0000 L CNN
 F 2 "TinyTiM_Lib:c_0805" H 10250 5050 50  0001 C CNN
@@
 Connection ~ 10150 5250
 Connection ~ 1400 2500
+Wire Wire Line
+	3150 4750 3150 5250
+Connection ~ 3150 5250
 $EndSCHEMATC

Commit message: Board layout updated
Parts:
- removed U86, U87, U88, U89, U90, U91, U92, U93, U94, U95, U96, U97, U98, U99: RGB_WS2812B, symbol RGB_WS2812B
- added LED85, LED86, LED87, LED88, LED89, LED90, LED91, LED92, LED93, LED94, LED95, LED96, LED97, LED98: RGB_WS2812B, ~, symbol RGB_WS2812B

Commit message: Board layout updated
Matrix placed and wired. Added RTC.
Parts:
- removed C95: 100n, TinyTiM_Lib:c_0805, symbol C2
- removed LED85, LED86, LED87, LED88, LED89, LED90, LED91, LED92, LED93, LED94, LED95, LED96, LED97, LED98: RGB_WS2812B, ~, symbol RGB_WS2812B
- added C109: 100n, TinyTiM_Lib:c_0805, symbol C2
- added LED85, LED86, LED87, LED88, LED89, LED90, LED91, LED92, LED93, LED94, LED95, LED96, LED97, LED98: WS2812B, ~, symbol WS2812B
- C100, C102, C104, C106, C108, C96, C98: Field5 100nF, 25V -> 100n, 25V
- C101, C103, C105, C107, C97, C99: Field5 100n, 25V -> 100nF, 25V
