File: KiCad/Row_G.sch (KiCad schematic (older format))
At the start: 28 parts

Commit message: PCB layout, work in progress
Parts:
- C100, C101, C102, C103, C104, C105, C106, C107, C108, C109, C96, C97, C98, C99: footprint TinyTiM_Lib:c_0805 -> C4_Pretty:c_0805
- LED85, LED86, LED87, LED88, LED89, LED90, LED91, LED92, LED93, LED94, LED95, LED96, LED97, LED98: footprint ~ -> C4_Pretty:RGB_WS2811B
Changed lines of the file:
@@
 F 0 "C96" H 1875 2900 50  0000 L CNN
 F 1 "100n" H 1875 2700 50  0000 L CNN
-F 2 "TinyTiM_Lib:c_0805" H 1850 2800 50  0001 C CNN
+F 2 "C4_Pretty:c_0805" H 1850 2800 50  0001 C CNN
 F 3 "" H 1850 2800 60  0001 C CNN
 F 4 "CAP CER 0.1UF 25V 10% X7R 0805" H 1850 3000 60  0001 L CNN "Field4"
@@
 F 0 "C97" H 3275 2900 50  0000 L CNN
 F 1 "100n" H 3275 2700 50  0000 L CNN
-F 2 "TinyTiM_Lib:c_0805" H 3250 2800 50  0001 C CNN
+F 2 "C4_Pretty:c_0805" H 3250 2800 50  0001 C CNN
 F 3 "" H 3250 2800 60  0001 C CNN
 F 4 "CAP CER 0.1UF 25V 10% X7R 0805" H 3250 3000 60  0001 L CNN "Field4"
@@
 F 0 "C98" H 4675 2900 50  0000 L CNN
 F 1 "100n" H 4675 2700 50  0000 L CNN
-F 2 "TinyTiM_Lib:c_0805" H 4650 2800 50  0001 C CNN
+F 2 "C4_Pretty:c_0805" H 4650 2800 50  0001 C CNN
 F 3 "" H 4650 2800 60  0001 C CNN
 F 4 "CAP CER 0.1UF 25V 10% X7R 0805" H 4650 3000 60  0001 L CNN "Field4"
@@
 F 0 "C99" H 6075 2900 50  0000 L CNN
 F 1 "100n" H 6075 2700 50  0000 L CNN
-F 2 "TinyTiM_Lib:c_0805" H 6050 2800 50  0001 C CNN
+F 2 "C4_Pretty:c_0805" H 6050 2800 50  0001 C CNN
 F 3 "" H 6050 2800 60  0001 C CNN
 F 4 "CAP CER 0.1UF 25V 10% X7R 0805" H 6050 3000 60  0001 L CNN "Field4"
@@
 F 0 "C100" H 7475 2900 50  0000 L CNN
 F 1 "100n" H 7475 2700 50  0000 L CNN
-F 2 "TinyTiM_Lib:c_0805" H 7450 2800 50  0001 C CNN
+F 2 "C4_Pretty:c_0805" H 7450 2800 50  0001 C CNN
 F 3 "" H 7450 2800 60  0001 C CNN
 F 4 "CAP CER 0.1UF 25V 10% X7R 0805" H 7450 3000 60  0001 L CNN "Field4"
@@
 F 0 "C101" H 8875 2900 50  0000 L CNN
 F 1 "100n" H 8875 2700 50  0000 L CNN
-F 2 "TinyTiM_Lib:c_0805" H 8850 2800 50  0001 C CNN
+F 2 "C4_Pretty:c_0805" H 8850 2800 50  0001 C CNN
 F 3 "" H 8850 2800 60  0001 C CNN
 F 4 "CAP CER 0.1UF 25V 10% X7R 0805" H 8850 3000 60  0001 L CNN "Field4"
@@
 F 0 "C102" H 10275 2900 50  0000 L CNN
 F 1 "100n" H 10275 2700 50  0000 L CNN
-F 2 "TinyTiM_Lib:c_0805" H 10250 2800 50  0001 C CNN
+F 2 "C4_Pretty:c_0805" H 10250 2800 50  0001 C CNN
 F 3 "" H 10250 2800 60  0001 C CNN
 F 4 "CAP CER 0.1UF 25V 10% X7R 0805" H 10250 3000 60  0001 L CNN "Field4"
@@
 F 0 "C103" H 1875 5250 50  0000 L CNN
 F 1 "100n" H 1875 5050 50  0000 L CNN
-F 2 "TinyTiM_Lib:c_0805" H 1850 5150 50  0001 C CNN
+F 2 "C4_Pretty:c_0805" H 1850 5150 50  0001 C CNN
 F 3 "" H 1850 5150 60  0001 C CNN
 F 4 "CAP CER 0.1UF 25V 10% X7R 0805" H 1850 5350 60  0001 L CNN "Field4"
@@
 F 0 "C104" H 3275 5250 50  0000 L CNN
 F 1 "100n" H 3275 5050 50  0000 L CNN
-F 2 "TinyTiM_Lib:c_0805" H 3250 5150 50  0001 C CNN
+F 2 "C4_Pretty:c_0805" H 3250 5150 50  0001 C CNN
 F 3 "" H 3250 5150 60  0001 C CNN
 F 4 "CAP CER 0.1UF 25V 10% X7R 0805" H 3250 5350 60  0001 L CNN "Field4"
@@
 F 0 "C105" H 4675 5250 50  0000 L CNN
 F 1 "100n" H 4675 5050 50  0000 L CNN
-F 2 "TinyTiM_Lib:c_0805" H 4650 5150 50  0001 C CNN
+F 2 "C4_Pretty:c_0805" H 4650 5150 50  0001 C CNN
 F 3 "" H 4650 5150 60  0001 C CNN
 F 4 "CAP CER 0.1UF 25V 10% X7R 0805" H 4650 5350 60  0001 L CNN "Field4"
@@
 F 0 "C106" H 6075 5250 50  0000 L CNN
 F 1 "100n" H 6075 5050 50  0000 L CNN
-F 2 "TinyTiM_Lib:c_0805" H 6050 5150 50  0001 C CNN
+F 2 "C4_Pretty:c_0805" H 6050 5150 50  0001 C CNN
 F 3 "" H 6050 5150 60  0001 C CNN
 F 4 "CAP CER 0.1UF 25V 10% X7R 0805" H 6050 5350 60  0001 L CNN "Field4"
@@
 F 0 "C107" H 7475 5250 50  0000 L CNN
 F 1 "100n" H 7475 5050 50  0000 L CNN
-F 2 "TinyTiM_Lib:c_0805" H 7450 5150 50  0001 C CNN
+F 2 "C4_Pretty:c_0805" H 7450 5150 50  0001 C CNN
 F 3 "" H 7450 5150 60  0001 C CNN
 F 4 "CAP CER 0.1UF 25V 10% X7R 0805" H 7450 5350 60  0001 L CNN "Field4"
@@
 F 0 "C108" H 8875 5250 50  0000 L CNN
 F 1 "100n" H 8875 5050 50  0000 L CNN
-F 2 "TinyTiM_Lib:c_0805" H 8850 5150 50  0001 C CNN
+F 2 "C4_Pretty:c_0805" H 8850 5150 50  0001 C CNN
 F 3 "" H 8850 5150 60  0001 C CNN
 F 4 "CAP CER 0.1UF 25V 10% X7R 0805" H 8850 5350 60  0001 L CNN "Field4"
@@
 F 0 "C109" H 10275 5250 50  0000 L CNN
 F 1 "100n" H 10275 5050 50  0000 L CNN
-F 2 "TinyTiM_Lib:c_0805" H 10250 5150 50  0001 C CNN
+F 2 "C4_Pretty:c_0805" H 10250 5150 50  0001 C CNN
 F 3 "" H 10250 5150 60  0001 C CNN
 F 4 "CAP CER 0.1UF 25V 10% X7R 0805" H 10250 5350 60  0001 L CNN "Field4"
@@
 F 0 "LED85" V 1425 1825 60  0000 C CNN
 F 1 "WS2812B" V 2075 1825 60  0001 C CNN
-F 2 "~" H 1675 1825 60  0000 C CNN
+F 2 "C4_Pretty:RGB_WS2811B" H 1675 1825 60  0001 C CNN
 F 3 "~" H 1675 1825 60  0000 C CNN
 	1    1675 1825
@@
 F 0 "LED86" V 2825 1825 60  0000 C CNN
 F 1 "WS2812B" V 3475 1825 60  0001 C CNN
-F 2 "~" H 3075 1825 60  0000 C CNN
+F 2 "C4_Pretty:RGB_WS2811B" H 3075 1825 60  0001 C CNN
 F 3 "~" H 3075 1825 60  0000 C CNN
 	1    3075 1825
@@
 F 0 "LED87" V 4225 1825 60  0000 C CNN
 F 1 "WS2812B" V 4875 1825 60  0001 C CNN
-F 2 "~" H 4475 1825 60  0000 C CNN
+F 2 "C4_Pretty:RGB_WS2811B" H 4475 1825 60  0001 C CNN
 F 3 "~" H 4475 1825 60  0000 C CNN
 	1    4475 1825
@@
 F 0 "LED88" V 5625 1825 60  0000 C CNN
 F 1 "WS2812B" V 6275 1825 60  0001 C CNN
-F 2 "~" H 5875 1825 60  0000 C CNN
+F 2 "C4_Pretty:RGB_WS2811B" H 5875 1825 60  0001 C CNN
 F 3 "~" H 5875 1825 60  0000 C CNN
 	1    5875 1825
@@
 F 0 "LED89" V 7025 1825 60  0000 C CNN
 F 1 "WS2812B" V 7675 1825 60  0001 C CNN
-F 2 "~" H 7275 1825 60  0000 C CNN
+F 2 "C4_Pretty:RGB_WS2811B" H 7275 1825 60  0001 C CNN
 F 3 "~" H 7275 1825 60  0000 C CNN
 	1    7275 1825
@@
 F 0 "LED90" V 8425 1825 60  0000 C CNN
 F 1 "WS2812B" V 9075 1825 60  0001 C CNN
-F 2 "~" H 8675 1825 60  0000 C CNN
+F 2 "C4_Pretty:RGB_WS2811B" H 8675 1825 60  0001 C CNN
 F 3 "~" H 8675 1825 60  0000 C CNN
 	1    8675 1825
@@
 F 0 "LED91" V 9825 1825 60  0000 C CNN
 F 1 "WS2812B" V 10475 1825 60  0001 C CNN
-F 2 "~" H 10075 1825 60  0000 C CNN
+F 2 "C4_Pretty:RGB_WS2811B" H 10075 1825 60  0001 C CNN
 F 3 "~" H 10075 1825 60  0000 C CNN
 	1    10075 1825
@@
 F 0 "LED92" V 1425 4225 60  0000 C CNN
 F 1 "WS2812B" V 2075 4225 60  0001 C CNN
-F 2 "~" H 1675 4225 60  0000 C CNN
+F 2 "C4_Pretty:RGB_WS2811B" H 1675 4225 60  0001 C CNN
 F 3 "~" H 1675 4225 60  0000 C CNN
 	1    1675 4225
@@
 F 0 "LED93" V 2825 4225 60  0000 C CNN
 F 1 "WS2812B" V 3475 4225 60  0001 C CNN
-F 2 "~" H 3075 4225 60  0000 C CNN
+F 2 "C4_Pretty:RGB_WS2811B" H 3075 4225 60  0001 C CNN
 F 3 "~" H 3075 4225 60  0000 C CNN
 	1    3075 4225
@@
 F 0 "LED94" V 4225 4225 60  0000 C CNN
 F 1 "WS2812B" V 4875 4225 60  0001 C CNN
-F 2 "~" H 4475 4225 60  0000 C CNN
+F 2 "C4_Pretty:RGB_WS2811B" H 4475 4225 60  0001 C CNN
 F 3 "~" H 4475 4225 60  0000 C CNN
 	1    4475 4225
@@
 F 0 "LED95" V 5625 4225 60  0000 C CNN
 F 1 "WS2812B" V 6275 4225 60  0001 C CNN
-F 2 "~" H 5875 4225 60  0000 C CNN
+F 2 "C4_Pretty:RGB_WS2811B" H 5875 4225 60  0001 C CNN
 F 3 "~" H 5875 4225 60  0000 C CNN
 	1    5875 4225
@@
 F 0 "LED96" V 7025 4225 60  0000 C CNN
 F 1 "WS2812B" V 7675 4225 60  0001 C CNN
-F 2 "~" H 7275 4225 60  0000 C CNN
+F 2 "C4_Pretty:RGB_WS2811B" H 7275 4225 60  0001 C CNN
 F 3 "~" H 7275 4225 60  0000 C CNN
 	1    7275 4225
@@
 F 0 "LED97" V 8425 4225 60  0000 C CNN
 F 1 "WS2812B" V 9075 4225 60  0001 C CNN
-F 2 "~" H 8675 4225 60  0000 C CNN
+F 2 "C4_Pretty:RGB_WS2811B" H 8675 4225 60  0001 C CNN
 F 3 "~" H 8675 4225 60  0000 C CNN
 	1    8675 4225
@@
 F 0 "LED98" V 9825 4225 60  0000 C CNN
 F 1 "WS2812B" V 10475 4225 60  0001 C CNN
-F 2 "~" H 10075 4225 60  0000 C CNN
+F 2 "C4_Pretty:RGB_WS2811B" H 10075 4225 60  0001 C CNN
 F 3 "~" H 10075 4225 60  0000 C CNN
 	1    10075 4225

Commit message: C4 PCB layout complete. Added Gerbers
Parts:
- C100, C101, C102, C103, C104, C105, C106, C107, C108, C109, C96, C97, C98, C99: footprint C4_Pretty:c_0805 -> C4_Pretty:c_0805_led
Changed lines of the file:
@@
 EESchema Schematic File Version 2
 LIBS:ClockFOUR
+LIBS:RowGB_sym
 LIBS:ClockFOUR-cache
 EELAYER 24 0
@@
 F 0 "C96" H 1875 2900 50  0000 L CNN
 F 1 "100n" H 1875 2700 50  0000 L CNN
-F 2 "C4_Pretty:c_0805" H 1850 2800 50  0001 C CNN
+F 2 "C4_Pretty:c_0805_led" H 1850 2800 50  0001 C CNN
 F 3 "" H 1850 2800 60  0001 C CNN
 F 4 "CAP CER 0.1UF 25V 10% X7R 0805" H 1850 3000 60  0001 L CNN "Field4"
@@
 F 0 "C97" H 3275 2900 50  0000 L CNN
 F 1 "100n" H 3275 2700 50  0000 L CNN
-F 2 "C4_Pretty:c_0805" H 3250 2800 50  0001 C CNN
+F 2 "C4_Pretty:c_0805_led" H 3250 2800 50  0001 C CNN
 F 3 "" H 3250 2800 60  0001 C CNN
 F 4 "CAP CER 0.1UF 25V 10% X7R 0805" H 3250 3000 60  0001 L CNN "Field4"
@@
 F 0 "C98" H 4675 2900 50  0000 L CNN
 F 1 "100n" H 4675 2700 50  0000 L CNN
-F 2 "C4_Pretty:c_0805" H 4650 2800 50  0001 C CNN
+F 2 "C4_Pretty:c_0805_led" H 4650 2800 50  0001 C CNN
 F 3 "" H 4650 2800 60  0001 C CNN
 F 4 "CAP CER 0.1UF 25V 10% X7R 0805" H 4650 3000 60  0001 L CNN "Field4"
@@
 F 0 "C99" H 6075 2900 50  0000 L CNN
 F 1 "100n" H 6075 2700 50  0000 L CNN
-F 2 "C4_Pretty:c_0805" H 6050 2800 50  0001 C CNN
+F 2 "C4_Pretty:c_0805_led" H 6050 2800 50  0001 C CNN
 F 3 "" H 6050 2800 60  0001 C CNN
 F 4 "CAP CER 0.1UF 25V 10% X7R 0805" H 6050 3000 60  0001 L CNN "Field4"
@@
 F 0 "C100" H 7475 2900 50  0000 L CNN
 F 1 "100n" H 7475 2700 50  0000 L CNN
-F 2 "C4_Pretty:c_0805" H 7450 2800 50  0001 C CNN
+F 2 "C4_Pretty:c_0805_led" H 7450 2800 50  0001 C CNN
 F 3 "" H 7450 2800 60  0001 C CNN
 F 4 "CAP CER 0.1UF 25V 10% X7R 0805" H 7450 3000 60  0001 L CNN "Field4"
@@
 F 0 "C101" H 8875 2900 50  0000 L CNN
 F 1 "100n" H 8875 2700 50  0000 L CNN
-F 2 "C4_Pretty:c_0805" H 8850 2800 50  0001 C CNN
+F 2 "C4_Pretty:c_0805_led" H 8850 2800 50  0001 C CNN
 F 3 "" H 8850 2800 60  0001 C CNN
 F 4 "CAP CER 0.1UF 25V 10% X7R 0805" H 8850 3000 60  0001 L CNN "Field4"
@@
 F 0 "C102" H 10275 2900 50  0000 L CNN
 F 1 "100n" H 10275 2700 50  0000 L CNN
-F 2 "C4_Pretty:c_0805" H 10250 2800 50  0001 C CNN
+F 2 "C4_Pretty:c_0805_led" H 10250 2800 50  0001 C CNN
 F 3 "" H 10250 2800 60  0001 C CNN
 F 4 "CAP CER 0.1UF 25V 10% X7R 0805" H 10250 3000 60  0001 L CNN "Field4"
@@
 F 0 "C103" H 1875 5250 50  0000 L CNN
 F 1 "100n" H 1875 5050 50  0000 L CNN
-F 2 "C4_Pretty:c_0805" H 1850 5150 50  0001 C CNN
+F 2 "C4_Pretty:c_0805_led" H 1850 5150 50  0001 C CNN
 F 3 "" H 1850 5150 60  0001 C CNN
 F 4 "CAP CER 0.1UF 25V 10% X7R 0805" H 1850 5350 60  0001 L CNN "Field4"
@@
 F 0 "C104" H 3275 5250 50  0000 L CNN
 F 1 "100n" H 3275 5050 50  0000 L CNN
-F 2 "C4_Pretty:c_0805" H 3250 5150 50  0001 C CNN
+F 2 "C4_Pretty:c_0805_led" H 3250 5150 50  0001 C CNN
 F 3 "" H 3250 5150 60  0001 C CNN
 F 4 "CAP CER 0.1UF 25V 10% X7R 0805" H 3250 5350 60  0001 L CNN "Field4"
@@
 F 0 "C105" H 4675 5250 50  0000 L CNN
 F 1 "100n" H 4675 5050 50  0000 L CNN
-F 2 "C4_Pretty:c_0805" H 4650 5150 50  0001 C CNN
+F 2 "C4_Pretty:c_0805_led" H 4650 5150 50  0001 C CNN
 F 3 "" H 4650 5150 60  0001 C CNN
 F 4 "CAP CER 0.1UF 25V 10% X7R 0805" H 4650 5350 60  0001 L CNN "Field4"
@@
 F 0 "C106" H 6075 5250 50  0000 L CNN
 F 1 "100n" H 6075 5050 50  0000 L CNN
-F 2 "C4_Pretty:c_0805" H 6050 5150 50  0001 C CNN
+F 2 "C4_Pretty:c_0805_led" H 6050 5150 50  0001 C CNN
 F 3 "" H 6050 5150 60  0001 C CNN
 F 4 "CAP CER 0.1UF 25V 10% X7R 0805" H 6050 5350 60  0001 L CNN "Field4"
@@
 F 0 "C107" H 7475 5250 50  0000 L CNN
 F 1 "100n" H 7475 5050 50  0000 L CNN
-F 2 "C4_Pretty:c_0805" H 7450 5150 50  0001 C CNN
+F 2 "C4_Pretty:c_0805_led" H 7450 5150 50  0001 C CNN
 F 3 "" H 7450 5150 60  0001 C CNN
 F 4 "CAP CER 0.1UF 25V 10% X7R 0805" H 7450 5350 60  0001 L CNN "Field4"
@@
 F 0 "C108" H 8875 5250 50  0000 L CNN
 F 1 "100n" H 8875 5050 50  0000 L CNN
-F 2 "C4_Pretty:c_0805" H 8850 5150 50  0001 C CNN
+F 2 "C4_Pretty:c_0805_led" H 8850 5150 50  0001 C CNN
 F 3 "" H 8850 5150 60  0001 C CNN
 F 4 "CAP CER 0.1UF 25V 10% X7R 0805" H 8850 5350 60  0001 L CNN "Field4"
@@
 F 0 "C109" H 10275 5250 50  0000 L CNN
 F 1 "100n" H 10275 5050 50  0000 L CNN
-F 2 "C4_Pretty:c_0805" H 10250 5150 50  0001 C CNN
+F 2 "C4_Pretty:c_0805_led" H 10250 5150 50  0001 C CNN
 F 3 "" H 10250 5150 60  0001 C CNN
 F 4 "CAP CER 0.1UF 25V 10% X7R 0805" H 10250 5350 60  0001 L CNN "Field4"
