File: KiCad/Row_H.sch (KiCad schematic (older format))
At the start: 14 parts, among them U101 RGB_WS2811B, U102 RGB_WS2811B, U103 RGB_WS2811B, U104 RGB_WS2811B, U105 RGB_WS2811B, U106 RGB_WS2811B, U107 RGB_WS2811B, U108 RGB_WS2811B

Commit message: Schematic updated
Parts:
- removed C101: 100n, TinyTiM_Lib:c_0805, symbol C2
- removed C117: 47u,8V, TinyTiM_Lib:c_2917, symbol C_POL_1
- removed S101, S102, S103, S104: CONN_1, TinyTiM_Lib:Screw, symbol CONN_1
- removed U101, U102, U103, U104, U105, U106, U107, U108: RGB_WS2811B, TinyTiM_Lib:RGB_WS2811B, symbol RGB_WS2811B
Connections:
- net labels removed: 5V, A_02, A_03, A_04, A_05, A_06, A_07, A_08, A_09, DI_A, DO_A, GND
- wire segments 49 -> 0
- no-connect marks 4 -> 0
Other:
- note removed: "Mounting Screws"

Commit message: Schematic updated
Parts:
- added C108, C109, C110, C111, C112, C113, C114, C115, C116, C117, C118, C119, C120, C121: 100n, TinyTiM_Lib:c_0805, symbol C2
- added U102, U103, U104, U105, U106, U107, U108, U109, U110, U111, U112, U113, U114, U115: RGB_WS2812B, symbol RGB_WS2812B
Connections:
- net labels added: 5V, DI_H, DO_H, GND
- wire segments 0 -> 82

Commit message: Schematic updated, board started
Parts:
- C109: renamed from C108; Field5 100nF, 25V -> 100n, 25V
- C111: renamed from C112; Field5 100nF, 25V -> 100n, 25V
- C113: renamed from C116; Field5 100nF, 25V -> 100n, 25V
- C115: renamed from C120; Field5 100nF, 25V -> 100n, 25V
- C117: renamed from C111; Field5 100nF, 25V -> 100n, 25V
- C119: renamed from C115; Field5 100nF, 25V -> 100n, 25V
- C121: renamed from C119; Field5 100nF, 25V -> 100n, 25V
- renumbered C114 to C112, C118 to C114, C109 to C116, C113 to C118, C117 to C120, C121 to C122, U102 to U100, U104 to U101, U106 to U102, U108 to U103, U110 to U104, U112 to U105, U114 to U106, U103 to U107, U105 to U108, U107 to U109, U109 to U110, U113 to U112, U115 to U113
Changed lines of the file:
@@
 LIBS:contrib
 LIBS:valves
-LIBS:TinyTiM-cache
-LIBS:TiNA_sym
+LIBS:ClockFOUR
 LIBS:ClockFOUR-cache
 EELAYER 27 0
@@
 Sheet 9 14
 Title "ClockFOUR"
-Date "30 sep 2014"
+Date "1 oct 2014"
 Rev ""
 Comp "WyoLum"
@@
 5V
 $Comp
-L GND #PWR019
+L GND #PWR021
 U 1 1 542C113F
 P 1350 2550
-F 0 "#PWR019" H 1350 2550 30  0001 C CNN
+F 0 "#PWR021" H 1350 2550 30  0001 C CNN
 F 1 "GND" H 1350 2480 30  0001 C CNN
 F 2 "" H 1350 2550 60  0001 C CNN
@@
 $EndComp
 $Comp
-L C2 C108
+L C2 C109
 U 1 1 542C114D
 P 1900 2700
-F 0 "C108" H 1925 2800 50  0000 L CNN
+F 0 "C109" H 1925 2800 50  0000 L CNN
 F 1 "100n" H 1925 2600 50  0000 L CNN
 F 2 "TinyTiM_Lib:c_0805" H 1900 2700 50  0001 C CNN
 F 3 "" H 1900 2700 60  0001 C CNN
 F 4 "CAP CER 0.1UF 25V 10% X7R 0805" H 1900 2900 60  0001 L CNN "Field4"
-F 5 "100nF, 25V" H 1900 3000 60  0001 L CNN "Field5"
+F 5 "100n, 25V" H 1900 3000 60  0001 L CNN "Field5"
 F 6 "Surface Mount, MLCC" H 1900 3100 60  0001 L CNN "Field6"
 F 7 "Kemet" H 1900 3200 60  0001 L CNN "Field7"
@@
 $EndComp
 $Comp
-L RGB_WS2812B U102
+L RGB_WS2812B U100
 U 1 1 542C1153
 P 1725 1725
-F 0 "U102" V 1475 1725 60  0000 C CNN
+F 0 "U100" V 1475 1725 60  0000 C CNN
 F 1 "RGB_WS2812B" V 2125 1725 60  0000 C CNN
 F 2 "" H 1725 1725 60  0000 C CNN
@@
 $EndComp
 $Comp
-L RGB_WS2812B U104
+L RGB_WS2812B U101
 U 1 1 542C1159
 P 3125 1725
-F 0 "U104" V 2875 1725 60  0000 C CNN
+F 0 "U101" V 2875 1725 60  0000 C CNN
 F 1 "RGB_WS2812B" V 3525 1725 60  0000 C CNN
 F 2 "" H 3125 1725 60  0000 C CNN
@@
 $EndComp
 $Comp
-L RGB_WS2812B U106
+L RGB_WS2812B U102
 U 1 1 542C115F
 P 4525 1725
-F 0 "U106" V 4275 1725 60  0000 C CNN
+F 0 "U102" V 4275 1725 60  0000 C CNN
 F 1 "RGB_WS2812B" V 4925 1725 60  0000 C CNN
 F 2 "" H 4525 1725 60  0000 C CNN
@@
 $EndComp
 $Comp
-L RGB_WS2812B U108
+L RGB_WS2812B U103
 U 1 1 542C1165
 P 5925 1725
-F 0 "U108" V 5675 1725 60  0000 C CNN
+F 0 "U103" V 5675 1725 60  0000 C CNN
 F 1 "RGB_WS2812B" V 6325 1725 60  0000 C CNN
 F 2 "" H 5925 1725 60  0000 C CNN
@@
 $EndComp
 $Comp
-L RGB_WS2812B U110
+L RGB_WS2812B U104
 U 1 1 542C116B
 P 7325 1725
-F 0 "U110" V 7075 1725 60  0000 C CNN
+F 0 "U104" V 7075 1725 60  0000 C CNN
 F 1 "RGB_WS2812B" V 7725 1725 60  0000 C CNN
 F 2 "" H 7325 1725 60  0000 C CNN
@@
 $EndComp
 $Comp
-L RGB_WS2812B U112
+L RGB_WS2812B U105
 U 1 1 542C1171
 P 8725 1725
-F 0 "U112" V 8475 1725 60  0000 C CNN
+F 0 "U105" V 8475 1725 60  0000 C CNN
 F 1 "RGB_WS2812B" V 9125 1725 60  0000 C CNN
 F 2 "" H 8725 1725 60  0000 C CNN
@@
 $EndComp
 $Comp
-L RGB_WS2812B U114
+L RGB_WS2812B U106
 U 1 1 542C1177
 P 10125 1725
-F 0 "U114" V 9875 1725 60  0000 C CNN
+F 0 "U106" V 9875 1725 60  0000 C CNN
 F 1 "RGB_WS2812B" V 10525 1725 60  0000 C CNN
 F 2 "" H 10125 1725 60  0000 C CNN
@@
 $EndComp
 $Comp
-L RGB_WS2812B U103
+L RGB_WS2812B U107
 U 1 1 542C117D
 P 1725 4125
-F 0 "U103" V 1475 4125 60  0000 C CNN
+F 0 "U107" V 1475 4125 60  0000 C CNN
 F 1 "RGB_WS2812B" V 2125 4125 60  0000 C CNN
 F 2 "" H 1725 4125 60  0000 C CNN
@@
 $EndComp
 $Comp
-L RGB_WS2812B U105
+L RGB_WS2812B U108
 U 1 1 542C1183
 P 3125 4125
-F 0 "U105" V 2875 4125 60  0000 C CNN
+F 0 "U108" V 2875 4125 60  0000 C CNN
 F 1 "RGB_WS2812B" V 3525 4125 60  0000 C CNN
 F 2 "" H 3125 4125 60  0000 C CNN
@@
 $EndComp
 $Comp
-L RGB_WS2812B U107
+L RGB_WS2812B U109
 U 1 1 542C1189
 P 4525 4125
-F 0 "U107" V 4275 4125 60  0000 C CNN
+F 0 "U109" V 4275 4125 60  0000 C CNN
 F 1 "RGB_WS2812B" V 4925 4125 60  0000 C CNN
 F 2 "" H 4525 4125 60  0000 C CNN
@@
 $EndComp
 $Comp
-L RGB_WS2812B U109
+L RGB_WS2812B U110
 U 1 1 542C118F
 P 5925 4125
-F 0 "U109" V 5675 4125 60  0000 C CNN
+F 0 "U110" V 5675 4125 60  0000 C CNN
 F 1 "RGB_WS2812B" V 6325 4125 60  0000 C CNN
 F 2 "" H 5925 4125 60  0000 C CNN
@@
 $EndComp
 $Comp
-L RGB_WS2812B U113
+L RGB_WS2812B U112
 U 1 1 542C119B
 P 8725 4125
-F 0 "U113" V 8475 4125 60  0000 C CNN
+F 0 "U112" V 8475 4125 60  0000 C CNN
 F 1 "RGB_WS2812B" V 9125 4125 60  0000 C CNN
 F 2 "" H 8725 4125 60  0000 C CNN
@@
 $EndComp
 $Comp
-L RGB_WS2812B U115
+L RGB_WS2812B U113
 U 1 1 542C11A1
 P 10125 4125
-F 0 "U115" V 9875 4125 60  0000 C CNN
+F 0 "U113" V 9875 4125 60  0000 C CNN
 F 1 "RGB_WS2812B" V 10525 4125 60  0000 C CNN
 F 2 "" H 10125 4125 60  0000 C CNN
@@
 $EndComp
 $Comp
-L C2 C112
+L C2 C111
 U 1 1 542C120A
 P 4700 2700
-F 0 "C112" H 4725 2800 50  0000 L CNN
+F 0 "C111" H 4725 2800 50  0000 L CNN
 F 1 "100n" H 4725 2600 50  0000 L CNN
 F 2 "TinyTiM_Lib:c_0805" H 4700 2700 50  0001 C CNN
 F 3 "" H 4700 2700 60  0001 C CNN
 F 4 "CAP CER 0.1UF 25V 10% X7R 0805" H 4700 2900 60  0001 L CNN "Field4"
-F 5 "100nF, 25V" H 4700 3000 60  0001 L CNN "Field5"
+F 5 "100n, 25V" H 4700 3000 60  0001 L CNN "Field5"
 F 6 "Surface Mount, MLCC" H 4700 3100 60  0001 L CNN "Field6"
 F 7 "Kemet" H 4700 3200 60  0001 L CNN "Field7"
@@
 $EndComp
 $Comp
-L C2 C114
+L C2 C112
 U 1 1 542C1218
 P 6100 2700
-F 0 "C114" H 6125 2800 50  0000 L CNN
+F 0 "C112" H 6125 2800 50  0000 L CNN
 F 1 "100n" H 6125 2600 50  0000 L CNN
 F 2 "TinyTiM_Lib:c_0805" H 6100 2700 50  0001 C CNN
@@
 $EndComp
 $Comp
-L C2 C116
+L C2 C113
 U 1 1 542C1226
 P 7500 2700
-F 0 "C116" H 7525 2800 50  0000 L CNN
+F 0 "C113" H 7525 2800 50  0000 L CNN
 F 1 "100n" H 7525 2600 50  0000 L CNN
 F 2 "TinyTiM_Lib:c_0805" H 7500 2700 50  0001 C CNN
 F 3 "" H 7500 2700 60  0001 C CNN
 F 4 "CAP CER 0.1UF 25V 10% X7R 0805" H 7500 2900 60  0001 L CNN "Field4"
-F 5 "100nF, 25V" H 7500 3000 60  0001 L CNN "Field5"
+F 5 "100n, 25V" H 7500 3000 60  0001 L CNN "Field5"
 F 6 "Surface Mount, MLCC" H 7500 3100 60  0001 L CNN "Field6"
 F 7 "Kemet" H 7500 3200 60  0001 L CNN "Field7"
@@
 $EndComp
 $Comp
-L C2 C118
+L C2 C114
 U 1 1 542C1234
 P 8900 2700
-F 0 "C118" H 8925 2800 50  0000 L CNN
+F 0 "C114" H 8925 2800 50  0000 L CNN
 F 1 "100n" H 8925 2600 50  0000 L CNN
 F 2 "TinyTiM_Lib:c_0805" H 8900 2700 50  0001 C CNN
@@
 $EndComp
 $Comp
-L C2 C120
+L C2 C115
 U 1 1 542C1242
 P 10300 2700
-F 0 "C120" H 10325 2800 50  0000 L CNN
+F 0 "C115" H 10325 2800 50  0000 L CNN
 F 1 "100n" H 10325 2600 50  0000 L CNN
 F 2 "TinyTiM_Lib:c_0805" H 10300 2700 50  0001 C CNN
 F 3 "" H 10300 2700 60  0001 C CNN
 F 4 "CAP CER 0.1UF 25V 10% X7R 0805" H 10300 2900 60  0001 L CNN "Field4"
-F 5 "100nF, 25V" H 10300 3000 60  0001 L CNN "Field5"
+F 5 "100n, 25V" H 10300 3000 60  0001 L CNN "Field5"
 F 6 "Surface Mount, MLCC" H 10300 3100 60  0001 L CNN "Field6"
 F 7 "Kemet" H 10300 3200 60  0001 L CNN "Field7"
@@
 Connection ~ 10200 2900
 $Comp
-L C2 C109
+L C2 C116
 U 1 1 542C1251
 P 1900 5050
-F 0 "C109" H 1925 5150 50  0000 L CNN
+F 0 "C116" H 1925 5150 50  0000 L CNN
 F 1 "100n" H 1925 4950 50  0000 L CNN
 F 2 "TinyTiM_Lib:c_0805" H 1900 5050 50  0001 C CNN
@@
 Connection ~ 1800 5250
 $Comp
-L C2 C111
+L C2 C117
 U 1 1 542C128E
 P 3300 5050
-F 0 "C111" H 3325 5150 50  0000 L CNN
+F 0 "C117" H 3325 5150 50  0000 L CNN
 F 1 "100n" H 3325 4950 50  0000 L CNN
 F 2 "TinyTiM_Lib:c_0805" H 3300 5050 50  0001 C CNN
 F 3 "" H 3300 5050 60  0001 C CNN
 F 4 "CAP CER 0.1UF 25V 10% X7R 0805" H 3300 5250 60  0001 L CNN "Field4"
-F 5 "100nF, 25V" H 3300 5350 60  0001 L CNN "Field5"
+F 5 "100n, 25V" H 3300 5350 60  0001 L CNN "Field5"
 F 6 "Surface Mount, MLCC" H 3300 5450 60  0001 L CNN "Field6"
 F 7 "Kemet" H 3300 5550 60  0001 L CNN "Field7"
@@
 $EndComp
 $Comp
-L C2 C113
+L C2 C118
 U 1 1 542C129C
 P 4700 5050
-F 0 "C113" H 4725 5150 50  0000 L CNN
+F 0 "C118" H 4725 5150 50  0000 L CNN
 F 1 "100n" H 4725 4950 50  0000 L CNN
 F 2 "TinyTiM_Lib:c_0805" H 4700 5050 50  0001 C CNN
@@
 $EndComp
 $Comp
-L C2 C115
+L C2 C119
 U 1 1 542C12AA
 P 6100 5050
-F 0 "C115" H 6125 5150 50  0000 L CNN
+F 0 "C119" H 6125 5150 50  0000 L CNN
 F 1 "100n" H 6125 4950 50  0000 L CNN
 F 2 "TinyTiM_Lib:c_0805" H 6100 5050 50  0001 C CNN
 F 3 "" H 6100 5050 60  0001 C CNN
 F 4 "CAP CER 0.1UF 25V 10% X7R 0805" H 6100 5250 60  0001 L CNN "Field4"
-F 5 "100nF, 25V" H 6100 5350 60  0001 L CNN "Field5"
+F 5 "100n, 25V" H 6100 5350 60  0001 L CNN "Field5"
 F 6 "Surface Mount, MLCC" H 6100 5450 60  0001 L CNN "Field6"
 F 7 "Kemet" H 6100 5550 60  0001 L CNN "Field7"
@@
 $EndComp
 $Comp
-L C2 C117
+L C2 C120
 U 1 1 542C12B8
 P 7500 5050
-F 0 "C117" H 7525 5150 50  0000 L CNN
+F 0 "C120" H 7525 5150 50  0000 L CNN
 F 1 "100n" H 7525 4950 50  0000 L CNN
 F 2 "TinyTiM_Lib:c_0805" H 7500 5050 50  0001 C CNN
@@
 $EndComp
 $Comp
-L C2 C119
+L C2 C121
 U 1 1 542C12C6
 P 8900 5050
-F 0 "C119" H 8925 5150 50  0000 L CNN
+F 0 "C121" H 8925 5150 50  0000 L CNN
 F 1 "100n" H 8925 4950 50  0000 L CNN
 F 2 "TinyTiM_Lib:c_0805" H 8900 5050 50  0001 C CNN
 F 3 "" H 8900 5050 60  0001 C CNN
 F 4 "CAP CER 0.1UF 25V 10% X7R 0805" H 8900 5250 60  0001 L CNN "Field4"
-F 5 "100nF, 25V" H 8900 5350 60  0001 L CNN "Field5"
+F 5 "100n, 25V" H 8900 5350 60  0001 L CNN "Field5"
 F 6 "Surface Mount, MLCC" H 8900 5450 60  0001 L CNN "Field6"
 F 7 "Kemet" H 8900 5550 60  0001 L CNN "Field7"
@@
 $EndComp
 $Comp
-L C2 C121
+L C2 C122
 U 1 1 542C12D4
 P 10300 5050
-F 0 "C121" H 10325 5150 50  0000 L CNN
+F 0 "C122" H 10325 5150 50  0000 L CNN
 F 1 "100n" H 10325 4950 50  0000 L CNN
 F 2 "TinyTiM_Lib:c_0805" H 10300 5050 50  0001 C CNN

Commit message: Board layout updated
Parts:
- removed U100, U101, U102, U103, U104, U105, U106, U107, U108, U109, U110, U111, U112, U113: RGB_WS2812B, symbol RGB_WS2812B
- added LED100, LED101, LED102, LED103, LED104, LED105, LED106, LED107, LED108, LED109, LED110, LED111, LED112, LED99: RGB_WS2812B, ~, symbol RGB_WS2812B

Commit message: Board layout updated
Matrix placed and wired. Added RTC.
Parts:
- removed C109: 100n, TinyTiM_Lib:c_0805, symbol C2
- removed LED100, LED101, LED102, LED103, LED104, LED105, LED106, LED107, LED108, LED109, LED110, LED111, LED112, LED99: RGB_WS2812B, ~, symbol RGB_WS2812B
- added C123: 100n, TinyTiM_Lib:c_0805, symbol C2
- added LED100, LED101, LED102, LED103, LED104, LED105, LED106, LED107, LED108, LED109, LED110, LED111, LED112, LED99: WS2812B, ~, symbol WS2812B
- C110, C112, C114, C116, C118, C120, C122: Field5 100nF, 25V -> 100n, 25V
- C111, C113, C115, C117, C119, C121: Field5 100n, 25V -> 100nF, 25V
