File: KiCad/Row_H.sch (KiCad schematic (older format))
At the start: 28 parts

Commit message: PCB layout, work in progress
Parts:
- C110, C111, C112, C113, C114, C115, C116, C117, C118, C119, C120, C121, C122, C123: footprint TinyTiM_Lib:c_0805 -> C4_Pretty:c_0805
- LED100, LED101, LED102, LED103, LED104, LED105, LED106, LED107, LED108, LED109, LED110, LED111, LED112, LED99: footprint ~ -> C4_Pretty:RGB_WS2811B
Changed lines of the file:
@@
 F 0 "C110" H 1875 2750 50  0000 L CNN
 F 1 "100n" H 1875 2550 50  0000 L CNN
-F 2 "TinyTiM_Lib:c_0805" H 1850 2650 50  0001 C CNN
+F 2 "C4_Pretty:c_0805" H 1850 2650 50  0001 C CNN
 F 3 "" H 1850 2650 60  0001 C CNN
 F 4 "CAP CER 0.1UF 25V 10% X7R 0805" H 1850 2850 60  0001 L CNN "Field4"
@@
 F 0 "C111" H 3275 2750 50  0000 L CNN
 F 1 "100n" H 3275 2550 50  0000 L CNN
-F 2 "TinyTiM_Lib:c_0805" H 3250 2650 50  0001 C CNN
+F 2 "C4_Pretty:c_0805" H 3250 2650 50  0001 C CNN
 F 3 "" H 3250 2650 60  0001 C CNN
 F 4 "CAP CER 0.1UF 25V 10% X7R 0805" H 3250 2850 60  0001 L CNN "Field4"
@@
 F 0 "C112" H 4675 2750 50  0000 L CNN
 F 1 "100n" H 4675 2550 50  0000 L CNN
-F 2 "TinyTiM_Lib:c_0805" H 4650 2650 50  0001 C CNN
+F 2 "C4_Pretty:c_0805" H 4650 2650 50  0001 C CNN
 F 3 "" H 4650 2650 60  0001 C CNN
 F 4 "CAP CER 0.1UF 25V 10% X7R 0805" H 4650 2850 60  0001 L CNN "Field4"
@@
 F 0 "C113" H 6075 2750 50  0000 L CNN
 F 1 "100n" H 6075 2550 50  0000 L CNN
-F 2 "TinyTiM_Lib:c_0805" H 6050 2650 50  0001 C CNN
+F 2 "C4_Pretty:c_0805" H 6050 2650 50  0001 C CNN
 F 3 "" H 6050 2650 60  0001 C CNN
 F 4 "CAP CER 0.1UF 25V 10% X7R 0805" H 6050 2850 60  0001 L CNN "Field4"
@@
 F 0 "C114" H 7475 2750 50  0000 L CNN
 F 1 "100n" H 7475 2550 50  0000 L CNN
-F 2 "TinyTiM_Lib:c_0805" H 7450 2650 50  0001 C CNN
+F 2 "C4_Pretty:c_0805" H 7450 2650 50  0001 C CNN
 F 3 "" H 7450 2650 60  0001 C CNN
 F 4 "CAP CER 0.1UF 25V 10% X7R 0805" H 7450 2850 60  0001 L CNN "Field4"
@@
 F 0 "C115" H 8875 2750 50  0000 L CNN
 F 1 "100n" H 8875 2550 50  0000 L CNN
-F 2 "TinyTiM_Lib:c_0805" H 8850 2650 50  0001 C CNN
+F 2 "C4_Pretty:c_0805" H 8850 2650 50  0001 C CNN
 F 3 "" H 8850 2650 60  0001 C CNN
 F 4 "CAP CER 0.1UF 25V 10% X7R 0805" H 8850 2850 60  0001 L CNN "Field4"
@@
 F 0 "C116" H 10275 2750 50  0000 L CNN
 F 1 "100n" H 10275 2550 50  0000 L CNN
-F 2 "TinyTiM_Lib:c_0805" H 10250 2650 50  0001 C CNN
+F 2 "C4_Pretty:c_0805" H 10250 2650 50  0001 C CNN
 F 3 "" H 10250 2650 60  0001 C CNN
 F 4 "CAP CER 0.1UF 25V 10% X7R 0805" H 10250 2850 60  0001 L CNN "Field4"
@@
 F 0 "C117" H 1875 5100 50  0000 L CNN
 F 1 "100n" H 1875 4900 50  0000 L CNN
-F 2 "TinyTiM_Lib:c_0805" H 1850 5000 50  0001 C CNN
+F 2 "C4_Pretty:c_0805" H 1850 5000 50  0001 C CNN
 F 3 "" H 1850 5000 60  0001 C CNN
 F 4 "CAP CER 0.1UF 25V 10% X7R 0805" H 1850 5200 60  0001 L CNN "Field4"
@@
 F 0 "C118" H 3275 5100 50  0000 L CNN
 F 1 "100n" H 3275 4900 50  0000 L CNN
-F 2 "TinyTiM_Lib:c_0805" H 3250 5000 50  0001 C CNN
+F 2 "C4_Pretty:c_0805" H 3250 5000 50  0001 C CNN
 F 3 "" H 3250 5000 60  0001 C CNN
 F 4 "CAP CER 0.1UF 25V 10% X7R 0805" H 3250 5200 60  0001 L CNN "Field4"
@@
 F 0 "C119" H 4675 5100 50  0000 L CNN
 F 1 "100n" H 4675 4900 50  0000 L CNN
-F 2 "TinyTiM_Lib:c_0805" H 4650 5000 50  0001 C CNN
+F 2 "C4_Pretty:c_0805" H 4650 5000 50  0001 C CNN
 F 3 "" H 4650 5000 60  0001 C CNN
 F 4 "CAP CER 0.1UF 25V 10% X7R 0805" H 4650 5200 60  0001 L CNN "Field4"
@@
 F 0 "C120" H 6075 5100 50  0000 L CNN
 F 1 "100n" H 6075 4900 50  0000 L CNN
-F 2 "TinyTiM_Lib:c_0805" H 6050 5000 50  0001 C CNN
+F 2 "C4_Pretty:c_0805" H 6050 5000 50  0001 C CNN
 F 3 "" H 6050 5000 60  0001 C CNN
 F 4 "CAP CER 0.1UF 25V 10% X7R 0805" H 6050 5200 60  0001 L CNN "Field4"
@@
 F 0 "C121" H 7475 5100 50  0000 L CNN
 F 1 "100n" H 7475 4900 50  0000 L CNN
-F 2 "TinyTiM_Lib:c_0805" H 7450 5000 50  0001 C CNN
+F 2 "C4_Pretty:c_0805" H 7450 5000 50  0001 C CNN
 F 3 "" H 7450 5000 60  0001 C CNN
 F 4 "CAP CER 0.1UF 25V 10% X7R 0805" H 7450 5200 60  0001 L CNN "Field4"
@@
 F 0 "C122" H 8875 5100 50  0000 L CNN
 F 1 "100n" H 8875 4900 50  0000 L CNN
-F 2 "TinyTiM_Lib:c_0805" H 8850 5000 50  0001 C CNN
+F 2 "C4_Pretty:c_0805" H 8850 5000 50  0001 C CNN
 F 3 "" H 8850 5000 60  0001 C CNN
 F 4 "CAP CER 0.1UF 25V 10% X7R 0805" H 8850 5200 60  0001 L CNN "Field4"
@@
 F 0 "C123" H 10275 5100 50  0000 L CNN
 F 1 "100n" H 10275 4900 50  0000 L CNN
-F 2 "TinyTiM_Lib:c_0805" H 10250 5000 50  0001 C CNN
+F 2 "C4_Pretty:c_0805" H 10250 5000 50  0001 C CNN
 F 3 "" H 10250 5000 60  0001 C CNN
 F 4 "CAP CER 0.1UF 25V 10% X7R 0805" H 10250 5200 60  0001 L CNN "Field4"
@@
 F 0 "LED99" V 1425 1675 60  0000 C CNN
 F 1 "WS2812B" V 2075 1675 60  0001 C CNN
-F 2 "~" H 1675 1675 60  0000 C CNN
+F 2 "C4_Pretty:RGB_WS2811B" H 1675 1675 60  0001 C CNN
 F 3 "~" H 1675 1675 60  0000 C CNN
 	1    1675 1675
@@
 F 0 "LED100" V 2825 1675 60  0000 C CNN
 F 1 "WS2812B" V 3475 1675 60  0001 C CNN
-F 2 "~" H 3075 1675 60  0000 C CNN
+F 2 "C4_Pretty:RGB_WS2811B" H 3075 1675 60  0001 C CNN
 F 3 "~" H 3075 1675 60  0000 C CNN
 	1    3075 1675
@@
 F 0 "LED101" V 4225 1675 60  0000 C CNN
 F 1 "WS2812B" V 4875 1675 60  0001 C CNN
-F 2 "~" H 4475 1675 60  0000 C CNN
+F 2 "C4_Pretty:RGB_WS2811B" H 4475 1675 60  0001 C CNN
 F 3 "~" H 4475 1675 60  0000 C CNN
 	1    4475 1675
@@
 F 0 "LED102" V 5625 1675 60  0000 C CNN
 F 1 "WS2812B" V 6275 1675 60  0001 C CNN
-F 2 "~" H 5875 1675 60  0000 C CNN
+F 2 "C4_Pretty:RGB_WS2811B" H 5875 1675 60  0001 C CNN
 F 3 "~" H 5875 1675 60  0000 C CNN
 	1    5875 1675
@@
 F 0 "LED103" V 7025 1675 60  0000 C CNN
 F 1 "WS2812B" V 7675 1675 60  0001 C CNN
-F 2 "~" H 7275 1675 60  0000 C CNN
+F 2 "C4_Pretty:RGB_WS2811B" H 7275 1675 60  0001 C CNN
 F 3 "~" H 7275 1675 60  0000 C CNN
 	1    7275 1675
@@
 F 0 "LED104" V 8425 1675 60  0000 C CNN
 F 1 "WS2812B" V 9075 1675 60  0001 C CNN
-F 2 "~" H 8675 1675 60  0000 C CNN
+F 2 "C4_Pretty:RGB_WS2811B" H 8675 1675 60  0001 C CNN
 F 3 "~" H 8675 1675 60  0000 C CNN
 	1    8675 1675
@@
 F 0 "LED105" V 9825 1675 60  0000 C CNN
 F 1 "WS2812B" V 10475 1675 60  0001 C CNN
-F 2 "~" H 10075 1675 60  0000 C CNN
+F 2 "C4_Pretty:RGB_WS2811B" H 10075 1675 60  0001 C CNN
 F 3 "~" H 10075 1675 60  0000 C CNN
 	1    10075 1675
@@
 F 0 "LED106" V 1425 4075 60  0000 C CNN
 F 1 "WS2812B" V 2075 4075 60  0001 C CNN
-F 2 "~" H 1675 4075 60  0000 C CNN
+F 2 "C4_Pretty:RGB_WS2811B" H 1675 4075 60  0001 C CNN
 F 3 "~" H 1675 4075 60  0000 C CNN
 	1    1675 4075
@@
 F 0 "LED107" V 2825 4075 60  0000 C CNN
 F 1 "WS2812B" V 3475 4075 60  0001 C CNN
-F 2 "~" H 3075 4075 60  0000 C CNN
+F 2 "C4_Pretty:RGB_WS2811B" H 3075 4075 60  0001 C CNN
 F 3 "~" H 3075 4075 60  0000 C CNN
 	1    3075 4075
@@
 F 0 "LED108" V 4225 4075 60  0000 C CNN
 F 1 "WS2812B" V 4875 4075 60  0001 C CNN
-F 2 "~" H 4475 4075 60  0000 C CNN
+F 2 "C4_Pretty:RGB_WS2811B" H 4475 4075 60  0001 C CNN
 F 3 "~" H 4475 4075 60  0000 C CNN
 	1    4475 4075
@@
 F 0 "LED109" V 5625 4075 60  0000 C CNN
 F 1 "WS2812B" V 6275 4075 60  0001 C CNN
-F 2 "~" H 5875 4075 60  0000 C CNN
+F 2 "C4_Pretty:RGB_WS2811B" H 5875 4075 60  0001 C CNN
 F 3 "~" H 5875 4075 60  0000 C CNN
 	1    5875 4075
@@
 F 0 "LED110" V 7025 4075 60  0000 C CNN
 F 1 "WS2812B" V 7675 4075 60  0001 C CNN
-F 2 "~" H 7275 4075 60  0000 C CNN
+F 2 "C4_Pretty:RGB_WS2811B" H 7275 4075 60  0001 C CNN
 F 3 "~" H 7275 4075 60  0000 C CNN
 	1    7275 4075
@@
 F 0 "LED111" V 8425 4075 60  0000 C CNN
 F 1 "WS2812B" V 9075 4075 60  0001 C CNN
-F 2 "~" H 8675 4075 60  0000 C CNN
+F 2 "C4_Pretty:RGB_WS2811B" H 8675 4075 60  0001 C CNN
 F 3 "~" H 8675 4075 60  0000 C CNN
 	1    8675 4075
@@
 F 0 "LED112" V 9825 4075 60  0000 C CNN
 F 1 "WS2812B" V 10475 4075 60  0001 C CNN
-F 2 "~" H 10075 4075 60  0000 C CNN
+F 2 "C4_Pretty:RGB_WS2811B" H 10075 4075 60  0001 C CNN
 F 3 "~" H 10075 4075 60  0000 C CNN
 	1    10075 4075

Commit message: C4 PCB layout complete. Added Gerbers
Parts:
- C110, C111, C112, C113, C114, C115, C116, C117, C118, C119, C120, C121, C122, C123: footprint C4_Pretty:c_0805 -> C4_Pretty:c_0805_led
Changed lines of the file:
@@
 EESchema Schematic File Version 2
 LIBS:ClockFOUR
+LIBS:RowGB_sym
 LIBS:ClockFOUR-cache
 EELAYER 24 0
@@
 F 0 "C110" H 1875 2750 50  0000 L CNN
 F 1 "100n" H 1875 2550 50  0000 L CNN
-F 2 "C4_Pretty:c_0805" H 1850 2650 50  0001 C CNN
+F 2 "C4_Pretty:c_0805_led" H 1850 2650 50  0001 C CNN
 F 3 "" H 1850 2650 60  0001 C CNN
 F 4 "CAP CER 0.1UF 25V 10% X7R 0805" H 1850 2850 60  0001 L CNN "Field4"
@@
 F 0 "C111" H 3275 2750 50  0000 L CNN
 F 1 "100n" H 3275 2550 50  0000 L CNN
-F 2 "C4_Pretty:c_0805" H 3250 2650 50  0001 C CNN
+F 2 "C4_Pretty:c_0805_led" H 3250 2650 50  0001 C CNN
 F 3 "" H 3250 2650 60  0001 C CNN
 F 4 "CAP CER 0.1UF 25V 10% X7R 0805" H 3250 2850 60  0001 L CNN "Field4"
@@
 F 0 "C112" H 4675 2750 50  0000 L CNN
 F 1 "100n" H 4675 2550 50  0000 L CNN
-F 2 "C4_Pretty:c_0805" H 4650 2650 50  0001 C CNN
+F 2 "C4_Pretty:c_0805_led" H 4650 2650 50  0001 C CNN
 F 3 "" H 4650 2650 60  0001 C CNN
 F 4 "CAP CER 0.1UF 25V 10% X7R 0805" H 4650 2850 60  0001 L CNN "Field4"
@@
 F 0 "C113" H 6075 2750 50  0000 L CNN
 F 1 "100n" H 6075 2550 50  0000 L CNN
-F 2 "C4_Pretty:c_0805" H 6050 2650 50  0001 C CNN
+F 2 "C4_Pretty:c_0805_led" H 6050 2650 50  0001 C CNN
 F 3 "" H 6050 2650 60  0001 C CNN
 F 4 "CAP CER 0.1UF 25V 10% X7R 0805" H 6050 2850 60  0001 L CNN "Field4"
@@
 F 0 "C114" H 7475 2750 50  0000 L CNN
 F 1 "100n" H 7475 2550 50  0000 L CNN
-F 2 "C4_Pretty:c_0805" H 7450 2650 50  0001 C CNN
+F 2 "C4_Pretty:c_0805_led" H 7450 2650 50  0001 C CNN
 F 3 "" H 7450 2650 60  0001 C CNN
 F 4 "CAP CER 0.1UF 25V 10% X7R 0805" H 7450 2850 60  0001 L CNN "Field4"
@@
 F 0 "C115" H 8875 2750 50  0000 L CNN
 F 1 "100n" H 8875 2550 50  0000 L CNN
-F 2 "C4_Pretty:c_0805" H 8850 2650 50  0001 C CNN
+F 2 "C4_Pretty:c_0805_led" H 8850 2650 50  0001 C CNN
 F 3 "" H 8850 2650 60  0001 C CNN
 F 4 "CAP CER 0.1UF 25V 10% X7R 0805" H 8850 2850 60  0001 L CNN "Field4"
@@
 F 0 "C116" H 10275 2750 50  0000 L CNN
 F 1 "100n" H 10275 2550 50  0000 L CNN
-F 2 "C4_Pretty:c_0805" H 10250 2650 50  0001 C CNN
+F 2 "C4_Pretty:c_0805_led" H 10250 2650 50  0001 C CNN
 F 3 "" H 10250 2650 60  0001 C CNN
 F 4 "CAP CER 0.1UF 25V 10% X7R 0805" H 10250 2850 60  0001 L CNN "Field4"
@@
 F 0 "C117" H 1875 5100 50  0000 L CNN
 F 1 "100n" H 1875 4900 50  0000 L CNN
-F 2 "C4_Pretty:c_0805" H 1850 5000 50  0001 C CNN
+F 2 "C4_Pretty:c_0805_led" H 1850 5000 50  0001 C CNN
 F 3 "" H 1850 5000 60  0001 C CNN
 F 4 "CAP CER 0.1UF 25V 10% X7R 0805" H 1850 5200 60  0001 L CNN "Field4"
@@
 F 0 "C118" H 3275 5100 50  0000 L CNN
 F 1 "100n" H 3275 4900 50  0000 L CNN
-F 2 "C4_Pretty:c_0805" H 3250 5000 50  0001 C CNN
+F 2 "C4_Pretty:c_0805_led" H 3250 5000 50  0001 C CNN
 F 3 "" H 3250 5000 60  0001 C CNN
 F 4 "CAP CER 0.1UF 25V 10% X7R 0805" H 3250 5200 60  0001 L CNN "Field4"
@@
 F 0 "C119" H 4675 5100 50  0000 L CNN
 F 1 "100n" H 4675 4900 50  0000 L CNN
-F 2 "C4_Pretty:c_0805" H 4650 5000 50  0001 C CNN
+F 2 "C4_Pretty:c_0805_led" H 4650 5000 50  0001 C CNN
 F 3 "" H 4650 5000 60  0001 C CNN
 F 4 "CAP CER 0.1UF 25V 10% X7R 0805" H 4650 5200 60  0001 L CNN "Field4"
@@
 F 0 "C120" H 6075 5100 50  0000 L CNN
 F 1 "100n" H 6075 4900 50  0000 L CNN
-F 2 "C4_Pretty:c_0805" H 6050 5000 50  0001 C CNN
+F 2 "C4_Pretty:c_0805_led" H 6050 5000 50  0001 C CNN
 F 3 "" H 6050 5000 60  0001 C CNN
 F 4 "CAP CER 0.1UF 25V 10% X7R 0805" H 6050 5200 60  0001 L CNN "Field4"
@@
 F 0 "C121" H 7475 5100 50  0000 L CNN
 F 1 "100n" H 7475 4900 50  0000 L CNN
-F 2 "C4_Pretty:c_0805" H 7450 5000 50  0001 C CNN
+F 2 "C4_Pretty:c_0805_led" H 7450 5000 50  0001 C CNN
 F 3 "" H 7450 5000 60  0001 C CNN
 F 4 "CAP CER 0.1UF 25V 10% X7R 0805" H 7450 5200 60  0001 L CNN "Field4"
@@
 F 0 "C122" H 8875 5100 50  0000 L CNN
 F 1 "100n" H 8875 4900 50  0000 L CNN
-F 2 "C4_Pretty:c_0805" H 8850 5000 50  0001 C CNN
+F 2 "C4_Pretty:c_0805_led" H 8850 5000 50  0001 C CNN
 F 3 "" H 8850 5000 60  0001 C CNN
 F 4 "CAP CER 0.1UF 25V 10% X7R 0805" H 8850 5200 60  0001 L CNN "Field4"
@@
 F 0 "C123" H 10275 5100 50  0000 L CNN
 F 1 "100n" H 10275 4900 50  0000 L CNN
-F 2 "C4_Pretty:c_0805" H 10250 5000 50  0001 C CNN
+F 2 "C4_Pretty:c_0805_led" H 10250 5000 50  0001 C CNN
 F 3 "" H 10250 5000 60  0001 C CNN
 F 4 "CAP CER 0.1UF 25V 10% X7R 0805" H 10250 5200 60  0001 L CNN "Field4"
