File: KiCad/Row_I.sch (KiCad schematic (older format))
At the start: 14 parts, among them U101 RGB_WS2811B, U102 RGB_WS2811B, U103 RGB_WS2811B, U104 RGB_WS2811B, U105 RGB_WS2811B, U106 RGB_WS2811B, U107 RGB_WS2811B, U108 RGB_WS2811B

Commit message: Schematic updated
Parts:
- removed C101: 100n, TinyTiM_Lib:c_0805, symbol C2
- removed C117: 47u,8V, TinyTiM_Lib:c_2917, symbol C_POL_1
- removed S101, S102, S103, S104: CONN_1, TinyTiM_Lib:Screw, symbol CONN_1
- removed U101, U102, U103, U104, U105, U106, U107, U108: RGB_WS2811B, TinyTiM_Lib:RGB_WS2811B, symbol RGB_WS2811B
Connections:
- net labels removed: 5V, A_02, A_03, A_04, A_05, A_06, A_07, A_08, A_09, DI_A, DO_A, GND
- wire segments 49 -> 0
- no-connect marks 4 -> 0
Other:
- note removed: "Mounting Screws"

Commit message: Schematic updated
Parts:
- added C122, C123, C124, C125, C126, C127, C128, C129, C130, C131, C132, C133, C134, C135: 100n, TinyTiM_Lib:c_0805, symbol C2
- added U116, U117, U118, U119, U120, U121, U122, U123, U124, U125, U126, U127, U128, U129: RGB_WS2812B, symbol RGB_WS2812B
Connections:
- net labels added: 5V, DI_I, DO_I, GND
- wire segments 0 -> 82

Commit message: Schematic updated, board started
Parts:
- removed U126: RGB_WS2812B, symbol RGB_WS2812B
- added U119: RGB_WS2812B, ~, symbol RGB_WS2812B
- C123: renamed from C122; Field5 100nF, 25V -> 100n, 25V
- C125: renamed from C126; Field5 100nF, 25V -> 100n, 25V
- C127: renamed from C130; Field5 100nF, 25V -> 100n, 25V
- C129: renamed from C134; Field5 100nF, 25V -> 100n, 25V
- C131: renamed from C125; Field5 100nF, 25V -> 100n, 25V
- C133: renamed from C129; Field5 100nF, 25V -> 100n, 25V
- C135: renamed from C133; Field5 100nF, 25V -> 100n, 25V
- renumbered C128 to C126, C132 to C128, C123 to C130, C127 to C132, C131 to C134, C135 to C136, U116 to U114, U118 to U115, U120 to U116, U122 to U117, U124 to U118, U128 to U120, U117 to U121, U119 to U122, U121 to U123, U123 to U124, U127 to U126, U129 to U127

Commit message: Board layout updated
Parts:
- removed U114, U115, U116, U117, U118, U120, U121, U122, U123, U124, U125, U126, U127: RGB_WS2812B, symbol RGB_WS2812B
- removed U119: RGB_WS2812B, ~, symbol RGB_WS2812B
- added LED113, LED114, LED115, LED116, LED117, LED118, LED119, LED120, LED121, LED122, LED123, LED124, LED125, LED126: RGB_WS2812B, ~, symbol RGB_WS2812B

Commit message: Board layout updated
Matrix placed and wired. Added RTC.
Parts:
- removed C123: 100n, TinyTiM_Lib:c_0805, symbol C2
- removed LED113, LED114, LED115, LED116, LED117, LED118, LED119, LED120, LED121, LED122, LED123, LED124, LED125, LED126: RGB_WS2812B, ~, symbol RGB_WS2812B
- added C137: 100n, TinyTiM_Lib:c_0805, symbol C2
- added LED113, LED114, LED115, LED116, LED117, LED118, LED119, LED120, LED121, LED122, LED123, LED124, LED125, LED126: WS2812B, ~, symbol WS2812B
- C124, C126, C128, C130, C132, C134, C136: Field5 100nF, 25V -> 100n, 25V
- C125, C127, C129, C131, C133, C135: Field5 100n, 25V -> 100nF, 25V
