File: KiCad/Row_I.sch (KiCad schematic (older format))
At the start: 28 parts

Commit message: PCB layout, work in progress
Parts:
- C124, C125, C126, C127, C128, C129, C130, C131, C132, C133, C134, C135, C136, C137: footprint TinyTiM_Lib:c_0805 -> C4_Pretty:c_0805
- LED113, LED114, LED115, LED116, LED117, LED118, LED119, LED120, LED121, LED122, LED123, LED124, LED125, LED126: footprint ~ -> C4_Pretty:RGB_WS2811B
Changed lines of the file:
@@
 F 0 "C124" H 1825 2800 50  0000 L CNN
 F 1 "100n" H 1825 2600 50  0000 L CNN
-F 2 "TinyTiM_Lib:c_0805" H 1800 2700 50  0001 C CNN
+F 2 "C4_Pretty:c_0805" H 1800 2700 50  0001 C CNN
 F 3 "" H 1800 2700 60  0001 C CNN
 F 4 "CAP CER 0.1UF 25V 10% X7R 0805" H 1800 2900 60  0001 L CNN "Field4"
@@
 F 0 "C125" H 3225 2800 50  0000 L CNN
 F 1 "100n" H 3225 2600 50  0000 L CNN
-F 2 "TinyTiM_Lib:c_0805" H 3200 2700 50  0001 C CNN
+F 2 "C4_Pretty:c_0805" H 3200 2700 50  0001 C CNN
 F 3 "" H 3200 2700 60  0001 C CNN
 F 4 "CAP CER 0.1UF 25V 10% X7R 0805" H 3200 2900 60  0001 L CNN "Field4"
@@
 F 0 "C126" H 4625 2800 50  0000 L CNN
 F 1 "100n" H 4625 2600 50  0000 L CNN
-F 2 "TinyTiM_Lib:c_0805" H 4600 2700 50  0001 C CNN
+F 2 "C4_Pretty:c_0805" H 4600 2700 50  0001 C CNN
 F 3 "" H 4600 2700 60  0001 C CNN
 F 4 "CAP CER 0.1UF 25V 10% X7R 0805" H 4600 2900 60  0001 L CNN "Field4"
@@
 F 0 "C127" H 6025 2800 50  0000 L CNN
 F 1 "100n" H 6025 2600 50  0000 L CNN
-F 2 "TinyTiM_Lib:c_0805" H 6000 2700 50  0001 C CNN
+F 2 "C4_Pretty:c_0805" H 6000 2700 50  0001 C CNN
 F 3 "" H 6000 2700 60  0001 C CNN
 F 4 "CAP CER 0.1UF 25V 10% X7R 0805" H 6000 2900 60  0001 L CNN "Field4"
@@
 F 0 "C128" H 7425 2800 50  0000 L CNN
 F 1 "100n" H 7425 2600 50  0000 L CNN
-F 2 "TinyTiM_Lib:c_0805" H 7400 2700 50  0001 C CNN
+F 2 "C4_Pretty:c_0805" H 7400 2700 50  0001 C CNN
 F 3 "" H 7400 2700 60  0001 C CNN
 F 4 "CAP CER 0.1UF 25V 10% X7R 0805" H 7400 2900 60  0001 L CNN "Field4"
@@
 F 0 "C129" H 8825 2800 50  0000 L CNN
 F 1 "100n" H 8825 2600 50  0000 L CNN
-F 2 "TinyTiM_Lib:c_0805" H 8800 2700 50  0001 C CNN
+F 2 "C4_Pretty:c_0805" H 8800 2700 50  0001 C CNN
 F 3 "" H 8800 2700 60  0001 C CNN
 F 4 "CAP CER 0.1UF 25V 10% X7R 0805" H 8800 2900 60  0001 L CNN "Field4"
@@
 F 0 "C130" H 10225 2800 50  0000 L CNN
 F 1 "100n" H 10225 2600 50  0000 L CNN
-F 2 "TinyTiM_Lib:c_0805" H 10200 2700 50  0001 C CNN
+F 2 "C4_Pretty:c_0805" H 10200 2700 50  0001 C CNN
 F 3 "" H 10200 2700 60  0001 C CNN
 F 4 "CAP CER 0.1UF 25V 10% X7R 0805" H 10200 2900 60  0001 L CNN "Field4"
@@
 F 0 "C131" H 1825 5150 50  0000 L CNN
 F 1 "100n" H 1825 4950 50  0000 L CNN
-F 2 "TinyTiM_Lib:c_0805" H 1800 5050 50  0001 C CNN
+F 2 "C4_Pretty:c_0805" H 1800 5050 50  0001 C CNN
 F 3 "" H 1800 5050 60  0001 C CNN
 F 4 "CAP CER 0.1UF 25V 10% X7R 0805" H 1800 5250 60  0001 L CNN "Field4"
@@
 F 0 "C132" H 3225 5150 50  0000 L CNN
 F 1 "100n" H 3225 4950 50  0000 L CNN
-F 2 "TinyTiM_Lib:c_0805" H 3200 5050 50  0001 C CNN
+F 2 "C4_Pretty:c_0805" H 3200 5050 50  0001 C CNN
 F 3 "" H 3200 5050 60  0001 C CNN
 F 4 "CAP CER 0.1UF 25V 10% X7R 0805" H 3200 5250 60  0001 L CNN "Field4"
@@
 F 0 "C133" H 4625 5150 50  0000 L CNN
 F 1 "100n" H 4625 4950 50  0000 L CNN
-F 2 "TinyTiM_Lib:c_0805" H 4600 5050 50  0001 C CNN
+F 2 "C4_Pretty:c_0805" H 4600 5050 50  0001 C CNN
 F 3 "" H 4600 5050 60  0001 C CNN
 F 4 "CAP CER 0.1UF 25V 10% X7R 0805" H 4600 5250 60  0001 L CNN "Field4"
@@
 F 0 "C134" H 6025 5150 50  0000 L CNN
 F 1 "100n" H 6025 4950 50  0000 L CNN
-F 2 "TinyTiM_Lib:c_0805" H 6000 5050 50  0001 C CNN
+F 2 "C4_Pretty:c_0805" H 6000 5050 50  0001 C CNN
 F 3 "" H 6000 5050 60  0001 C CNN
 F 4 "CAP CER 0.1UF 25V 10% X7R 0805" H 6000 5250 60  0001 L CNN "Field4"
@@
 F 0 "C135" H 7425 5150 50  0000 L CNN
 F 1 "100n" H 7425 4950 50  0000 L CNN
-F 2 "TinyTiM_Lib:c_0805" H 7400 5050 50  0001 C CNN
+F 2 "C4_Pretty:c_0805" H 7400 5050 50  0001 C CNN
 F 3 "" H 7400 5050 60  0001 C CNN
 F 4 "CAP CER 0.1UF 25V 10% X7R 0805" H 7400 5250 60  0001 L CNN "Field4"
@@
 F 0 "C136" H 8825 5150 50  0000 L CNN
 F 1 "100n" H 8825 4950 50  0000 L CNN
-F 2 "TinyTiM_Lib:c_0805" H 8800 5050 50  0001 C CNN
+F 2 "C4_Pretty:c_0805" H 8800 5050 50  0001 C CNN
 F 3 "" H 8800 5050 60  0001 C CNN
 F 4 "CAP CER 0.1UF 25V 10% X7R 0805" H 8800 5250 60  0001 L CNN "Field4"
@@
 F 0 "C137" H 10225 5150 50  0000 L CNN
 F 1 "100n" H 10225 4950 50  0000 L CNN
-F 2 "TinyTiM_Lib:c_0805" H 10200 5050 50  0001 C CNN
+F 2 "C4_Pretty:c_0805" H 10200 5050 50  0001 C CNN
 F 3 "" H 10200 5050 60  0001 C CNN
 F 4 "CAP CER 0.1UF 25V 10% X7R 0805" H 10200 5250 60  0001 L CNN "Field4"
@@
 F 0 "LED113" V 1375 1725 60  0000 C CNN
 F 1 "WS2812B" V 2025 1725 60  0001 C CNN
-F 2 "~" H 1625 1725 60  0000 C CNN
+F 2 "C4_Pretty:RGB_WS2811B" H 1625 1725 60  0001 C CNN
 F 3 "~" H 1625 1725 60  0000 C CNN
 	1    1625 1725
@@
 F 0 "LED114" V 2775 1725 60  0000 C CNN
 F 1 "WS2812B" V 3425 1725 60  0001 C CNN
-F 2 "~" H 3025 1725 60  0000 C CNN
+F 2 "C4_Pretty:RGB_WS2811B" H 3025 1725 60  0001 C CNN
 F 3 "~" H 3025 1725 60  0000 C CNN
 	1    3025 1725
@@
 F 0 "LED115" V 4175 1725 60  0000 C CNN
 F 1 "WS2812B" V 4825 1725 60  0001 C CNN
-F 2 "~" H 4425 1725 60  0000 C CNN
+F 2 "C4_Pretty:RGB_WS2811B" H 4425 1725 60  0001 C CNN
 F 3 "~" H 4425 1725 60  0000 C CNN
 	1    4425 1725
@@
 F 0 "LED116" V 5575 1725 60  0000 C CNN
 F 1 "WS2812B" V 6225 1725 60  0001 C CNN
-F 2 "~" H 5825 1725 60  0000 C CNN
+F 2 "C4_Pretty:RGB_WS2811B" H 5825 1725 60  0001 C CNN
 F 3 "~" H 5825 1725 60  0000 C CNN
 	1    5825 1725
@@
 F 0 "LED117" V 6975 1725 60  0000 C CNN
 F 1 "WS2812B" V 7625 1725 60  0001 C CNN
-F 2 "~" H 7225 1725 60  0000 C CNN
+F 2 "C4_Pretty:RGB_WS2811B" H 7225 1725 60  0001 C CNN
 F 3 "~" H 7225 1725 60  0000 C CNN
 	1    7225 1725
@@
 F 0 "LED118" V 8375 1725 60  0000 C CNN
 F 1 "WS2812B" V 9025 1725 60  0001 C CNN
-F 2 "~" H 8625 1725 60  0000 C CNN
+F 2 "C4_Pretty:RGB_WS2811B" H 8625 1725 60  0001 C CNN
 F 3 "~" H 8625 1725 60  0000 C CNN
 	1    8625 1725
@@
 F 0 "LED119" V 9775 1725 60  0000 C CNN
 F 1 "WS2812B" V 10425 1725 60  0001 C CNN
-F 2 "~" H 10025 1725 60  0000 C CNN
+F 2 "C4_Pretty:RGB_WS2811B" H 10025 1725 60  0001 C CNN
 F 3 "~" H 10025 1725 60  0000 C CNN
 	1    10025 1725
@@
 F 0 "LED120" V 1375 4125 60  0000 C CNN
 F 1 "WS2812B" V 2025 4125 60  0001 C CNN
-F 2 "~" H 1625 4125 60  0000 C CNN
+F 2 "C4_Pretty:RGB_WS2811B" H 1625 4125 60  0001 C CNN
 F 3 "~" H 1625 4125 60  0000 C CNN
 	1    1625 4125
@@
 F 0 "LED121" V 2775 4125 60  0000 C CNN
 F 1 "WS2812B" V 3425 4125 60  0001 C CNN
-F 2 "~" H 3025 4125 60  0000 C CNN
+F 2 "C4_Pretty:RGB_WS2811B" H 3025 4125 60  0001 C CNN
 F 3 "~" H 3025 4125 60  0000 C CNN
 	1    3025 4125
@@
 F 0 "LED122" V 4175 4125 60  0000 C CNN
 F 1 "WS2812B" V 4825 4125 60  0001 C CNN
-F 2 "~" H 4425 4125 60  0000 C CNN
+F 2 "C4_Pretty:RGB_WS2811B" H 4425 4125 60  0001 C CNN
 F 3 "~" H 4425 4125 60  0000 C CNN
 	1    4425 4125
@@
 F 0 "LED123" V 5575 4125 60  0000 C CNN
 F 1 "WS2812B" V 6225 4125 60  0001 C CNN
-F 2 "~" H 5825 4125 60  0000 C CNN
+F 2 "C4_Pretty:RGB_WS2811B" H 5825 4125 60  0001 C CNN
 F 3 "~" H 5825 4125 60  0000 C CNN
 	1    5825 4125
@@
 F 0 "LED124" V 6975 4125 60  0000 C CNN
 F 1 "WS2812B" V 7625 4125 60  0001 C CNN
-F 2 "~" H 7225 4125 60  0000 C CNN
+F 2 "C4_Pretty:RGB_WS2811B" H 7225 4125 60  0001 C CNN
 F 3 "~" H 7225 4125 60  0000 C CNN
 	1    7225 4125
@@
 F 0 "LED125" V 8375 4125 60  0000 C CNN
 F 1 "WS2812B" V 9025 4125 60  0001 C CNN
-F 2 "~" H 8625 4125 60  0000 C CNN
+F 2 "C4_Pretty:RGB_WS2811B" H 8625 4125 60  0001 C CNN
 F 3 "~" H 8625 4125 60  0000 C CNN
 	1    8625 4125
@@
 F 0 "LED126" V 9775 4125 60  0000 C CNN
 F 1 "WS2812B" V 10425 4125 60  0001 C CNN
-F 2 "~" H 10025 4125 60  0000 C CNN
+F 2 "C4_Pretty:RGB_WS2811B" H 10025 4125 60  0001 C CNN
 F 3 "~" H 10025 4125 60  0000 C CNN
 	1    10025 4125

Commit message: C4 PCB layout complete. Added Gerbers
Parts:
- C124, C125, C126, C127, C128, C129, C130, C131, C132, C133, C134, C135, C136, C137: footprint C4_Pretty:c_0805 -> C4_Pretty:c_0805_led
Changed lines of the file:
@@
 EESchema Schematic File Version 2
 LIBS:ClockFOUR
+LIBS:RowGB_sym
 LIBS:ClockFOUR-cache
 EELAYER 24 0
@@
 F 0 "C124" H 1825 2800 50  0000 L CNN
 F 1 "100n" H 1825 2600 50  0000 L CNN
-F 2 "C4_Pretty:c_0805" H 1800 2700 50  0001 C CNN
+F 2 "C4_Pretty:c_0805_led" H 1800 2700 50  0001 C CNN
 F 3 "" H 1800 2700 60  0001 C CNN
 F 4 "CAP CER 0.1UF 25V 10% X7R 0805" H 1800 2900 60  0001 L CNN "Field4"
@@
 F 0 "C125" H 3225 2800 50  0000 L CNN
 F 1 "100n" H 3225 2600 50  0000 L CNN
-F 2 "C4_Pretty:c_0805" H 3200 2700 50  0001 C CNN
+F 2 "C4_Pretty:c_0805_led" H 3200 2700 50  0001 C CNN
 F 3 "" H 3200 2700 60  0001 C CNN
 F 4 "CAP CER 0.1UF 25V 10% X7R 0805" H 3200 2900 60  0001 L CNN "Field4"
@@
 F 0 "C126" H 4625 2800 50  0000 L CNN
 F 1 "100n" H 4625 2600 50  0000 L CNN
-F 2 "C4_Pretty:c_0805" H 4600 2700 50  0001 C CNN
+F 2 "C4_Pretty:c_0805_led" H 4600 2700 50  0001 C CNN
 F 3 "" H 4600 2700 60  0001 C CNN
 F 4 "CAP CER 0.1UF 25V 10% X7R 0805" H 4600 2900 60  0001 L CNN "Field4"
@@
 F 0 "C127" H 6025 2800 50  0000 L CNN
 F 1 "100n" H 6025 2600 50  0000 L CNN
-F 2 "C4_Pretty:c_0805" H 6000 2700 50  0001 C CNN
+F 2 "C4_Pretty:c_0805_led" H 6000 2700 50  0001 C CNN
 F 3 "" H 6000 2700 60  0001 C CNN
 F 4 "CAP CER 0.1UF 25V 10% X7R 0805" H 6000 2900 60  0001 L CNN "Field4"
@@
 F 0 "C128" H 7425 2800 50  0000 L CNN
 F 1 "100n" H 7425 2600 50  0000 L CNN
-F 2 "C4_Pretty:c_0805" H 7400 2700 50  0001 C CNN
+F 2 "C4_Pretty:c_0805_led" H 7400 2700 50  0001 C CNN
 F 3 "" H 7400 2700 60  0001 C CNN
 F 4 "CAP CER 0.1UF 25V 10% X7R 0805" H 7400 2900 60  0001 L CNN "Field4"
@@
 F 0 "C129" H 8825 2800 50  0000 L CNN
 F 1 "100n" H 8825 2600 50  0000 L CNN
-F 2 "C4_Pretty:c_0805" H 8800 2700 50  0001 C CNN
+F 2 "C4_Pretty:c_0805_led" H 8800 2700 50  0001 C CNN
 F 3 "" H 8800 2700 60  0001 C CNN
 F 4 "CAP CER 0.1UF 25V 10% X7R 0805" H 8800 2900 60  0001 L CNN "Field4"
@@
 F 0 "C130" H 10225 2800 50  0000 L CNN
 F 1 "100n" H 10225 2600 50  0000 L CNN
-F 2 "C4_Pretty:c_0805" H 10200 2700 50  0001 C CNN
+F 2 "C4_Pretty:c_0805_led" H 10200 2700 50  0001 C CNN
 F 3 "" H 10200 2700 60  0001 C CNN
 F 4 "CAP CER 0.1UF 25V 10% X7R 0805" H 10200 2900 60  0001 L CNN "Field4"
@@
 F 0 "C131" H 1825 5150 50  0000 L CNN
 F 1 "100n" H 1825 4950 50  0000 L CNN
-F 2 "C4_Pretty:c_0805" H 1800 5050 50  0001 C CNN
+F 2 "C4_Pretty:c_0805_led" H 1800 5050 50  0001 C CNN
 F 3 "" H 1800 5050 60  0001 C CNN
 F 4 "CAP CER 0.1UF 25V 10% X7R 0805" H 1800 5250 60  0001 L CNN "Field4"
@@
 F 0 "C132" H 3225 5150 50  0000 L CNN
 F 1 "100n" H 3225 4950 50  0000 L CNN
-F 2 "C4_Pretty:c_0805" H 3200 5050 50  0001 C CNN
+F 2 "C4_Pretty:c_0805_led" H 3200 5050 50  0001 C CNN
 F 3 "" H 3200 5050 60  0001 C CNN
 F 4 "CAP CER 0.1UF 25V 10% X7R 0805" H 3200 5250 60  0001 L CNN "Field4"
@@
 F 0 "C133" H 4625 5150 50  0000 L CNN
 F 1 "100n" H 4625 4950 50  0000 L CNN
-F 2 "C4_Pretty:c_0805" H 4600 5050 50  0001 C CNN
+F 2 "C4_Pretty:c_0805_led" H 4600 5050 50  0001 C CNN
 F 3 "" H 4600 5050 60  0001 C CNN
 F 4 "CAP CER 0.1UF 25V 10% X7R 0805" H 4600 5250 60  0001 L CNN "Field4"
@@
 F 0 "C134" H 6025 5150 50  0000 L CNN
 F 1 "100n" H 6025 4950 50  0000 L CNN
-F 2 "C4_Pretty:c_0805" H 6000 5050 50  0001 C CNN
+F 2 "C4_Pretty:c_0805_led" H 6000 5050 50  0001 C CNN
 F 3 "" H 6000 5050 60  0001 C CNN
 F 4 "CAP CER 0.1UF 25V 10% X7R 0805" H 6000 5250 60  0001 L CNN "Field4"
@@
 F 0 "C135" H 7425 5150 50  0000 L CNN
 F 1 "100n" H 7425 4950 50  0000 L CNN
-F 2 "C4_Pretty:c_0805" H 7400 5050 50  0001 C CNN
+F 2 "C4_Pretty:c_0805_led" H 7400 5050 50  0001 C CNN
 F 3 "" H 7400 5050 60  0001 C CNN
 F 4 "CAP CER 0.1UF 25V 10% X7R 0805" H 7400 5250 60  0001 L CNN "Field4"
@@
 F 0 "C136" H 8825 5150 50  0000 L CNN
 F 1 "100n" H 8825 4950 50  0000 L CNN
-F 2 "C4_Pretty:c_0805" H 8800 5050 50  0001 C CNN
+F 2 "C4_Pretty:c_0805_led" H 8800 5050 50  0001 C CNN
 F 3 "" H 8800 5050 60  0001 C CNN
 F 4 "CAP CER 0.1UF 25V 10% X7R 0805" H 8800 5250 60  0001 L CNN "Field4"
@@
 F 0 "C137" H 10225 5150 50  0000 L CNN
 F 1 "100n" H 10225 4950 50  0000 L CNN
-F 2 "C4_Pretty:c_0805" H 10200 5050 50  0001 C CNN
+F 2 "C4_Pretty:c_0805_led" H 10200 5050 50  0001 C CNN
 F 3 "" H 10200 5050 60  0001 C CNN
 F 4 "CAP CER 0.1UF 25V 10% X7R 0805" H 10200 5250 60  0001 L CNN "Field4"
