File: KiCad/Row_J.sch (KiCad schematic (older format))
At the start: 14 parts, among them U101 RGB_WS2811B, U102 RGB_WS2811B, U103 RGB_WS2811B, U104 RGB_WS2811B, U105 RGB_WS2811B, U106 RGB_WS2811B, U107 RGB_WS2811B, U108 RGB_WS2811B

Commit message: Schematic updated
Parts:
- removed C101: 100n, TinyTiM_Lib:c_0805, symbol C2
- removed C117: 47u,8V, TinyTiM_Lib:c_2917, symbol C_POL_1
- removed S101, S102, S103, S104: CONN_1, TinyTiM_Lib:Screw, symbol CONN_1
- removed U101, U102, U103, U104, U105, U106, U107, U108: RGB_WS2811B, TinyTiM_Lib:RGB_WS2811B, symbol RGB_WS2811B
Connections:
- net labels removed: 5V, A_02, A_03, A_04, A_05, A_06, A_07, A_08, A_09, DI_A, DO_A, GND
- wire segments 49 -> 0
- no-connect marks 4 -> 0
Other:
- note removed: "Mounting Screws"

Commit message: Schematic updated
Parts:
- added C136, C137, C138, C139, C140, C141, C142, C143, C144, C145, C146, C147, C148, C149: 100n, TinyTiM_Lib:c_0805, symbol C2
- added U130, U131, U132, U133, U134, U135, U136, U137, U138, U139, U140, U141, U142, U143: RGB_WS2812B, symbol RGB_WS2812B
Connections:
- net labels added: 5V, DI_J, DO_J, GND
- wire segments 0 -> 82

Commit message: Schematic updated, board started
Parts:
- C137: renamed from C136; Field5 100nF, 25V -> 100n, 25V
- C139: renamed from C140; Field5 100nF, 25V -> 100n, 25V
- C141: renamed from C144; Field5 100nF, 25V -> 100n, 25V
- C143: renamed from C148; Field5 100nF, 25V -> 100n, 25V
- C145: renamed from C139; Field5 100nF, 25V -> 100n, 25V
- C147: renamed from C143; Field5 100nF, 25V -> 100n, 25V
- C149: renamed from C147; Field5 100nF, 25V -> 100n, 25V
- renumbered C142 to C140, C146 to C142, C137 to C144, C141 to C146, C145 to C148, C149 to C150, U130 to U128, U132 to U129, U134 to U130, U136 to U131, U138 to U132, U140 to U133, U142 to U134, U131 to U135, U133 to U136, U135 to U137, U137 to U138, U141 to U140, U143 to U141
Changed lines of the file:
@@
 LIBS:contrib
 LIBS:valves
-LIBS:TinyTiM-cache
-LIBS:TiNA_sym
+LIBS:ClockFOUR
 LIBS:ClockFOUR-cache
 EELAYER 27 0
@@
 Sheet 11 14
 Title "ClockFOUR"
-Date "30 sep 2014"
+Date "1 oct 2014"
 Rev ""
 Comp "WyoLum"
@@
 5V
 $Comp
-L GND #PWR021
+L GND #PWR023
 U 1 1 542C15F9
 P 1350 2700
-F 0 "#PWR021" H 1350 2700 30  0001 C CNN
+F 0 "#PWR023" H 1350 2700 30  0001 C CNN
 F 1 "GND" H 1350 2630 30  0001 C CNN
 F 2 "" H 1350 2700 60  0001 C CNN
@@
 $EndComp
 $Comp
-L C2 C136
+L C2 C137
 U 1 1 542C1607
 P 1900 2850
-F 0 "C136" H 1925 2950 50  0000 L CNN
+F 0 "C137" H 1925 2950 50  0000 L CNN
 F 1 "100n" H 1925 2750 50  0000 L CNN
 F 2 "TinyTiM_Lib:c_0805" H 1900 2850 50  0001 C CNN
 F 3 "" H 1900 2850 60  0001 C CNN
 F 4 "CAP CER 0.1UF 25V 10% X7R 0805" H 1900 3050 60  0001 L CNN "Field4"
-F 5 "100nF, 25V" H 1900 3150 60  0001 L CNN "Field5"
+F 5 "100n, 25V" H 1900 3150 60  0001 L CNN "Field5"
 F 6 "Surface Mount, MLCC" H 1900 3250 60  0001 L CNN "Field6"
 F 7 "Kemet" H 1900 3350 60  0001 L CNN "Field7"
@@
 $EndComp
 $Comp
-L RGB_WS2812B U130
+L RGB_WS2812B U128
 U 1 1 542C160D
 P 1725 1875
-F 0 "U130" V 1475 1875 60  0000 C CNN
+F 0 "U128" V 1475 1875 60  0000 C CNN
 F 1 "RGB_WS2812B" V 2125 1875 60  0000 C CNN
 F 2 "" H 1725 1875 60  0000 C CNN
@@
 $EndComp
 $Comp
-L RGB_WS2812B U132
+L RGB_WS2812B U129
 U 1 1 542C1613
 P 3125 1875
-F 0 "U132" V 2875 1875 60  0000 C CNN
+F 0 "U129" V 2875 1875 60  0000 C CNN
 F 1 "RGB_WS2812B" V 3525 1875 60  0000 C CNN
 F 2 "" H 3125 1875 60  0000 C CNN
@@
 $EndComp
 $Comp
-L RGB_WS2812B U134
+L RGB_WS2812B U130
 U 1 1 542C1619
 P 4525 1875
-F 0 "U134" V 4275 1875 60  0000 C CNN
+F 0 "U130" V 4275 1875 60  0000 C CNN
 F 1 "RGB_WS2812B" V 4925 1875 60  0000 C CNN
 F 2 "" H 4525 1875 60  0000 C CNN
@@
 $EndComp
 $Comp
-L RGB_WS2812B U136
+L RGB_WS2812B U131
 U 1 1 542C161F
 P 5925 1875
-F 0 "U136" V 5675 1875 60  0000 C CNN
+F 0 "U131" V 5675 1875 60  0000 C CNN
 F 1 "RGB_WS2812B" V 6325 1875 60  0000 C CNN
 F 2 "" H 5925 1875 60  0000 C CNN
@@
 $EndComp
 $Comp
-L RGB_WS2812B U138
+L RGB_WS2812B U132
 U 1 1 542C1625
 P 7325 1875
-F 0 "U138" V 7075 1875 60  0000 C CNN
+F 0 "U132" V 7075 1875 60  0000 C CNN
 F 1 "RGB_WS2812B" V 7725 1875 60  0000 C CNN
 F 2 "" H 7325 1875 60  0000 C CNN
@@
 $EndComp
 $Comp
-L RGB_WS2812B U140
+L RGB_WS2812B U133
 U 1 1 542C162B
 P 8725 1875
-F 0 "U140" V 8475 1875 60  0000 C CNN
+F 0 "U133" V 8475 1875 60  0000 C CNN
 F 1 "RGB_WS2812B" V 9125 1875 60  0000 C CNN
 F 2 "" H 8725 1875 60  0000 C CNN
@@
 $EndComp
 $Comp
-L RGB_WS2812B U142
+L RGB_WS2812B U134
 U 1 1 542C1631
 P 10125 1875
-F 0 "U142" V 9875 1875 60  0000 C CNN
+F 0 "U134" V 9875 1875 60  0000 C CNN
 F 1 "RGB_WS2812B" V 10525 1875 60  0000 C CNN
 F 2 "" H 10125 1875 60  0000 C CNN
@@
 $EndComp
 $Comp
-L RGB_WS2812B U131
+L RGB_WS2812B U135
 U 1 1 542C1637
 P 1725 4275
-F 0 "U131" V 1475 4275 60  0000 C CNN
+F 0 "U135" V 1475 4275 60  0000 C CNN
 F 1 "RGB_WS2812B" V 2125 4275 60  0000 C CNN
 F 2 "" H 1725 4275 60  0000 C CNN
@@
 $EndComp
 $Comp
-L RGB_WS2812B U133
+L RGB_WS2812B U136
 U 1 1 542C163D
 P 3125 4275
-F 0 "U133" V 2875 4275 60  0000 C CNN
+F 0 "U136" V 2875 4275 60  0000 C CNN
 F 1 "RGB_WS2812B" V 3525 4275 60  0000 C CNN
 F 2 "" H 3125 4275 60  0000 C CNN
@@
 $EndComp
 $Comp
-L RGB_WS2812B U135
+L RGB_WS2812B U137
 U 1 1 542C1643
 P 4525 4275
-F 0 "U135" V 4275 4275 60  0000 C CNN
+F 0 "U137" V 4275 4275 60  0000 C CNN
 F 1 "RGB_WS2812B" V 4925 4275 60  0000 C CNN
 F 2 "" H 4525 4275 60  0000 C CNN
@@
 $EndComp
 $Comp
-L RGB_WS2812B U137
+L RGB_WS2812B U138
 U 1 1 542C1649
 P 5925 4275
-F 0 "U137" V 5675 4275 60  0000 C CNN
+F 0 "U138" V 5675 4275 60  0000 C CNN
 F 1 "RGB_WS2812B" V 6325 4275 60  0000 C CNN
 F 2 "" H 5925 4275 60  0000 C CNN
@@
 $EndComp
 $Comp
-L RGB_WS2812B U141
+L RGB_WS2812B U140
 U 1 1 542C1655
 P 8725 4275
-F 0 "U141" V 8475 4275 60  0000 C CNN
+F 0 "U140" V 8475 4275 60  0000 C CNN
 F 1 "RGB_WS2812B" V 9125 4275 60  0000 C CNN
 F 2 "" H 8725 4275 60  0000 C CNN
@@
 $EndComp
 $Comp
-L RGB_WS2812B U143
+L RGB_WS2812B U141
 U 1 1 542C165B
 P 10125 4275
-F 0 "U143" V 9875 4275 60  0000 C CNN
+F 0 "U141" V 9875 4275 60  0000 C CNN
 F 1 "RGB_WS2812B" V 10525 4275 60  0000 C CNN
 F 2 "" H 10125 4275 60  0000 C CNN
@@
 $EndComp
 $Comp
-L C2 C140
+L C2 C139
 U 1 1 542C16C4
 P 4700 2850
-F 0 "C140" H 4725 2950 50  0000 L CNN
+F 0 "C139" H 4725 2950 50  0000 L CNN
 F 1 "100n" H 4725 2750 50  0000 L CNN
 F 2 "TinyTiM_Lib:c_0805" H 4700 2850 50  0001 C CNN
 F 3 "" H 4700 2850 60  0001 C CNN
 F 4 "CAP CER 0.1UF 25V 10% X7R 0805" H 4700 3050 60  0001 L CNN "Field4"
-F 5 "100nF, 25V" H 4700 3150 60  0001 L CNN "Field5"
+F 5 "100n, 25V" H 4700 3150 60  0001 L CNN "Field5"
 F 6 "Surface Mount, MLCC" H 4700 3250 60  0001 L CNN "Field6"
 F 7 "Kemet" H 4700 3350 60  0001 L CNN "Field7"
@@
 $EndComp
 $Comp
-L C2 C142
+L C2 C140
 U 1 1 542C16D2
 P 6100 2850
-F 0 "C142" H 6125 2950 50  0000 L CNN
+F 0 "C140" H 6125 2950 50  0000 L CNN
 F 1 "100n" H 6125 2750 50  0000 L CNN
 F 2 "TinyTiM_Lib:c_0805" H 6100 2850 50  0001 C CNN
@@
 $EndComp
 $Comp
-L C2 C144
+L C2 C141
 U 1 1 542C16E0
 P 7500 2850
-F 0 "C144" H 7525 2950 50  0000 L CNN
+F 0 "C141" H 7525 2950 50  0000 L CNN
 F 1 "100n" H 7525 2750 50  0000 L CNN
 F 2 "TinyTiM_Lib:c_0805" H 7500 2850 50  0001 C CNN
 F 3 "" H 7500 2850 60  0001 C CNN
 F 4 "CAP CER 0.1UF 25V 10% X7R 0805" H 7500 3050 60  0001 L CNN "Field4"
-F 5 "100nF, 25V" H 7500 3150 60  0001 L CNN "Field5"
+F 5 "100n, 25V" H 7500 3150 60  0001 L CNN "Field5"
 F 6 "Surface Mount, MLCC" H 7500 3250 60  0001 L CNN "Field6"
 F 7 "Kemet" H 7500 3350 60  0001 L CNN "Field7"
@@
 $EndComp
 $Comp
-L C2 C146
+L C2 C142
 U 1 1 542C16EE
 P 8900 2850
-F 0 "C146" H 8925 2950 50  0000 L CNN
+F 0 "C142" H 8925 2950 50  0000 L CNN
 F 1 "100n" H 8925 2750 50  0000 L CNN
 F 2 "TinyTiM_Lib:c_0805" H 8900 2850 50  0001 C CNN
@@
 $EndComp
 $Comp
-L C2 C148
+L C2 C143
 U 1 1 542C16FC
 P 10300 2850
-F 0 "C148" H 10325 2950 50  0000 L CNN
+F 0 "C143" H 10325 2950 50  0000 L CNN
 F 1 "100n" H 10325 2750 50  0000 L CNN
 F 2 "TinyTiM_Lib:c_0805" H 10300 2850 50  0001 C CNN
 F 3 "" H 10300 2850 60  0001 C CNN
 F 4 "CAP CER 0.1UF 25V 10% X7R 0805" H 10300 3050 60  0001 L CNN "Field4"
-F 5 "100nF, 25V" H 10300 3150 60  0001 L CNN "Field5"
+F 5 "100n, 25V" H 10300 3150 60  0001 L CNN "Field5"
 F 6 "Surface Mount, MLCC" H 10300 3250 60  0001 L CNN "Field6"
 F 7 "Kemet" H 10300 3350 60  0001 L CNN "Field7"
@@
 Connection ~ 10200 3050
 $Comp
-L C2 C137
+L C2 C144
 U 1 1 542C170B
 P 1900 5200
-F 0 "C137" H 1925 5300 50  0000 L CNN
+F 0 "C144" H 1925 5300 50  0000 L CNN
 F 1 "100n" H 1925 5100 50  0000 L CNN
 F 2 "TinyTiM_Lib:c_0805" H 1900 5200 50  0001 C CNN
@@
 Connection ~ 1800 5400
 $Comp
-L C2 C139
+L C2 C145
 U 1 1 542C1748
 P 3300 5200
-F 0 "C139" H 3325 5300 50  0000 L CNN
+F 0 "C145" H 3325 5300 50  0000 L CNN
 F 1 "100n" H 3325 5100 50  0000 L CNN
 F 2 "TinyTiM_Lib:c_0805" H 3300 5200 50  0001 C CNN
 F 3 "" H 3300 5200 60  0001 C CNN
 F 4 "CAP CER 0.1UF 25V 10% X7R 0805" H 3300 5400 60  0001 L CNN "Field4"
-F 5 "100nF, 25V" H 3300 5500 60  0001 L CNN "Field5"
+F 5 "100n, 25V" H 3300 5500 60  0001 L CNN "Field5"
 F 6 "Surface Mount, MLCC" H 3300 5600 60  0001 L CNN "Field6"
 F 7 "Kemet" H 3300 5700 60  0001 L CNN "Field7"
@@
 $EndComp
 $Comp
-L C2 C141
+L C2 C146
 U 1 1 542C1756
 P 4700 5200
-F 0 "C141" H 4725 5300 50  0000 L CNN
+F 0 "C146" H 4725 5300 50  0000 L CNN
 F 1 "100n" H 4725 5100 50  0000 L CNN
 F 2 "TinyTiM_Lib:c_0805" H 4700 5200 50  0001 C CNN
@@
 $EndComp
 $Comp
-L C2 C143
+L C2 C147
 U 1 1 542C1764
 P 6100 5200
-F 0 "C143" H 6125 5300 50  0000 L CNN
+F 0 "C147" H 6125 5300 50  0000 L CNN
 F 1 "100n" H 6125 5100 50  0000 L CNN
 F 2 "TinyTiM_Lib:c_0805" H 6100 5200 50  0001 C CNN
 F 3 "" H 6100 5200 60  0001 C CNN
 F 4 "CAP CER 0.1UF 25V 10% X7R 0805" H 6100 5400 60  0001 L CNN "Field4"
-F 5 "100nF, 25V" H 6100 5500 60  0001 L CNN "Field5"
+F 5 "100n, 25V" H 6100 5500 60  0001 L CNN "Field5"
 F 6 "Surface Mount, MLCC" H 6100 5600 60  0001 L CNN "Field6"
 F 7 "Kemet" H 6100 5700 60  0001 L CNN "Field7"
@@
 $EndComp
 $Comp
-L C2 C145
+L C2 C148
 U 1 1 542C1772
 P 7500 5200
-F 0 "C145" H 7525 5300 50  0000 L CNN
+F 0 "C148" H 7525 5300 50  0000 L CNN
 F 1 "100n" H 7525 5100 50  0000 L CNN
 F 2 "TinyTiM_Lib:c_0805" H 7500 5200 50  0001 C CNN
@@
 $EndComp
 $Comp
-L C2 C147
+L C2 C149
 U 1 1 542C1780
 P 8900 5200
-F 0 "C147" H 8925 5300 50  0000 L CNN
+F 0 "C149" H 8925 5300 50  0000 L CNN
 F 1 "100n" H 8925 5100 50  0000 L CNN
 F 2 "TinyTiM_Lib:c_0805" H 8900 5200 50  0001 C CNN
 F 3 "" H 8900 5200 60  0001 C CNN
 F 4 "CAP CER 0.1UF 25V 10% X7R 0805" H 8900 5400 60  0001 L CNN "Field4"
-F 5 "100nF, 25V" H 8900 5500 60  0001 L CNN "Field5"
+F 5 "100n, 25V" H 8900 5500 60  0001 L CNN "Field5"
 F 6 "Surface Mount, MLCC" H 8900 5600 60  0001 L CNN "Field6"
 F 7 "Kemet" H 8900 5700 60  0001 L CNN "Field7"
@@
 $EndComp
 $Comp
-L C2 C149
+L C2 C150
 U 1 1 542C178E
 P 10300 5200
-F 0 "C149" H 10325 5300 50  0000 L CNN
+F 0 "C150" H 10325 5300 50  0000 L CNN
 F 1 "100n" H 10325 5100 50  0000 L CNN
 F 2 "TinyTiM_Lib:c_0805" H 10300 5200 50  0001 C CNN

Commit message: Board layout updated
Parts:
- removed U128, U129, U130, U131, U132, U133, U134, U135, U136, U137, U138, U139, U140, U141: RGB_WS2812B, symbol RGB_WS2812B
- added LED127, LED128, LED129, LED130, LED131, LED132, LED133, LED134, LED135, LED136, LED137, LED138, LED139, LED140: RGB_WS2812B, ~, symbol RGB_WS2812B

Commit message: Board layout updated
Matrix placed and wired. Added RTC.
Parts:
- removed C137: 100n, TinyTiM_Lib:c_0805, symbol C2
- removed LED127, LED128, LED129, LED130, LED131, LED132, LED133, LED134, LED135, LED136, LED137, LED138, LED139, LED140: RGB_WS2812B, ~, symbol RGB_WS2812B
- added C151: 100n, TinyTiM_Lib:c_0805, symbol C2
- added LED127, LED128, LED129, LED130, LED131, LED132, LED133, LED134, LED135, LED136, LED137, LED138, LED139, LED140: WS2812B, ~, symbol WS2812B
- C138, C140, C142, C144, C146, C148, C150: Field5 100nF, 25V -> 100n, 25V
- C139, C141, C143, C145, C147, C149: Field5 100n, 25V -> 100nF, 25V
