File: KiCad/Row_J.sch (KiCad schematic (older format))
At the start: 28 parts

Commit message: PCB layout, work in progress
Parts:
- C138, C139, C140, C141, C142, C143, C144, C145, C146, C147, C148, C149, C150, C151: footprint TinyTiM_Lib:c_0805 -> C4_Pretty:c_0805
- LED127, LED128, LED129, LED130, LED131, LED132, LED133, LED134, LED135, LED136, LED137, LED138, LED139, LED140: footprint ~ -> C4_Pretty:RGB_WS2811B
Changed lines of the file:
@@
 F 0 "C138" H 1975 3100 50  0000 L CNN
 F 1 "100n" H 1975 2900 50  0000 L CNN
-F 2 "TinyTiM_Lib:c_0805" H 1950 3000 50  0001 C CNN
+F 2 "C4_Pretty:c_0805" H 1950 3000 50  0001 C CNN
 F 3 "" H 1950 3000 60  0001 C CNN
 F 4 "CAP CER 0.1UF 25V 10% X7R 0805" H 1950 3200 60  0001 L CNN "Field4"
@@
 F 0 "C139" H 3375 3100 50  0000 L CNN
 F 1 "100n" H 3375 2900 50  0000 L CNN
-F 2 "TinyTiM_Lib:c_0805" H 3350 3000 50  0001 C CNN
+F 2 "C4_Pretty:c_0805" H 3350 3000 50  0001 C CNN
 F 3 "" H 3350 3000 60  0001 C CNN
 F 4 "CAP CER 0.1UF 25V 10% X7R 0805" H 3350 3200 60  0001 L CNN "Field4"
@@
 F 0 "C140" H 4775 3100 50  0000 L CNN
 F 1 "100n" H 4775 2900 50  0000 L CNN
-F 2 "TinyTiM_Lib:c_0805" H 4750 3000 50  0001 C CNN
+F 2 "C4_Pretty:c_0805" H 4750 3000 50  0001 C CNN
 F 3 "" H 4750 3000 60  0001 C CNN
 F 4 "CAP CER 0.1UF 25V 10% X7R 0805" H 4750 3200 60  0001 L CNN "Field4"
@@
 F 0 "C141" H 6175 3100 50  0000 L CNN
 F 1 "100n" H 6175 2900 50  0000 L CNN
-F 2 "TinyTiM_Lib:c_0805" H 6150 3000 50  0001 C CNN
+F 2 "C4_Pretty:c_0805" H 6150 3000 50  0001 C CNN
 F 3 "" H 6150 3000 60  0001 C CNN
 F 4 "CAP CER 0.1UF 25V 10% X7R 0805" H 6150 3200 60  0001 L CNN "Field4"
@@
 F 0 "C142" H 7575 3100 50  0000 L CNN
 F 1 "100n" H 7575 2900 50  0000 L CNN
-F 2 "TinyTiM_Lib:c_0805" H 7550 3000 50  0001 C CNN
+F 2 "C4_Pretty:c_0805" H 7550 3000 50  0001 C CNN
 F 3 "" H 7550 3000 60  0001 C CNN
 F 4 "CAP CER 0.1UF 25V 10% X7R 0805" H 7550 3200 60  0001 L CNN "Field4"
@@
 F 0 "C143" H 8975 3100 50  0000 L CNN
 F 1 "100n" H 8975 2900 50  0000 L CNN
-F 2 "TinyTiM_Lib:c_0805" H 8950 3000 50  0001 C CNN
+F 2 "C4_Pretty:c_0805" H 8950 3000 50  0001 C CNN
 F 3 "" H 8950 3000 60  0001 C CNN
 F 4 "CAP CER 0.1UF 25V 10% X7R 0805" H 8950 3200 60  0001 L CNN "Field4"
@@
 F 0 "C144" H 10375 3100 50  0000 L CNN
 F 1 "100n" H 10375 2900 50  0000 L CNN
-F 2 "TinyTiM_Lib:c_0805" H 10350 3000 50  0001 C CNN
+F 2 "C4_Pretty:c_0805" H 10350 3000 50  0001 C CNN
 F 3 "" H 10350 3000 60  0001 C CNN
 F 4 "CAP CER 0.1UF 25V 10% X7R 0805" H 10350 3200 60  0001 L CNN "Field4"
@@
 F 0 "C145" H 1975 5450 50  0000 L CNN
 F 1 "100n" H 1975 5250 50  0000 L CNN
-F 2 "TinyTiM_Lib:c_0805" H 1950 5350 50  0001 C CNN
+F 2 "C4_Pretty:c_0805" H 1950 5350 50  0001 C CNN
 F 3 "" H 1950 5350 60  0001 C CNN
 F 4 "CAP CER 0.1UF 25V 10% X7R 0805" H 1950 5550 60  0001 L CNN "Field4"
@@
 F 0 "C146" H 3375 5450 50  0000 L CNN
 F 1 "100n" H 3375 5250 50  0000 L CNN
-F 2 "TinyTiM_Lib:c_0805" H 3350 5350 50  0001 C CNN
+F 2 "C4_Pretty:c_0805" H 3350 5350 50  0001 C CNN
 F 3 "" H 3350 5350 60  0001 C CNN
 F 4 "CAP CER 0.1UF 25V 10% X7R 0805" H 3350 5550 60  0001 L CNN "Field4"
@@
 F 0 "C147" H 4775 5450 50  0000 L CNN
 F 1 "100n" H 4775 5250 50  0000 L CNN
-F 2 "TinyTiM_Lib:c_0805" H 4750 5350 50  0001 C CNN
+F 2 "C4_Pretty:c_0805" H 4750 5350 50  0001 C CNN
 F 3 "" H 4750 5350 60  0001 C CNN
 F 4 "CAP CER 0.1UF 25V 10% X7R 0805" H 4750 5550 60  0001 L CNN "Field4"
@@
 F 0 "C148" H 6175 5450 50  0000 L CNN
 F 1 "100n" H 6175 5250 50  0000 L CNN
-F 2 "TinyTiM_Lib:c_0805" H 6150 5350 50  0001 C CNN
+F 2 "C4_Pretty:c_0805" H 6150 5350 50  0001 C CNN
 F 3 "" H 6150 5350 60  0001 C CNN
 F 4 "CAP CER 0.1UF 25V 10% X7R 0805" H 6150 5550 60  0001 L CNN "Field4"
@@
 F 0 "C149" H 7575 5450 50  0000 L CNN
 F 1 "100n" H 7575 5250 50  0000 L CNN
-F 2 "TinyTiM_Lib:c_0805" H 7550 5350 50  0001 C CNN
+F 2 "C4_Pretty:c_0805" H 7550 5350 50  0001 C CNN
 F 3 "" H 7550 5350 60  0001 C CNN
 F 4 "CAP CER 0.1UF 25V 10% X7R 0805" H 7550 5550 60  0001 L CNN "Field4"
@@
 F 0 "C150" H 8975 5450 50  0000 L CNN
 F 1 "100n" H 8975 5250 50  0000 L CNN
-F 2 "TinyTiM_Lib:c_0805" H 8950 5350 50  0001 C CNN
+F 2 "C4_Pretty:c_0805" H 8950 5350 50  0001 C CNN
 F 3 "" H 8950 5350 60  0001 C CNN
 F 4 "CAP CER 0.1UF 25V 10% X7R 0805" H 8950 5550 60  0001 L CNN "Field4"
@@
 F 0 "C151" H 10375 5450 50  0000 L CNN
 F 1 "100n" H 10375 5250 50  0000 L CNN
-F 2 "TinyTiM_Lib:c_0805" H 10350 5350 50  0001 C CNN
+F 2 "C4_Pretty:c_0805" H 10350 5350 50  0001 C CNN
 F 3 "" H 10350 5350 60  0001 C CNN
 F 4 "CAP CER 0.1UF 25V 10% X7R 0805" H 10350 5550 60  0001 L CNN "Field4"
@@
 F 0 "LED127" V 1525 2025 60  0000 C CNN
 F 1 "WS2812B" V 2175 2025 60  0001 C CNN
-F 2 "~" H 1775 2025 60  0000 C CNN
+F 2 "C4_Pretty:RGB_WS2811B" H 1775 2025 60  0001 C CNN
 F 3 "~" H 1775 2025 60  0000 C CNN
 	1    1775 2025
@@
 F 0 "LED128" V 2925 2025 60  0000 C CNN
 F 1 "WS2812B" V 3575 2025 60  0001 C CNN
-F 2 "~" H 3175 2025 60  0000 C CNN
+F 2 "C4_Pretty:RGB_WS2811B" H 3175 2025 60  0001 C CNN
 F 3 "~" H 3175 2025 60  0000 C CNN
 	1    3175 2025
@@
 F 0 "LED129" V 4325 2025 60  0000 C CNN
 F 1 "WS2812B" V 4975 2025 60  0001 C CNN
-F 2 "~" H 4575 2025 60  0000 C CNN
+F 2 "C4_Pretty:RGB_WS2811B" H 4575 2025 60  0001 C CNN
 F 3 "~" H 4575 2025 60  0000 C CNN
 	1    4575 2025
@@
 F 0 "LED130" V 5725 2025 60  0000 C CNN
 F 1 "WS2812B" V 6375 2025 60  0001 C CNN
-F 2 "~" H 5975 2025 60  0000 C CNN
+F 2 "C4_Pretty:RGB_WS2811B" H 5975 2025 60  0001 C CNN
 F 3 "~" H 5975 2025 60  0000 C CNN
 	1    5975 2025
@@
 F 0 "LED131" V 7125 2025 60  0000 C CNN
 F 1 "WS2812B" V 7775 2025 60  0001 C CNN
-F 2 "~" H 7375 2025 60  0000 C CNN
+F 2 "C4_Pretty:RGB_WS2811B" H 7375 2025 60  0001 C CNN
 F 3 "~" H 7375 2025 60  0000 C CNN
 	1    7375 2025
@@
 F 0 "LED132" V 8525 2025 60  0000 C CNN
 F 1 "WS2812B" V 9175 2025 60  0001 C CNN
-F 2 "~" H 8775 2025 60  0000 C CNN
+F 2 "C4_Pretty:RGB_WS2811B" H 8775 2025 60  0001 C CNN
 F 3 "~" H 8775 2025 60  0000 C CNN
 	1    8775 2025
@@
 F 0 "LED133" V 9925 2025 60  0000 C CNN
 F 1 "WS2812B" V 10575 2025 60  0001 C CNN
-F 2 "~" H 10175 2025 60  0000 C CNN
+F 2 "C4_Pretty:RGB_WS2811B" H 10175 2025 60  0001 C CNN
 F 3 "~" H 10175 2025 60  0000 C CNN
 	1    10175 2025
@@
 F 0 "LED134" V 1525 4425 60  0000 C CNN
 F 1 "WS2812B" V 2175 4425 60  0001 C CNN
-F 2 "~" H 1775 4425 60  0000 C CNN
+F 2 "C4_Pretty:RGB_WS2811B" H 1775 4425 60  0001 C CNN
 F 3 "~" H 1775 4425 60  0000 C CNN
 	1    1775 4425
@@
 F 0 "LED135" V 2925 4425 60  0000 C CNN
 F 1 "WS2812B" V 3575 4425 60  0001 C CNN
-F 2 "~" H 3175 4425 60  0000 C CNN
+F 2 "C4_Pretty:RGB_WS2811B" H 3175 4425 60  0001 C CNN
 F 3 "~" H 3175 4425 60  0000 C CNN
 	1    3175 4425
@@
 F 0 "LED136" V 4325 4425 60  0000 C CNN
 F 1 "WS2812B" V 4975 4425 60  0001 C CNN
-F 2 "~" H 4575 4425 60  0000 C CNN
+F 2 "C4_Pretty:RGB_WS2811B" H 4575 4425 60  0001 C CNN
 F 3 "~" H 4575 4425 60  0000 C CNN
 	1    4575 4425
@@
 F 0 "LED137" V 5725 4425 60  0000 C CNN
 F 1 "WS2812B" V 6375 4425 60  0001 C CNN
-F 2 "~" H 5975 4425 60  0000 C CNN
+F 2 "C4_Pretty:RGB_WS2811B" H 5975 4425 60  0001 C CNN
 F 3 "~" H 5975 4425 60  0000 C CNN
 	1    5975 4425
@@
 F 0 "LED138" V 7125 4425 60  0000 C CNN
 F 1 "WS2812B" V 7775 4425 60  0001 C CNN
-F 2 "~" H 7375 4425 60  0000 C CNN
+F 2 "C4_Pretty:RGB_WS2811B" H 7375 4425 60  0001 C CNN
 F 3 "~" H 7375 4425 60  0000 C CNN
 	1    7375 4425
@@
 F 0 "LED139" V 8525 4425 60  0000 C CNN
 F 1 "WS2812B" V 9175 4425 60  0001 C CNN
-F 2 "~" H 8775 4425 60  0000 C CNN
+F 2 "C4_Pretty:RGB_WS2811B" H 8775 4425 60  0001 C CNN
 F 3 "~" H 8775 4425 60  0000 C CNN
 	1    8775 4425
@@
 F 0 "LED140" V 9925 4425 60  0000 C CNN
 F 1 "WS2812B" V 10575 4425 60  0001 C CNN
-F 2 "~" H 10175 4425 60  0000 C CNN
+F 2 "C4_Pretty:RGB_WS2811B" H 10175 4425 60  0001 C CNN
 F 3 "~" H 10175 4425 60  0000 C CNN
 	1    10175 4425

Commit message: C4 PCB layout complete. Added Gerbers
Parts:
- C138, C139, C140, C141, C142, C143, C144, C145, C146, C147, C148, C149, C150, C151: footprint C4_Pretty:c_0805 -> C4_Pretty:c_0805_led
Changed lines of the file:
@@
 EESchema Schematic File Version 2
 LIBS:ClockFOUR
+LIBS:RowGB_sym
 LIBS:ClockFOUR-cache
 EELAYER 24 0
@@
 F 0 "C138" H 1975 3100 50  0000 L CNN
 F 1 "100n" H 1975 2900 50  0000 L CNN
-F 2 "C4_Pretty:c_0805" H 1950 3000 50  0001 C CNN
+F 2 "C4_Pretty:c_0805_led" H 1950 3000 50  0001 C CNN
 F 3 "" H 1950 3000 60  0001 C CNN
 F 4 "CAP CER 0.1UF 25V 10% X7R 0805" H 1950 3200 60  0001 L CNN "Field4"
@@
 F 0 "C139" H 3375 3100 50  0000 L CNN
 F 1 "100n" H 3375 2900 50  0000 L CNN
-F 2 "C4_Pretty:c_0805" H 3350 3000 50  0001 C CNN
+F 2 "C4_Pretty:c_0805_led" H 3350 3000 50  0001 C CNN
 F 3 "" H 3350 3000 60  0001 C CNN
 F 4 "CAP CER 0.1UF 25V 10% X7R 0805" H 3350 3200 60  0001 L CNN "Field4"
@@
 F 0 "C140" H 4775 3100 50  0000 L CNN
 F 1 "100n" H 4775 2900 50  0000 L CNN
-F 2 "C4_Pretty:c_0805" H 4750 3000 50  0001 C CNN
+F 2 "C4_Pretty:c_0805_led" H 4750 3000 50  0001 C CNN
 F 3 "" H 4750 3000 60  0001 C CNN
 F 4 "CAP CER 0.1UF 25V 10% X7R 0805" H 4750 3200 60  0001 L CNN "Field4"
@@
 F 0 "C141" H 6175 3100 50  0000 L CNN
 F 1 "100n" H 6175 2900 50  0000 L CNN
-F 2 "C4_Pretty:c_0805" H 6150 3000 50  0001 C CNN
+F 2 "C4_Pretty:c_0805_led" H 6150 3000 50  0001 C CNN
 F 3 "" H 6150 3000 60  0001 C CNN
 F 4 "CAP CER 0.1UF 25V 10% X7R 0805" H 6150 3200 60  0001 L CNN "Field4"
@@
 F 0 "C142" H 7575 3100 50  0000 L CNN
 F 1 "100n" H 7575 2900 50  0000 L CNN
-F 2 "C4_Pretty:c_0805" H 7550 3000 50  0001 C CNN
+F 2 "C4_Pretty:c_0805_led" H 7550 3000 50  0001 C CNN
 F 3 "" H 7550 3000 60  0001 C CNN
 F 4 "CAP CER 0.1UF 25V 10% X7R 0805" H 7550 3200 60  0001 L CNN "Field4"
@@
 F 0 "C143" H 8975 3100 50  0000 L CNN
 F 1 "100n" H 8975 2900 50  0000 L CNN
-F 2 "C4_Pretty:c_0805" H 8950 3000 50  0001 C CNN
+F 2 "C4_Pretty:c_0805_led" H 8950 3000 50  0001 C CNN
 F 3 "" H 8950 3000 60  0001 C CNN
 F 4 "CAP CER 0.1UF 25V 10% X7R 0805" H 8950 3200 60  0001 L CNN "Field4"
@@
 F 0 "C144" H 10375 3100 50  0000 L CNN
 F 1 "100n" H 10375 2900 50  0000 L CNN
-F 2 "C4_Pretty:c_0805" H 10350 3000 50  0001 C CNN
+F 2 "C4_Pretty:c_0805_led" H 10350 3000 50  0001 C CNN
 F 3 "" H 10350 3000 60  0001 C CNN
 F 4 "CAP CER 0.1UF 25V 10% X7R 0805" H 10350 3200 60  0001 L CNN "Field4"
@@
 F 0 "C145" H 1975 5450 50  0000 L CNN
 F 1 "100n" H 1975 5250 50  0000 L CNN
-F 2 "C4_Pretty:c_0805" H 1950 5350 50  0001 C CNN
+F 2 "C4_Pretty:c_0805_led" H 1950 5350 50  0001 C CNN
 F 3 "" H 1950 5350 60  0001 C CNN
 F 4 "CAP CER 0.1UF 25V 10% X7R 0805" H 1950 5550 60  0001 L CNN "Field4"
@@
 F 0 "C146" H 3375 5450 50  0000 L CNN
 F 1 "100n" H 3375 5250 50  0000 L CNN
-F 2 "C4_Pretty:c_0805" H 3350 5350 50  0001 C CNN
+F 2 "C4_Pretty:c_0805_led" H 3350 5350 50  0001 C CNN
 F 3 "" H 3350 5350 60  0001 C CNN
 F 4 "CAP CER 0.1UF 25V 10% X7R 0805" H 3350 5550 60  0001 L CNN "Field4"
@@
 F 0 "C147" H 4775 5450 50  0000 L CNN
 F 1 "100n" H 4775 5250 50  0000 L CNN
-F 2 "C4_Pretty:c_0805" H 4750 5350 50  0001 C CNN
+F 2 "C4_Pretty:c_0805_led" H 4750 5350 50  0001 C CNN
 F 3 "" H 4750 5350 60  0001 C CNN
 F 4 "CAP CER 0.1UF 25V 10% X7R 0805" H 4750 5550 60  0001 L CNN "Field4"
@@
 F 0 "C148" H 6175 5450 50  0000 L CNN
 F 1 "100n" H 6175 5250 50  0000 L CNN
-F 2 "C4_Pretty:c_0805" H 6150 5350 50  0001 C CNN
+F 2 "C4_Pretty:c_0805_led" H 6150 5350 50  0001 C CNN
 F 3 "" H 6150 5350 60  0001 C CNN
 F 4 "CAP CER 0.1UF 25V 10% X7R 0805" H 6150 5550 60  0001 L CNN "Field4"
@@
 F 0 "C149" H 7575 5450 50  0000 L CNN
 F 1 "100n" H 7575 5250 50  0000 L CNN
-F 2 "C4_Pretty:c_0805" H 7550 5350 50  0001 C CNN
+F 2 "C4_Pretty:c_0805_led" H 7550 5350 50  0001 C CNN
 F 3 "" H 7550 5350 60  0001 C CNN
 F 4 "CAP CER 0.1UF 25V 10% X7R 0805" H 7550 5550 60  0001 L CNN "Field4"
@@
 F 0 "C150" H 8975 5450 50  0000 L CNN
 F 1 "100n" H 8975 5250 50  0000 L CNN
-F 2 "C4_Pretty:c_0805" H 8950 5350 50  0001 C CNN
+F 2 "C4_Pretty:c_0805_led" H 8950 5350 50  0001 C CNN
 F 3 "" H 8950 5350 60  0001 C CNN
 F 4 "CAP CER 0.1UF 25V 10% X7R 0805" H 8950 5550 60  0001 L CNN "Field4"
@@
 F 0 "C151" H 10375 5450 50  0000 L CNN
 F 1 "100n" H 10375 5250 50  0000 L CNN
-F 2 "C4_Pretty:c_0805" H 10350 5350 50  0001 C CNN
+F 2 "C4_Pretty:c_0805_led" H 10350 5350 50  0001 C CNN
 F 3 "" H 10350 5350 60  0001 C CNN
 F 4 "CAP CER 0.1UF 25V 10% X7R 0805" H 10350 5550 60  0001 L CNN "Field4"
