File: KiCad/Row_K.sch (KiCad schematic (older format))
At the start: 14 parts, among them U101 RGB_WS2811B, U102 RGB_WS2811B, U103 RGB_WS2811B, U104 RGB_WS2811B, U105 RGB_WS2811B, U106 RGB_WS2811B, U107 RGB_WS2811B, U108 RGB_WS2811B

Commit message: Schematic updated
Parts:
- removed C101: 100n, TinyTiM_Lib:c_0805, symbol C2
- removed C117: 47u,8V, TinyTiM_Lib:c_2917, symbol C_POL_1
- removed S101, S102, S103, S104: CONN_1, TinyTiM_Lib:Screw, symbol CONN_1
- removed U101, U102, U103, U104, U105, U106, U107, U108: RGB_WS2811B, TinyTiM_Lib:RGB_WS2811B, symbol RGB_WS2811B
Connections:
- net labels removed: 5V, A_02, A_03, A_04, A_05, A_06, A_07, A_08, A_09, DI_A, DO_A, GND
- wire segments 49 -> 0
- no-connect marks 4 -> 0
Other:
- note removed: "Mounting Screws"

Commit message: Schematic updated
Parts:
- added C150, C151, C152, C153, C154, C155, C156, C157, C158, C159, C160, C161, C162, C163: 100n, TinyTiM_Lib:c_0805, symbol C2
- added U144, U145, U146, U147, U148, U149, U150, U151, U152, U153, U154, U155, U156, U157: RGB_WS2812B, symbol RGB_WS2812B
Connections:
- net labels added: 5V, DI_K, DO_K, GND
- wire segments 0 -> 82

Commit message: Schematic updated, board started
Parts:
- C151: renamed from C150; Field5 100nF, 25V -> 100n, 25V
- C153: renamed from C154; Field5 100nF, 25V -> 100n, 25V
- C155: renamed from C158; Field5 100nF, 25V -> 100n, 25V
- C157: renamed from C162; Field5 100nF, 25V -> 100n, 25V
- C159: renamed from C153; Field5 100nF, 25V -> 100n, 25V
- C161: renamed from C157; Field5 100nF, 25V -> 100n, 25V
- C163: renamed from C161; Field5 100nF, 25V -> 100n, 25V
- renumbered C156 to C154, C160 to C156, C151 to C158, C155 to C160, C159 to C162, C163 to C164, U144 to U142, U146 to U143, U148 to U144, U150 to U145, U152 to U146, U154 to U147, U156 to U148, U145 to U149, U147 to U150, U149 to U151, U151 to U152, U155 to U154, U157 to U155
Changed lines of the file:
@@
 LIBS:contrib
 LIBS:valves
-LIBS:TinyTiM-cache
-LIBS:TiNA_sym
+LIBS:ClockFOUR
 LIBS:ClockFOUR-cache
 EELAYER 27 0
@@
 Sheet 12 14
 Title "ClockFOUR"
-Date "30 sep 2014"
+Date "1 oct 2014"
 Rev ""
 Comp "WyoLum"
@@
 5V
 $Comp
-L GND #PWR022
+L GND #PWR024
 U 1 1 542C17A6
 P 1350 2800
-F 0 "#PWR022" H 1350 2800 30  0001 C CNN
+F 0 "#PWR024" H 1350 2800 30  0001 C CNN
 F 1 "GND" H 1350 2730 30  0001 C CNN
 F 2 "" H 1350 2800 60  0001 C CNN
@@
 $EndComp
 $Comp
-L C2 C150
+L C2 C151
 U 1 1 542C17B4
 P 1900 2950
-F 0 "C150" H 1925 3050 50  0000 L CNN
+F 0 "C151" H 1925 3050 50  0000 L CNN
 F 1 "100n" H 1925 2850 50  0000 L CNN
 F 2 "TinyTiM_Lib:c_0805" H 1900 2950 50  0001 C CNN
 F 3 "" H 1900 2950 60  0001 C CNN
 F 4 "CAP CER 0.1UF 25V 10% X7R 0805" H 1900 3150 60  0001 L CNN "Field4"
-F 5 "100nF, 25V" H 1900 3250 60  0001 L CNN "Field5"
+F 5 "100n, 25V" H 1900 3250 60  0001 L CNN "Field5"
 F 6 "Surface Mount, MLCC" H 1900 3350 60  0001 L CNN "Field6"
 F 7 "Kemet" H 1900 3450 60  0001 L CNN "Field7"
@@
 $EndComp
 $Comp
-L RGB_WS2812B U144
+L RGB_WS2812B U142
 U 1 1 542C17BA
 P 1725 1975
-F 0 "U144" V 1475 1975 60  0000 C CNN
+F 0 "U142" V 1475 1975 60  0000 C CNN
 F 1 "RGB_WS2812B" V 2125 1975 60  0000 C CNN
 F 2 "" H 1725 1975 60  0000 C CNN
@@
 $EndComp
 $Comp
-L RGB_WS2812B U146
+L RGB_WS2812B U143
 U 1 1 542C17C0
 P 3125 1975
-F 0 "U146" V 2875 1975 60  0000 C CNN
+F 0 "U143" V 2875 1975 60  0000 C CNN
 F 1 "RGB_WS2812B" V 3525 1975 60  0000 C CNN
 F 2 "" H 3125 1975 60  0000 C CNN
@@
 $EndComp
 $Comp
-L RGB_WS2812B U148
+L RGB_WS2812B U144
 U 1 1 542C17C6
 P 4525 1975
-F 0 "U148" V 4275 1975 60  0000 C CNN
+F 0 "U144" V 4275 1975 60  0000 C CNN
 F 1 "RGB_WS2812B" V 4925 1975 60  0000 C CNN
 F 2 "" H 4525 1975 60  0000 C CNN
@@
 $EndComp
 $Comp
-L RGB_WS2812B U150
+L RGB_WS2812B U145
 U 1 1 542C17CC
 P 5925 1975
-F 0 "U150" V 5675 1975 60  0000 C CNN
+F 0 "U145" V 5675 1975 60  0000 C CNN
 F 1 "RGB_WS2812B" V 6325 1975 60  0000 C CNN
 F 2 "" H 5925 1975 60  0000 C CNN
@@
 $EndComp
 $Comp
-L RGB_WS2812B U152
+L RGB_WS2812B U146
 U 1 1 542C17D2
 P 7325 1975
-F 0 "U152" V 7075 1975 60  0000 C CNN
+F 0 "U146" V 7075 1975 60  0000 C CNN
 F 1 "RGB_WS2812B" V 7725 1975 60  0000 C CNN
 F 2 "" H 7325 1975 60  0000 C CNN
@@
 $EndComp
 $Comp
-L RGB_WS2812B U154
+L RGB_WS2812B U147
 U 1 1 542C17D8
 P 8725 1975
-F 0 "U154" V 8475 1975 60  0000 C CNN
+F 0 "U147" V 8475 1975 60  0000 C CNN
 F 1 "RGB_WS2812B" V 9125 1975 60  0000 C CNN
 F 2 "" H 8725 1975 60  0000 C CNN
@@
 $EndComp
 $Comp
-L RGB_WS2812B U156
+L RGB_WS2812B U148
 U 1 1 542C17DE
 P 10125 1975
-F 0 "U156" V 9875 1975 60  0000 C CNN
+F 0 "U148" V 9875 1975 60  0000 C CNN
 F 1 "RGB_WS2812B" V 10525 1975 60  0000 C CNN
 F 2 "" H 10125 1975 60  0000 C CNN
@@
 $EndComp
 $Comp
-L RGB_WS2812B U145
+L RGB_WS2812B U149
 U 1 1 542C17E4
 P 1725 4375
-F 0 "U145" V 1475 4375 60  0000 C CNN
+F 0 "U149" V 1475 4375 60  0000 C CNN
 F 1 "RGB_WS2812B" V 2125 4375 60  0000 C CNN
 F 2 "" H 1725 4375 60  0000 C CNN
@@
 $EndComp
 $Comp
-L RGB_WS2812B U147
+L RGB_WS2812B U150
 U 1 1 542C17EA
 P 3125 4375
-F 0 "U147" V 2875 4375 60  0000 C CNN
+F 0 "U150" V 2875 4375 60  0000 C CNN
 F 1 "RGB_WS2812B" V 3525 4375 60  0000 C CNN
 F 2 "" H 3125 4375 60  0000 C CNN
@@
 $EndComp
 $Comp
-L RGB_WS2812B U149
+L RGB_WS2812B U151
 U 1 1 542C17F0
 P 4525 4375
-F 0 "U149" V 4275 4375 60  0000 C CNN
+F 0 "U151" V 4275 4375 60  0000 C CNN
 F 1 "RGB_WS2812B" V 4925 4375 60  0000 C CNN
 F 2 "" H 4525 4375 60  0000 C CNN
@@
 $EndComp
 $Comp
-L RGB_WS2812B U151
+L RGB_WS2812B U152
 U 1 1 542C17F6
 P 5925 4375
-F 0 "U151" V 5675 4375 60  0000 C CNN
+F 0 "U152" V 5675 4375 60  0000 C CNN
 F 1 "RGB_WS2812B" V 6325 4375 60  0000 C CNN
 F 2 "" H 5925 4375 60  0000 C CNN
@@
 $EndComp
 $Comp
-L RGB_WS2812B U155
+L RGB_WS2812B U154
 U 1 1 542C1802
 P 8725 4375
-F 0 "U155" V 8475 4375 60  0000 C CNN
+F 0 "U154" V 8475 4375 60  0000 C CNN
 F 1 "RGB_WS2812B" V 9125 4375 60  0000 C CNN
 F 2 "" H 8725 4375 60  0000 C CNN
@@
 $EndComp
 $Comp
-L RGB_WS2812B U157
+L RGB_WS2812B U155
 U 1 1 542C1808
 P 10125 4375
-F 0 "U157" V 9875 4375 60  0000 C CNN
+F 0 "U155" V 9875 4375 60  0000 C CNN
 F 1 "RGB_WS2812B" V 10525 4375 60  0000 C CNN
 F 2 "" H 10125 4375 60  0000 C CNN
@@
 $EndComp
 $Comp
-L C2 C154
+L C2 C153
 U 1 1 542C1871
 P 4700 2950
-F 0 "C154" H 4725 3050 50  0000 L CNN
+F 0 "C153" H 4725 3050 50  0000 L CNN
 F 1 "100n" H 4725 2850 50  0000 L CNN
 F 2 "TinyTiM_Lib:c_0805" H 4700 2950 50  0001 C CNN
 F 3 "" H 4700 2950 60  0001 C CNN
 F 4 "CAP CER 0.1UF 25V 10% X7R 0805" H 4700 3150 60  0001 L CNN "Field4"
-F 5 "100nF, 25V" H 4700 3250 60  0001 L CNN "Field5"
+F 5 "100n, 25V" H 4700 3250 60  0001 L CNN "Field5"
 F 6 "Surface Mount, MLCC" H 4700 3350 60  0001 L CNN "Field6"
 F 7 "Kemet" H 4700 3450 60  0001 L CNN "Field7"
@@
 $EndComp
 $Comp
-L C2 C156
+L C2 C154
 U 1 1 542C187F
 P 6100 2950
-F 0 "C156" H 6125 3050 50  0000 L CNN
+F 0 "C154" H 6125 3050 50  0000 L CNN
 F 1 "100n" H 6125 2850 50  0000 L CNN
 F 2 "TinyTiM_Lib:c_0805" H 6100 2950 50  0001 C CNN
@@
 $EndComp
 $Comp
-L C2 C158
+L C2 C155
 U 1 1 542C188D
 P 7500 2950
-F 0 "C158" H 7525 3050 50  0000 L CNN
+F 0 "C155" H 7525 3050 50  0000 L CNN
 F 1 "100n" H 7525 2850 50  0000 L CNN
 F 2 "TinyTiM_Lib:c_0805" H 7500 2950 50  0001 C CNN
 F 3 "" H 7500 2950 60  0001 C CNN
 F 4 "CAP CER 0.1UF 25V 10% X7R 0805" H 7500 3150 60  0001 L CNN "Field4"
-F 5 "100nF, 25V" H 7500 3250 60  0001 L CNN "Field5"
+F 5 "100n, 25V" H 7500 3250 60  0001 L CNN "Field5"
 F 6 "Surface Mount, MLCC" H 7500 3350 60  0001 L CNN "Field6"
 F 7 "Kemet" H 7500 3450 60  0001 L CNN "Field7"
@@
 $EndComp
 $Comp
-L C2 C160
+L C2 C156
 U 1 1 542C189B
 P 8900 2950
-F 0 "C160" H 8925 3050 50  0000 L CNN
+F 0 "C156" H 8925 3050 50  0000 L CNN
 F 1 "100n" H 8925 2850 50  0000 L CNN
 F 2 "TinyTiM_Lib:c_0805" H 8900 2950 50  0001 C CNN
@@
 $EndComp
 $Comp
-L C2 C162
+L C2 C157
 U 1 1 542C18A9
 P 10300 2950
-F 0 "C162" H 10325 3050 50  0000 L CNN
+F 0 "C157" H 10325 3050 50  0000 L CNN
 F 1 "100n" H 10325 2850 50  0000 L CNN
 F 2 "TinyTiM_Lib:c_0805" H 10300 2950 50  0001 C CNN
 F 3 "" H 10300 2950 60  0001 C CNN
 F 4 "CAP CER 0.1UF 25V 10% X7R 0805" H 10300 3150 60  0001 L CNN "Field4"
-F 5 "100nF, 25V" H 10300 3250 60  0001 L CNN "Field5"
+F 5 "100n, 25V" H 10300 3250 60  0001 L CNN "Field5"
 F 6 "Surface Mount, MLCC" H 10300 3350 60  0001 L CNN "Field6"
 F 7 "Kemet" H 10300 3450 60  0001 L CNN "Field7"
@@
 Connection ~ 10200 3150
 $Comp
-L C2 C151
+L C2 C158
 U 1 1 542C18B8
 P 1900 5300
-F 0 "C151" H 1925 5400 50  0000 L CNN
+F 0 "C158" H 1925 5400 50  0000 L CNN
 F 1 "100n" H 1925 5200 50  0000 L CNN
 F 2 "TinyTiM_Lib:c_0805" H 1900 5300 50  0001 C CNN
@@
 Connection ~ 1800 5500
 $Comp
-L C2 C153
+L C2 C159
 U 1 1 542C18F5
 P 3300 5300
-F 0 "C153" H 3325 5400 50  0000 L CNN
+F 0 "C159" H 3325 5400 50  0000 L CNN
 F 1 "100n" H 3325 5200 50  0000 L CNN
 F 2 "TinyTiM_Lib:c_0805" H 3300 5300 50  0001 C CNN
 F 3 "" H 3300 5300 60  0001 C CNN
 F 4 "CAP CER 0.1UF 25V 10% X7R 0805" H 3300 5500 60  0001 L CNN "Field4"
-F 5 "100nF, 25V" H 3300 5600 60  0001 L CNN "Field5"
+F 5 "100n, 25V" H 3300 5600 60  0001 L CNN "Field5"
 F 6 "Surface Mount, MLCC" H 3300 5700 60  0001 L CNN "Field6"
 F 7 "Kemet" H 3300 5800 60  0001 L CNN "Field7"
@@
 $EndComp
 $Comp
-L C2 C155
+L C2 C160
 U 1 1 542C1903
 P 4700 5300
-F 0 "C155" H 4725 5400 50  0000 L CNN
+F 0 "C160" H 4725 5400 50  0000 L CNN
 F 1 "100n" H 4725 5200 50  0000 L CNN
 F 2 "TinyTiM_Lib:c_0805" H 4700 5300 50  0001 C CNN
@@
 $EndComp
 $Comp
-L C2 C157
+L C2 C161
 U 1 1 542C1911
 P 6100 5300
-F 0 "C157" H 6125 5400 50  0000 L CNN
+F 0 "C161" H 6125 5400 50  0000 L CNN
 F 1 "100n" H 6125 5200 50  0000 L CNN
 F 2 "TinyTiM_Lib:c_0805" H 6100 5300 50  0001 C CNN
 F 3 "" H 6100 5300 60  0001 C CNN
 F 4 "CAP CER 0.1UF 25V 10% X7R 0805" H 6100 5500 60  0001 L CNN "Field4"
-F 5 "100nF, 25V" H 6100 5600 60  0001 L CNN "Field5"
+F 5 "100n, 25V" H 6100 5600 60  0001 L CNN "Field5"
 F 6 "Surface Mount, MLCC" H 6100 5700 60  0001 L CNN "Field6"
 F 7 "Kemet" H 6100 5800 60  0001 L CNN "Field7"
@@
 $EndComp
 $Comp
-L C2 C159
+L C2 C162
 U 1 1 542C191F
 P 7500 5300
-F 0 "C159" H 7525 5400 50  0000 L CNN
+F 0 "C162" H 7525 5400 50  0000 L CNN
 F 1 "100n" H 7525 5200 50  0000 L CNN
 F 2 "TinyTiM_Lib:c_0805" H 7500 5300 50  0001 C CNN
@@
 $EndComp
 $Comp
-L C2 C161
+L C2 C163
 U 1 1 542C192D
 P 8900 5300
-F 0 "C161" H 8925 5400 50  0000 L CNN
+F 0 "C163" H 8925 5400 50  0000 L CNN
 F 1 "100n" H 8925 5200 50  0000 L CNN
 F 2 "TinyTiM_Lib:c_0805" H 8900 5300 50  0001 C CNN
 F 3 "" H 8900 5300 60  0001 C CNN
 F 4 "CAP CER 0.1UF 25V 10% X7R 0805" H 8900 5500 60  0001 L CNN "Field4"
-F 5 "100nF, 25V" H 8900 5600 60  0001 L CNN "Field5"
+F 5 "100n, 25V" H 8900 5600 60  0001 L CNN "Field5"
 F 6 "Surface Mount, MLCC" H 8900 5700 60  0001 L CNN "Field6"
 F 7 "Kemet" H 8900 5800 60  0001 L CNN "Field7"
@@
 $EndComp
 $Comp
-L C2 C163
+L C2 C164
 U 1 1 542C193B
 P 10300 5300
-F 0 "C163" H 10325 5400 50  0000 L CNN
+F 0 "C164" H 10325 5400 50  0000 L CNN
 F 1 "100n" H 10325 5200 50  0000 L CNN
 F 2 "TinyTiM_Lib:c_0805" H 10300 5300 50  0001 C CNN

Commit message: Board layout updated
Parts:
- removed U142, U143, U144, U145, U146, U147, U148, U149, U150, U151, U152, U153, U154, U155: RGB_WS2812B, symbol RGB_WS2812B
- added LED141, LED142, LED143, LED144, LED145, LED146, LED147, LED148, LED149, LED150, LED151, LED152, LED153, LED154: RGB_WS2812B, ~, symbol RGB_WS2812B

Commit message: Board layout updated
Matrix placed and wired. Added RTC.
Parts:
- removed C151: 100n, TinyTiM_Lib:c_0805, symbol C2
- removed LED141, LED142, LED143, LED144, LED145, LED146, LED147, LED148, LED149, LED150, LED151, LED152, LED153, LED154: RGB_WS2812B, ~, symbol RGB_WS2812B
- added C165: 100n, TinyTiM_Lib:c_0805, symbol C2
- added LED141, LED142, LED143, LED144, LED145, LED146, LED147, LED148, LED149, LED150, LED151, LED152, LED153, LED154: WS2812B, ~, symbol WS2812B
- C152, C154, C156, C158, C160, C162, C164: Field5 100nF, 25V -> 100n, 25V
- C153, C155, C157, C159, C161, C163: Field5 100n, 25V -> 100nF, 25V
