File: KiCad/Row_K.sch (KiCad schematic (older format))
At the start: 28 parts

Commit message: PCB layout, work in progress
Parts:
- C152, C153, C154, C155, C156, C157, C158, C159, C160, C161, C162, C163, C164, C165: footprint TinyTiM_Lib:c_0805 -> C4_Pretty:c_0805
- LED141, LED142, LED143, LED144, LED145, LED146, LED147, LED148, LED149, LED150, LED151, LED152, LED153, LED154: footprint ~ -> C4_Pretty:RGB_WS2811B
Changed lines of the file:
@@
 F 0 "C152" H 1825 3250 50  0000 L CNN
 F 1 "100n" H 1825 3050 50  0000 L CNN
-F 2 "TinyTiM_Lib:c_0805" H 1800 3150 50  0001 C CNN
+F 2 "C4_Pretty:c_0805" H 1800 3150 50  0001 C CNN
 F 3 "" H 1800 3150 60  0001 C CNN
 F 4 "CAP CER 0.1UF 25V 10% X7R 0805" H 1800 3350 60  0001 L CNN "Field4"
@@
 F 0 "C153" H 3225 3250 50  0000 L CNN
 F 1 "100n" H 3225 3050 50  0000 L CNN
-F 2 "TinyTiM_Lib:c_0805" H 3200 3150 50  0001 C CNN
+F 2 "C4_Pretty:c_0805" H 3200 3150 50  0001 C CNN
 F 3 "" H 3200 3150 60  0001 C CNN
 F 4 "CAP CER 0.1UF 25V 10% X7R 0805" H 3200 3350 60  0001 L CNN "Field4"
@@
 F 0 "C154" H 4625 3250 50  0000 L CNN
 F 1 "100n" H 4625 3050 50  0000 L CNN
-F 2 "TinyTiM_Lib:c_0805" H 4600 3150 50  0001 C CNN
+F 2 "C4_Pretty:c_0805" H 4600 3150 50  0001 C CNN
 F 3 "" H 4600 3150 60  0001 C CNN
 F 4 "CAP CER 0.1UF 25V 10% X7R 0805" H 4600 3350 60  0001 L CNN "Field4"
@@
 F 0 "C155" H 6025 3250 50  0000 L CNN
 F 1 "100n" H 6025 3050 50  0000 L CNN
-F 2 "TinyTiM_Lib:c_0805" H 6000 3150 50  0001 C CNN
+F 2 "C4_Pretty:c_0805" H 6000 3150 50  0001 C CNN
 F 3 "" H 6000 3150 60  0001 C CNN
 F 4 "CAP CER 0.1UF 25V 10% X7R 0805" H 6000 3350 60  0001 L CNN "Field4"
@@
 F 0 "C156" H 7425 3250 50  0000 L CNN
 F 1 "100n" H 7425 3050 50  0000 L CNN
-F 2 "TinyTiM_Lib:c_0805" H 7400 3150 50  0001 C CNN
+F 2 "C4_Pretty:c_0805" H 7400 3150 50  0001 C CNN
 F 3 "" H 7400 3150 60  0001 C CNN
 F 4 "CAP CER 0.1UF 25V 10% X7R 0805" H 7400 3350 60  0001 L CNN "Field4"
@@
 F 0 "C157" H 8825 3250 50  0000 L CNN
 F 1 "100n" H 8825 3050 50  0000 L CNN
-F 2 "TinyTiM_Lib:c_0805" H 8800 3150 50  0001 C CNN
+F 2 "C4_Pretty:c_0805" H 8800 3150 50  0001 C CNN
 F 3 "" H 8800 3150 60  0001 C CNN
 F 4 "CAP CER 0.1UF 25V 10% X7R 0805" H 8800 3350 60  0001 L CNN "Field4"
@@
 F 0 "C158" H 10225 3250 50  0000 L CNN
 F 1 "100n" H 10225 3050 50  0000 L CNN
-F 2 "TinyTiM_Lib:c_0805" H 10200 3150 50  0001 C CNN
+F 2 "C4_Pretty:c_0805" H 10200 3150 50  0001 C CNN
 F 3 "" H 10200 3150 60  0001 C CNN
 F 4 "CAP CER 0.1UF 25V 10% X7R 0805" H 10200 3350 60  0001 L CNN "Field4"
@@
 F 0 "C159" H 1825 5600 50  0000 L CNN
 F 1 "100n" H 1825 5400 50  0000 L CNN
-F 2 "TinyTiM_Lib:c_0805" H 1800 5500 50  0001 C CNN
+F 2 "C4_Pretty:c_0805" H 1800 5500 50  0001 C CNN
 F 3 "" H 1800 5500 60  0001 C CNN
 F 4 "CAP CER 0.1UF 25V 10% X7R 0805" H 1800 5700 60  0001 L CNN "Field4"
@@
 F 0 "C160" H 3225 5600 50  0000 L CNN
 F 1 "100n" H 3225 5400 50  0000 L CNN
-F 2 "TinyTiM_Lib:c_0805" H 3200 5500 50  0001 C CNN
+F 2 "C4_Pretty:c_0805" H 3200 5500 50  0001 C CNN
 F 3 "" H 3200 5500 60  0001 C CNN
 F 4 "CAP CER 0.1UF 25V 10% X7R 0805" H 3200 5700 60  0001 L CNN "Field4"
@@
 F 0 "C161" H 4625 5600 50  0000 L CNN
 F 1 "100n" H 4625 5400 50  0000 L CNN
-F 2 "TinyTiM_Lib:c_0805" H 4600 5500 50  0001 C CNN
+F 2 "C4_Pretty:c_0805" H 4600 5500 50  0001 C CNN
 F 3 "" H 4600 5500 60  0001 C CNN
 F 4 "CAP CER 0.1UF 25V 10% X7R 0805" H 4600 5700 60  0001 L CNN "Field4"
@@
 F 0 "C162" H 6025 5600 50  0000 L CNN
 F 1 "100n" H 6025 5400 50  0000 L CNN
-F 2 "TinyTiM_Lib:c_0805" H 6000 5500 50  0001 C CNN
+F 2 "C4_Pretty:c_0805" H 6000 5500 50  0001 C CNN
 F 3 "" H 6000 5500 60  0001 C CNN
 F 4 "CAP CER 0.1UF 25V 10% X7R 0805" H 6000 5700 60  0001 L CNN "Field4"
@@
 F 0 "C163" H 7425 5600 50  0000 L CNN
 F 1 "100n" H 7425 5400 50  0000 L CNN
-F 2 "TinyTiM_Lib:c_0805" H 7400 5500 50  0001 C CNN
+F 2 "C4_Pretty:c_0805" H 7400 5500 50  0001 C CNN
 F 3 "" H 7400 5500 60  0001 C CNN
 F 4 "CAP CER 0.1UF 25V 10% X7R 0805" H 7400 5700 60  0001 L CNN "Field4"
@@
 F 0 "C164" H 8825 5600 50  0000 L CNN
 F 1 "100n" H 8825 5400 50  0000 L CNN
-F 2 "TinyTiM_Lib:c_0805" H 8800 5500 50  0001 C CNN
+F 2 "C4_Pretty:c_0805" H 8800 5500 50  0001 C CNN
 F 3 "" H 8800 5500 60  0001 C CNN
 F 4 "CAP CER 0.1UF 25V 10% X7R 0805" H 8800 5700 60  0001 L CNN "Field4"
@@
 F 0 "C165" H 10225 5600 50  0000 L CNN
 F 1 "100n" H 10225 5400 50  0000 L CNN
-F 2 "TinyTiM_Lib:c_0805" H 10200 5500 50  0001 C CNN
+F 2 "C4_Pretty:c_0805" H 10200 5500 50  0001 C CNN
 F 3 "" H 10200 5500 60  0001 C CNN
 F 4 "CAP CER 0.1UF 25V 10% X7R 0805" H 10200 5700 60  0001 L CNN "Field4"
@@
 F 0 "LED141" V 1375 2175 60  0000 C CNN
 F 1 "WS2812B" V 2025 2175 60  0001 C CNN
-F 2 "~" H 1625 2175 60  0000 C CNN
+F 2 "C4_Pretty:RGB_WS2811B" H 1625 2175 60  0001 C CNN
 F 3 "~" H 1625 2175 60  0000 C CNN
 	1    1625 2175
@@
 F 0 "LED142" V 2775 2175 60  0000 C CNN
 F 1 "WS2812B" V 3425 2175 60  0001 C CNN
-F 2 "~" H 3025 2175 60  0000 C CNN
+F 2 "C4_Pretty:RGB_WS2811B" H 3025 2175 60  0001 C CNN
 F 3 "~" H 3025 2175 60  0000 C CNN
 	1    3025 2175
@@
 F 0 "LED143" V 4175 2175 60  0000 C CNN
 F 1 "WS2812B" V 4825 2175 60  0001 C CNN
-F 2 "~" H 4425 2175 60  0000 C CNN
+F 2 "C4_Pretty:RGB_WS2811B" H 4425 2175 60  0001 C CNN
 F 3 "~" H 4425 2175 60  0000 C CNN
 	1    4425 2175
@@
 F 0 "LED144" V 5575 2175 60  0000 C CNN
 F 1 "WS2812B" V 6225 2175 60  0001 C CNN
-F 2 "~" H 5825 2175 60  0000 C CNN
+F 2 "C4_Pretty:RGB_WS2811B" H 5825 2175 60  0001 C CNN
 F 3 "~" H 5825 2175 60  0000 C CNN
 	1    5825 2175
@@
 F 0 "LED145" V 6975 2175 60  0000 C CNN
 F 1 "WS2812B" V 7625 2175 60  0001 C CNN
-F 2 "~" H 7225 2175 60  0000 C CNN
+F 2 "C4_Pretty:RGB_WS2811B" H 7225 2175 60  0001 C CNN
 F 3 "~" H 7225 2175 60  0000 C CNN
 	1    7225 2175
@@
 F 0 "LED146" V 8375 2175 60  0000 C CNN
 F 1 "WS2812B" V 9025 2175 60  0001 C CNN
-F 2 "~" H 8625 2175 60  0000 C CNN
+F 2 "C4_Pretty:RGB_WS2811B" H 8625 2175 60  0001 C CNN
 F 3 "~" H 8625 2175 60  0000 C CNN
 	1    8625 2175
@@
 F 0 "LED147" V 9775 2175 60  0000 C CNN
 F 1 "WS2812B" V 10425 2175 60  0001 C CNN
-F 2 "~" H 10025 2175 60  0000 C CNN
+F 2 "C4_Pretty:RGB_WS2811B" H 10025 2175 60  0001 C CNN
 F 3 "~" H 10025 2175 60  0000 C CNN
 	1    10025 2175
@@
 F 0 "LED148" V 1375 4575 60  0000 C CNN
 F 1 "WS2812B" V 2025 4575 60  0001 C CNN
-F 2 "~" H 1625 4575 60  0000 C CNN
+F 2 "C4_Pretty:RGB_WS2811B" H 1625 4575 60  0001 C CNN
 F 3 "~" H 1625 4575 60  0000 C CNN
 	1    1625 4575
@@
 F 0 "LED149" V 2775 4575 60  0000 C CNN
 F 1 "WS2812B" V 3425 4575 60  0001 C CNN
-F 2 "~" H 3025 4575 60  0000 C CNN
+F 2 "C4_Pretty:RGB_WS2811B" H 3025 4575 60  0001 C CNN
 F 3 "~" H 3025 4575 60  0000 C CNN
 	1    3025 4575
@@
 F 0 "LED150" V 4175 4575 60  0000 C CNN
 F 1 "WS2812B" V 4825 4575 60  0001 C CNN
-F 2 "~" H 4425 4575 60  0000 C CNN
+F 2 "C4_Pretty:RGB_WS2811B" H 4425 4575 60  0001 C CNN
 F 3 "~" H 4425 4575 60  0000 C CNN
 	1    4425 4575
@@
 F 0 "LED151" V 5575 4575 60  0000 C CNN
 F 1 "WS2812B" V 6225 4575 60  0001 C CNN
-F 2 "~" H 5825 4575 60  0000 C CNN
+F 2 "C4_Pretty:RGB_WS2811B" H 5825 4575 60  0001 C CNN
 F 3 "~" H 5825 4575 60  0000 C CNN
 	1    5825 4575
@@
 F 0 "LED152" V 6975 4575 60  0000 C CNN
 F 1 "WS2812B" V 7625 4575 60  0001 C CNN
-F 2 "~" H 7225 4575 60  0000 C CNN
+F 2 "C4_Pretty:RGB_WS2811B" H 7225 4575 60  0001 C CNN
 F 3 "~" H 7225 4575 60  0000 C CNN
 	1    7225 4575
@@
 F 0 "LED153" V 8375 4575 60  0000 C CNN
 F 1 "WS2812B" V 9025 4575 60  0001 C CNN
-F 2 "~" H 8625 4575 60  0000 C CNN
+F 2 "C4_Pretty:RGB_WS2811B" H 8625 4575 60  0001 C CNN
 F 3 "~" H 8625 4575 60  0000 C CNN
 	1    8625 4575
@@
 F 0 "LED154" V 9775 4575 60  0000 C CNN
 F 1 "WS2812B" V 10425 4575 60  0001 C CNN
-F 2 "~" H 10025 4575 60  0000 C CNN
+F 2 "C4_Pretty:RGB_WS2811B" H 10025 4575 60  0001 C CNN
 F 3 "~" H 10025 4575 60  0000 C CNN
 	1    10025 4575

Commit message: C4 PCB layout complete. Added Gerbers
Parts:
- C152, C153, C154, C155, C156, C157, C158, C159, C160, C161, C162, C163, C164, C165: footprint C4_Pretty:c_0805 -> C4_Pretty:c_0805_led
Changed lines of the file:
@@
 EESchema Schematic File Version 2
 LIBS:ClockFOUR
+LIBS:RowGB_sym
 LIBS:ClockFOUR-cache
 EELAYER 24 0
@@
 F 0 "C152" H 1825 3250 50  0000 L CNN
 F 1 "100n" H 1825 3050 50  0000 L CNN
-F 2 "C4_Pretty:c_0805" H 1800 3150 50  0001 C CNN
+F 2 "C4_Pretty:c_0805_led" H 1800 3150 50  0001 C CNN
 F 3 "" H 1800 3150 60  0001 C CNN
 F 4 "CAP CER 0.1UF 25V 10% X7R 0805" H 1800 3350 60  0001 L CNN "Field4"
@@
 F 0 "C153" H 3225 3250 50  0000 L CNN
 F 1 "100n" H 3225 3050 50  0000 L CNN
-F 2 "C4_Pretty:c_0805" H 3200 3150 50  0001 C CNN
+F 2 "C4_Pretty:c_0805_led" H 3200 3150 50  0001 C CNN
 F 3 "" H 3200 3150 60  0001 C CNN
 F 4 "CAP CER 0.1UF 25V 10% X7R 0805" H 3200 3350 60  0001 L CNN "Field4"
@@
 F 0 "C154" H 4625 3250 50  0000 L CNN
 F 1 "100n" H 4625 3050 50  0000 L CNN
-F 2 "C4_Pretty:c_0805" H 4600 3150 50  0001 C CNN
+F 2 "C4_Pretty:c_0805_led" H 4600 3150 50  0001 C CNN
 F 3 "" H 4600 3150 60  0001 C CNN
 F 4 "CAP CER 0.1UF 25V 10% X7R 0805" H 4600 3350 60  0001 L CNN "Field4"
@@
 F 0 "C155" H 6025 3250 50  0000 L CNN
 F 1 "100n" H 6025 3050 50  0000 L CNN
-F 2 "C4_Pretty:c_0805" H 6000 3150 50  0001 C CNN
+F 2 "C4_Pretty:c_0805_led" H 6000 3150 50  0001 C CNN
 F 3 "" H 6000 3150 60  0001 C CNN
 F 4 "CAP CER 0.1UF 25V 10% X7R 0805" H 6000 3350 60  0001 L CNN "Field4"
@@
 F 0 "C156" H 7425 3250 50  0000 L CNN
 F 1 "100n" H 7425 3050 50  0000 L CNN
-F 2 "C4_Pretty:c_0805" H 7400 3150 50  0001 C CNN
+F 2 "C4_Pretty:c_0805_led" H 7400 3150 50  0001 C CNN
 F 3 "" H 7400 3150 60  0001 C CNN
 F 4 "CAP CER 0.1UF 25V 10% X7R 0805" H 7400 3350 60  0001 L CNN "Field4"
@@
 F 0 "C157" H 8825 3250 50  0000 L CNN
 F 1 "100n" H 8825 3050 50  0000 L CNN
-F 2 "C4_Pretty:c_0805" H 8800 3150 50  0001 C CNN
+F 2 "C4_Pretty:c_0805_led" H 8800 3150 50  0001 C CNN
 F 3 "" H 8800 3150 60  0001 C CNN
 F 4 "CAP CER 0.1UF 25V 10% X7R 0805" H 8800 3350 60  0001 L CNN "Field4"
@@
 F 0 "C158" H 10225 3250 50  0000 L CNN
 F 1 "100n" H 10225 3050 50  0000 L CNN
-F 2 "C4_Pretty:c_0805" H 10200 3150 50  0001 C CNN
+F 2 "C4_Pretty:c_0805_led" H 10200 3150 50  0001 C CNN
 F 3 "" H 10200 3150 60  0001 C CNN
 F 4 "CAP CER 0.1UF 25V 10% X7R 0805" H 10200 3350 60  0001 L CNN "Field4"
@@
 F 0 "C159" H 1825 5600 50  0000 L CNN
 F 1 "100n" H 1825 5400 50  0000 L CNN
-F 2 "C4_Pretty:c_0805" H 1800 5500 50  0001 C CNN
+F 2 "C4_Pretty:c_0805_led" H 1800 5500 50  0001 C CNN
 F 3 "" H 1800 5500 60  0001 C CNN
 F 4 "CAP CER 0.1UF 25V 10% X7R 0805" H 1800 5700 60  0001 L CNN "Field4"
@@
 F 0 "C160" H 3225 5600 50  0000 L CNN
 F 1 "100n" H 3225 5400 50  0000 L CNN
-F 2 "C4_Pretty:c_0805" H 3200 5500 50  0001 C CNN
+F 2 "C4_Pretty:c_0805_led" H 3200 5500 50  0001 C CNN
 F 3 "" H 3200 5500 60  0001 C CNN
 F 4 "CAP CER 0.1UF 25V 10% X7R 0805" H 3200 5700 60  0001 L CNN "Field4"
@@
 F 0 "C161" H 4625 5600 50  0000 L CNN
 F 1 "100n" H 4625 5400 50  0000 L CNN
-F 2 "C4_Pretty:c_0805" H 4600 5500 50  0001 C CNN
+F 2 "C4_Pretty:c_0805_led" H 4600 5500 50  0001 C CNN
 F 3 "" H 4600 5500 60  0001 C CNN
 F 4 "CAP CER 0.1UF 25V 10% X7R 0805" H 4600 5700 60  0001 L CNN "Field4"
@@
 F 0 "C162" H 6025 5600 50  0000 L CNN
 F 1 "100n" H 6025 5400 50  0000 L CNN
-F 2 "C4_Pretty:c_0805" H 6000 5500 50  0001 C CNN
+F 2 "C4_Pretty:c_0805_led" H 6000 5500 50  0001 C CNN
 F 3 "" H 6000 5500 60  0001 C CNN
 F 4 "CAP CER 0.1UF 25V 10% X7R 0805" H 6000 5700 60  0001 L CNN "Field4"
@@
 F 0 "C163" H 7425 5600 50  0000 L CNN
 F 1 "100n" H 7425 5400 50  0000 L CNN
-F 2 "C4_Pretty:c_0805" H 7400 5500 50  0001 C CNN
+F 2 "C4_Pretty:c_0805_led" H 7400 5500 50  0001 C CNN
 F 3 "" H 7400 5500 60  0001 C CNN
 F 4 "CAP CER 0.1UF 25V 10% X7R 0805" H 7400 5700 60  0001 L CNN "Field4"
@@
 F 0 "C164" H 8825 5600 50  0000 L CNN
 F 1 "100n" H 8825 5400 50  0000 L CNN
-F 2 "C4_Pretty:c_0805" H 8800 5500 50  0001 C CNN
+F 2 "C4_Pretty:c_0805_led" H 8800 5500 50  0001 C CNN
 F 3 "" H 8800 5500 60  0001 C CNN
 F 4 "CAP CER 0.1UF 25V 10% X7R 0805" H 8800 5700 60  0001 L CNN "Field4"
@@
 F 0 "C165" H 10225 5600 50  0000 L CNN
 F 1 "100n" H 10225 5400 50  0000 L CNN
-F 2 "C4_Pretty:c_0805" H 10200 5500 50  0001 C CNN
+F 2 "C4_Pretty:c_0805_led" H 10200 5500 50  0001 C CNN
 F 3 "" H 10200 5500 60  0001 C CNN
 F 4 "CAP CER 0.1UF 25V 10% X7R 0805" H 10200 5700 60  0001 L CNN "Field4"
