File: KiCad/Row_L.sch (KiCad schematic (older format))
At the start: 14 parts, among them U101 RGB_WS2811B, U102 RGB_WS2811B, U103 RGB_WS2811B, U104 RGB_WS2811B, U105 RGB_WS2811B, U106 RGB_WS2811B, U107 RGB_WS2811B, U108 RGB_WS2811B

Commit message: Schematic updated
Parts:
- removed C101: 100n, TinyTiM_Lib:c_0805, symbol C2
- removed C117: 47u,8V, TinyTiM_Lib:c_2917, symbol C_POL_1
- removed S101, S102, S103, S104: CONN_1, TinyTiM_Lib:Screw, symbol CONN_1
- removed U101, U102, U103, U104, U105, U106, U107, U108: RGB_WS2811B, TinyTiM_Lib:RGB_WS2811B, symbol RGB_WS2811B
Connections:
- net labels removed: 5V, A_02, A_03, A_04, A_05, A_06, A_07, A_08, A_09, DI_A, DO_A, GND
- wire segments 49 -> 0
- no-connect marks 4 -> 0
Other:
- note removed: "Mounting Screws"

Commit message: Schematic updated
Parts:
- added C164, C165, C166, C167, C168, C169, C170, C171, C172, C173, C174, C175, C176, C177: 100n, TinyTiM_Lib:c_0805, symbol C2
- added U158, U159, U160, U161, U162, U163, U164, U165, U166, U167, U168, U169, U170, U171: RGB_WS2812B, symbol RGB_WS2812B
Connections:
- net labels added: 5V, DI_L, DO_L, GND
- wire segments 0 -> 82

Commit message: Schematic updated, board started
Parts:
- C165: renamed from C164; Field5 100nF, 25V -> 100n, 25V
- C167: renamed from C168; Field5 100nF, 25V -> 100n, 25V
- C169: renamed from C172; Field5 100nF, 25V -> 100n, 25V
- C171: renamed from C176; Field5 100nF, 25V -> 100n, 25V
- C173: renamed from C167; Field5 100nF, 25V -> 100n, 25V
- C175: renamed from C171; Field5 100nF, 25V -> 100n, 25V
- C177: renamed from C175; Field5 100nF, 25V -> 100n, 25V
- renumbered C170 to C168, C174 to C170, C165 to C172, C169 to C174, C173 to C176, C177 to C178, U158 to U156, U160 to U157, U162 to U158, U164 to U159, U166 to U160, U168 to U161, U170 to U162, U159 to U163, U161 to U164, U163 to U165, U165 to U166, U169 to U168, U171 to U169
Changed lines of the file:
@@
 LIBS:contrib
 LIBS:valves
-LIBS:TinyTiM-cache
-LIBS:TiNA_sym
+LIBS:ClockFOUR
 LIBS:ClockFOUR-cache
 EELAYER 27 0
@@
 Sheet 13 14
 Title "ClockFOUR"
-Date "30 sep 2014"
+Date "1 oct 2014"
 Rev ""
 Comp "WyoLum"
@@
 5V
 $Comp
-L GND #PWR023
+L GND #PWR025
 U 1 1 542C1953
 P 1300 2750
-F 0 "#PWR023" H 1300 2750 30  0001 C CNN
+F 0 "#PWR025" H 1300 2750 30  0001 C CNN
 F 1 "GND" H 1300 2680 30  0001 C CNN
 F 2 "" H 1300 2750 60  0001 C CNN
@@
 $EndComp
 $Comp
-L C2 C164
+L C2 C165
 U 1 1 542C1961
 P 1850 2900
-F 0 "C164" H 1875 3000 50  0000 L CNN
+F 0 "C165" H 1875 3000 50  0000 L CNN
 F 1 "100n" H 1875 2800 50  0000 L CNN
 F 2 "TinyTiM_Lib:c_0805" H 1850 2900 50  0001 C CNN
 F 3 "" H 1850 2900 60  0001 C CNN
 F 4 "CAP CER 0.1UF 25V 10% X7R 0805" H 1850 3100 60  0001 L CNN "Field4"
-F 5 "100nF, 25V" H 1850 3200 60  0001 L CNN "Field5"
+F 5 "100n, 25V" H 1850 3200 60  0001 L CNN "Field5"
 F 6 "Surface Mount, MLCC" H 1850 3300 60  0001 L CNN "Field6"
 F 7 "Kemet" H 1850 3400 60  0001 L CNN "Field7"
@@
 $EndComp
 $Comp
-L RGB_WS2812B U158
+L RGB_WS2812B U156
 U 1 1 542C1967
 P 1675 1925
-F 0 "U158" V 1425 1925 60  0000 C CNN
+F 0 "U156" V 1425 1925 60  0000 C CNN
 F 1 "RGB_WS2812B" V 2075 1925 60  0000 C CNN
 F 2 "" H 1675 1925 60  0000 C CNN
@@
 $EndComp
 $Comp
-L RGB_WS2812B U160
+L RGB_WS2812B U157
 U 1 1 542C196D
 P 3075 1925
-F 0 "U160" V 2825 1925 60  0000 C CNN
+F 0 "U157" V 2825 1925 60  0000 C CNN
 F 1 "RGB_WS2812B" V 3475 1925 60  0000 C CNN
 F 2 "" H 3075 1925 60  0000 C CNN
@@
 $EndComp
 $Comp
-L RGB_WS2812B U162
+L RGB_WS2812B U158
 U 1 1 542C1973
 P 4475 1925
-F 0 "U162" V 4225 1925 60  0000 C CNN
+F 0 "U158" V 4225 1925 60  0000 C CNN
 F 1 "RGB_WS2812B" V 4875 1925 60  0000 C CNN
 F 2 "" H 4475 1925 60  0000 C CNN
@@
 $EndComp
 $Comp
-L RGB_WS2812B U164
+L RGB_WS2812B U159
 U 1 1 542C1979
 P 5875 1925
-F 0 "U164" V 5625 1925 60  0000 C CNN
+F 0 "U159" V 5625 1925 60  0000 C CNN
 F 1 "RGB_WS2812B" V 6275 1925 60  0000 C CNN
 F 2 "" H 5875 1925 60  0000 C CNN
@@
 $EndComp
 $Comp
-L RGB_WS2812B U166
+L RGB_WS2812B U160
 U 1 1 542C197F
 P 7275 1925
-F 0 "U166" V 7025 1925 60  0000 C CNN
+F 0 "U160" V 7025 1925 60  0000 C CNN
 F 1 "RGB_WS2812B" V 7675 1925 60  0000 C CNN
 F 2 "" H 7275 1925 60  0000 C CNN
@@
 $EndComp
 $Comp
-L RGB_WS2812B U168
+L RGB_WS2812B U161
 U 1 1 542C1985
 P 8675 1925
-F 0 "U168" V 8425 1925 60  0000 C CNN
+F 0 "U161" V 8425 1925 60  0000 C CNN
 F 1 "RGB_WS2812B" V 9075 1925 60  0000 C CNN
 F 2 "" H 8675 1925 60  0000 C CNN
@@
 $EndComp
 $Comp
-L RGB_WS2812B U170
+L RGB_WS2812B U162
 U 1 1 542C198B
 P 10075 1925
-F 0 "U170" V 9825 1925 60  0000 C CNN
+F 0 "U162" V 9825 1925 60  0000 C CNN
 F 1 "RGB_WS2812B" V 10475 1925 60  0000 C CNN
 F 2 "" H 10075 1925 60  0000 C CNN
@@
 $EndComp
 $Comp
-L RGB_WS2812B U159
+L RGB_WS2812B U163
 U 1 1 542C1991
 P 1675 4325
-F 0 "U159" V 1425 4325 60  0000 C CNN
+F 0 "U163" V 1425 4325 60  0000 C CNN
 F 1 "RGB_WS2812B" V 2075 4325 60  0000 C CNN
 F 2 "" H 1675 4325 60  0000 C CNN
@@
 $EndComp
 $Comp
-L RGB_WS2812B U161
+L RGB_WS2812B U164
 U 1 1 542C1997
 P 3075 4325
-F 0 "U161" V 2825 4325 60  0000 C CNN
+F 0 "U164" V 2825 4325 60  0000 C CNN
 F 1 "RGB_WS2812B" V 3475 4325 60  0000 C CNN
 F 2 "" H 3075 4325 60  0000 C CNN
@@
 $EndComp
 $Comp
-L RGB_WS2812B U163
+L RGB_WS2812B U165
 U 1 1 542C199D
 P 4475 4325
-F 0 "U163" V 4225 4325 60  0000 C CNN
+F 0 "U165" V 4225 4325 60  0000 C CNN
 F 1 "RGB_WS2812B" V 4875 4325 60  0000 C CNN
 F 2 "" H 4475 4325 60  0000 C CNN
@@
 $EndComp
 $Comp
-L RGB_WS2812B U165
+L RGB_WS2812B U166
 U 1 1 542C19A3
 P 5875 4325
-F 0 "U165" V 5625 4325 60  0000 C CNN
+F 0 "U166" V 5625 4325 60  0000 C CNN
 F 1 "RGB_WS2812B" V 6275 4325 60  0000 C CNN
 F 2 "" H 5875 4325 60  0000 C CNN
@@
 $EndComp
 $Comp
-L RGB_WS2812B U169
+L RGB_WS2812B U168
 U 1 1 542C19AF
 P 8675 4325
-F 0 "U169" V 8425 4325 60  0000 C CNN
+F 0 "U168" V 8425 4325 60  0000 C CNN
 F 1 "RGB_WS2812B" V 9075 4325 60  0000 C CNN
 F 2 "" H 8675 4325 60  0000 C CNN
@@
 $EndComp
 $Comp
-L RGB_WS2812B U171
+L RGB_WS2812B U169
 U 1 1 542C19B5
 P 10075 4325
-F 0 "U171" V 9825 4325 60  0000 C CNN
+F 0 "U169" V 9825 4325 60  0000 C CNN
 F 1 "RGB_WS2812B" V 10475 4325 60  0000 C CNN
 F 2 "" H 10075 4325 60  0000 C CNN
@@
 $EndComp
 $Comp
-L C2 C168
+L C2 C167
 U 1 1 542C1A1E
 P 4650 2900
-F 0 "C168" H 4675 3000 50  0000 L CNN
+F 0 "C167" H 4675 3000 50  0000 L CNN
 F 1 "100n" H 4675 2800 50  0000 L CNN
 F 2 "TinyTiM_Lib:c_0805" H 4650 2900 50  0001 C CNN
 F 3 "" H 4650 2900 60  0001 C CNN
 F 4 "CAP CER 0.1UF 25V 10% X7R 0805" H 4650 3100 60  0001 L CNN "Field4"
-F 5 "100nF, 25V" H 4650 3200 60  0001 L CNN "Field5"
+F 5 "100n, 25V" H 4650 3200 60  0001 L CNN "Field5"
 F 6 "Surface Mount, MLCC" H 4650 3300 60  0001 L CNN "Field6"
 F 7 "Kemet" H 4650 3400 60  0001 L CNN "Field7"
@@
 $EndComp
 $Comp
-L C2 C170
+L C2 C168
 U 1 1 542C1A2C
 P 6050 2900
-F 0 "C170" H 6075 3000 50  0000 L CNN
+F 0 "C168" H 6075 3000 50  0000 L CNN
 F 1 "100n" H 6075 2800 50  0000 L CNN
 F 2 "TinyTiM_Lib:c_0805" H 6050 2900 50  0001 C CNN
@@
 $EndComp
 $Comp
-L C2 C172
+L C2 C169
 U 1 1 542C1A3A
 P 7450 2900
-F 0 "C172" H 7475 3000 50  0000 L CNN
+F 0 "C169" H 7475 3000 50  0000 L CNN
 F 1 "100n" H 7475 2800 50  0000 L CNN
 F 2 "TinyTiM_Lib:c_0805" H 7450 2900 50  0001 C CNN
 F 3 "" H 7450 2900 60  0001 C CNN
 F 4 "CAP CER 0.1UF 25V 10% X7R 0805" H 7450 3100 60  0001 L CNN "Field4"
-F 5 "100nF, 25V" H 7450 3200 60  0001 L CNN "Field5"
+F 5 "100n, 25V" H 7450 3200 60  0001 L CNN "Field5"
 F 6 "Surface Mount, MLCC" H 7450 3300 60  0001 L CNN "Field6"
 F 7 "Kemet" H 7450 3400 60  0001 L CNN "Field7"
@@
 $EndComp
 $Comp
-L C2 C174
+L C2 C170
 U 1 1 542C1A48
 P 8850 2900
-F 0 "C174" H 8875 3000 50  0000 L CNN
+F 0 "C170" H 8875 3000 50  0000 L CNN
 F 1 "100n" H 8875 2800 50  0000 L CNN
 F 2 "TinyTiM_Lib:c_0805" H 8850 2900 50  0001 C CNN
@@
 $EndComp
 $Comp
-L C2 C176
+L C2 C171
 U 1 1 542C1A56
 P 10250 2900
-F 0 "C176" H 10275 3000 50  0000 L CNN
+F 0 "C171" H 10275 3000 50  0000 L CNN
 F 1 "100n" H 10275 2800 50  0000 L CNN
 F 2 "TinyTiM_Lib:c_0805" H 10250 2900 50  0001 C CNN
 F 3 "" H 10250 2900 60  0001 C CNN
 F 4 "CAP CER 0.1UF 25V 10% X7R 0805" H 10250 3100 60  0001 L CNN "Field4"
-F 5 "100nF, 25V" H 10250 3200 60  0001 L CNN "Field5"
+F 5 "100n, 25V" H 10250 3200 60  0001 L CNN "Field5"
 F 6 "Surface Mount, MLCC" H 10250 3300 60  0001 L CNN "Field6"
 F 7 "Kemet" H 10250 3400 60  0001 L CNN "Field7"
@@
 Connection ~ 10150 3100
 $Comp
-L C2 C165
+L C2 C172
 U 1 1 542C1A65
 P 1850 5250
-F 0 "C165" H 1875 5350 50  0000 L CNN
+F 0 "C172" H 1875 5350 50  0000 L CNN
 F 1 "100n" H 1875 5150 50  0000 L CNN
 F 2 "TinyTiM_Lib:c_0805" H 1850 5250 50  0001 C CNN
@@
 Connection ~ 1750 5450
 $Comp
-L C2 C167
+L C2 C173
 U 1 1 542C1AA2
 P 3250 5250
-F 0 "C167" H 3275 5350 50  0000 L CNN
+F 0 "C173" H 3275 5350 50  0000 L CNN
 F 1 "100n" H 3275 5150 50  0000 L CNN
 F 2 "TinyTiM_Lib:c_0805" H 3250 5250 50  0001 C CNN
 F 3 "" H 3250 5250 60  0001 C CNN
 F 4 "CAP CER 0.1UF 25V 10% X7R 0805" H 3250 5450 60  0001 L CNN "Field4"
-F 5 "100nF, 25V" H 3250 5550 60  0001 L CNN "Field5"
+F 5 "100n, 25V" H 3250 5550 60  0001 L CNN "Field5"
 F 6 "Surface Mount, MLCC" H 3250 5650 60  0001 L CNN "Field6"
 F 7 "Kemet" H 3250 5750 60  0001 L CNN "Field7"
@@
 $EndComp
 $Comp
-L C2 C169
+L C2 C174
 U 1 1 542C1AB0
 P 4650 5250
-F 0 "C169" H 4675 5350 50  0000 L CNN
+F 0 "C174" H 4675 5350 50  0000 L CNN
 F 1 "100n" H 4675 5150 50  0000 L CNN
 F 2 "TinyTiM_Lib:c_0805" H 4650 5250 50  0001 C CNN
@@
 $EndComp
 $Comp
-L C2 C171
+L C2 C175
 U 1 1 542C1ABE
 P 6050 5250
-F 0 "C171" H 6075 5350 50  0000 L CNN
+F 0 "C175" H 6075 5350 50  0000 L CNN
 F 1 "100n" H 6075 5150 50  0000 L CNN
 F 2 "TinyTiM_Lib:c_0805" H 6050 5250 50  0001 C CNN
 F 3 "" H 6050 5250 60  0001 C CNN
 F 4 "CAP CER 0.1UF 25V 10% X7R 0805" H 6050 5450 60  0001 L CNN "Field4"
-F 5 "100nF, 25V" H 6050 5550 60  0001 L CNN "Field5"
+F 5 "100n, 25V" H 6050 5550 60  0001 L CNN "Field5"
 F 6 "Surface Mount, MLCC" H 6050 5650 60  0001 L CNN "Field6"
 F 7 "Kemet" H 6050 5750 60  0001 L CNN "Field7"
@@
 $EndComp
 $Comp
-L C2 C173
+L C2 C176
 U 1 1 542C1ACC
 P 7450 5250
-F 0 "C173" H 7475 5350 50  0000 L CNN
+F 0 "C176" H 7475 5350 50  0000 L CNN
 F 1 "100n" H 7475 5150 50  0000 L CNN
 F 2 "TinyTiM_Lib:c_0805" H 7450 5250 50  0001 C CNN
@@
 $EndComp
 $Comp
-L C2 C175
+L C2 C177
 U 1 1 542C1ADA
 P 8850 5250
-F 0 "C175" H 8875 5350 50  0000 L CNN
+F 0 "C177" H 8875 5350 50  0000 L CNN
 F 1 "100n" H 8875 5150 50  0000 L CNN
 F 2 "TinyTiM_Lib:c_0805" H 8850 5250 50  0001 C CNN
 F 3 "" H 8850 5250 60  0001 C CNN
 F 4 "CAP CER 0.1UF 25V 10% X7R 0805" H 8850 5450 60  0001 L CNN "Field4"
-F 5 "100nF, 25V" H 8850 5550 60  0001 L CNN "Field5"
+F 5 "100n, 25V" H 8850 5550 60  0001 L CNN "Field5"
 F 6 "Surface Mount, MLCC" H 8850 5650 60  0001 L CNN "Field6"
 F 7 "Kemet" H 8850 5750 60  0001 L CNN "Field7"
@@
 $EndComp
 $Comp
-L C2 C177
+L C2 C178
 U 1 1 542C1AE8
 P 10250 5250
-F 0 "C177" H 10275 5350 50  0000 L CNN
+F 0 "C178" H 10275 5350 50  0000 L CNN
 F 1 "100n" H 10275 5150 50  0000 L CNN
 F 2 "TinyTiM_Lib:c_0805" H 10250 5250 50  0001 C CNN

Commit message: Board layout updated
Parts:
- removed U156, U157, U158, U159, U160, U161, U162, U163, U164, U165, U166, U167, U168, U169: RGB_WS2812B, symbol RGB_WS2812B
- added LED155, LED156, LED157, LED158, LED159, LED160, LED161, LED162, LED163, LED164, LED165, LED166, LED167, LED168: RGB_WS2812B, ~, symbol RGB_WS2812B

Commit message: Board layout updated
Matrix placed and wired. Added RTC.
Parts:
- removed C165: 100n, TinyTiM_Lib:c_0805, symbol C2
- removed LED155, LED156, LED157, LED158, LED159, LED160, LED161, LED162, LED163, LED164, LED165, LED166, LED167, LED168: RGB_WS2812B, ~, symbol RGB_WS2812B
- added C179: 100n, TinyTiM_Lib:c_0805, symbol C2
- added LED155, LED156, LED157, LED158, LED159, LED160, LED161, LED162, LED163, LED164, LED165, LED166, LED167, LED168: WS2812B, ~, symbol WS2812B
- C166, C168, C170, C172, C174, C176, C178: Field5 100nF, 25V -> 100n, 25V
- C167, C169, C171, C173, C175, C177: Field5 100n, 25V -> 100nF, 25V
