File: KiCad/Row_L.sch (KiCad schematic (older format))
At the start: 28 parts

Commit message: PCB layout, work in progress
Parts:
- C166, C167, C168, C169, C170, C171, C172, C173, C174, C175, C176, C177, C178, C179: footprint TinyTiM_Lib:c_0805 -> C4_Pretty:c_0805
- LED155, LED156, LED157, LED158, LED159, LED160, LED161, LED162, LED163, LED164, LED165, LED166, LED167, LED168: footprint ~ -> C4_Pretty:RGB_WS2811B
Changed lines of the file:
@@
 F 0 "C166" H 1875 3100 50  0000 L CNN
 F 1 "100n" H 1875 2900 50  0000 L CNN
-F 2 "TinyTiM_Lib:c_0805" H 1850 3000 50  0001 C CNN
+F 2 "C4_Pretty:c_0805" H 1850 3000 50  0001 C CNN
 F 3 "" H 1850 3000 60  0001 C CNN
 F 4 "CAP CER 0.1UF 25V 10% X7R 0805" H 1850 3200 60  0001 L CNN "Field4"
@@
 F 0 "C167" H 3275 3100 50  0000 L CNN
 F 1 "100n" H 3275 2900 50  0000 L CNN
-F 2 "TinyTiM_Lib:c_0805" H 3250 3000 50  0001 C CNN
+F 2 "C4_Pretty:c_0805" H 3250 3000 50  0001 C CNN
 F 3 "" H 3250 3000 60  0001 C CNN
 F 4 "CAP CER 0.1UF 25V 10% X7R 0805" H 3250 3200 60  0001 L CNN "Field4"
@@
 F 0 "C168" H 4675 3100 50  0000 L CNN
 F 1 "100n" H 4675 2900 50  0000 L CNN
-F 2 "TinyTiM_Lib:c_0805" H 4650 3000 50  0001 C CNN
+F 2 "C4_Pretty:c_0805" H 4650 3000 50  0001 C CNN
 F 3 "" H 4650 3000 60  0001 C CNN
 F 4 "CAP CER 0.1UF 25V 10% X7R 0805" H 4650 3200 60  0001 L CNN "Field4"
@@
 F 0 "C169" H 6075 3100 50  0000 L CNN
 F 1 "100n" H 6075 2900 50  0000 L CNN
-F 2 "TinyTiM_Lib:c_0805" H 6050 3000 50  0001 C CNN
+F 2 "C4_Pretty:c_0805" H 6050 3000 50  0001 C CNN
 F 3 "" H 6050 3000 60  0001 C CNN
 F 4 "CAP CER 0.1UF 25V 10% X7R 0805" H 6050 3200 60  0001 L CNN "Field4"
@@
 F 0 "C170" H 7475 3100 50  0000 L CNN
 F 1 "100n" H 7475 2900 50  0000 L CNN
-F 2 "TinyTiM_Lib:c_0805" H 7450 3000 50  0001 C CNN
+F 2 "C4_Pretty:c_0805" H 7450 3000 50  0001 C CNN
 F 3 "" H 7450 3000 60  0001 C CNN
 F 4 "CAP CER 0.1UF 25V 10% X7R 0805" H 7450 3200 60  0001 L CNN "Field4"
@@
 F 0 "C171" H 8875 3100 50  0000 L CNN
 F 1 "100n" H 8875 2900 50  0000 L CNN
-F 2 "TinyTiM_Lib:c_0805" H 8850 3000 50  0001 C CNN
+F 2 "C4_Pretty:c_0805" H 8850 3000 50  0001 C CNN
 F 3 "" H 8850 3000 60  0001 C CNN
 F 4 "CAP CER 0.1UF 25V 10% X7R 0805" H 8850 3200 60  0001 L CNN "Field4"
@@
 F 0 "C172" H 10275 3100 50  0000 L CNN
 F 1 "100n" H 10275 2900 50  0000 L CNN
-F 2 "TinyTiM_Lib:c_0805" H 10250 3000 50  0001 C CNN
+F 2 "C4_Pretty:c_0805" H 10250 3000 50  0001 C CNN
 F 3 "" H 10250 3000 60  0001 C CNN
 F 4 "CAP CER 0.1UF 25V 10% X7R 0805" H 10250 3200 60  0001 L CNN "Field4"
@@
 F 0 "C173" H 1875 5450 50  0000 L CNN
 F 1 "100n" H 1875 5250 50  0000 L CNN
-F 2 "TinyTiM_Lib:c_0805" H 1850 5350 50  0001 C CNN
+F 2 "C4_Pretty:c_0805" H 1850 5350 50  0001 C CNN
 F 3 "" H 1850 5350 60  0001 C CNN
 F 4 "CAP CER 0.1UF 25V 10% X7R 0805" H 1850 5550 60  0001 L CNN "Field4"
@@
 F 0 "C174" H 3275 5450 50  0000 L CNN
 F 1 "100n" H 3275 5250 50  0000 L CNN
-F 2 "TinyTiM_Lib:c_0805" H 3250 5350 50  0001 C CNN
+F 2 "C4_Pretty:c_0805" H 3250 5350 50  0001 C CNN
 F 3 "" H 3250 5350 60  0001 C CNN
 F 4 "CAP CER 0.1UF 25V 10% X7R 0805" H 3250 5550 60  0001 L CNN "Field4"
@@
 F 0 "C175" H 4675 5450 50  0000 L CNN
 F 1 "100n" H 4675 5250 50  0000 L CNN
-F 2 "TinyTiM_Lib:c_0805" H 4650 5350 50  0001 C CNN
+F 2 "C4_Pretty:c_0805" H 4650 5350 50  0001 C CNN
 F 3 "" H 4650 5350 60  0001 C CNN
 F 4 "CAP CER 0.1UF 25V 10% X7R 0805" H 4650 5550 60  0001 L CNN "Field4"
@@
 F 0 "C176" H 6075 5450 50  0000 L CNN
 F 1 "100n" H 6075 5250 50  0000 L CNN
-F 2 "TinyTiM_Lib:c_0805" H 6050 5350 50  0001 C CNN
+F 2 "C4_Pretty:c_0805" H 6050 5350 50  0001 C CNN
 F 3 "" H 6050 5350 60  0001 C CNN
 F 4 "CAP CER 0.1UF 25V 10% X7R 0805" H 6050 5550 60  0001 L CNN "Field4"
@@
 F 0 "C177" H 7475 5450 50  0000 L CNN
 F 1 "100n" H 7475 5250 50  0000 L CNN
-F 2 "TinyTiM_Lib:c_0805" H 7450 5350 50  0001 C CNN
+F 2 "C4_Pretty:c_0805" H 7450 5350 50  0001 C CNN
 F 3 "" H 7450 5350 60  0001 C CNN
 F 4 "CAP CER 0.1UF 25V 10% X7R 0805" H 7450 5550 60  0001 L CNN "Field4"
@@
 F 0 "C178" H 8875 5450 50  0000 L CNN
 F 1 "100n" H 8875 5250 50  0000 L CNN
-F 2 "TinyTiM_Lib:c_0805" H 8850 5350 50  0001 C CNN
+F 2 "C4_Pretty:c_0805" H 8850 5350 50  0001 C CNN
 F 3 "" H 8850 5350 60  0001 C CNN
 F 4 "CAP CER 0.1UF 25V 10% X7R 0805" H 8850 5550 60  0001 L CNN "Field4"
@@
 F 0 "C179" H 10275 5450 50  0000 L CNN
 F 1 "100n" H 10275 5250 50  0000 L CNN
-F 2 "TinyTiM_Lib:c_0805" H 10250 5350 50  0001 C CNN
+F 2 "C4_Pretty:c_0805" H 10250 5350 50  0001 C CNN
 F 3 "" H 10250 5350 60  0001 C CNN
 F 4 "CAP CER 0.1UF 25V 10% X7R 0805" H 10250 5550 60  0001 L CNN "Field4"
@@
 F 0 "LED155" V 1425 2025 60  0000 C CNN
 F 1 "WS2812B" V 2075 2025 60  0001 C CNN
-F 2 "~" H 1675 2025 60  0000 C CNN
+F 2 "C4_Pretty:RGB_WS2811B" H 1675 2025 60  0001 C CNN
 F 3 "~" H 1675 2025 60  0000 C CNN
 	1    1675 2025
@@
 F 0 "LED156" V 2825 2025 60  0000 C CNN
 F 1 "WS2812B" V 3475 2025 60  0001 C CNN
-F 2 "~" H 3075 2025 60  0000 C CNN
+F 2 "C4_Pretty:RGB_WS2811B" H 3075 2025 60  0001 C CNN
 F 3 "~" H 3075 2025 60  0000 C CNN
 	1    3075 2025
@@
 F 0 "LED157" V 4225 2025 60  0000 C CNN
 F 1 "WS2812B" V 4875 2025 60  0001 C CNN
-F 2 "~" H 4475 2025 60  0000 C CNN
+F 2 "C4_Pretty:RGB_WS2811B" H 4475 2025 60  0001 C CNN
 F 3 "~" H 4475 2025 60  0000 C CNN
 	1    4475 2025
@@
 F 0 "LED158" V 5625 2025 60  0000 C CNN
 F 1 "WS2812B" V 6275 2025 60  0001 C CNN
-F 2 "~" H 5875 2025 60  0000 C CNN
+F 2 "C4_Pretty:RGB_WS2811B" H 5875 2025 60  0001 C CNN
 F 3 "~" H 5875 2025 60  0000 C CNN
 	1    5875 2025
@@
 F 0 "LED159" V 7025 2025 60  0000 C CNN
 F 1 "WS2812B" V 7675 2025 60  0001 C CNN
-F 2 "~" H 7275 2025 60  0000 C CNN
+F 2 "C4_Pretty:RGB_WS2811B" H 7275 2025 60  0001 C CNN
 F 3 "~" H 7275 2025 60  0000 C CNN
 	1    7275 2025
@@
 F 0 "LED160" V 8425 2025 60  0000 C CNN
 F 1 "WS2812B" V 9075 2025 60  0001 C CNN
-F 2 "~" H 8675 2025 60  0000 C CNN
+F 2 "C4_Pretty:RGB_WS2811B" H 8675 2025 60  0001 C CNN
 F 3 "~" H 8675 2025 60  0000 C CNN
 	1    8675 2025
@@
 F 0 "LED161" V 9825 2025 60  0000 C CNN
 F 1 "WS2812B" V 10475 2025 60  0001 C CNN
-F 2 "~" H 10075 2025 60  0000 C CNN
+F 2 "C4_Pretty:RGB_WS2811B" H 10075 2025 60  0001 C CNN
 F 3 "~" H 10075 2025 60  0000 C CNN
 	1    10075 2025
@@
 F 0 "LED162" V 1425 4425 60  0000 C CNN
 F 1 "WS2812B" V 2075 4425 60  0001 C CNN
-F 2 "~" H 1675 4425 60  0000 C CNN
+F 2 "C4_Pretty:RGB_WS2811B" H 1675 4425 60  0001 C CNN
 F 3 "~" H 1675 4425 60  0000 C CNN
 	1    1675 4425
@@
 F 0 "LED163" V 2825 4425 60  0000 C CNN
 F 1 "WS2812B" V 3475 4425 60  0001 C CNN
-F 2 "~" H 3075 4425 60  0000 C CNN
+F 2 "C4_Pretty:RGB_WS2811B" H 3075 4425 60  0001 C CNN
 F 3 "~" H 3075 4425 60  0000 C CNN
 	1    3075 4425
@@
 F 0 "LED164" V 4225 4425 60  0000 C CNN
 F 1 "WS2812B" V 4875 4425 60  0001 C CNN
-F 2 "~" H 4475 4425 60  0000 C CNN
+F 2 "C4_Pretty:RGB_WS2811B" H 4475 4425 60  0001 C CNN
 F 3 "~" H 4475 4425 60  0000 C CNN
 	1    4475 4425
@@
 F 0 "LED165" V 5625 4425 60  0000 C CNN
 F 1 "WS2812B" V 6275 4425 60  0001 C CNN
-F 2 "~" H 5875 4425 60  0000 C CNN
+F 2 "C4_Pretty:RGB_WS2811B" H 5875 4425 60  0001 C CNN
 F 3 "~" H 5875 4425 60  0000 C CNN
 	1    5875 4425
@@
 F 0 "LED166" V 7025 4425 60  0000 C CNN
 F 1 "WS2812B" V 7675 4425 60  0001 C CNN
-F 2 "~" H 7275 4425 60  0000 C CNN
+F 2 "C4_Pretty:RGB_WS2811B" H 7275 4425 60  0001 C CNN
 F 3 "~" H 7275 4425 60  0000 C CNN
 	1    7275 4425
@@
 F 0 "LED167" V 8425 4425 60  0000 C CNN
 F 1 "WS2812B" V 9075 4425 60  0001 C CNN
-F 2 "~" H 8675 4425 60  0000 C CNN
+F 2 "C4_Pretty:RGB_WS2811B" H 8675 4425 60  0001 C CNN
 F 3 "~" H 8675 4425 60  0000 C CNN
 	1    8675 4425
@@
 F 0 "LED168" V 9825 4425 60  0000 C CNN
 F 1 "WS2812B" V 10475 4425 60  0001 C CNN
-F 2 "~" H 10075 4425 60  0000 C CNN
+F 2 "C4_Pretty:RGB_WS2811B" H 10075 4425 60  0001 C CNN
 F 3 "~" H 10075 4425 60  0000 C CNN
 	1    10075 4425

Commit message: C4 PCB layout complete. Added Gerbers
Parts:
- C166, C167, C168, C169, C170, C171, C172, C173, C174, C175, C176, C177, C178, C179: footprint C4_Pretty:c_0805 -> C4_Pretty:c_0805_led
Changed lines of the file:
@@
 EESchema Schematic File Version 2
 LIBS:ClockFOUR
+LIBS:RowGB_sym
 LIBS:ClockFOUR-cache
 EELAYER 24 0
@@
 F 0 "C166" H 1875 3100 50  0000 L CNN
 F 1 "100n" H 1875 2900 50  0000 L CNN
-F 2 "C4_Pretty:c_0805" H 1850 3000 50  0001 C CNN
+F 2 "C4_Pretty:c_0805_led" H 1850 3000 50  0001 C CNN
 F 3 "" H 1850 3000 60  0001 C CNN
 F 4 "CAP CER 0.1UF 25V 10% X7R 0805" H 1850 3200 60  0001 L CNN "Field4"
@@
 F 0 "C167" H 3275 3100 50  0000 L CNN
 F 1 "100n" H 3275 2900 50  0000 L CNN
-F 2 "C4_Pretty:c_0805" H 3250 3000 50  0001 C CNN
+F 2 "C4_Pretty:c_0805_led" H 3250 3000 50  0001 C CNN
 F 3 "" H 3250 3000 60  0001 C CNN
 F 4 "CAP CER 0.1UF 25V 10% X7R 0805" H 3250 3200 60  0001 L CNN "Field4"
@@
 F 0 "C168" H 4675 3100 50  0000 L CNN
 F 1 "100n" H 4675 2900 50  0000 L CNN
-F 2 "C4_Pretty:c_0805" H 4650 3000 50  0001 C CNN
+F 2 "C4_Pretty:c_0805_led" H 4650 3000 50  0001 C CNN
 F 3 "" H 4650 3000 60  0001 C CNN
 F 4 "CAP CER 0.1UF 25V 10% X7R 0805" H 4650 3200 60  0001 L CNN "Field4"
@@
 F 0 "C169" H 6075 3100 50  0000 L CNN
 F 1 "100n" H 6075 2900 50  0000 L CNN
-F 2 "C4_Pretty:c_0805" H 6050 3000 50  0001 C CNN
+F 2 "C4_Pretty:c_0805_led" H 6050 3000 50  0001 C CNN
 F 3 "" H 6050 3000 60  0001 C CNN
 F 4 "CAP CER 0.1UF 25V 10% X7R 0805" H 6050 3200 60  0001 L CNN "Field4"
@@
 F 0 "C170" H 7475 3100 50  0000 L CNN
 F 1 "100n" H 7475 2900 50  0000 L CNN
-F 2 "C4_Pretty:c_0805" H 7450 3000 50  0001 C CNN
+F 2 "C4_Pretty:c_0805_led" H 7450 3000 50  0001 C CNN
 F 3 "" H 7450 3000 60  0001 C CNN
 F 4 "CAP CER 0.1UF 25V 10% X7R 0805" H 7450 3200 60  0001 L CNN "Field4"
@@
 F 0 "C171" H 8875 3100 50  0000 L CNN
 F 1 "100n" H 8875 2900 50  0000 L CNN
-F 2 "C4_Pretty:c_0805" H 8850 3000 50  0001 C CNN
+F 2 "C4_Pretty:c_0805_led" H 8850 3000 50  0001 C CNN
 F 3 "" H 8850 3000 60  0001 C CNN
 F 4 "CAP CER 0.1UF 25V 10% X7R 0805" H 8850 3200 60  0001 L CNN "Field4"
@@
 F 0 "C172" H 10275 3100 50  0000 L CNN
 F 1 "100n" H 10275 2900 50  0000 L CNN
-F 2 "C4_Pretty:c_0805" H 10250 3000 50  0001 C CNN
+F 2 "C4_Pretty:c_0805_led" H 10250 3000 50  0001 C CNN
 F 3 "" H 10250 3000 60  0001 C CNN
 F 4 "CAP CER 0.1UF 25V 10% X7R 0805" H 10250 3200 60  0001 L CNN "Field4"
@@
 F 0 "C173" H 1875 5450 50  0000 L CNN
 F 1 "100n" H 1875 5250 50  0000 L CNN
-F 2 "C4_Pretty:c_0805" H 1850 5350 50  0001 C CNN
+F 2 "C4_Pretty:c_0805_led" H 1850 5350 50  0001 C CNN
 F 3 "" H 1850 5350 60  0001 C CNN
 F 4 "CAP CER 0.1UF 25V 10% X7R 0805" H 1850 5550 60  0001 L CNN "Field4"
@@
 F 0 "C174" H 3275 5450 50  0000 L CNN
 F 1 "100n" H 3275 5250 50  0000 L CNN
-F 2 "C4_Pretty:c_0805" H 3250 5350 50  0001 C CNN
+F 2 "C4_Pretty:c_0805_led" H 3250 5350 50  0001 C CNN
 F 3 "" H 3250 5350 60  0001 C CNN
 F 4 "CAP CER 0.1UF 25V 10% X7R 0805" H 3250 5550 60  0001 L CNN "Field4"
@@
 F 0 "C175" H 4675 5450 50  0000 L CNN
 F 1 "100n" H 4675 5250 50  0000 L CNN
-F 2 "C4_Pretty:c_0805" H 4650 5350 50  0001 C CNN
+F 2 "C4_Pretty:c_0805_led" H 4650 5350 50  0001 C CNN
 F 3 "" H 4650 5350 60  0001 C CNN
 F 4 "CAP CER 0.1UF 25V 10% X7R 0805" H 4650 5550 60  0001 L CNN "Field4"
@@
 F 0 "C176" H 6075 5450 50  0000 L CNN
 F 1 "100n" H 6075 5250 50  0000 L CNN
-F 2 "C4_Pretty:c_0805" H 6050 5350 50  0001 C CNN
+F 2 "C4_Pretty:c_0805_led" H 6050 5350 50  0001 C CNN
 F 3 "" H 6050 5350 60  0001 C CNN
 F 4 "CAP CER 0.1UF 25V 10% X7R 0805" H 6050 5550 60  0001 L CNN "Field4"
@@
 F 0 "C177" H 7475 5450 50  0000 L CNN
 F 1 "100n" H 7475 5250 50  0000 L CNN
-F 2 "C4_Pretty:c_0805" H 7450 5350 50  0001 C CNN
+F 2 "C4_Pretty:c_0805_led" H 7450 5350 50  0001 C CNN
 F 3 "" H 7450 5350 60  0001 C CNN
 F 4 "CAP CER 0.1UF 25V 10% X7R 0805" H 7450 5550 60  0001 L CNN "Field4"
@@
 F 0 "C178" H 8875 5450 50  0000 L CNN
 F 1 "100n" H 8875 5250 50  0000 L CNN
-F 2 "C4_Pretty:c_0805" H 8850 5350 50  0001 C CNN
+F 2 "C4_Pretty:c_0805_led" H 8850 5350 50  0001 C CNN
 F 3 "" H 8850 5350 60  0001 C CNN
 F 4 "CAP CER 0.1UF 25V 10% X7R 0805" H 8850 5550 60  0001 L CNN "Field4"
@@
 F 0 "C179" H 10275 5450 50  0000 L CNN
 F 1 "100n" H 10275 5250 50  0000 L CNN
-F 2 "C4_Pretty:c_0805" H 10250 5350 50  0001 C CNN
+F 2 "C4_Pretty:c_0805_led" H 10250 5350 50  0001 C CNN
 F 3 "" H 10250 5350 60  0001 C CNN
 F 4 "CAP CER 0.1UF 25V 10% X7R 0805" H 10250 5550 60  0001 L CNN "Field4"
