File: KiCad/Row_M.sch (KiCad schematic (older format))
At the start: 14 parts, among them U101 RGB_WS2811B, U102 RGB_WS2811B, U103 RGB_WS2811B, U104 RGB_WS2811B, U105 RGB_WS2811B, U106 RGB_WS2811B, U107 RGB_WS2811B, U108 RGB_WS2811B

Commit message: Schematic updated
Parts:
- removed C101: 100n, TinyTiM_Lib:c_0805, symbol C2
- removed C117: 47u,8V, TinyTiM_Lib:c_2917, symbol C_POL_1
- removed S101, S102, S103, S104: CONN_1, TinyTiM_Lib:Screw, symbol CONN_1
- removed U101, U102, U103, U104, U105, U106, U107, U108: RGB_WS2811B, TinyTiM_Lib:RGB_WS2811B, symbol RGB_WS2811B
Connections:
- net labels removed: 5V, A_02, A_03, A_04, A_05, A_06, A_07, A_08, A_09, DI_A, DO_A, GND
- wire segments 49 -> 0
- no-connect marks 4 -> 0
Other:
- note removed: "Mounting Screws"

Commit message: Schematic updated
Parts:
- added C178, C179, C180, C181, C182, C183, C184, C185, C186, C187, C188, C189, C190, C191: 100n, TinyTiM_Lib:c_0805, symbol C2
- added U172, U173, U174, U175, U176, U177, U178, U179, U180, U181, U182, U183, U184, U185: RGB_WS2812B, symbol RGB_WS2812B
Connections:
- net labels added: 5V, DI_M, DO_M, GND
- wire segments 0 -> 82

Commit message: Schematic updated, board started
Parts:
- C179: renamed from C178; Field5 100nF, 25V -> 100n, 25V
- C181: renamed from C182; Field5 100nF, 25V -> 100n, 25V
- C183: renamed from C186; Field5 100nF, 25V -> 100n, 25V
- C185: renamed from C190; Field5 100nF, 25V -> 100n, 25V
- C187: renamed from C181; Field5 100nF, 25V -> 100n, 25V
- C189: renamed from C185; Field5 100nF, 25V -> 100n, 25V
- C191: renamed from C189; Field5 100nF, 25V -> 100n, 25V
- renumbered C184 to C182, C188 to C184, C179 to C186, C183 to C188, C187 to C190, C191 to C192, U172 to U170, U174 to U171, U176 to U172, U178 to U173, U180 to U174, U182 to U175, U184 to U176, U173 to U177, U175 to U178, U177 to U179, U179 to U180, U183 to U182, U185 to U183
Changed lines of the file:
@@
 LIBS:contrib
 LIBS:valves
-LIBS:TinyTiM-cache
-LIBS:TiNA_sym
+LIBS:ClockFOUR
 LIBS:ClockFOUR-cache
 EELAYER 27 0
@@
 Sheet 14 14
 Title "ClockFOUR"
-Date "30 sep 2014"
+Date "1 oct 2014"
 Rev ""
 Comp "WyoLum"
@@
 5V
 $Comp
-L GND #PWR024
+L GND #PWR026
 U 1 1 542C1B00
 P 1400 2950
-F 0 "#PWR024" H 1400 2950 30  0001 C CNN
+F 0 "#PWR026" H 1400 2950 30  0001 C CNN
 F 1 "GND" H 1400 2880 30  0001 C CNN
 F 2 "" H 1400 2950 60  0001 C CNN
@@
 $EndComp
 $Comp
-L C2 C178
+L C2 C179
 U 1 1 542C1B0E
 P 1950 3100
-F 0 "C178" H 1975 3200 50  0000 L CNN
+F 0 "C179" H 1975 3200 50  0000 L CNN
 F 1 "100n" H 1975 3000 50  0000 L CNN
 F 2 "TinyTiM_Lib:c_0805" H 1950 3100 50  0001 C CNN
 F 3 "" H 1950 3100 60  0001 C CNN
 F 4 "CAP CER 0.1UF 25V 10% X7R 0805" H 1950 3300 60  0001 L CNN "Field4"
-F 5 "100nF, 25V" H 1950 3400 60  0001 L CNN "Field5"
+F 5 "100n, 25V" H 1950 3400 60  0001 L CNN "Field5"
 F 6 "Surface Mount, MLCC" H 1950 3500 60  0001 L CNN "Field6"
 F 7 "Kemet" H 1950 3600 60  0001 L CNN "Field7"
@@
 $EndComp
 $Comp
-L RGB_WS2812B U172
+L RGB_WS2812B U170
 U 1 1 542C1B14
 P 1775 2125
-F 0 "U172" V 1525 2125 60  0000 C CNN
+F 0 "U170" V 1525 2125 60  0000 C CNN
 F 1 "RGB_WS2812B" V 2175 2125 60  0000 C CNN
 F 2 "" H 1775 2125 60  0000 C CNN
@@
 $EndComp
 $Comp
-L RGB_WS2812B U174
+L RGB_WS2812B U171
 U 1 1 542C1B1A
 P 3175 2125
-F 0 "U174" V 2925 2125 60  0000 C CNN
+F 0 "U171" V 2925 2125 60  0000 C CNN
 F 1 "RGB_WS2812B" V 3575 2125 60  0000 C CNN
 F 2 "" H 3175 2125 60  0000 C CNN
@@
 $EndComp
 $Comp
-L RGB_WS2812B U176
+L RGB_WS2812B U172
 U 1 1 542C1B20
 P 4575 2125
-F 0 "U176" V 4325 2125 60  0000 C CNN
+F 0 "U172" V 4325 2125 60  0000 C CNN
 F 1 "RGB_WS2812B" V 4975 2125 60  0000 C CNN
 F 2 "" H 4575 2125 60  0000 C CNN
@@
 $EndComp
 $Comp
-L RGB_WS2812B U178
+L RGB_WS2812B U173
 U 1 1 542C1B26
 P 5975 2125
-F 0 "U178" V 5725 2125 60  0000 C CNN
+F 0 "U173" V 5725 2125 60  0000 C CNN
 F 1 "RGB_WS2812B" V 6375 2125 60  0000 C CNN
 F 2 "" H 5975 2125 60  0000 C CNN
@@
 $EndComp
 $Comp
-L RGB_WS2812B U180
+L RGB_WS2812B U174
 U 1 1 542C1B2C
 P 7375 2125
-F 0 "U180" V 7125 2125 60  0000 C CNN
+F 0 "U174" V 7125 2125 60  0000 C CNN
 F 1 "RGB_WS2812B" V 7775 2125 60  0000 C CNN
 F 2 "" H 7375 2125 60  0000 C CNN
@@
 $EndComp
 $Comp
-L RGB_WS2812B U182
+L RGB_WS2812B U175
 U 1 1 542C1B32
 P 8775 2125
-F 0 "U182" V 8525 2125 60  0000 C CNN
+F 0 "U175" V 8525 2125 60  0000 C CNN
 F 1 "RGB_WS2812B" V 9175 2125 60  0000 C CNN
 F 2 "" H 8775 2125 60  0000 C CNN
@@
 $EndComp
 $Comp
-L RGB_WS2812B U184
+L RGB_WS2812B U176
 U 1 1 542C1B38
 P 10175 2125
-F 0 "U184" V 9925 2125 60  0000 C CNN
+F 0 "U176" V 9925 2125 60  0000 C CNN
 F 1 "RGB_WS2812B" V 10575 2125 60  0000 C CNN
 F 2 "" H 10175 2125 60  0000 C CNN
@@
 $EndComp
 $Comp
-L RGB_WS2812B U173
+L RGB_WS2812B U177
 U 1 1 542C1B3E
 P 1775 4525
-F 0 "U173" V 1525 4525 60  0000 C CNN
+F 0 "U177" V 1525 4525 60  0000 C CNN
 F 1 "RGB_WS2812B" V 2175 4525 60  0000 C CNN
 F 2 "" H 1775 4525 60  0000 C CNN
@@
 $EndComp
 $Comp
-L RGB_WS2812B U175
+L RGB_WS2812B U178
 U 1 1 542C1B44
 P 3175 4525
-F 0 "U175" V 2925 4525 60  0000 C CNN
+F 0 "U178" V 2925 4525 60  0000 C CNN
 F 1 "RGB_WS2812B" V 3575 4525 60  0000 C CNN
 F 2 "" H 3175 4525 60  0000 C CNN
@@
 $EndComp
 $Comp
-L RGB_WS2812B U177
+L RGB_WS2812B U179
 U 1 1 542C1B4A
 P 4575 4525
-F 0 "U177" V 4325 4525 60  0000 C CNN
+F 0 "U179" V 4325 4525 60  0000 C CNN
 F 1 "RGB_WS2812B" V 4975 4525 60  0000 C CNN
 F 2 "" H 4575 4525 60  0000 C CNN
@@
 $EndComp
 $Comp
-L RGB_WS2812B U179
+L RGB_WS2812B U180
 U 1 1 542C1B50
 P 5975 4525
-F 0 "U179" V 5725 4525 60  0000 C CNN
+F 0 "U180" V 5725 4525 60  0000 C CNN
 F 1 "RGB_WS2812B" V 6375 4525 60  0000 C CNN
 F 2 "" H 5975 4525 60  0000 C CNN
@@
 $EndComp
 $Comp
-L RGB_WS2812B U183
+L RGB_WS2812B U182
 U 1 1 542C1B5C
 P 8775 4525
-F 0 "U183" V 8525 4525 60  0000 C CNN
+F 0 "U182" V 8525 4525 60  0000 C CNN
 F 1 "RGB_WS2812B" V 9175 4525 60  0000 C CNN
 F 2 "" H 8775 4525 60  0000 C CNN
@@
 $EndComp
 $Comp
-L RGB_WS2812B U185
+L RGB_WS2812B U183
 U 1 1 542C1B62
 P 10175 4525
-F 0 "U185" V 9925 4525 60  0000 C CNN
+F 0 "U183" V 9925 4525 60  0000 C CNN
 F 1 "RGB_WS2812B" V 10575 4525 60  0000 C CNN
 F 2 "" H 10175 4525 60  0000 C CNN
@@
 $EndComp
 $Comp
-L C2 C182
+L C2 C181
 U 1 1 542C1BCB
 P 4750 3100
-F 0 "C182" H 4775 3200 50  0000 L CNN
+F 0 "C181" H 4775 3200 50  0000 L CNN
 F 1 "100n" H 4775 3000 50  0000 L CNN
 F 2 "TinyTiM_Lib:c_0805" H 4750 3100 50  0001 C CNN
 F 3 "" H 4750 3100 60  0001 C CNN
 F 4 "CAP CER 0.1UF 25V 10% X7R 0805" H 4750 3300 60  0001 L CNN "Field4"
-F 5 "100nF, 25V" H 4750 3400 60  0001 L CNN "Field5"
+F 5 "100n, 25V" H 4750 3400 60  0001 L CNN "Field5"
 F 6 "Surface Mount, MLCC" H 4750 3500 60  0001 L CNN "Field6"
 F 7 "Kemet" H 4750 3600 60  0001 L CNN "Field7"
@@
 $EndComp
 $Comp
-L C2 C184
+L C2 C182
 U 1 1 542C1BD9
 P 6150 3100
-F 0 "C184" H 6175 3200 50  0000 L CNN
+F 0 "C182" H 6175 3200 50  0000 L CNN
 F 1 "100n" H 6175 3000 50  0000 L CNN
 F 2 "TinyTiM_Lib:c_0805" H 6150 3100 50  0001 C CNN
@@
 $EndComp
 $Comp
-L C2 C186
+L C2 C183
 U 1 1 542C1BE7
 P 7550 3100
-F 0 "C186" H 7575 3200 50  0000 L CNN
+F 0 "C183" H 7575 3200 50  0000 L CNN
 F 1 "100n" H 7575 3000 50  0000 L CNN
 F 2 "TinyTiM_Lib:c_0805" H 7550 3100 50  0001 C CNN
 F 3 "" H 7550 3100 60  0001 C CNN
 F 4 "CAP CER 0.1UF 25V 10% X7R 0805" H 7550 3300 60  0001 L CNN "Field4"
-F 5 "100nF, 25V" H 7550 3400 60  0001 L CNN "Field5"
+F 5 "100n, 25V" H 7550 3400 60  0001 L CNN "Field5"
 F 6 "Surface Mount, MLCC" H 7550 3500 60  0001 L CNN "Field6"
 F 7 "Kemet" H 7550 3600 60  0001 L CNN "Field7"
@@
 $EndComp
 $Comp
-L C2 C188
+L C2 C184
 U 1 1 542C1BF5
 P 8950 3100
-F 0 "C188" H 8975 3200 50  0000 L CNN
+F 0 "C184" H 8975 3200 50  0000 L CNN
 F 1 "100n" H 8975 3000 50  0000 L CNN
 F 2 "TinyTiM_Lib:c_0805" H 8950 3100 50  0001 C CNN
@@
 $EndComp
 $Comp
-L C2 C190
+L C2 C185
 U 1 1 542C1C03
 P 10350 3100
-F 0 "C190" H 10375 3200 50  0000 L CNN
+F 0 "C185" H 10375 3200 50  0000 L CNN
 F 1 "100n" H 10375 3000 50  0000 L CNN
 F 2 "TinyTiM_Lib:c_0805" H 10350 3100 50  0001 C CNN
 F 3 "" H 10350 3100 60  0001 C CNN
 F 4 "CAP CER 0.1UF 25V 10% X7R 0805" H 10350 3300 60  0001 L CNN "Field4"
-F 5 "100nF, 25V" H 10350 3400 60  0001 L CNN "Field5"
+F 5 "100n, 25V" H 10350 3400 60  0001 L CNN "Field5"
 F 6 "Surface Mount, MLCC" H 10350 3500 60  0001 L CNN "Field6"
 F 7 "Kemet" H 10350 3600 60  0001 L CNN "Field7"
@@
 Connection ~ 10250 3300
 $Comp
-L C2 C179
+L C2 C186
 U 1 1 542C1C12
 P 1950 5450
-F 0 "C179" H 1975 5550 50  0000 L CNN
+F 0 "C186" H 1975 5550 50  0000 L CNN
 F 1 "100n" H 1975 5350 50  0000 L CNN
 F 2 "TinyTiM_Lib:c_0805" H 1950 5450 50  0001 C CNN
@@
 Connection ~ 1850 5650
 $Comp
-L C2 C181
+L C2 C187
 U 1 1 542C1C4F
 P 3350 5450
-F 0 "C181" H 3375 5550 50  0000 L CNN
+F 0 "C187" H 3375 5550 50  0000 L CNN
 F 1 "100n" H 3375 5350 50  0000 L CNN
 F 2 "TinyTiM_Lib:c_0805" H 3350 5450 50  0001 C CNN
 F 3 "" H 3350 5450 60  0001 C CNN
 F 4 "CAP CER 0.1UF 25V 10% X7R 0805" H 3350 5650 60  0001 L CNN "Field4"
-F 5 "100nF, 25V" H 3350 5750 60  0001 L CNN "Field5"
+F 5 "100n, 25V" H 3350 5750 60  0001 L CNN "Field5"
 F 6 "Surface Mount, MLCC" H 3350 5850 60  0001 L CNN "Field6"
 F 7 "Kemet" H 3350 5950 60  0001 L CNN "Field7"
@@
 $EndComp
 $Comp
-L C2 C183
+L C2 C188
 U 1 1 542C1C5D
 P 4750 5450
-F 0 "C183" H 4775 5550 50  0000 L CNN
+F 0 "C188" H 4775 5550 50  0000 L CNN
 F 1 "100n" H 4775 5350 50  0000 L CNN
 F 2 "TinyTiM_Lib:c_0805" H 4750 5450 50  0001 C CNN
@@
 $EndComp
 $Comp
-L C2 C185
+L C2 C189
 U 1 1 542C1C6B
 P 6150 5450
-F 0 "C185" H 6175 5550 50  0000 L CNN
+F 0 "C189" H 6175 5550 50  0000 L CNN
 F 1 "100n" H 6175 5350 50  0000 L CNN
 F 2 "TinyTiM_Lib:c_0805" H 6150 5450 50  0001 C CNN
 F 3 "" H 6150 5450 60  0001 C CNN
 F 4 "CAP CER 0.1UF 25V 10% X7R 0805" H 6150 5650 60  0001 L CNN "Field4"
-F 5 "100nF, 25V" H 6150 5750 60  0001 L CNN "Field5"
+F 5 "100n, 25V" H 6150 5750 60  0001 L CNN "Field5"
 F 6 "Surface Mount, MLCC" H 6150 5850 60  0001 L CNN "Field6"
 F 7 "Kemet" H 6150 5950 60  0001 L CNN "Field7"
@@
 $EndComp
 $Comp
-L C2 C187
+L C2 C190
 U 1 1 542C1C79
 P 7550 5450
-F 0 "C187" H 7575 5550 50  0000 L CNN
+F 0 "C190" H 7575 5550 50  0000 L CNN
 F 1 "100n" H 7575 5350 50  0000 L CNN
 F 2 "TinyTiM_Lib:c_0805" H 7550 5450 50  0001 C CNN
@@
 $EndComp
 $Comp
-L C2 C189
+L C2 C191
 U 1 1 542C1C87
 P 8950 5450
-F 0 "C189" H 8975 5550 50  0000 L CNN
+F 0 "C191" H 8975 5550 50  0000 L CNN
 F 1 "100n" H 8975 5350 50  0000 L CNN
 F 2 "TinyTiM_Lib:c_0805" H 8950 5450 50  0001 C CNN
 F 3 "" H 8950 5450 60  0001 C CNN
 F 4 "CAP CER 0.1UF 25V 10% X7R 0805" H 8950 5650 60  0001 L CNN "Field4"
-F 5 "100nF, 25V" H 8950 5750 60  0001 L CNN "Field5"
+F 5 "100n, 25V" H 8950 5750 60  0001 L CNN "Field5"
 F 6 "Surface Mount, MLCC" H 8950 5850 60  0001 L CNN "Field6"
 F 7 "Kemet" H 8950 5950 60  0001 L CNN "Field7"
@@
 $EndComp
 $Comp
-L C2 C191
+L C2 C192
 U 1 1 542C1C95
 P 10350 5450
-F 0 "C191" H 10375 5550 50  0000 L CNN
+F 0 "C192" H 10375 5550 50  0000 L CNN
 F 1 "100n" H 10375 5350 50  0000 L CNN
 F 2 "TinyTiM_Lib:c_0805" H 10350 5450 50  0001 C CNN

Commit message: Board layout updated
Parts:
- removed U170, U171, U172, U173, U174, U175, U176, U177, U178, U179, U180, U181, U182, U183: RGB_WS2812B, symbol RGB_WS2812B
- added LED169, LED170, LED171, LED172, LED173, LED174, LED175, LED176, LED177, LED178, LED179, LED180, LED181, LED182: RGB_WS2812B, ~, symbol RGB_WS2812B

Commit message: Board layout updated
Matrix placed and wired. Added RTC.
Parts:
- removed C179: 100n, TinyTiM_Lib:c_0805, symbol C2
- removed LED169, LED170, LED171, LED172, LED173, LED174, LED175, LED176, LED177, LED178, LED179, LED180, LED181, LED182: RGB_WS2812B, ~, symbol RGB_WS2812B
- added C193: 100n, TinyTiM_Lib:c_0805, symbol C2
- added LED169, LED170, LED171, LED172, LED173, LED174, LED175, LED176, LED177, LED178, LED179, LED180, LED181, LED182: WS2812B, ~, symbol WS2812B
- C180, C182, C184, C186, C188, C190, C192: Field5 100nF, 25V -> 100n, 25V
- C181, C183, C185, C187, C189, C191: Field5 100n, 25V -> 100nF, 25V
