File: KiCad/Row_B.sch (KiCad schematic (older format))
At the start: 28 parts

Commit message: PCB layout, work in progress
Parts:
- C26, C27, C28, C29, C30, C31, C32, C33, C34, C35, C36, C37, C38, C39: footprint TinyTiM_Lib:c_0805 -> C4_Pretty:c_0805
- LED15, LED16, LED17, LED18, LED19, LED20, LED21, LED22, LED23, LED24, LED25, LED26, LED27, LED28: footprint ~ -> C4_Pretty:RGB_WS2811B
Changed lines of the file:
@@
 F 0 "C26" H 1925 2850 50  0000 L CNN
 F 1 "100n" H 1925 2650 50  0000 L CNN
-F 2 "TinyTiM_Lib:c_0805" H 1900 2750 50  0001 C CNN
+F 2 "C4_Pretty:c_0805" H 1900 2750 50  0001 C CNN
 F 3 "" H 1900 2750 60  0001 C CNN
 F 4 "CAP CER 0.1UF 25V 10% X7R 0805" H 1900 2950 60  0001 L CNN "Field4"
@@
 F 0 "C27" H 3325 2850 50  0000 L CNN
 F 1 "100n" H 3325 2650 50  0000 L CNN
-F 2 "TinyTiM_Lib:c_0805" H 3300 2750 50  0001 C CNN
+F 2 "C4_Pretty:c_0805" H 3300 2750 50  0001 C CNN
 F 3 "" H 3300 2750 60  0001 C CNN
 F 4 "CAP CER 0.1UF 25V 10% X7R 0805" H 3300 2950 60  0001 L CNN "Field4"
@@
 F 0 "C28" H 4725 2850 50  0000 L CNN
 F 1 "100n" H 4725 2650 50  0000 L CNN
-F 2 "TinyTiM_Lib:c_0805" H 4700 2750 50  0001 C CNN
+F 2 "C4_Pretty:c_0805" H 4700 2750 50  0001 C CNN
 F 3 "" H 4700 2750 60  0001 C CNN
 F 4 "CAP CER 0.1UF 25V 10% X7R 0805" H 4700 2950 60  0001 L CNN "Field4"
@@
 F 0 "C29" H 6125 2850 50  0000 L CNN
 F 1 "100n" H 6125 2650 50  0000 L CNN
-F 2 "TinyTiM_Lib:c_0805" H 6100 2750 50  0001 C CNN
+F 2 "C4_Pretty:c_0805" H 6100 2750 50  0001 C CNN
 F 3 "" H 6100 2750 60  0001 C CNN
 F 4 "CAP CER 0.1UF 25V 10% X7R 0805" H 6100 2950 60  0001 L CNN "Field4"
@@
 F 0 "C30" H 7525 2850 50  0000 L CNN
 F 1 "100n" H 7525 2650 50  0000 L CNN
-F 2 "TinyTiM_Lib:c_0805" H 7500 2750 50  0001 C CNN
+F 2 "C4_Pretty:c_0805" H 7500 2750 50  0001 C CNN
 F 3 "" H 7500 2750 60  0001 C CNN
 F 4 "CAP CER 0.1UF 25V 10% X7R 0805" H 7500 2950 60  0001 L CNN "Field4"
@@
 F 0 "C31" H 8925 2850 50  0000 L CNN
 F 1 "100n" H 8925 2650 50  0000 L CNN
-F 2 "TinyTiM_Lib:c_0805" H 8900 2750 50  0001 C CNN
+F 2 "C4_Pretty:c_0805" H 8900 2750 50  0001 C CNN
 F 3 "" H 8900 2750 60  0001 C CNN
 F 4 "CAP CER 0.1UF 25V 10% X7R 0805" H 8900 2950 60  0001 L CNN "Field4"
@@
 F 0 "C32" H 10325 2850 50  0000 L CNN
 F 1 "100n" H 10325 2650 50  0000 L CNN
-F 2 "TinyTiM_Lib:c_0805" H 10300 2750 50  0001 C CNN
+F 2 "C4_Pretty:c_0805" H 10300 2750 50  0001 C CNN
 F 3 "" H 10300 2750 60  0001 C CNN
 F 4 "CAP CER 0.1UF 25V 10% X7R 0805" H 10300 2950 60  0001 L CNN "Field4"
@@
 F 0 "C33" H 1925 5200 50  0000 L CNN
 F 1 "100n" H 1925 5000 50  0000 L CNN
-F 2 "TinyTiM_Lib:c_0805" H 1900 5100 50  0001 C CNN
+F 2 "C4_Pretty:c_0805" H 1900 5100 50  0001 C CNN
 F 3 "" H 1900 5100 60  0001 C CNN
 F 4 "CAP CER 0.1UF 25V 10% X7R 0805" H 1900 5300 60  0001 L CNN "Field4"
@@
 F 0 "C34" H 3325 5200 50  0000 L CNN
 F 1 "100n" H 3325 5000 50  0000 L CNN
-F 2 "TinyTiM_Lib:c_0805" H 3300 5100 50  0001 C CNN
+F 2 "C4_Pretty:c_0805" H 3300 5100 50  0001 C CNN
 F 3 "" H 3300 5100 60  0001 C CNN
 F 4 "CAP CER 0.1UF 25V 10% X7R 0805" H 3300 5300 60  0001 L CNN "Field4"
@@
 F 0 "C35" H 4725 5200 50  0000 L CNN
 F 1 "100n" H 4725 5000 50  0000 L CNN
-F 2 "TinyTiM_Lib:c_0805" H 4700 5100 50  0001 C CNN
+F 2 "C4_Pretty:c_0805" H 4700 5100 50  0001 C CNN
 F 3 "" H 4700 5100 60  0001 C CNN
 F 4 "CAP CER 0.1UF 25V 10% X7R 0805" H 4700 5300 60  0001 L CNN "Field4"
@@
 F 0 "C36" H 6125 5200 50  0000 L CNN
 F 1 "100n" H 6125 5000 50  0000 L CNN
-F 2 "TinyTiM_Lib:c_0805" H 6100 5100 50  0001 C CNN
+F 2 "C4_Pretty:c_0805" H 6100 5100 50  0001 C CNN
 F 3 "" H 6100 5100 60  0001 C CNN
 F 4 "CAP CER 0.1UF 25V 10% X7R 0805" H 6100 5300 60  0001 L CNN "Field4"
@@
 F 0 "C37" H 7525 5200 50  0000 L CNN
 F 1 "100n" H 7525 5000 50  0000 L CNN
-F 2 "TinyTiM_Lib:c_0805" H 7500 5100 50  0001 C CNN
+F 2 "C4_Pretty:c_0805" H 7500 5100 50  0001 C CNN
 F 3 "" H 7500 5100 60  0001 C CNN
 F 4 "CAP CER 0.1UF 25V 10% X7R 0805" H 7500 5300 60  0001 L CNN "Field4"
@@
 F 0 "C38" H 8925 5200 50  0000 L CNN
 F 1 "100n" H 8925 5000 50  0000 L CNN
-F 2 "TinyTiM_Lib:c_0805" H 8900 5100 50  0001 C CNN
+F 2 "C4_Pretty:c_0805" H 8900 5100 50  0001 C CNN
 F 3 "" H 8900 5100 60  0001 C CNN
 F 4 "CAP CER 0.1UF 25V 10% X7R 0805" H 8900 5300 60  0001 L CNN "Field4"
@@
 F 0 "C39" H 10325 5200 50  0000 L CNN
 F 1 "100n" H 10325 5000 50  0000 L CNN
-F 2 "TinyTiM_Lib:c_0805" H 10300 5100 50  0001 C CNN
+F 2 "C4_Pretty:c_0805" H 10300 5100 50  0001 C CNN
 F 3 "" H 10300 5100 60  0001 C CNN
 F 4 "CAP CER 0.1UF 25V 10% X7R 0805" H 10300 5300 60  0001 L CNN "Field4"
@@
 F 0 "LED15" V 1475 1775 60  0000 C CNN
 F 1 "WS2812B" V 2125 1775 60  0001 C CNN
-F 2 "~" H 1725 1775 60  0000 C CNN
+F 2 "C4_Pretty:RGB_WS2811B" H 1725 1775 60  0001 C CNN
 F 3 "~" H 1725 1775 60  0000 C CNN
 	1    1725 1775
@@
 F 0 "LED16" V 2875 1775 60  0000 C CNN
 F 1 "WS2812B" V 3525 1775 60  0001 C CNN
-F 2 "~" H 3125 1775 60  0000 C CNN
+F 2 "C4_Pretty:RGB_WS2811B" H 3125 1775 60  0001 C CNN
 F 3 "~" H 3125 1775 60  0000 C CNN
 	1    3125 1775
@@
 F 0 "LED17" V 4275 1775 60  0000 C CNN
 F 1 "WS2812B" V 4925 1775 60  0001 C CNN
-F 2 "~" H 4525 1775 60  0000 C CNN
+F 2 "C4_Pretty:RGB_WS2811B" H 4525 1775 60  0001 C CNN
 F 3 "~" H 4525 1775 60  0000 C CNN
 	1    4525 1775
@@
 F 0 "LED18" V 5675 1775 60  0000 C CNN
 F 1 "WS2812B" V 6325 1775 60  0001 C CNN
-F 2 "~" H 5925 1775 60  0000 C CNN
+F 2 "C4_Pretty:RGB_WS2811B" H 5925 1775 60  0001 C CNN
 F 3 "~" H 5925 1775 60  0000 C CNN
 	1    5925 1775
@@
 F 0 "LED19" V 7075 1775 60  0000 C CNN
 F 1 "WS2812B" V 7725 1775 60  0001 C CNN
-F 2 "~" H 7325 1775 60  0000 C CNN
+F 2 "C4_Pretty:RGB_WS2811B" H 7325 1775 60  0001 C CNN
 F 3 "~" H 7325 1775 60  0000 C CNN
 	1    7325 1775
@@
 F 0 "LED20" V 8475 1775 60  0000 C CNN
 F 1 "WS2812B" V 9125 1775 60  0001 C CNN
-F 2 "~" H 8725 1775 60  0000 C CNN
+F 2 "C4_Pretty:RGB_WS2811B" H 8725 1775 60  0001 C CNN
 F 3 "~" H 8725 1775 60  0000 C CNN
 	1    8725 1775
@@
 F 0 "LED21" V 9875 1775 60  0000 C CNN
 F 1 "WS2812B" V 10525 1775 60  0001 C CNN
-F 2 "~" H 10125 1775 60  0000 C CNN
+F 2 "C4_Pretty:RGB_WS2811B" H 10125 1775 60  0001 C CNN
 F 3 "~" H 10125 1775 60  0000 C CNN
 	1    10125 1775
@@
 F 0 "LED22" V 1475 4175 60  0000 C CNN
 F 1 "WS2812B" V 2125 4175 60  0001 C CNN
-F 2 "~" H 1725 4175 60  0000 C CNN
+F 2 "C4_Pretty:RGB_WS2811B" H 1725 4175 60  0001 C CNN
 F 3 "~" H 1725 4175 60  0000 C CNN
 	1    1725 4175
@@
 F 0 "LED23" V 2875 4175 60  0000 C CNN
 F 1 "WS2812B" V 3525 4175 60  0001 C CNN
-F 2 "~" H 3125 4175 60  0000 C CNN
+F 2 "C4_Pretty:RGB_WS2811B" H 3125 4175 60  0001 C CNN
 F 3 "~" H 3125 4175 60  0000 C CNN
 	1    3125 4175
@@
 F 0 "LED24" V 4275 4175 60  0000 C CNN
 F 1 "WS2812B" V 4925 4175 60  0001 C CNN
-F 2 "~" H 4525 4175 60  0000 C CNN
+F 2 "C4_Pretty:RGB_WS2811B" H 4525 4175 60  0001 C CNN
 F 3 "~" H 4525 4175 60  0000 C CNN
 	1    4525 4175
@@
 F 0 "LED25" V 5675 4175 60  0000 C CNN
 F 1 "WS2812B" V 6325 4175 60  0001 C CNN
-F 2 "~" H 5925 4175 60  0000 C CNN
+F 2 "C4_Pretty:RGB_WS2811B" H 5925 4175 60  0001 C CNN
 F 3 "~" H 5925 4175 60  0000 C CNN
 	1    5925 4175
@@
 F 0 "LED26" V 7075 4175 60  0000 C CNN
 F 1 "WS2812B" V 7725 4175 60  0001 C CNN
-F 2 "~" H 7325 4175 60  0000 C CNN
+F 2 "C4_Pretty:RGB_WS2811B" H 7325 4175 60  0001 C CNN
 F 3 "~" H 7325 4175 60  0000 C CNN
 	1    7325 4175
@@
 F 0 "LED27" V 8475 4175 60  0000 C CNN
 F 1 "WS2812B" V 9125 4175 60  0001 C CNN
-F 2 "~" H 8725 4175 60  0000 C CNN
+F 2 "C4_Pretty:RGB_WS2811B" H 8725 4175 60  0001 C CNN
 F 3 "~" H 8725 4175 60  0000 C CNN
 	1    8725 4175
@@
 F 0 "LED28" V 9875 4175 60  0000 C CNN
 F 1 "WS2812B" V 10525 4175 60  0001 C CNN
-F 2 "~" H 10125 4175 60  0000 C CNN
+F 2 "C4_Pretty:RGB_WS2811B" H 10125 4175 60  0001 C CNN
 F 3 "~" H 10125 4175 60  0000 C CNN
 	1    10125 4175

Commit message: C4 PCB layout complete. Added Gerbers
Parts:
- C26, C27, C28, C29, C30, C31, C32, C33, C34, C35, C36, C37, C38, C39: footprint C4_Pretty:c_0805 -> C4_Pretty:c_0805_led
Changed lines of the file:
@@
 EESchema Schematic File Version 2
 LIBS:ClockFOUR
+LIBS:RowGB_sym
 LIBS:ClockFOUR-cache
 EELAYER 24 0
@@
 F 0 "C26" H 1925 2850 50  0000 L CNN
 F 1 "100n" H 1925 2650 50  0000 L CNN
-F 2 "C4_Pretty:c_0805" H 1900 2750 50  0001 C CNN
+F 2 "C4_Pretty:c_0805_led" H 1900 2750 50  0001 C CNN
 F 3 "" H 1900 2750 60  0001 C CNN
 F 4 "CAP CER 0.1UF 25V 10% X7R 0805" H 1900 2950 60  0001 L CNN "Field4"
@@
 F 0 "C27" H 3325 2850 50  0000 L CNN
 F 1 "100n" H 3325 2650 50  0000 L CNN
-F 2 "C4_Pretty:c_0805" H 3300 2750 50  0001 C CNN
+F 2 "C4_Pretty:c_0805_led" H 3300 2750 50  0001 C CNN
 F 3 "" H 3300 2750 60  0001 C CNN
 F 4 "CAP CER 0.1UF 25V 10% X7R 0805" H 3300 2950 60  0001 L CNN "Field4"
@@
 F 0 "C28" H 4725 2850 50  0000 L CNN
 F 1 "100n" H 4725 2650 50  0000 L CNN
-F 2 "C4_Pretty:c_0805" H 4700 2750 50  0001 C CNN
+F 2 "C4_Pretty:c_0805_led" H 4700 2750 50  0001 C CNN
 F 3 "" H 4700 2750 60  0001 C CNN
 F 4 "CAP CER 0.1UF 25V 10% X7R 0805" H 4700 2950 60  0001 L CNN "Field4"
@@
 F 0 "C29" H 6125 2850 50  0000 L CNN
 F 1 "100n" H 6125 2650 50  0000 L CNN
-F 2 "C4_Pretty:c_0805" H 6100 2750 50  0001 C CNN
+F 2 "C4_Pretty:c_0805_led" H 6100 2750 50  0001 C CNN
 F 3 "" H 6100 2750 60  0001 C CNN
 F 4 "CAP CER 0.1UF 25V 10% X7R 0805" H 6100 2950 60  0001 L CNN "Field4"
@@
 F 0 "C30" H 7525 2850 50  0000 L CNN
 F 1 "100n" H 7525 2650 50  0000 L CNN
-F 2 "C4_Pretty:c_0805" H 7500 2750 50  0001 C CNN
+F 2 "C4_Pretty:c_0805_led" H 7500 2750 50  0001 C CNN
 F 3 "" H 7500 2750 60  0001 C CNN
 F 4 "CAP CER 0.1UF 25V 10% X7R 0805" H 7500 2950 60  0001 L CNN "Field4"
@@
 F 0 "C31" H 8925 2850 50  0000 L CNN
 F 1 "100n" H 8925 2650 50  0000 L CNN
-F 2 "C4_Pretty:c_0805" H 8900 2750 50  0001 C CNN
+F 2 "C4_Pretty:c_0805_led" H 8900 2750 50  0001 C CNN
 F 3 "" H 8900 2750 60  0001 C CNN
 F 4 "CAP CER 0.1UF 25V 10% X7R 0805" H 8900 2950 60  0001 L CNN "Field4"
@@
 F 0 "C32" H 10325 2850 50  0000 L CNN
 F 1 "100n" H 10325 2650 50  0000 L CNN
-F 2 "C4_Pretty:c_0805" H 10300 2750 50  0001 C CNN
+F 2 "C4_Pretty:c_0805_led" H 10300 2750 50  0001 C CNN
 F 3 "" H 10300 2750 60  0001 C CNN
 F 4 "CAP CER 0.1UF 25V 10% X7R 0805" H 10300 2950 60  0001 L CNN "Field4"
@@
 F 0 "C33" H 1925 5200 50  0000 L CNN
 F 1 "100n" H 1925 5000 50  0000 L CNN
-F 2 "C4_Pretty:c_0805" H 1900 5100 50  0001 C CNN
+F 2 "C4_Pretty:c_0805_led" H 1900 5100 50  0001 C CNN
 F 3 "" H 1900 5100 60  0001 C CNN
 F 4 "CAP CER 0.1UF 25V 10% X7R 0805" H 1900 5300 60  0001 L CNN "Field4"
@@
 F 0 "C34" H 3325 5200 50  0000 L CNN
 F 1 "100n" H 3325 5000 50  0000 L CNN
-F 2 "C4_Pretty:c_0805" H 3300 5100 50  0001 C CNN
+F 2 "C4_Pretty:c_0805_led" H 3300 5100 50  0001 C CNN
 F 3 "" H 3300 5100 60  0001 C CNN
 F 4 "CAP CER 0.1UF 25V 10% X7R 0805" H 3300 5300 60  0001 L CNN "Field4"
@@
 F 0 "C35" H 4725 5200 50  0000 L CNN
 F 1 "100n" H 4725 5000 50  0000 L CNN
-F 2 "C4_Pretty:c_0805" H 4700 5100 50  0001 C CNN
+F 2 "C4_Pretty:c_0805_led" H 4700 5100 50  0001 C CNN
 F 3 "" H 4700 5100 60  0001 C CNN
 F 4 "CAP CER 0.1UF 25V 10% X7R 0805" H 4700 5300 60  0001 L CNN "Field4"
@@
 F 0 "C36" H 6125 5200 50  0000 L CNN
 F 1 "100n" H 6125 5000 50  0000 L CNN
-F 2 "C4_Pretty:c_0805" H 6100 5100 50  0001 C CNN
+F 2 "C4_Pretty:c_0805_led" H 6100 5100 50  0001 C CNN
 F 3 "" H 6100 5100 60  0001 C CNN
 F 4 "CAP CER 0.1UF 25V 10% X7R 0805" H 6100 5300 60  0001 L CNN "Field4"
@@
 F 0 "C37" H 7525 5200 50  0000 L CNN
 F 1 "100n" H 7525 5000 50  0000 L CNN
-F 2 "C4_Pretty:c_0805" H 7500 5100 50  0001 C CNN
+F 2 "C4_Pretty:c_0805_led" H 7500 5100 50  0001 C CNN
 F 3 "" H 7500 5100 60  0001 C CNN
 F 4 "CAP CER 0.1UF 25V 10% X7R 0805" H 7500 5300 60  0001 L CNN "Field4"
@@
 F 0 "C38" H 8925 5200 50  0000 L CNN
 F 1 "100n" H 8925 5000 50  0000 L CNN
-F 2 "C4_Pretty:c_0805" H 8900 5100 50  0001 C CNN
+F 2 "C4_Pretty:c_0805_led" H 8900 5100 50  0001 C CNN
 F 3 "" H 8900 5100 60  0001 C CNN
 F 4 "CAP CER 0.1UF 25V 10% X7R 0805" H 8900 5300 60  0001 L CNN "Field4"
@@
 F 0 "C39" H 10325 5200 50  0000 L CNN
 F 1 "100n" H 10325 5000 50  0000 L CNN
-F 2 "C4_Pretty:c_0805" H 10300 5100 50  0001 C CNN
+F 2 "C4_Pretty:c_0805_led" H 10300 5100 50  0001 C CNN
 F 3 "" H 10300 5100 60  0001 C CNN
 F 4 "CAP CER 0.1UF 25V 10% X7R 0805" H 10300 5300 60  0001 L CNN "Field4"
